File: hdw/Pulse_Oximeter/PIC32MZ.sch (KiCad schematic (older format))
At the start: 1 part

Commit message: Added display circuits
Connections:
- net LCD_PMP_DB5: now reaches U?.1 (RE5/AN17/ETXEN/RPE5/PMD5)
- net LCD_PMP_DB6: now reaches U?.2 (RE6/AN16/ETXD0/PMD6)
- net LCD_PMP_DB7: now reaches U?.3 (RE7/AN15/ETXD1/PMD7)
- net LCD_PMP_RS: now reaches U?.30 (RB15/AN10/EMDC/AEMDC/RPB15/OCFB/PMA0)
- net MCU_REFCLK: now reaches U?.47 (RC13/SOSCI/RPC13)
- net LCD_PMP_E: now reaches U?.52 (RD4/SQICS0/RPD4/PMWR)
- net LCD_PMP_R_W: now reaches U?.53 (RD5/SQICS1/RPD5/PMRD)
- net LCD_PMP_DB0: now reaches U?.58 (RE0/TRD0/SQID0/ERXD1/PMD0)
- net LCD_BACKLIGHT_PWM: now reaches U?.6 (RG8/AN12/C2IND/RPG8/SCL4/PMA3)
- net LCD_PMP_DB1: now reaches U?.61 (RE1/TRD1/SQID1/ERXD0/PMD1)
- net LCD_PMP_DB2: now reaches U?.62 (RE2/TRD2/SQID2/ERXDV/ECRSDV/AECRSDV/PMD2)
- net LCD_PMP_DB3: now reaches U?.63 (RE3/TRD3/SQID3/ERXCLK/EREFCLK/RPE3/PMD3)
- net LCD_PMP_DB4: now reaches U?.64 (RE4/AN18/ERXERR/PMD4)
Changed lines of the file:
@@
 EESchema Schematic File Version 4
+LIBS:Pulse_Oximeter-cache
 EELAYER 30 0
 EELAYER END
@@
 NoConn ~ 3360 5510
 NoConn ~ 3360 5610
-Text Notes 4280 4510 0    250  ~ 50
+Text Notes 5170 4510 0    250  ~ 50
 VERIFY PINOUT
 $Comp
@@
 	1    0    0    -1
 $EndComp
+Text GLabel 7560 3310 2    50   Output ~ 0
+LCD_BACKLIGHT_PWM
+Text GLabel 3360 3010 0    50   Output ~ 0
+LCD_PMP_RS
+Text GLabel 3360 4610 0    50   Output ~ 0
+LCD_PMP_R_W
+Text GLabel 3360 4510 0    50   Output ~ 0
+LCD_PMP_E
+Text GLabel 7560 1210 2    50   Output ~ 0
+LCD_PMP_DB0
+Text GLabel 7560 1310 2    50   Output ~ 0
+LCD_PMP_DB1
+Text GLabel 7560 1410 2    50   Output ~ 0
+LCD_PMP_DB2
+Text GLabel 7560 1510 2    50   Output ~ 0
+LCD_PMP_DB3
+Text GLabel 7560 1610 2    50   Output ~ 0
+LCD_PMP_DB4
+Text GLabel 7560 1710 2    50   Output ~ 0
+LCD_PMP_DB5
+Text GLabel 7560 1810 2    50   Output ~ 0
+LCD_PMP_DB6
+Text GLabel 7560 1910 2    50   Output ~ 0
+LCD_PMP_DB7
+Text GLabel 3360 3510 0    50   Output ~ 0
+MCU_REFCLK
 $EndSCHEMATC

Commit message: few sch additions
Connections:
- net PIC32MZ_REFCLK1: now reaches U?.5 (RG7/AN13/C1INC/RPG7/SDA4/PMA4)
- net ICSPCLK renamed PIC32MZ_ICSPCLK
- net ICSPDAT renamed PIC32MZ_ICSPDAT
- net MCU_POSC renamed PIC32MZ_POSC_EC
- net MCU_POSC_Enable renamed PIC32MZ_POSC_EC_Enable
- net MCU_REFCLK renamed PIC32MZ_REFCLK
- net MCU_SOSC renamed PIC32MZ_SOSC
- net ~MCLR renamed ~PIC32MZ_MCLR
Changed lines of the file:
@@
 	4810 880  4810 960
 Text GLabel 3360 5910 0    40   Input ~ 0
-~MCLR
+~PIC32MZ_MCLR
 $Comp
 L power:GND #PWR?
@@
 	3250 5410 3360 5410
 Text GLabel 3360 3410 0    50   Input ~ 0
-MCU_POSC
+PIC32MZ_POSC_EC
 Text GLabel 3360 3610 0    50   Input ~ 0
-MCU_SOSC
+PIC32MZ_SOSC
 Text GLabel 3360 2210 0    50   BiDi ~ 0
-ICSPDAT
+PIC32MZ_ICSPDAT
 Text GLabel 3360 2110 0    50   Input ~ 0
-ICSPCLK
+PIC32MZ_ICSPCLK
 Text GLabel 3360 3710 0    50   Output ~ 0
-MCU_POSC_Enable
+PIC32MZ_POSC_EC_Enable
 Text GLabel 3360 4310 0    50   Input ~ 0
 USB_UART_RX
@@
 LCD_PMP_DB7
 Text GLabel 3360 3510 0    50   Output ~ 0
-MCU_REFCLK
+PIC32MZ_REFCLK
+Text GLabel 7560 3210 2    50   Output ~ 0
+PIC32MZ_REFCLK1
 $EndSCHEMATC

Commit message: More sch work
Other:
- note added: "DON'T FORGET I2C PULLUPS"
Changed lines of the file:
@@
 Text GLabel 7560 3210 2    50   Output ~ 0
 PIC32MZ_REFCLK1
+Text Notes 5180 5380 0    250  ~ 50
+DON'T FORGET I2C PULLUPS
 $EndSCHEMATC

Commit message: Added I2C to PIC32MZ
Parts:
- added R? (x2): 10k, Resistors_SMD:R_0402, symbol Custom_Library:R_Custom
Connections:
- net +3V3: now also R?.1, R?.1
- net I2C_SDA: now reaches U?.41 (RF4/RPF4/SDA5/PMA9)
- net I2C_SDA: now also R?.2
- net I2C_SCL: now reaches U?.42 (RF5/RPF5/SCL5/PMA8)
- net I2C_SCL: now also R?.2
Other:
- note removed: "DON'T FORGET I2C PULLUPS"
Changed lines of the file:
@@
 Text GLabel 7560 3210 2    50   Output ~ 0
 PIC32MZ_REFCLK1
-Text Notes 5180 5380 0    250  ~ 50
-DON'T FORGET I2C PULLUPS
+Text GLabel 9670 2710 2    50   Output ~ 0
+I2C_SCL
+Text GLabel 9670 2610 2    50   BiDi ~ 0
+I2C_SDA
+Wire Wire Line
+	7560 2610 8780 2610
+Wire Wire Line
+	7560 2710 9370 2710
+$Comp
+L Custom_Library:R_Custom R?
+U 1 1 5EB7DAD1
+P 9370 2380
+AR Path="/5BB27BA3/5EB7DAD1" Ref="R?"  Part="1"
+AR Path="/5BB27BF7/5EB7DAD1" Ref="R?"  Part="1"
+AR Path="/5C1DE17A/5EB7DAD1" Ref="R?"  Part="1"
+AR Path="/5C1E3A08/5EB7DAD1" Ref="R?"  Part="1"
+AR Path="/5D779AE1/5EB7DAD1" Ref="R?"  Part="1"
+AR Path="/5CB7718D/5EB7DAD1" Ref="R?"  Part="1"
+AR Path="/5E0DC082/5EB7DAD1" Ref="R?"  Part="1"
+AR Path="/5E0F9110/5EB7DAD1" Ref="R?"  Part="1"
+AR Path="/5E9E0EA5/5EB7DAD1" Ref="R?"  Part="1"
+AR Path="/5E9E0E87/5EB7DAD1" Ref="R?"  Part="1"
+AR Path="/5EAE2D66/5EB7DAD1" Ref="R?"  Part="1"
+AR Path="/5EAE4A89/5EB7DAD1" Ref="R?"  Part="1"
+F 0 "R?" H 9290 2380 50  0000 R CNN
+F 1 "10k" V 9370 2380 50  0000 C CNN
+F 2 "Resistors_SMD:R_0402" H 9370 2380 50  0001 C CNN
+F 3 "" H 9370 2380 50  0001 C CNN
+F 4 "0402" H 9470 2460 50  0000 L CNN "display_footprint"
+F 5 "1%" H 9470 2380 50  0000 L CNN "Tolerance"
+F 6 "1/16W" H 9480 2300 50  0000 L CNN "Wattage"
+	1    9370 2380
+	1    0    0    -1
+$EndComp
+$Comp
+L power:+3.3V #PWR?
+U 1 1 5EB7DAD7
+P 9370 2230
+F 0 "#PWR?" H 9370 2080 50  0001 C CNN
+F 1 "+3.3V" H 9370 2370 50  0000 C CNN
+F 2 "" H 9370 2230 50  0001 C CNN
+F 3 "" H 9370 2230 50  0001 C CNN
+	1    9370 2230
+	1    0    0    -1
+$EndComp
+$Comp
+L Custom_Library:R_Custom R?
+U 1 1 5EB7DEAB
+P 8780 2380
+AR Path="/5BB27BA3/5EB7DEAB" Ref="R?"  Part="1"
+AR Path="/5BB27BF7/5EB7DEAB" Ref="R?"  Part="1"
+AR Path="/5C1DE17A/5EB7DEAB" Ref="R?"  Part="1"
+AR Path="/5C1E3A08/5EB7DEAB" Ref="R?"  Part="1"
+AR Path="/5D779AE1/5EB7DEAB" Ref="R?"  Part="1"
+AR Path="/5CB7718D/5EB7DEAB" Ref="R?"  Part="1"
+AR Path="/5E0DC082/5EB7DEAB" Ref="R?"  Part="1"
+AR Path="/5E0F9110/5EB7DEAB" Ref="R?"  Part="1"
+AR Path="/5E9E0EA5/5EB7DEAB" Ref="R?"  Part="1"
+AR Path="/5E9E0E87/5EB7DEAB" Ref="R?"  Part="1"
+AR Path="/5EAE2D66/5EB7DEAB" Ref="R?"  Part="1"
+AR Path="/5EAE4A89/5EB7DEAB" Ref="R?"  Part="1"
+F 0 "R?" H 8700 2380 50  0000 R CNN
+F 1 "10k" V 8780 2380 50  0000 C CNN
+F 2 "Resistors_SMD:R_0402" H 8780 2380 50  0001 C CNN
+F 3 "" H 8780 2380 50  0001 C CNN
+F 4 "0402" H 8880 2460 50  0000 L CNN "display_footprint"
+F 5 "1%" H 8880 2380 50  0000 L CNN "Tolerance"
+F 6 "1/16W" H 8890 2300 50  0000 L CNN "Wattage"
+	1    8780 2380
+	1    0    0    -1
+$EndComp
+$Comp
+L power:+3.3V #PWR?
+U 1 1 5EB7DEB5
+P 8780 2230
+F 0 "#PWR?" H 8780 2080 50  0001 C CNN
+F 1 "+3.3V" H 8780 2370 50  0000 C CNN
+F 2 "" H 8780 2230 50  0001 C CNN
+F 3 "" H 8780 2230 50  0001 C CNN
+	1    8780 2230
+	1    0    0    -1
+$EndComp
+Wire Wire Line
+	8780 2530 8780 2610
+Connection ~ 8780 2610
+Wire Wire Line
+	8780 2610 9670 2610
+Wire Wire Line
+	9370 2530 9370 2710
+Connection ~ 9370 2710
+Wire Wire Line
+	9370 2710 9670 2710
 $EndSCHEMATC

Commit message: Added more stuff to sch
Changed lines of the file:
@@
 $Descr A 11000 8500
 encoding utf-8
-Sheet 11 19
-Title "VFD Clock"
+Sheet 11 20
+Title "Pulse Oximeter"
 Date "2019-04-11"
 Rev "A"
@@
 AR Path="/5EAE2D66/5EB7DAD1" Ref="R?"  Part="1"
 AR Path="/5EAE4A89/5EB7DAD1" Ref="R?"  Part="1"
+AR Path="/5EAE2F23/5EB7DAD1" Ref="R?"  Part="1"
 F 0 "R?" H 9290 2380 50  0000 R CNN
 F 1 "10k" V 9370 2380 50  0000 C CNN
@@
 AR Path="/5EAE2D66/5EB7DEAB" Ref="R?"  Part="1"
 AR Path="/5EAE4A89/5EB7DEAB" Ref="R?"  Part="1"
+AR Path="/5EAE2F23/5EB7DEAB" Ref="R?"  Part="1"
 F 0 "R?" H 8700 2380 50  0000 R CNN
 F 1 "10k" V 8780 2380 50  0000 C CNN
@@
 Wire Wire Line
 	9370 2710 9670 2710
+Text GLabel 8630 5200 2    50   UnSpc ~ 0
+Telemetry_Config
 $EndSCHEMATC

Commit message: Added SD card slot and backup RTC
Changed lines of the file:
@@
 $Descr A 11000 8500
 encoding utf-8
-Sheet 11 20
+Sheet 11 22
 Title "Pulse Oximeter"
 Date "2019-04-11"
@@
 Text GLabel 8630 5200 2    50   UnSpc ~ 0
 Telemetry_Config
+Text GLabel 9580 4790 0    40   Output ~ 0
+~SD_CARD_DETECT
+Text GLabel 9580 4090 0    50   Input ~ 0
+SD_SPI_CS
+Text GLabel 9580 4190 0    50   Input ~ 0
+SD_SPI_MOSI
+Text GLabel 9580 4390 0    50   Input ~ 0
+SD_SPI_SCLK
+Text GLabel 9580 4590 0    50   Output ~ 0
+SD_SPI_MISO
 $EndSCHEMATC

Commit message: Added digikey pn's, footprints
Parts:
- R1101, R1102: renamed from R?; Digi-Key PN (none) -> RMCF0402FT10K0CT-ND
- gave numbers to parts that had none: 1
Changed lines of the file:
@@
 Sheet 11 23
 Title "Pulse Oximeter"
-Date "2019-04-11"
+Date "2019-01-03"
 Rev "A"
 Comp "Drew Maatman"
@@
 	5660 920  5560 920
 $Comp
-L power:GND #PWR?
+L power:GND #PWR01105
 U 1 1 5CB03EF2
 P 5460 6240
-F 0 "#PWR?" H 5460 5990 50  0001 C CNN
+F 0 "#PWR01105" H 5460 5990 50  0001 C CNN
 F 1 "GND" H 5460 6090 50  0000 C CNN
 F 2 "" H 5460 6240 50  0001 C CNN
@@
 ~PIC32MZ_MCLR
 $Comp
-L power:GND #PWR?
+L power:GND #PWR01101
 U 1 1 5CB14B21
 P 3250 5490
-F 0 "#PWR?" H 3250 5240 50  0001 C CNN
+F 0 "#PWR01101" H 3250 5240 50  0001 C CNN
 F 1 "GND" H 3250 5340 50  0000 C CNN
 F 2 "" H 3250 5490 50  0001 C CNN
@@
 USB_UART_TX
 $Comp
-L power:+3.3V #PWR?
+L power:+3.3V #PWR01104
 U 1 1 5E6E7B25
 P 5460 880
-F 0 "#PWR?" H 5460 730 50  0001 C CNN
+F 0 "#PWR01104" H 5460 730 50  0001 C CNN
 F 1 "+3.3V" H 5460 1020 50  0000 C CNN
 F 2 "" H 5460 880 50  0001 C CNN
@@
 $EndComp
 $Comp
-L Custom_Library:+3.3VA_MZ #PWR?
+L Custom_Library:+3.3VA_MZ #PWR01102
 U 1 1 5EB1FED1
 P 4810 880
-F 0 "#PWR?" H 4810 730 50  0001 C CNN
+F 0 "#PWR01102" H 4810 730 50  0001 C CNN
 F 1 "+3.3VA_MZ" H 4810 1020 50  0000 C CNN
 F 2 "" H 4810 880 50  0001 C CNN
@@
 $EndComp
 $Comp
-L Custom_Library:GNDA_MZ #PWR?
+L Custom_Library:GNDA_MZ #PWR01103
 U 1 1 5EB20397
 P 4810 6240
-F 0 "#PWR?" H 4810 5990 50  0001 C CNN
+F 0 "#PWR01103" H 4810 5990 50  0001 C CNN
 F 1 "GNDA_MZ" H 4810 6090 50  0000 C CNN
 F 2 "" H 4810 6240 50  0001 C CNN
@@
 VERIFY PINOUT
 $Comp
-L Custom_Library:PIC32MZ0512EFE064T-I_PT U?
+L Custom_Library:PIC32MZ0512EFE064T-I_PT U1101
 U 1 1 5EB2446C
 P 5460 3560
-F 0 "U?" H 7260 1060 50  0000 R CNN
+F 0 "U1101" H 7260 1060 50  0000 R CNN
 F 1 "PIC32MZ0512EFE064T-I_PT" H 5460 3560 50  0000 C CNN
 F 2 "Package_QFP:TQFP-64_10x10mm_P0.5mm" H 5460 3560 50  0001 C CNN
@@
 AR Path="/5EAE2D66/5EB7DAD1" Ref="R?"  Part="1"
 AR Path="/5EAE4A89/5EB7DAD1" Ref="R?"  Part="1"
-AR Path="/5EAE2F23/5EB7DAD1" Ref="R?"  Part="1"
-F 0 "R?" H 9290 2380 50  0000 R CNN
+AR Path="/5EAE2F23/5EB7DAD1" Ref="R1102"  Part="1"
+F 0 "R1102" H 9290 2380 50  0000 R CNN
 F 1 "10k" V 9370 2380 50  0000 C CNN
 F 2 "Resistors_SMD:R_0402" H 9370 2380 50  0001 C CNN
@@
 F 5 "1%" H 9470 2380 50  0000 L CNN "Tolerance"
 F 6 "1/16W" H 9480 2300 50  0000 L CNN "Wattage"
+F 7 "RMCF0402FT10K0CT-ND" H 9370 2380 50  0001 C CNN "Digi-Key PN"
 	1    9370 2380
 	1    0    0    -1
 $EndComp
 $Comp
-L power:+3.3V #PWR?
+L power:+3.3V #PWR01107
 U 1 1 5EB7DAD7
 P 9370 2230
-F 0 "#PWR?" H 9370 2080 50  0001 C CNN
+F 0 "#PWR01107" H 9370 2080 50  0001 C CNN
 F 1 "+3.3V" H 9370 2370 50  0000 C CNN
 F 2 "" H 9370 2230 50  0001 C CNN
@@
 AR Path="/5EAE2D66/5EB7DEAB" Ref="R?"  Part="1"
 AR Path="/5EAE4A89/5EB7DEAB" Ref="R?"  Part="1"
-AR Path="/5EAE2F23/5EB7DEAB" Ref="R?"  Part="1"
-F 0 "R?" H 8700 2380 50  0000 R CNN
+AR Path="/5EAE2F23/5EB7DEAB" Ref="R1101"  Part="1"
+F 0 "R1101" H 8700 2380 50  0000 R CNN
 F 1 "10k" V 8780 2380 50  0000 C CNN
 F 2 "Resistors_SMD:R_0402" H 8780 2380 50  0001 C CNN
@@
 F 5 "1%" H 8880 2380 50  0000 L CNN "Tolerance"
 F 6 "1/16W" H 8890 2300 50  0000 L CNN "Wattage"
+F 7 "RMCF0402FT10K0CT-ND" H 8780 2380 50  0001 C CNN "Digi-Key PN"
 	1    8780 2380
 	1    0    0    -1
 $EndComp
 $Comp
-L power:+3.3V #PWR?
+L power:+3.3V #PWR01106
 U 1 1 5EB7DEB5
 P 8780 2230
-F 0 "#PWR?" H 8780 2080 50  0001 C CNN
+F 0 "#PWR01106" H 8780 2080 50  0001 C CNN
 F 1 "+3.3V" H 8780 2370 50  0000 C CNN
 F 2 "" H 8780 2230 50  0001 C CNN
