File: hdw/Pulse_Oximeter/PIC32MZ_Clocking.sch (KiCad schematic (older format))
At the start: 15 parts

Commit message: Added display circuits
Parts:
- added TP?: TP, Custom Footprints Library:Test_Point, symbol Custom_Library:TP
Connections:
- new net MCU_REFCLK: TP?.1 (TP)
Changed lines of the file:
@@
 EESchema Schematic File Version 4
+LIBS:Pulse_Oximeter-cache
 EELAYER 30 0
 EELAYER END
@@
 	1    0    0    -1
 $EndComp
+$Comp
+L Custom_Library:TP TP?
+U 1 1 5EBAE156
+P 2550 4610
+AR Path="/5C1D5CD8/5EBAE156" Ref="TP?"  Part="1"
+AR Path="/5C1D5C9E/5EBAE156" Ref="TP?"  Part="1"
+AR Path="/5CB6F1ED/5EBAE156" Ref="TP?"  Part="1"
+AR Path="/5E939CFF/5EBAE156" Ref="TP?"  Part="1"
+AR Path="/5E9E0E87/5EBAE156" Ref="TP?"  Part="1"
+AR Path="/5EAE2D66/5EBAE156" Ref="TP?"  Part="1"
+F 0 "TP?" H 2550 4760 50  0000 C CNN
+F 1 "TP" H 2550 4760 50  0001 C CNN
+F 2 "Custom Footprints Library:Test_Point" H 2550 4610 60  0001 C CNN
+F 3 "" H 2550 4610 60  0000 C CNN
+	1    2550 4610
+	1    0    0    -1
+$EndComp
+Text GLabel 2550 4610 3    50   UnSpc ~ 0
+MCU_REFCLK
 $EndSCHEMATC

Commit message: few sch additions
Connections:
- net MCU_POSC renamed PIC32MZ_POSC_EC
- net MCU_POSC_Enable renamed PIC32MZ_POSC_EC_Enable
- net MCU_REFCLK renamed PIC32MZ_REFCLK1
- net MCU_SOSC renamed PIC32MZ_SOSC
Other:
- moved on the sheet: TP?
Changed lines of the file:
@@
 $EndComp
 Text GLabel 6810 2700 2    50   Output ~ 0
-MCU_POSC
+PIC32MZ_POSC_EC
 $Comp
 L Custom_Library:R_Custom R?
@@
 	4660 2700 4960 2700
 Text GLabel 4660 2700 0    50   Input ~ 0
-MCU_POSC_Enable
+PIC32MZ_POSC_EC_Enable
 $Comp
 L power:GND #PWR?
@@
 $EndComp
 Text GLabel 6810 5190 2    50   Output ~ 0
-MCU_SOSC
+PIC32MZ_SOSC
 $Comp
 L Custom_Library:R_Custom R?
@@
 L Custom_Library:TP TP?
 U 1 1 5EBAE156
-P 2550 4610
+P 2460 4680
 AR Path="/5C1D5CD8/5EBAE156" Ref="TP?"  Part="1"
 AR Path="/5C1D5C9E/5EBAE156" Ref="TP?"  Part="1"
@@
 AR Path="/5E9E0E87/5EBAE156" Ref="TP?"  Part="1"
 AR Path="/5EAE2D66/5EBAE156" Ref="TP?"  Part="1"
-F 0 "TP?" H 2550 4760 50  0000 C CNN
-F 1 "TP" H 2550 4760 50  0001 C CNN
-F 2 "Custom Footprints Library:Test_Point" H 2550 4610 60  0001 C CNN
-F 3 "" H 2550 4610 60  0000 C CNN
-	1    2550 4610
-	1    0    0    -1
-$EndComp
-Text GLabel 2550 4610 3    50   UnSpc ~ 0
-MCU_REFCLK
+AR Path="/5EAE2F15/5EBAE156" Ref="TP?"  Part="1"
+F 0 "TP?" V 2460 4830 50  0000 L CNN
+F 1 "TP" H 2460 4830 50  0001 C CNN
+F 2 "Custom Footprints Library:Test_Point" H 2460 4680 60  0001 C CNN
+F 3 "" H 2460 4680 60  0000 C CNN
+	1    2460 4680
+	0    1    1    0
+$EndComp
+Text GLabel 2460 4680 0    50   UnSpc ~ 0
+PIC32MZ_REFCLK1
 $EndSCHEMATC

Commit message: More sch work
Parts:
- removed R? (x2): 100, Resistors_SMD:R_0402, symbol Custom_Library:R_Custom
- added R? (x2): 10, Resistors_SMD:R_0402, symbol Custom_Library:R_Custom
Connections:
- net PIC32MZ_POSC_EC: now also R?.2
- net PIC32MZ_SOSC: now also R?.2
- net at X?.3 (OUT): now also R?.1 (x2)
Other:
- moved on the sheet: TP?
Changed lines of the file:
@@
 	6560 2700 6560 2780
 Connection ~ 6560 2700
-$Comp
-L Custom_Library:R_Custom R?
-U 1 1 5E024C29
-P 6110 2700
-AR Path="/5BAAE2B6/5E024C29" Ref="R?"  Part="1"
-AR Path="/5BB6CF6D/5E024C29" Ref="R?"  Part="1"
-AR Path="/5BBE424C/5E024C29" Ref="R?"  Part="1"
-AR Path="/5BAAE1DC/5E024C29" Ref="R?"  Part="1"
-AR Path="/5CAD2DA3/5E024C29" Ref="R?"  Part="1"
-AR Path="/5E01BCC3/5E024C29" Ref="R?"  Part="1"
-AR Path="/5E697952/5E024C29" Ref="R?"  Part="1"
-AR Path="/5EAE2F15/5E024C29" Ref="R?"  Part="1"
-F 0 "R?" V 6070 2560 50  0000 R CNN
-F 1 "100" V 6110 2700 50  0000 C CNN
-F 2 "Resistors_SMD:R_0402" H 6110 2700 50  0001 C CNN
-F 3 "" H 6110 2700 50  0001 C CNN
-F 4 "0402" V 6210 2700 50  0001 C CNN "display_footprint"
-F 5 "1%" V 6310 2700 50  0001 C CNN "Tolerance"
-F 6 "1/16W" V 6410 2700 50  0001 C CNN "Wattage"
-F 7 "541-100LCT-ND" H 6410 3100 60  0001 C CNN "Digi-Key PN"
-	1    6110 2700
-	0    -1   1    0
-$EndComp
 Wire Wire Line
 	5960 2700 5810 2700
@@
 	6560 5190 6560 5270
 Connection ~ 6560 5190
-$Comp
-L Custom_Library:R_Custom R?
-U 1 1 5E0562C1
-P 6110 5190
-AR Path="/5BAAE2B6/5E0562C1" Ref="R?"  Part="1"
-AR Path="/5BB6CF6D/5E0562C1" Ref="R?"  Part="1"
-AR Path="/5BBE424C/5E0562C1" Ref="R?"  Part="1"
-AR Path="/5BAAE1DC/5E0562C1" Ref="R?"  Part="1"
-AR Path="/5CAD2DA3/5E0562C1" Ref="R?"  Part="1"
-AR Path="/5E01BCC3/5E0562C1" Ref="R?"  Part="1"
-AR Path="/5E697952/5E0562C1" Ref="R?"  Part="1"
-AR Path="/5EAE2F15/5E0562C1" Ref="R?"  Part="1"
-F 0 "R?" V 6070 5050 50  0000 R CNN
-F 1 "100" V 6110 5190 50  0000 C CNN
-F 2 "Resistors_SMD:R_0402" H 6110 5190 50  0001 C CNN
-F 3 "" H 6110 5190 50  0001 C CNN
-F 4 "0402" V 6210 5190 50  0001 C CNN "display_footprint"
-F 5 "1%" V 6310 5190 50  0001 C CNN "Tolerance"
-F 6 "1/16W" V 6410 5190 50  0001 C CNN "Wattage"
-F 7 "541-100LCT-ND" H 6410 5590 60  0001 C CNN "Digi-Key PN"
-	1    6110 5190
-	0    -1   1    0
-$EndComp
 Wire Wire Line
 	5960 5190 5810 5190
@@
 L Custom_Library:TP TP?
 U 1 1 5EBAE156
-P 2460 4680
+P 3170 5190
 AR Path="/5C1D5CD8/5EBAE156" Ref="TP?"  Part="1"
 AR Path="/5C1D5C9E/5EBAE156" Ref="TP?"  Part="1"
@@
 AR Path="/5EAE2D66/5EBAE156" Ref="TP?"  Part="1"
 AR Path="/5EAE2F15/5EBAE156" Ref="TP?"  Part="1"
-F 0 "TP?" V 2460 4830 50  0000 L CNN
-F 1 "TP" H 2460 4830 50  0001 C CNN
-F 2 "Custom Footprints Library:Test_Point" H 2460 4680 60  0001 C CNN
-F 3 "" H 2460 4680 60  0000 C CNN
-	1    2460 4680
+F 0 "TP?" V 3170 5340 50  0000 L CNN
+F 1 "TP" H 3170 5340 50  0001 C CNN
+F 2 "Custom Footprints Library:Test_Point" H 3170 5190 60  0001 C CNN
+F 3 "" H 3170 5190 60  0000 C CNN
+	1    3170 5190
 	0    1    1    0
 $EndComp
-Text GLabel 2460 4680 0    50   UnSpc ~ 0
+Text GLabel 3170 5190 0    50   UnSpc ~ 0
 PIC32MZ_REFCLK1
+$Comp
+L Custom_Library:R_Custom R?
+U 1 1 5EB9D3C3
+P 6110 5190
+AR Path="/5EAE2EF2/5EB9D3C3" Ref="R?"  Part="1"
+AR Path="/5EAE2F15/5EB9D3C3" Ref="R?"  Part="1"
+F 0 "R?" V 6010 5190 50  0000 C CNN
+F 1 "10" V 6110 5190 50  0000 C CNN
+F 2 "Resistors_SMD:R_0402" H 6110 5190 50  0001 C CNN
+F 3 "" H 6110 5190 50  0001 C CNN
+F 4 "0402" V 6210 5190 50  0000 C CNN "display_footprint"
+F 5 "1%" V 6310 5190 50  0000 C CNN "Tolerance"
+F 6 "1/16W" V 6410 5190 50  0000 C CNN "Wattage"
+F 7 "541-3964-1-ND" H 6410 5590 60  0001 C CNN "Digi-Key PN"
+	1    6110 5190
+	0    -1   -1   0
+$EndComp
+$Comp
+L Custom_Library:R_Custom R?
+U 1 1 5EB9DF29
+P 6110 2700
+AR Path="/5EAE2EF2/5EB9DF29" Ref="R?"  Part="1"
+AR Path="/5EAE2F15/5EB9DF29" Ref="R?"  Part="1"
+F 0 "R?" V 6010 2700 50  0000 C CNN
+F 1 "10" V 6110 2700 50  0000 C CNN
+F 2 "Resistors_SMD:R_0402" H 6110 2700 50  0001 C CNN
+F 3 "" H 6110 2700 50  0001 C CNN
+F 4 "0402" V 6210 2700 50  0000 C CNN "display_footprint"
+F 5 "1%" V 6310 2700 50  0000 C CNN "Tolerance"
+F 6 "1/16W" V 6410 2700 50  0000 C CNN "Wattage"
+F 7 "541-3964-1-ND" H 6410 3100 60  0001 C CNN "Digi-Key PN"
+	1    6110 2700
+	0    -1   -1   0
+$EndComp
 $EndSCHEMATC

Commit message: Added I2C to PIC32MZ
Parts:
- added R?: 10k, Resistors_SMD:R_0402, symbol Custom_Library:R_Custom
Connections:
- net GND: now also R?.2
- net PIC32MZ_REFCLK1: now also R?.1
Other:
- moved on the sheet: TP?
Changed lines of the file:
@@
 L Custom_Library:TP TP?
 U 1 1 5EBAE156
-P 3170 5190
+P 3500 5190
 AR Path="/5C1D5CD8/5EBAE156" Ref="TP?"  Part="1"
 AR Path="/5C1D5C9E/5EBAE156" Ref="TP?"  Part="1"
@@
 AR Path="/5EAE2D66/5EBAE156" Ref="TP?"  Part="1"
 AR Path="/5EAE2F15/5EBAE156" Ref="TP?"  Part="1"
-F 0 "TP?" V 3170 5340 50  0000 L CNN
-F 1 "TP" H 3170 5340 50  0001 C CNN
-F 2 "Custom Footprints Library:Test_Point" H 3170 5190 60  0001 C CNN
-F 3 "" H 3170 5190 60  0000 C CNN
-	1    3170 5190
+F 0 "TP?" V 3500 5340 50  0000 L CNN
+F 1 "TP" H 3500 5340 50  0001 C CNN
+F 2 "Custom Footprints Library:Test_Point" H 3500 5190 60  0001 C CNN
+F 3 "" H 3500 5190 60  0000 C CNN
+	1    3500 5190
 	0    1    1    0
 $EndComp
-Text GLabel 3170 5190 0    50   UnSpc ~ 0
+Text GLabel 3170 5190 0    50   Input ~ 0
 PIC32MZ_REFCLK1
 $Comp
@@
 	0    -1   -1   0
 $EndComp
+$Comp
+L Custom_Library:R_Custom R?
+U 1 1 5EB723DB
+P 3420 5420
+AR Path="/5BAAE1F3/5EB723DB" Ref="R?"  Part="1"
+AR Path="/5BAAE1DC/5EB723DB" Ref="R?"  Part="1"
+AR Path="/5BAAE16C/5EB723DB" Ref="R?"  Part="1"
+AR Path="/5BB844FD/5EB723DB" Ref="R?"  Part="1"
+AR Path="/5BF346B3/5EB723DB" Ref="R?"  Part="1"
+AR Path="/5CAD2D97/5EB723DB" Ref="R?"  Part="1"
+AR Path="/5CB7A8BC/5EB723DB" Ref="R?"  Part="1"
+AR Path="/5E01BCC3/5EB723DB" Ref="R?"  Part="1"
+AR Path="/5E697952/5EB723DB" Ref="R?"  Part="1"
+AR Path="/5EAE2F15/5EB723DB" Ref="R?"  Part="1"
+F 0 "R?" H 3360 5420 50  0000 R CNN
+F 1 "10k" V 3420 5420 50  0000 C CNN
+F 2 "Resistors_SMD:R_0402" H 3420 5420 50  0001 C CNN
+F 3 "" H 3420 5420 50  0001 C CNN
+F 4 "0402" H 3490 5500 50  0000 L CNN "display_footprint"
+F 5 "1%" H 3490 5420 50  0000 L CNN "Tolerance"
+F 6 "1/16W" H 3490 5350 50  0000 L CNN "Wattage"
+F 7 "RMCF0402FT10K0CT-ND" H 3420 5420 50  0001 C CNN "Digi-Key PN"
+	1    3420 5420
+	-1   0    0    -1
+$EndComp
+Wire Wire Line
+	3500 5190 3420 5190
+Wire Wire Line
+	3420 5190 3420 5270
+Wire Wire Line
+	3420 5190 3170 5190
+Connection ~ 3420 5190
+$Comp
+L power:GND #PWR?
+U 1 1 5EB74E9C
+P 3420 5570
+F 0 "#PWR?" H 3420 5320 50  0001 C CNN
+F 1 "GND" H 3420 5420 50  0000 C CNN
+F 2 "" H 3420 5570 50  0001 C CNN
+F 3 "" H 3420 5570 50  0001 C CNN
+	1    3420 5570
+	1    0    0    -1
+$EndComp
 $EndSCHEMATC

Commit message: Added more stuff to sch
Parts:
- removed C?: 0.1uF, Capacitors_SMD:C_0402, symbol Custom_Library:C_Custom
- removed C?: 1nF, Capacitors_SMD:C_0402, symbol Custom_Library:C_Custom
- removed C?: 10nF, Capacitors_SMD:C_0402, symbol Custom_Library:C_Custom
- removed L?: 600R 0.5A, Inductors_SMD:L_0402, symbol Device:Ferrite_Bead
- removed R?: 10k, Resistors_SMD:R_0402, symbol Custom_Library:R_Custom
- removed R?: 10, Resistors_SMD:R_0402, symbol Custom_Library:R_Custom
- removed X?: ECS-327KE, Custom Footprints Library:ECS-327KE, symbol Custom_Library:ECS-327KE
- added C?: 10uF, Capacitors_SMD:C_0402, symbol Custom_Library:C_Custom
Connections:
- net GND: now also C?.2
- net at C?.1, C?.1, C?.1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: now also C?.1
Other:
- moved on the sheet: R?, TP?

Commit message: Added SD card slot and backup RTC
Parts:
- removed C?: 10uF, Capacitors_SMD:C_0402, symbol Custom_Library:C_Custom
- removed R?: 10k, Resistors_SMD:R_0402, symbol Custom_Library:R_Custom
- removed R?: 10, Resistors_SMD:R_0402, symbol Custom_Library:R_Custom
- removed TP?: TP, Custom Footprints Library:Test_Point, symbol Custom_Library:TP
- added C702: 0.1uF, Capacitors_SMD:C_0402, symbol Custom_Library:C_Custom
- added C704: 10nF, Capacitors_SMD:C_0402, symbol Custom_Library:C_Custom
- added C706: 1nF, Capacitors_SMD:C_0402, symbol Custom_Library:C_Custom
- added L702: 600R 0.5A, Inductors_SMD:L_0402, symbol Device:Ferrite_Bead
- added R702, R703: 100, Resistors_SMD:R_0402, symbol Custom_Library:R_Custom
- added R705: 10k, Resistors_SMD:R_0402, symbol Custom_Library:R_Custom
- added X702: ECS-327KE, Custom Footprints Library:ECS-327KE, symbol Custom_Library:ECS-327KE
- gave numbers to parts that had none: 7
Connections:
- net +3V3: now also L702.2
- net GND: now also C702.2, C704.2, C706.2, R705.2, X702.2 (GND)
- net PIC32MZ_POSC_EC: now also R702.2
- net at X701.3 (OUT): now also R702.1
- new net: R703.1, X702.3 (OUT)
- new net: C702.1, C704.1, C706.1, L702.1, X702.1 (EN), X702.4 (Vdd)
- new net PIC32MZ_SOSC: R703.2, R705.1

Commit message: Added mech sheet, more complicated bullshit you dont need
Parts:
- renumbered C701 to C?, C705 to C?, C703 to C?, C702 to C?, C706 to C?, C704 to C?, L701 to L?, L702 to L?, R704 to R?, R702 to R?, R701 to R?, R705 to R?, R703 to R?, X701 to X?, X702 to X?

Commit message: Added digikey pn's, footprints
Parts:
- gave numbers to parts that had none: 15
Changed lines of the file:
@@
 encoding utf-8
 Sheet 10 23
-Title ""
-Date ""
-Rev ""
-Comp ""
+Title "Pulse Oximeter"
+Date "2019-01-03"
+Rev "A"
+Comp "Drew Maatman"
 Comment1 ""
 Comment2 ""
@@
 $EndDescr
 $Comp
-L Oscillator:ASE-xxxMHz X?
+L Oscillator:ASE-xxxMHz X1001
 U 1 1 5E015C3C
 P 5510 2700
-F 0 "X?" H 5310 2950 50  0000 L CNN
+F 0 "X1001" H 5310 2950 50  0000 L CNN
 F 1 "ASE-8.000MHz" H 5560 2450 50  0000 L CNN
 F 2 "Oscillator:Oscillator_SMD_Abracon_ASE-4Pin_3.2x2.5mm" H 6210 2350 50  0001 C CNN
@@
 $EndComp
 $Comp
-L power:GND #PWR?
+L power:GND #PWR01004
 U 1 1 5E01A3D9
 P 5510 3000
-F 0 "#PWR?" H 5510 2750 50  0001 C CNN
+F 0 "#PWR01004" H 5510 2750 50  0001 C CNN
 F 1 "GND" H 5510 2850 50  0000 C CNN
 F 2 "" H 5510 3000 50  0001 C CNN
@@
 AR Path="/5E01BCC3/5E021EF5" Ref="R?"  Part="1"
 AR Path="/5E697952/5E021EF5" Ref="R?"  Part="1"
-AR Path="/5EAE2F15/5E021EF5" Ref="R?"  Part="1"
-F 0 "R?" H 6500 2930 50  0000 R CNN
+AR Path="/5EAE2F15/5E021EF5" Ref="R1004"  Part="1"
+F 0 "R1004" H 6500 2930 50  0000 R CNN
 F 1 "10k" V 6560 2930 50  0000 C CNN
 F 2 "Resistors_SMD:R_0402" H 6560 2930 50  0001 C CNN
@@
 AR Path="/5E01BCC3/5E021EFB" Ref="#PWR?"  Part="1"
 AR Path="/5E697952/5E021EFB" Ref="#PWR?"  Part="1"
-AR Path="/5EAE2F15/5E021EFB" Ref="#PWR?"  Part="1"
-F 0 "#PWR?" H 6560 2830 50  0001 C CNN
+AR Path="/5EAE2F15/5E021EFB" Ref="#PWR01008"  Part="1"
+F 0 "#PWR01008" H 6560 2830 50  0001 C CNN
 F 1 "GND" H 6560 2930 50  0000 C CNN
 F 2 "" H 6560 3080 50  0001 C CNN
@@
 AR Path="/5E01BCC3/5E024C29" Ref="R?"  Part="1"
 AR Path="/5E697952/5E024C29" Ref="R?"  Part="1"
-AR Path="/5EAE2F15/5E024C29" Ref="R?"  Part="1"
-F 0 "R?" V 6070 2560 50  0000 R CNN
+AR Path="/5EAE2F15/5E024C29" Ref="R1002"  Part="1"
+F 0 "R1002" V 6070 2560 50  0000 R CNN
 F 1 "100" V 6110 2700 50  0000 C CNN
 F 2 "Resistors_SMD:R_0402" H 6110 2700 50  0001 C CNN
@@
 AR Path="/5E01BCC3/5E0269C4" Ref="R?"  Part="1"
 AR Path="/5E697952/5E0269C4" Ref="R?"  Part="1"
-AR Path="/5EAE2F15/5E0269C4" Ref="R?"  Part="1"
-F 0 "R?" H 4900 2930 50  0000 R CNN
+AR Path="/5EAE2F15/5E0269C4" Ref="R1001"  Part="1"
+F 0 "R1001" H 4900 2930 50  0000 R CNN
 F 1 "10k" V 4960 2930 50  0000 C CNN
 F 2 "Resistors_SMD:R_0402" H 4960 2930 50  0001 C CNN
@@
 AR Path="/5E01BCC3/5E0269CA" Ref="#PWR?"  Part="1"
 AR Path="/5E697952/5E0269CA" Ref="#PWR?"  Part="1"
-AR Path="/5EAE2F15/5E0269CA" Ref="#PWR?"  Part="1"
-F 0 "#PWR?" H 4960 2830 50  0001 C CNN
+AR Path="/5EAE2F15/5E0269CA" Ref="#PWR01003"  Part="1"
+F 0 "#PWR01003" H 4960 2830 50  0001 C CNN
 F 1 "GND" H 4960 2930 50  0000 C CNN
 F 2 "" H 4960 3080 50  0001 C CNN
@@
 AR Path="/5E01BCC3/5E03ADCE" Ref="#PWR?"  Part="1"
 AR Path="/5E697952/5E03ADCE" Ref="#PWR?"  Part="1"
-AR Path="/5EAE2F15/5E03ADCE" Ref="#PWR?"  Part="1"
-F 0 "#PWR?" H 6400 2050 50  0001 C CNN
+AR Path="/5EAE2F15/5E03ADCE" Ref="#PWR01006"  Part="1"
+F 0 "#PWR01006" H 6400 2050 50  0001 C CNN
 F 1 "GND" H 6400 2150 50  0000 C CNN
 F 2 "" H 6400 2300 50  0000 C CNN
@@
 AR Path="/5E01BCC3/5E03ADD8" Ref="C?"  Part="1"
 AR Path="/5E697952/5E03ADD8" Ref="C?"  Part="1"
-AR Path="/5EAE2F15/5E03ADD8" Ref="C?"  Part="1"
-F 0 "C?" H 6105 2170 50  0000 L CNN
+AR Path="/5EAE2F15/5E03ADD8" Ref="C1001"  Part="1"
+F 0 "C1001" H 6105 2170 50  0000 L CNN
 F 1 "0.1uF" H 6105 1970 50  0000 L CNN
 F 2 "Capacitors_SMD:C_0402" H 6118 1920 50  0001 C CNN
@@
 AR Path="/5E01BCC3/5E03ADE2" Ref="C?"  Part="1"
 AR Path="/5E697952/5E03ADE2" Ref="C?"  Part="1"
-AR Path="/5EAE2F15/5E03ADE2" Ref="C?"  Part="1"
-F 0 "C?" H 6745 2170 50  0000 L CNN
+AR Path="/5EAE2F15/5E03ADE2" Ref="C1005"  Part="1"
+F 0 "C1005" H 6745 2170 50  0000 L CNN
 F 1 "1nF" H 6745 1970 50  0000 L CNN
 F 2 "Capacitors_SMD:C_0402" H 6758 1920 50  0001 C CNN
@@
 AR Path="/5E01BCC3/5E03ADEC" Ref="C?"  Part="1"
 AR Path="/5E697952/5E03ADEC" Ref="C?"  Part="1"
-AR Path="/5EAE2F15/5E03ADEC" Ref="C?"  Part="1"
-F 0 "C?" H 6425 2170 50  0000 L CNN
+AR Path="/5EAE2F15/5E03ADEC" Ref="C1003"  Part="1"
+F 0 "C1003" H 6425 2170 50  0000 L CNN
 F 1 "10nF" H 6425 1970 50  0000 L CNN
 F 2 "Capacitors_SMD:C_0402" H 6438 1920 50  0001 C CNN
@@
 AR Path="/5E01BCC3/5E053473" Ref="L?"  Part="1"
 AR Path="/5E697952/5E053473" Ref="L?"  Part="1"
-AR Path="/5EAE2F15/5E053473" Ref="L?"  Part="1"
-F 0 "L?" V 4890 1825 50  0000 C CNN
+AR Path="/5EAE2F15/5E053473" Ref="L1001"  Part="1"
+F 0 "L1001" V 4890 1825 50  0000 C CNN
 F 1 "600R 0.5A" V 5190 1800 50  0000 C CNN
 F 2 "Inductors_SMD:L_0402" V 4970 1800 50  0001 C CNN
@@
 	4530 1800 4890 1800
 $Comp
-L power:GND #PWR?
+L power:GND #PWR01005
 U 1 1 5E056297
 P 5510 5490
-F 0 "#PWR?" H 5510 5240 50  0001 C CNN
+F 0 "#PWR01005" H 5510 5240 50  0001 C CNN
 F 1 "GND" H 5510 5340 50  0000 C CNN
 F 2 "" H 5510 5490 50  0001 C CNN
@@
 AR Path="/5E01BCC3/5E0562A6" Ref="R?"  Part="1"
 AR Path="/5E697952/5E0562A6" Ref="R?"  Part="1"
-AR Path="/5EAE2F15/5E0562A6" Ref="R?"  Part="1"
-F 0 "R?" H 6500 5420 50  0000 R CNN
+AR Path="/5EAE2F15/5E0562A6" Ref="R1005"  Part="1"
+F 0 "R1005" H 6500 5420 50  0000 R CNN
 F 1 "10k" V 6560 5420 50  0000 C CNN
 F 2 "Resistors_SMD:R_0402" H 6560 5420 50  0001 C CNN
@@
 AR Path="/5E01BCC3/5E0562B0" Ref="#PWR?"  Part="1"
 AR Path="/5E697952/5E0562B0" Ref="#PWR?"  Part="1"
-AR Path="/5EAE2F15/5E0562B0" Ref="#PWR?"  Part="1"
-F 0 "#PWR?" H 6560 5320 50  0001 C CNN
+AR Path="/5EAE2F15/5E0562B0" Ref="#PWR01009"  Part="1"
+F 0 "#PWR01009" H 6560 5320 50  0001 C CNN
 F 1 "GND" H 6560 5420 50  0000 C CNN
 F 2 "" H 6560 5570 50  0001 C CNN
@@
 AR Path="/5E01BCC3/5E0562C1" Ref="R?"  Part="1"
 AR Path="/5E697952/5E0562C1" Ref="R?"  Part="1"
-AR Path="/5EAE2F15/5E0562C1" Ref="R?"  Part="1"
-F 0 "R?" V 6070 5050 50  0000 R CNN
+AR Path="/5EAE2F15/5E0562C1" Ref="R1003"  Part="1"
+F 0 "R1003" V 6070 5050 50  0000 R CNN
 F 1 "100" V 6110 5190 50  0000 C CNN
 F 2 "Resistors_SMD:R_0402" H 6110 5190 50  0001 C CNN
@@
 AR Path="/5E01BCC3/5E0562EA" Ref="#PWR?"  Part="1"
 AR Path="/5E697952/5E0562EA" Ref="#PWR?"  Part="1"
-AR Path="/5EAE2F15/5E0562EA" Ref="#PWR?"  Part="1"
-F 0 "#PWR?" H 6400 4540 50  0001 C CNN
+AR Path="/5EAE2F15/5E0562EA" Ref="#PWR01007"  Part="1"
+F 0 "#PWR01007" H 6400 4540 50  0001 C CNN
 F 1 "GND" H 6400 4640 50  0000 C CNN
 F 2 "" H 6400 4790 50  0000 C CNN
@@
 AR Path="/5E01BCC3/5E0562F8" Ref="C?"  Part="1"
 AR Path="/5E697952/5E0562F8" Ref="C?"  Part="1"
-AR Path="/5EAE2F15/5E0562F8" Ref="C?"  Part="1"
-F 0 "C?" H 6105 4660 50  0000 L CNN
+AR Path="/5EAE2F15/5E0562F8" Ref="C1002"  Part="1"
+F 0 "C1002" H 6105 4660 50  0000 L CNN
 F 1 "0.1uF" H 6105 4460 50  0000 L CNN
 F 2 "Capacitors_SMD:C_0402" H 6118 4410 50  0001 C CNN
@@
 AR Path="/5E01BCC3/5E056306" Ref="C?"  Part="1"
 AR Path="/5E697952/5E056306" Ref="C?"  Part="1"
-AR Path="/5EAE2F15/5E056306" Ref="C?"  Part="1"
-F 0 "C?" H 6745 4660 50  0000 L CNN
+AR Path="/5EAE2F15/5E056306" Ref="C1006"  Part="1"
+F 0 "C1006" H 6745 4660 50  0000 L CNN
 F 1 "1nF" H 6745 4460 50  0000 L CNN
 F 2 "Capacitors_SMD:C_0402" H 6758 4410 50  0001 C CNN
@@
 AR Path="/5E01BCC3/5E056314" Ref="C?"  Part="1"
 AR Path="/5E697952/5E056314" Ref="C?"  Part="1"
-AR Path="/5EAE2F15/5E056314" Ref="C?"  Part="1"
-F 0 "C?" H 6425 4660 50  0000 L CNN
+AR Path="/5EAE2F15/5E056314" Ref="C1004"  Part="1"
+F 0 "C1004" H 6425 4660 50  0000 L CNN
 F 1 "10nF" H 6425 4460 50  0000 L CNN
 F 2 "Capacitors_SMD:C_0402" H 6438 4410 50  0001 C CNN
@@
 AR Path="/5E01BCC3/5E05632C" Ref="L?"  Part="1"
 AR Path="/5E697952/5E05632C" Ref="L?"  Part="1"
-AR Path="/5EAE2F15/5E05632C" Ref="L?"  Part="1"
-F 0 "L?" V 4890 4315 50  0000 C CNN
+AR Path="/5EAE2F15/5E05632C" Ref="L1002"  Part="1"
+F 0 "L1002" V 4890 4315 50  0000 C CNN
 F 1 "600R 0.5A" V 5190 4290 50  0000 C CNN
 F 2 "Inductors_SMD:L_0402" V 4970 4290 50  0001 C CNN
@@
 	4530 4290 4890 4290
 $Comp
-L Custom_Library:ECS-327KE X?
+L Custom_Library:ECS-327KE X1002
 U 1 1 5E05D8E0
 P 5510 5190
-F 0 "X?" H 5310 5440 50  0000 L CNN
+F 0 "X1002" H 5310 5440 50  0000 L CNN
 F 1 "ECS-327KE" H 5560 4940 50  0000 L CNN
 F 2 "Custom Footprints Library:ECS-327KE" H 6210 4840 50  0001 C CNN
@@
 	5510 4750 5510 4890
 $Comp
-L power:PWR_FLAG #FLG?
+L power:PWR_FLAG #FLG01002
 U 1 1 5E43B375
 P 5510 4220
-F 0 "#FLG?" H 5510 4295 50  0001 C CNN
+F 0 "#FLG01002" H 5510 4295 50  0001 C CNN
 F 1 "PWR_FLAG" H 5510 4370 50  0000 C CNN
 F 2 "" H 5510 4220 50  0001 C CNN
@@
 	5510 4220 5510 4290
 $Comp
-L power:PWR_FLAG #FLG?
+L power:PWR_FLAG #FLG01001
 U 1 1 5E43F288
 P 5510 1730
-F 0 "#FLG?" H 5510 1805 50  0001 C CNN
+F 0 "#FLG01001" H 5510 1805 50  0001 C CNN
 F 1 "PWR_FLAG" H 5510 1880 50  0000 C CNN
 F 2 "" H 5510 1730 50  0001 C CNN
@@
 	5510 1730 5510 1800
 $Comp
-L power:+3.3V #PWR?
+L power:+3.3V #PWR01001
 U 1 1 5E6E8CA9
 P 4530 1720
-F 0 "#PWR?" H 4530 1570 50  0001 C CNN
+F 0 "#PWR01001" H 4530 1570 50  0001 C CNN
 F 1 "+3.3V" H 4530 1860 50  0000 C CNN
 F 2 "" H 4530 1720 50  0001 C CNN
@@
 $EndComp
 $Comp
-L power:+3.3V #PWR?
+L power:+3.3V #PWR01002
 U 1 1 5E6E96AD
 P 4530 4210
-F 0 "#PWR?" H 4530 4060 50  0001 C CNN
+F 0 "#PWR01002" H 4530 4060 50  0001 C CNN
 F 1 "+3.3V" H 4530 4350 50  0000 C CNN
 F 2 "" H 4530 4210 50  0001 C CNN
