File: hdw/Pulse_Oximeter/POS1P8_Power_Supply.sch (KiCad schematic (older format))
At the start: 0 parts

Commit message: Continued schematic development
Parts:
- added C? (x2): 0.1uF, Capacitors_SMD:C_0402, symbol Custom_Library:C_Custom
- added C? (x3): C_Custom, symbol Custom_Library:C_Custom
- added R? (x2): 10k, Resistors_SMD:R_0402, symbol Custom_Library:R_Custom
- added R? (x2): 0.02, Resistors_SMD:R_0612, symbol Custom_Library:R_Custom
- added R? (x4): 10, Resistors_SMD:R_0603, symbol Custom_Library:R_Custom
- added R? (x2): R, Resistors_SMD:R_0402, symbol Custom_Library:R_Custom
- added TP?: TP, Custom Footprints Library:Test_Point, symbol Custom_Library:TP
- added U?: TPS7A91, Package_DFN_QFN:Texas_S-PDSO-N10_EP1.2x2mm, symbol Custom_Library:TPS7A91
Connections:
- new net: C?.1, U?.8 (NR/SS)
- new net: C?.1, C?.1, R?.1, R?.2, U?.1 (OUT), U?.2 (OUT)
- new net: C?.1, R?.2, R?.2, U?.10 (IN), U?.9 (IN)
- new net: R?.1, R?.2, U?.3 (FB)
- new net +1.8V: C?.1, R?.1, R?.2, R?.2, TP?.1 (TP)
- new net +3V3: R?.1, R?.1, R?.2, U?.6 (SS_CTRL)
- new net GND: C?.2, C?.2, C?.2, C?.2, C?.2, R?.2, R?.2, U?.11 (GND), U?.4 (GND)
- new net OS1P8_PGOOD: R?.2, U?.5 (PG)
- new net POS1P8_RUN: R?.1, U?.7 (EN)
- new net POS1P8_SNS_IN+: R?.1
- new net POS1P8_SNS_IN-: R?.1
- new net POS1P8_SNS_OUT+: R?.1
- new net POS1P8_SNS_OUT-: R?.1
Other:
- note removed: "Probably a small footprint LDO"

Commit message: few sch additions
Parts:
- removed C? (x3): C_Custom, symbol Custom_Library:C_Custom
- added C? (x3): 10uF, Capacitors_SMD:C_0402, symbol Custom_Library:C_Custom
- R?: value R -> 1.87k
- R?: value R -> 1.5k
Connections:
- net GND: now also C?.2, C?.2, C?.2
- net at R?.1, R?.2, U?.1 (OUT)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: now also C?.1, C?.1
- net at R?.2, R?.2, U?.10 (IN)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: now also C?.1
Changed lines of the file:
@@
 	4360 4580 4360 4660
-$Comp
-L Custom_Library:C_Custom C?
-U 1 1 5EBB926B
-P 5780 3510
-F 0 "C?" H 5805 3610 50  0000 L CNN
-F 1 "C_Custom" H 5805 3410 50  0000 L CNN
-F 2 "" H 5818 3360 50  0001 C CNN
-F 3 "" H 5805 3610 50  0001 C CNN
-F 4 "Foot" H 5630 3610 50  0000 R CNN "display_footprint"
-F 5 "V" H 5630 3510 50  0000 R CNN "Voltage"
-F 6 "Er" H 5630 3410 50  0000 R CNN "Dielectric"
-F 7 "PN" H 6205 4010 60  0001 C CNN "Digi-Key PN"
-	1    5780 3510
-	1    0    0    -1
-$EndComp
-$Comp
-L Custom_Library:C_Custom C?
-U 1 1 5EBBA073
-P 6430 3510
-F 0 "C?" H 6455 3610 50  0000 L CNN
-F 1 "C_Custom" H 6455 3410 50  0000 L CNN
-F 2 "" H 6468 3360 50  0001 C CNN
-F 3 "" H 6455 3610 50  0001 C CNN
-F 4 "Foot" H 6280 3610 50  0000 R CNN "display_footprint"
-F 5 "V" H 6280 3510 50  0000 R CNN "Voltage"
-F 6 "Er" H 6280 3410 50  0000 R CNN "Dielectric"
-F 7 "PN" H 6855 4010 60  0001 C CNN "Digi-Key PN"
-	1    6430 3510
-	1    0    0    -1
-$EndComp
 $Comp
 L Custom_Library:TPS7A91 U?
@@
 $EndComp
 $Comp
-L Custom_Library:C_Custom C?
-U 1 1 5EBC7C91
-P 4360 3510
-F 0 "C?" H 4385 3610 50  0000 L CNN
-F 1 "C_Custom" H 4385 3410 50  0000 L CNN
-F 2 "" H 4398 3360 50  0001 C CNN
-F 3 "" H 4385 3610 50  0001 C CNN
-F 4 "Foot" H 4210 3610 50  0000 R CNN "display_footprint"
-F 5 "V" H 4210 3510 50  0000 R CNN "Voltage"
-F 6 "Er" H 4210 3410 50  0000 R CNN "Dielectric"
-F 7 "PN" H 4785 4010 60  0001 C CNN "Digi-Key PN"
-	1    4360 3510
-	1    0    0    -1
-$EndComp
-$Comp
 L Custom_Library:R_Custom R?
 U 1 1 5EBC99AE
@@
 Wire Wire Line
 	3040 3980 3040 4060
-$Comp
-L power:+3.3V #PWR?
-U 1 1 5EBCCCA8
-P 3040 3200
-F 0 "#PWR?" H 3040 3050 50  0001 C CNN
-F 1 "+3.3V" H 3040 3340 50  0000 C CNN
-F 2 "" H 3040 3200 50  0001 C CNN
-F 3 "" H 3040 3200 50  0001 C CNN
-	1    3040 3200
-	1    0    0    -1
-$EndComp
-Wire Wire Line
-	3040 3200 3040 3360
 Text GLabel 2960 3880 0    50   Output ~ 0
 OS1P8_PGOOD
@@
 AR Path="/5EAE2E5F/5EBE93DF" Ref="R?"  Part="1"
 F 0 "R?" H 7220 3510 50  0000 R CNN
-F 1 "R" V 7300 3510 50  0000 C CNN
+F 1 "1.87k" V 7300 3510 40  0000 C CNN
 F 2 "Resistors_SMD:R_0402" H 7300 3510 50  0001 C CNN
 F 3 "" H 7300 3510 50  0001 C CNN
@@
 AR Path="/5EAE2E5F/5EBEA0E2" Ref="R?"  Part="1"
 F 0 "R?" H 7220 4110 50  0000 R CNN
-F 1 "R" V 7300 4110 50  0000 C CNN
+F 1 "1.5k" V 7300 4110 50  0000 C CNN
 F 2 "Resistors_SMD:R_0402" H 7300 4110 50  0001 C CNN
 F 3 "" H 7300 4110 50  0001 C CNN
@@
 	4640 3980 3040 3980
 Connection ~ 3040 3980
+$Comp
+L Custom_Library:C_Custom C?
+U 1 1 5EB8DDAD
+P 4360 3510
+AR Path="/5CB7718D/5EB8DDAD" Ref="C?"  Part="1"
+AR Path="/5E0DC082/5EB8DDAD" Ref="C?"  Part="1"
+AR Path="/5E0F9110/5EB8DDAD" Ref="C?"  Part="1"
+AR Path="/5A557C58/5EB8DDAD" Ref="C?"  Part="1"
+AR Path="/5CB25152/5EB8DDAD" Ref="C?"  Part="1"
+AR Path="/5E697934/5EB8DDAD" Ref="C?"  Part="1"
+AR Path="/5EAE2F02/5EB8DDAD" Ref="C?"  Part="1"
+AR Path="/5EAE2E5F/5EB8DDAD" Ref="C?"  Part="1"
+F 0 "C?" H 4385 3610 50  0000 L CNN
+F 1 "10uF" H 4385 3410 50  0000 L CNN
+F 2 "Capacitors_SMD:C_0402" H 4398 3360 50  0001 C CNN
+F 3 "" H 4385 3610 50  0001 C CNN
+F 4 "0402" H 4210 3610 50  0000 R CNN "display_footprint"
+F 5 "6.3V" H 4210 3510 50  0000 R CNN "Voltage"
+F 6 "X5R" H 4210 3410 50  0000 R CNN "Dielectric"
+F 7 "490-13211-1-ND" H 4360 3510 50  0001 C CNN "Digi-Key PN"
+	1    4360 3510
+	1    0    0    -1
+$EndComp
+$Comp
+L Custom_Library:C_Custom C?
+U 1 1 5EB8E55F
+P 6430 3510
+AR Path="/5CB7718D/5EB8E55F" Ref="C?"  Part="1"
+AR Path="/5E0DC082/5EB8E55F" Ref="C?"  Part="1"
+AR Path="/5E0F9110/5EB8E55F" Ref="C?"  Part="1"
+AR Path="/5A557C58/5EB8E55F" Ref="C?"  Part="1"
+AR Path="/5CB25152/5EB8E55F" Ref="C?"  Part="1"
+AR Path="/5E697934/5EB8E55F" Ref="C?"  Part="1"
+AR Path="/5EAE2F02/5EB8E55F" Ref="C?"  Part="1"
+AR Path="/5EAE2E5F/5EB8E55F" Ref="C?"  Part="1"
+F 0 "C?" H 6455 3610 50  0000 L CNN
+F 1 "10uF" H 6455 3410 50  0000 L CNN
+F 2 "Capacitors_SMD:C_0402" H 6468 3360 50  0001 C CNN
+F 3 "" H 6455 3610 50  0001 C CNN
+F 4 "0402" H 6280 3610 50  0000 R CNN "display_footprint"
+F 5 "6.3V" H 6280 3510 50  0000 R CNN "Voltage"
+F 6 "X5R" H 6280 3410 50  0000 R CNN "Dielectric"
+F 7 "490-13211-1-ND" H 6430 3510 50  0001 C CNN "Digi-Key PN"
+	1    6430 3510
+	1    0    0    -1
+$EndComp
+$Comp
+L Custom_Library:C_Custom C?
+U 1 1 5EB8EF89
+P 5780 3510
+AR Path="/5CB7718D/5EB8EF89" Ref="C?"  Part="1"
+AR Path="/5E0DC082/5EB8EF89" Ref="C?"  Part="1"
+AR Path="/5E0F9110/5EB8EF89" Ref="C?"  Part="1"
+AR Path="/5A557C58/5EB8EF89" Ref="C?"  Part="1"
+AR Path="/5CB25152/5EB8EF89" Ref="C?"  Part="1"
+AR Path="/5E697934/5EB8EF89" Ref="C?"  Part="1"
+AR Path="/5EAE2F02/5EB8EF89" Ref="C?"  Part="1"
+AR Path="/5EAE2E5F/5EB8EF89" Ref="C?"  Part="1"
+F 0 "C?" H 5805 3610 50  0000 L CNN
+F 1 "10uF" H 5805 3410 50  0000 L CNN
+F 2 "Capacitors_SMD:C_0402" H 5818 3360 50  0001 C CNN
+F 3 "" H 5805 3610 50  0001 C CNN
+F 4 "0402" H 5630 3610 50  0000 R CNN "display_footprint"
+F 5 "6.3V" H 5630 3510 50  0000 R CNN "Voltage"
+F 6 "X5R" H 5630 3410 50  0000 R CNN "Dielectric"
+F 7 "490-13211-1-ND" H 5780 3510 50  0001 C CNN "Digi-Key PN"
+	1    5780 3510
+	1    0    0    -1
+$EndComp
+$Comp
+L power:+3.3V #PWR?
+U 1 1 5EBBDFFE
+P 3040 3360
+F 0 "#PWR?" H 3040 3210 50  0001 C CNN
+F 1 "+3.3V" H 3040 3500 50  0000 C CNN
+F 2 "" H 3040 3360 50  0001 C CNN
+F 3 "" H 3040 3360 50  0001 C CNN
+	1    3040 3360
+	1    0    0    -1
+$EndComp
 $EndSCHEMATC

Commit message: More sch work
Connections:
- net OS1P8_PGOOD renamed POS1P8_PGOOD
Changed lines of the file:
@@
 	3040 3980 3040 4060
 Text GLabel 2960 3880 0    50   Output ~ 0
-OS1P8_PGOOD
+POS1P8_PGOOD
 Text GLabel 2960 3980 0    50   Input ~ 0
 POS1P8_RUN

Commit message: Added more stuff to sch
Parts:
- R? (x4): footprint Resistors_SMD:R_0603 -> Resistors_SMD:R_0402; Digi-Key PN (none) -> 541-3964-1-ND; Wattage 1/10W -> 1/16W; display_footprint 0603 -> 0402
Changed lines of the file:
@@
 $Descr A 11000 8500
 encoding utf-8
-Sheet 6 19
-Title ""
+Sheet 6 20
+Title "Pulse Oximeter"
 Date "2020-05-02"
-Rev ""
-Comp ""
+Rev "A"
+Comp "Drew Maatman"
 Comment1 ""
 Comment2 ""
@@
 F 0 "R?" V 3800 2950 50  0000 C CNN
 F 1 "10" V 3900 2950 50  0000 C CNN
-F 2 "Resistors_SMD:R_0603" H 3900 2950 50  0001 C CNN
+F 2 "Resistors_SMD:R_0402" H 3900 2950 50  0001 C CNN
 F 3 "" H 3900 2950 50  0001 C CNN
-F 4 "0603" V 4000 2950 50  0001 C CNN "display_footprint"
+F 4 "0402" V 4000 2950 50  0001 C CNN "display_footprint"
 F 5 "1%" V 4100 2950 50  0001 C CNN "Tolerance"
-F 6 "1/10W" V 4200 2950 50  0001 C CNN "Wattage"
+F 6 "1/16W" V 4200 2950 50  0001 C CNN "Wattage"
+F 7 "541-3964-1-ND" H 3900 2950 50  0001 C CNN "Digi-Key PN"
 	1    3900 2950
 	1    0    0    -1
@@
 F 0 "R?" V 4260 2950 50  0000 C CNN
 F 1 "10" V 4360 2950 50  0000 C CNN
-F 2 "Resistors_SMD:R_0603" H 4360 2950 50  0001 C CNN
+F 2 "Resistors_SMD:R_0402" H 4360 2950 50  0001 C CNN
 F 3 "" H 4360 2950 50  0001 C CNN
-F 4 "0603" V 4460 2950 50  0001 C CNN "display_footprint"
+F 4 "0402" V 4460 2950 50  0001 C CNN "display_footprint"
 F 5 "1%" V 4560 2950 50  0001 C CNN "Tolerance"
-F 6 "1/10W" V 4660 2950 50  0001 C CNN "Wattage"
+F 6 "1/16W" V 4660 2950 50  0001 C CNN "Wattage"
+F 7 "541-3964-1-ND" H 4360 2950 50  0001 C CNN "Digi-Key PN"
 	1    4360 2950
 	-1   0    0    -1
@@
 F 0 "R?" V 6740 2950 50  0000 C CNN
 F 1 "10" V 6840 2950 50  0000 C CNN
-F 2 "Resistors_SMD:R_0603" H 6840 2950 50  0001 C CNN
+F 2 "Resistors_SMD:R_0402" H 6840 2950 50  0001 C CNN
 F 3 "" H 6840 2950 50  0001 C CNN
-F 4 "0603" V 6940 2950 50  0001 C CNN "display_footprint"
+F 4 "0402" V 6940 2950 50  0001 C CNN "display_footprint"
 F 5 "1%" V 7040 2950 50  0001 C CNN "Tolerance"
-F 6 "1/10W" V 7140 2950 50  0001 C CNN "Wattage"
+F 6 "1/16W" V 7140 2950 50  0001 C CNN "Wattage"
+F 7 "541-3964-1-ND" H 6840 2950 50  0001 C CNN "Digi-Key PN"
 	1    6840 2950
 	-1   0    0    -1
@@
 F 0 "R?" V 7200 2950 50  0000 C CNN
 F 1 "10" V 7300 2950 50  0000 C CNN
-F 2 "Resistors_SMD:R_0603" H 7300 2950 50  0001 C CNN
+F 2 "Resistors_SMD:R_0402" H 7300 2950 50  0001 C CNN
 F 3 "" H 7300 2950 50  0001 C CNN
-F 4 "0603" V 7400 2950 50  0001 C CNN "display_footprint"
+F 4 "0402" V 7400 2950 50  0001 C CNN "display_footprint"
 F 5 "1%" V 7500 2950 50  0001 C CNN "Tolerance"
-F 6 "1/10W" V 7600 2950 50  0001 C CNN "Wattage"
+F 6 "1/16W" V 7600 2950 50  0001 C CNN "Wattage"
+F 7 "541-3964-1-ND" H 7300 2950 50  0001 C CNN "Digi-Key PN"
 	1    7300 2950
 	-1   0    0    -1

Commit message: Added digikey pn's, footprints
Parts:
- R601, R602: renamed from R?; Digi-Key PN (none) -> RMCF0402FT10K0CT-ND
- R609: renamed from R?; Digi-Key PN (none) -> RMCF0402FT1K87CT-ND
- R610: renamed from R?; Digi-Key PN (none) -> 311-1.50KLRCT-ND
- gave numbers to parts that had none: 13
