File: hdw/Pulse_Oximeter/SD_Card_Slot.sch (KiCad schematic (older format))
At the start: 20 parts

Commit message: Added mech sheet, more complicated bullshit you dont need
Parts:
- removed D? (x5): PESD3V3L5UV, Package_TO_SOT_SMD:SOT-666, symbol Power_Protection:PESD3V3L5UV
- added D? (x5): PESD3V3L5UY, Package_TO_SOT_SMD:SOT-363_SC-70-6, symbol Power_Protection:PESD3V3L5UY
- J?: Configuration (none) -> SD Logging
Connections:
- net GND: now also D?.2 (A)
- net at J?.10 (DET_A), R?.1, R?.2: now also D?.6 (K5)
- net at J?.2 (DAT3/CD), R?.1, R?.2: now also D?.1 (K1)
- net at J?.3 (CMD), R?.1, R?.2: now also D?.3 (K2)
- net at J?.5 (CLK), R?.1, R?.2: now also D?.4 (K3)
- net at J?.7 (DAT0), R?.1, R?.2: now also D?.5 (K4)
Changed lines of the file:
@@
 $Descr A 11000 8500
 encoding utf-8
-Sheet 22 22
+Sheet 22 23
 Title ""
 Date ""
@@
 F 3 "https://www.hirose.com/product/en/download_file/key_name/DM3/category/Catalog/doc_file_id/49662/?file_category_id=4&item_id=195&is_series=1" H 6770 3990 50  0001 C CNN
 F 4 "WM6357CT-ND" H 6770 3890 50  0001 C CNN "Digi-Key PN"
+F 5 "SD Logging" H 6770 3180 50  0000 C CNN "Configuration"
 	1    6770 3890
 	1    0    0    -1
@@
 $EndComp
 $Comp
-L Power_Protection:PESD3V3L5UV D?
-U 1 1 5EBCE2AF
-P 4300 4580
-F 0 "D?" H 4300 4680 50  0000 C CNN
-F 1 "PESD3V3L5UV" V 4300 4480 50  0000 R CNN
-F 2 "Package_TO_SOT_SMD:SOT-666" H 4300 4580 50  0001 C CNN
-F 3 "https://assets.nexperia.com/documents/data-sheet/PESDXL5UF_V_Y.pdf" H 4300 4580 50  0001 C CNN
-	1    4300 4580
-	0    1    1    0
-$EndComp
-$Comp
-L Power_Protection:PESD3V3L5UV D?
-U 2 1 5EBCFE08
-P 4500 4580
-F 0 "D?" H 4500 4680 50  0000 C CNN
-F 1 "PESD3V3L5UV" V 4500 4480 50  0001 R CNN
-F 2 "Package_TO_SOT_SMD:SOT-666" H 4500 4580 50  0001 C CNN
-F 3 "https://assets.nexperia.com/documents/data-sheet/PESDXL5UF_V_Y.pdf" H 4500 4580 50  0001 C CNN
-	2    4500 4580
-	0    1    1    0
-$EndComp
-$Comp
 L Custom_Library:R_Custom R?
 U 1 1 5EBA2A9C
@@
 Wire Wire Line
 	3990 3590 4300 3590
-$Comp
-L Power_Protection:PESD3V3L5UV D?
-U 3 1 5EBD1F55
-P 4700 4580
-F 0 "D?" H 4700 4680 50  0000 C CNN
-F 1 "PESD3V3L5UV" V 4700 4480 50  0001 R CNN
-F 2 "Package_TO_SOT_SMD:SOT-666" H 4700 4580 50  0001 C CNN
-F 3 "https://assets.nexperia.com/documents/data-sheet/PESDXL5UF_V_Y.pdf" H 4700 4580 50  0001 C CNN
-	3    4700 4580
-	0    1    1    0
-$EndComp
-$Comp
-L Power_Protection:PESD3V3L5UV D?
-U 4 1 5EBD26EA
-P 4900 4580
-F 0 "D?" H 4900 4680 50  0000 C CNN
-F 1 "PESD3V3L5UV" V 4900 4480 50  0001 R CNN
-F 2 "Package_TO_SOT_SMD:SOT-666" H 4900 4580 50  0001 C CNN
-F 3 "https://assets.nexperia.com/documents/data-sheet/PESDXL5UF_V_Y.pdf" H 4900 4580 50  0001 C CNN
-	4    4900 4580
-	0    1    1    0
-$EndComp
-$Comp
-L Power_Protection:PESD3V3L5UV D?
-U 5 1 5EBD2E02
-P 5100 4580
-F 0 "D?" H 5100 4680 50  0000 C CNN
-F 1 "PESD3V3L5UV" V 5100 4480 50  0001 R CNN
-F 2 "Package_TO_SOT_SMD:SOT-666" H 5100 4580 50  0001 C CNN
-F 3 "https://assets.nexperia.com/documents/data-sheet/PESDXL5UF_V_Y.pdf" H 5100 4580 50  0001 C CNN
-	5    5100 4580
-	0    1    1    0
-$EndComp
 Wire Wire Line
 	4300 3510 4300 3590
@@
 Text GLabel 3690 4090 0    50   Output ~ 0
 SD_SPI_MISO
+$Comp
+L Power_Protection:PESD3V3L5UY D?
+U 1 1 5EBFF172
+P 4300 4580
+F 0 "D?" V 4220 4480 50  0000 R CNN
+F 1 "PESD3V3L5UY" V 4320 4480 50  0000 R CNN
+F 2 "Package_TO_SOT_SMD:SOT-363_SC-70-6" H 4300 4580 50  0001 C CNN
+F 3 "https://assets.nexperia.com/documents/data-sheet/PESDXL5UF_V_Y.pdf" H 4300 4580 50  0001 C CNN
+F 4 "1727-3828-1-ND" H 4300 4580 50  0001 C CNN "Digi-Key PN"
+F 5 "SD Logging" V 4430 4970 50  0000 C CNN "Configuration"
+	1    4300 4580
+	0    1    1    0
+$EndComp
+$Comp
+L Power_Protection:PESD3V3L5UY D?
+U 2 1 5EC01F12
+P 4500 4580
+F 0 "D?" V 4420 4480 50  0001 R CNN
+F 1 "PESD3V3L5UY" V 4520 4480 50  0001 R CNN
+F 2 "Package_TO_SOT_SMD:SOT-363_SC-70-6" H 4500 4580 50  0001 C CNN
+F 3 "https://assets.nexperia.com/documents/data-sheet/PESDXL5UF_V_Y.pdf" H 4500 4580 50  0001 C CNN
+	2    4500 4580
+	0    1    1    0
+$EndComp
+$Comp
+L Power_Protection:PESD3V3L5UY D?
+U 3 1 5EC02369
+P 4700 4580
+F 0 "D?" V 4620 4480 50  0001 R CNN
+F 1 "PESD3V3L5UY" V 4720 4480 50  0001 R CNN
+F 2 "Package_TO_SOT_SMD:SOT-363_SC-70-6" H 4700 4580 50  0001 C CNN
+F 3 "https://assets.nexperia.com/documents/data-sheet/PESDXL5UF_V_Y.pdf" H 4700 4580 50  0001 C CNN
+	3    4700 4580
+	0    1    1    0
+$EndComp
+$Comp
+L Power_Protection:PESD3V3L5UY D?
+U 4 1 5EC027AC
+P 4900 4580
+F 0 "D?" V 4820 4480 50  0001 R CNN
+F 1 "PESD3V3L5UY" V 4920 4480 50  0001 R CNN
+F 2 "Package_TO_SOT_SMD:SOT-363_SC-70-6" H 4900 4580 50  0001 C CNN
+F 3 "https://assets.nexperia.com/documents/data-sheet/PESDXL5UF_V_Y.pdf" H 4900 4580 50  0001 C CNN
+	4    4900 4580
+	0    1    1    0
+$EndComp
+$Comp
+L Power_Protection:PESD3V3L5UY D?
+U 5 1 5EC02BD8
+P 5100 4580
+F 0 "D?" V 5020 4480 50  0001 R CNN
+F 1 "PESD3V3L5UY" V 5120 4480 50  0001 R CNN
+F 2 "Package_TO_SOT_SMD:SOT-363_SC-70-6" H 5100 4580 50  0001 C CNN
+F 3 "https://assets.nexperia.com/documents/data-sheet/PESDXL5UF_V_Y.pdf" H 5100 4580 50  0001 C CNN
+	5    5100 4580
+	0    1    1    0
+$EndComp
 $EndSCHEMATC

Commit message: Added digikey pn's, footprints
Parts:
- D2201: renamed from D?; Configuration (none) -> SD Logging; Digi-Key PN (none) -> 1727-3828-1-ND
- R2206, R2207, R2208, R2209, R2210: renamed from R?; Digi-Key PN (none) -> RMCF0402FT10K0CT-ND
- gave numbers to parts that had none: 11
