File: hdw/Pulse_Oximeter/Backup_RTC.sch (KiCad schematic (older format))
At the start: 10 parts, among them J2101 CR2032 socket, Q2101 BSS214NW, U2101 DS3231MZ

Commit message: few sch additions
Parts:
- added TP2101: TP, Custom Footprints Library:Test_Point, symbol Custom_Library:TP
Connections:
- net VBAT: now also TP2101.1 (TP)
Changed lines of the file:
@@
 Text GLabel 4310 6030 0    50   Input ~ 0
 POS3P3_PGOOD
+$Comp
+L Custom_Library:TP TP?
+U 1 1 5EC3F1A9
+P 2910 5180
+AR Path="/5C1D5CD8/5EC3F1A9" Ref="TP?"  Part="1"
+AR Path="/5C1D5C9E/5EC3F1A9" Ref="TP?"  Part="1"
+AR Path="/5CB6F1ED/5EC3F1A9" Ref="TP?"  Part="1"
+AR Path="/5E939CFF/5EC3F1A9" Ref="TP?"  Part="1"
+AR Path="/5E9E0E87/5EC3F1A9" Ref="TP?"  Part="1"
+AR Path="/5EAE2D66/5EC3F1A9" Ref="TP?"  Part="1"
+AR Path="/5EB8C603/5EC3F1A9" Ref="TP2101"  Part="1"
+F 0 "TP2101" H 2910 5330 50  0000 C CNN
+F 1 "TP" H 2910 5330 50  0001 C CNN
+F 2 "Custom Footprints Library:Test_Point" H 2910 5180 60  0001 C CNN
+F 3 "" H 2910 5180 60  0000 C CNN
+	1    2910 5180
+	1    0    0    -1
+$EndComp
+Wire Wire Line
+	2910 5180 2910 5280
+Wire Wire Line
+	2910 5280 2580 5280
+Connection ~ 2580 5280
+$Comp
+L power:PWR_FLAG #FLG0103
+U 1 1 5EC3F51F
+P 3300 5180
+F 0 "#FLG0103" H 3300 5255 50  0001 C CNN
+F 1 "PWR_FLAG" H 3300 5330 50  0000 C CNN
+F 2 "" H 3300 5180 50  0001 C CNN
+F 3 "~" H 3300 5180 50  0001 C CNN
+	1    3300 5180
+	1    0    0    -1
+$EndComp
+Wire Wire Line
+	3300 5180 3300 5280
+Wire Wire Line
+	3300 5280 2910 5280
+Connection ~ 2910 5280
 $EndSCHEMATC
