File: hdw/Pulse_Oximeter/Display.sch (KiCad schematic (older format))
At the start: 0 parts

Commit message: Added display circuits
Parts:
- added C? (x3): 0.1uF, Capacitors_SMD:C_0402, symbol Custom_Library:C_Custom
- added C? (x2): 1nF, Capacitors_SMD:C_0402, symbol Custom_Library:C_Custom
- added C? (x2): 10nF, Capacitors_SMD:C_0402, symbol Custom_Library:C_Custom
- added C? (x2): 10uF, Capacitors_SMD:C_0402, symbol Custom_Library:C_Custom
- added DOC?: wkjeflkaj, symbol Custom_Library:I2C_Address
- added R?: 499, Resistors_SMD:R_0402, symbol Custom_Library:R_Custom
- added R? (x4): 10k, Resistors_SMD:R_0402, symbol Custom_Library:R_Custom
- added RN?: 10k, Resistors_SMD:R_Array_Convex_8x0602, symbol Device:R_Pack08
- added RV?: 10k, Potentiometer_SMD:Potentiometer_Vishay_TS53YL_Vertical, symbol Device:R_POT
- added U?: NHD-0420H1Z, Display:NHD-0420H1Z, symbol Display_Character:NHD-0420H1Z
- added U?: 74LVC1G17, TO_SOT_Packages_SMD:SOT-353_SC-70-5, symbol Custom_Library:74LVC1G17_Power
- added U?: TPL0401A-10-Q1, Package_TO_SOT_SMD:Texas_R-PDSO-G6, symbol Potentiometer_Digital:TPL0401A-10-Q1
Connections:
- net labels added: +3.3V, GND, I2C_SCL, I2C_SDA, LCD_BACKLIGHT, LCD_BACKLIGHT_PWM, LCD_CONTRAST, LCD_PMP_DB0, LCD_PMP_DB1, LCD_PMP_DB2, LCD_PMP_DB3, LCD_PMP_DB4, LCD_PMP_DB5, LCD_PMP_DB6, LCD_PMP_DB7, LCD_PMP_E, LCD_PMP_RS, LCD_PMP_R_W
- wire segments 0 -> 79

Commit message: More sch work
Parts:
- removed C?: 0.1uF, Capacitors_SMD:C_0402, symbol Custom_Library:C_Custom
- removed C?: 1nF, Capacitors_SMD:C_0402, symbol Custom_Library:C_Custom
- removed C?: 10nF, Capacitors_SMD:C_0402, symbol Custom_Library:C_Custom
- removed C?: 10uF, Capacitors_SMD:C_0402, symbol Custom_Library:C_Custom
- removed DOC?: wkjeflkaj, symbol Custom_Library:I2C_Address
- removed U?: TPL0401A-10-Q1, Package_TO_SOT_SMD:Texas_R-PDSO-G6, symbol Potentiometer_Digital:TPL0401A-10-Q1
- RV?: Digi-Key PN DNP -> TS53YL-10KCT-ND
Connections:
- net labels removed: I2C_SCL, I2C_SDA
- wire segments 79 -> 67
Other:
- moved on the sheet: RV?

Commit message: Added digikey pn's, footprints
Parts:
- R1601, R1602, R1603, R1605: renamed from R?; Digi-Key PN (none) -> RMCF0402FT10K0CT-ND
- R1604: renamed from R?; Digi-Key PN (none) -> RMCF0402FT499RCT-ND
- gave numbers to parts that had none: 9

Commit message: few sch additions
Parts:
- removed RN1601: 10k, Resistors_SMD:R_Array_Convex_8x0602, symbol Device:R_Pack08
- added R1606, R1607, R1608, R1609, R1610, R1611, R1612, R1613: 10k, Resistors_SMD:R_0402, symbol Custom_Library:R_Custom
Connections:
- net GND: now also R1606.2, R1607.2, R1608.2, R1609.2, R1610.2, R1611.2, R1612.2, R1613.2
- net LCD_PMP_DB0: now also R1606.1
- net LCD_PMP_DB1: now also R1607.1
- net LCD_PMP_DB2: now also R1608.1
- net LCD_PMP_DB3: now also R1609.1
- net LCD_PMP_DB4: now also R1610.1
- net LCD_PMP_DB5: now also R1611.1
- net LCD_PMP_DB6: now also R1612.1
- net LCD_PMP_DB7: now also R1613.1
Other:
- moved on the sheet: R1603
