File: hdw/Pulse_Oximeter/PIC32MZ_Programming.sch (KiCad schematic (older format))
At the start: 10 parts

Commit message: few sch additions
Connections:
- net ICSPCLK renamed PIC32MZ_ICSPCLK
- net ICSPDAT renamed PIC32MZ_ICSPDAT
- net ~MCLR renamed ~PIC32MZ_MCLR
Other:
- moved on the sheet: C?
Changed lines of the file:
@@
 $EndComp
 Text GLabel 1270 1790 2    50   UnSpc ~ 0
-~MCLR
+~PIC32MZ_MCLR
 Text GLabel 1270 2090 2    50   BiDi ~ 0
-ICSPDAT
+PIC32MZ_ICSPDAT
 Text GLabel 1270 2190 2    50   Output ~ 0
-ICSPCLK
+PIC32MZ_ICSPCLK
 $Comp
 L power:GND #PWR?
 U 1 1 5BB4A7C4
-P 1790 2040
-F 0 "#PWR?" H 1790 1790 50  0001 C CNN
-F 1 "GND" H 1790 1890 50  0000 C CNN
-F 2 "" H 1790 2040 50  0001 C CNN
-F 3 "" H 1790 2040 50  0001 C CNN
-	1    1790 2040
+P 2160 2040
+F 0 "#PWR?" H 2160 1790 50  0001 C CNN
+F 1 "GND" H 2160 1890 50  0000 C CNN
+F 2 "" H 2160 2040 50  0001 C CNN
+F 3 "" H 2160 2040 50  0001 C CNN
+	1    2160 2040
 	-1   0    0    -1
 $EndComp
 Wire Wire Line
-	1790 1820 1790 1890
-Wire Wire Line
-	1790 1890 1270 1890
-Wire Wire Line
-	1790 2040 1790 1990
-Wire Wire Line
-	1790 1990 1270 1990
+	2160 1820 2160 1890
+Wire Wire Line
+	2160 2040 2160 1990
 NoConn ~ 1270 2290
 $Comp
 L Custom_Library:C_Custom C?
 U 1 1 5BC13497
-P 2460 2030
-F 0 "C?" H 2485 2130 50  0000 L CNN
-F 1 "0.1uF" H 2485 1930 50  0000 L CNN
-F 2 "Capacitors_SMD:C_0402" H 2498 1880 50  0001 C CNN
-F 3 "" H 2485 2130 50  0001 C CNN
-F 4 "0402" H 2310 2130 50  0000 R CNN "display_footprint"
-F 5 "50V" H 2310 2030 50  0000 R CNN "Voltage"
-F 6 "X7R" H 2310 1930 50  0000 R CNN "Dielectric"
-F 7 "490-10701-1-ND" H 2885 2530 60  0001 C CNN "Digi-Key PN"
-	1    2460 2030
+P 2790 2030
+F 0 "C?" H 2815 2130 50  0000 L CNN
+F 1 "0.1uF" H 2815 1930 50  0000 L CNN
+F 2 "Capacitors_SMD:C_0402" H 2828 1880 50  0001 C CNN
+F 3 "" H 2815 2130 50  0001 C CNN
+F 4 "0402" H 2640 2130 50  0000 R CNN "display_footprint"
+F 5 "50V" H 2640 2030 50  0000 R CNN "Voltage"
+F 6 "X7R" H 2640 1930 50  0000 R CNN "Dielectric"
+F 7 "490-10701-1-ND" H 3215 2530 60  0001 C CNN "Digi-Key PN"
+	1    2790 2030
 	1    0    0    -1
 $EndComp
@@
 L power:GND #PWR?
 U 1 1 5BC1349E
-P 2460 2180
-F 0 "#PWR?" H 2460 1930 50  0001 C CNN
-F 1 "GND" H 2460 2030 50  0000 C CNN
-F 2 "" H 2460 2180 50  0001 C CNN
-F 3 "" H 2460 2180 50  0001 C CNN
-	1    2460 2180
+P 2790 2180
+F 0 "#PWR?" H 2790 1930 50  0001 C CNN
+F 1 "GND" H 2790 2030 50  0000 C CNN
+F 2 "" H 2790 2180 50  0001 C CNN
+F 3 "" H 2790 2180 50  0001 C CNN
+	1    2790 2180
 	1    0    0    -1
 $EndComp
@@
 Connection ~ 7550 2250
 Text GLabel 8230 2250 2    50   UnSpc ~ 0
-~MCLR
+~PIC32MZ_MCLR
 $Comp
 L Switch:SW_Push SW?
@@
 L power:+3.3V #PWR?
 U 1 1 5E6EC62F
-P 2460 1880
-F 0 "#PWR?" H 2460 1730 50  0001 C CNN
-F 1 "+3.3V" H 2460 2020 50  0000 C CNN
-F 2 "" H 2460 1880 50  0001 C CNN
-F 3 "" H 2460 1880 50  0001 C CNN
-	1    2460 1880
+P 2790 1880
+F 0 "#PWR?" H 2790 1730 50  0001 C CNN
+F 1 "+3.3V" H 2790 2020 50  0000 C CNN
+F 2 "" H 2790 1880 50  0001 C CNN
+F 3 "" H 2790 1880 50  0001 C CNN
+	1    2790 1880
 	1    0    0    -1
 $EndComp
@@
 L power:+3.3V #PWR?
 U 1 1 5E6ECA36
-P 1790 1820
-F 0 "#PWR?" H 1790 1670 50  0001 C CNN
-F 1 "+3.3V" H 1790 1960 50  0000 C CNN
-F 2 "" H 1790 1820 50  0001 C CNN
-F 3 "" H 1790 1820 50  0001 C CNN
-	1    1790 1820
+P 2160 1820
+F 0 "#PWR?" H 2160 1670 50  0001 C CNN
+F 1 "+3.3V" H 2160 1960 50  0000 C CNN
+F 2 "" H 2160 1820 50  0001 C CNN
+F 3 "" H 2160 1820 50  0001 C CNN
+	1    2160 1820
 	1    0    0    -1
 $EndComp
@@
 	1    0    0    -1
 $EndComp
+Wire Wire Line
+	1270 1890 2160 1890
+Wire Wire Line
+	1270 1990 2160 1990
 $EndSCHEMATC

Commit message: More sch work
Parts:
- removed R?: 100, Resistors_SMD:R_0402, symbol Custom_Library:R_Custom
- added R?: 10, Resistors_SMD:R_0402, symbol Custom_Library:R_Custom
Connections:
- net at C?.1, R?.2, R?.2: now also R?.2
- net at Q?.3 (D): now also R?.1
Changed lines of the file:
@@
 	1    0    0    -1
-$EndComp
-$Comp
-L Custom_Library:R_Custom R?
-U 1 1 5BC190FF
-P 6860 2250
-F 0 "R?" V 6760 2250 50  0000 C CNN
-F 1 "100" V 6860 2250 50  0000 C CNN
-F 2 "Resistors_SMD:R_0402" H 6860 2250 50  0001 C CNN
-F 3 "" H 6860 2250 50  0001 C CNN
-F 4 "0402" V 6960 2250 50  0000 C CNN "display_footprint"
-F 5 "1%" V 7060 2250 50  0000 C CNN "Tolerance"
-F 6 "1/16W" V 7160 2250 50  0000 C CNN "Wattage"
-F 7 "541-100LCT-ND" H 7160 2650 60  0001 C CNN "Digi-Key PN"
-	1    6860 2250
-	0    1    1    0
 $EndComp
 Wire Wire Line
@@
 Wire Wire Line
 	1270 1990 2160 1990
+$Comp
+L Custom_Library:R_Custom R?
+U 1 1 5EB9A4D9
+P 6860 2250
+F 0 "R?" V 6760 2250 50  0000 C CNN
+F 1 "10" V 6860 2250 50  0000 C CNN
+F 2 "Resistors_SMD:R_0402" H 6860 2250 50  0001 C CNN
+F 3 "" H 6860 2250 50  0001 C CNN
+F 4 "0402" V 6960 2250 50  0000 C CNN "display_footprint"
+F 5 "1%" V 7060 2250 50  0000 C CNN "Tolerance"
+F 6 "1/16W" V 7160 2250 50  0000 C CNN "Wattage"
+F 7 "541-3964-1-ND" H 7160 2650 60  0001 C CNN "Digi-Key PN"
+	1    6860 2250
+	0    -1   -1   0
+$EndComp
 $EndSCHEMATC

Commit message: Added digikey pn's, footprints
Parts:
- gave numbers to parts that had none: 10
Changed lines of the file:
@@
 Sheet 8 23
 Title "Pulse Oximeter"
-Date "2019-04-11"
+Date "2019-01-03"
 Rev "A"
 Comp "Drew Maatman"
@@
 $EndDescr
 $Comp
-L Connector_Generic:Conn_01x06 J?
+L Connector_Generic:Conn_01x06 J801
 U 1 1 5BB4A695
 P 1070 1990
-F 0 "J?" H 1160 1980 50  0000 L CNN
+F 0 "J801" H 1160 1980 50  0000 L CNN
 F 1 "PICKIT3" H 1160 1900 50  0000 L CNN
 F 2 "Custom Footprints Library:PICKIT3_Header" H 1070 1990 50  0001 C CNN
@@
 PIC32MZ_ICSPCLK
 $Comp
-L power:GND #PWR?
+L power:GND #PWR0802
 U 1 1 5BB4A7C4
 P 2160 2040
-F 0 "#PWR?" H 2160 1790 50  0001 C CNN
+F 0 "#PWR0802" H 2160 1790 50  0001 C CNN
 F 1 "GND" H 2160 1890 50  0000 C CNN
 F 2 "" H 2160 2040 50  0001 C CNN
@@
 NoConn ~ 1270 2290
 $Comp
-L Custom_Library:C_Custom C?
+L Custom_Library:C_Custom C801
 U 1 1 5BC13497
 P 2790 2030
-F 0 "C?" H 2815 2130 50  0000 L CNN
+F 0 "C801" H 2815 2130 50  0000 L CNN
 F 1 "0.1uF" H 2815 1930 50  0000 L CNN
 F 2 "Capacitors_SMD:C_0402" H 2828 1880 50  0001 C CNN
@@
 $EndComp
 $Comp
-L power:GND #PWR?
+L power:GND #PWR0804
 U 1 1 5BC1349E
 P 2790 2180
-F 0 "#PWR?" H 2790 1930 50  0001 C CNN
+F 0 "#PWR0804" H 2790 1930 50  0001 C CNN
 F 1 "GND" H 2790 2030 50  0000 C CNN
 F 2 "" H 2790 2180 50  0001 C CNN
@@
 AR Path="/5CB0BC26/5BC152E5" Ref="R?"  Part="1"
 AR Path="/5E697920/5BC152E5" Ref="R?"  Part="1"
-AR Path="/5EAE2EF2/5BC152E5" Ref="R?"  Part="1"
-F 0 "R?" H 7490 2020 50  0000 R CNN
+AR Path="/5EAE2EF2/5BC152E5" Ref="R804"  Part="1"
+F 0 "R804" H 7490 2020 50  0000 R CNN
 F 1 "10k" V 7550 2020 50  0000 C CNN
 F 2 "Resistors_SMD:R_0402" H 7550 2020 50  0001 C CNN
@@
 $EndComp
 $Comp
-L Custom_Library:C_Custom C?
+L Custom_Library:C_Custom C802
 U 1 1 5BC1574E
 P 7550 2830
-F 0 "C?" H 7575 2930 50  0000 L CNN
+F 0 "C802" H 7575 2930 50  0000 L CNN
 F 1 "0.1uF" H 7575 2730 50  0000 L CNN
 F 2 "Capacitors_SMD:C_0402" H 7588 2680 50  0001 C CNN
@@
 $EndComp
 $Comp
-L power:GND #PWR?
+L power:GND #PWR0809
 U 1 1 5BC15E18
 P 7550 2980
-F 0 "#PWR?" H 7550 2730 50  0001 C CNN
+F 0 "#PWR0809" H 7550 2730 50  0001 C CNN
 F 1 "GND" H 7550 2830 50  0000 C CNN
 F 2 "" H 7550 2980 50  0001 C CNN
@@
 $EndComp
 $Comp
-L Custom_Library:R_Custom R?
+L Custom_Library:R_Custom R805
 U 1 1 5BC16316
 P 8080 2250
-F 0 "R?" V 7980 2250 50  0000 C CNN
+F 0 "R805" V 7980 2250 50  0000 C CNN
 F 1 "1k" V 8080 2250 50  0000 C CNN
 F 2 "Resistors_SMD:R_0402" H 8080 2250 50  0001 C CNN
@@
 ~PIC32MZ_MCLR
 $Comp
-L Switch:SW_Push SW?
+L Switch:SW_Push SW801
 U 1 1 5BC17B44
 P 5020 2770
-F 0 "SW?" H 5020 3055 50  0000 C CNN
+F 0 "SW801" H 5020 3055 50  0000 C CNN
 F 1 "MRST" H 5020 2964 50  0000 C CNN
 F 2 "Buttons_Switches_THT:SW_PUSH_6mm" H 5020 2970 50  0001 C CNN
@@
 	7010 2250 7550 2250
 $Comp
-L power:GND #PWR?
+L power:GND #PWR0807
 U 1 1 5BE087C1
 P 6510 2970
-F 0 "#PWR?" H 6510 2720 50  0001 C CNN
+F 0 "#PWR0807" H 6510 2720 50  0001 C CNN
 F 1 "GND" H 6510 2820 50  0000 C CNN
 F 2 "" H 6510 2970 50  0001 C CNN
@@
 $EndComp
 $Comp
-L Custom_Library:R_Custom R?
+L Custom_Library:R_Custom R801
 U 1 1 5BE087CB
 P 5470 2770
-F 0 "R?" V 5370 2770 50  0000 C CNN
+F 0 "R801" V 5370 2770 50  0000 C CNN
 F 1 "10" V 5470 2770 50  0000 C CNN
 F 2 "Resistors_SMD:R_0402" H 5470 2770 50  0001 C CNN
@@
 AR Path="/5CB0BC26/5BE087D6" Ref="R?"  Part="1"
 AR Path="/5E697920/5BE087D6" Ref="R?"  Part="1"
-AR Path="/5EAE2EF2/5BE087D6" Ref="R?"  Part="1"
-F 0 "R?" H 5860 3000 50  0000 R CNN
+AR Path="/5EAE2EF2/5BE087D6" Ref="R802"  Part="1"
+F 0 "R802" H 5860 3000 50  0000 R CNN
 F 1 "10k" V 5920 3000 50  0000 C CNN
 F 2 "Resistors_SMD:R_0402" H 5920 3000 50  0001 C CNN
@@
 $EndComp
 $Comp
-L power:GND #PWR?
+L power:GND #PWR0806
 U 1 1 5BE087DD
 P 5920 3150
-F 0 "#PWR?" H 5920 2900 50  0001 C CNN
+F 0 "#PWR0806" H 5920 2900 50  0001 C CNN
 F 1 "GND" H 5920 3000 50  0000 C CNN
 F 2 "" H 5920 3150 50  0001 C CNN
@@
 	7550 2680 7550 2250
 $Comp
-L power:+3.3V #PWR?
+L power:+3.3V #PWR0805
 U 1 1 5E6EB62A
 P 4670 2720
-F 0 "#PWR?" H 4670 2570 50  0001 C CNN
+F 0 "#PWR0805" H 4670 2570 50  0001 C CNN
 F 1 "+3.3V" H 4670 2860 50  0000 C CNN
 F 2 "" H 4670 2720 50  0001 C CNN
@@
 $EndComp
 $Comp
-L power:+3.3V #PWR?
+L power:+3.3V #PWR0808
 U 1 1 5E6EBFA5
 P 7550 1870
-F 0 "#PWR?" H 7550 1720 50  0001 C CNN
+F 0 "#PWR0808" H 7550 1720 50  0001 C CNN
 F 1 "+3.3V" H 7550 2010 50  0000 C CNN
 F 2 "" H 7550 1870 50  0001 C CNN
@@
 $EndComp
 $Comp
-L power:+3.3V #PWR?
+L power:+3.3V #PWR0803
 U 1 1 5E6EC62F
 P 2790 1880
-F 0 "#PWR?" H 2790 1730 50  0001 C CNN
+F 0 "#PWR0803" H 2790 1730 50  0001 C CNN
 F 1 "+3.3V" H 2790 2020 50  0000 C CNN
 F 2 "" H 2790 1880 50  0001 C CNN
@@
 $EndComp
 $Comp
-L power:+3.3V #PWR?
+L power:+3.3V #PWR0801
 U 1 1 5E6ECA36
 P 2160 1820
-F 0 "#PWR?" H 2160 1670 50  0001 C CNN
+F 0 "#PWR0801" H 2160 1670 50  0001 C CNN
 F 1 "+3.3V" H 2160 1960 50  0000 C CNN
 F 2 "" H 2160 1820 50  0001 C CNN
@@
 $EndComp
 $Comp
-L Transistor_FET:BSS214NW Q?
+L Transistor_FET:BSS214NW Q801
 U 1 1 5E765004
 P 6410 2770
-F 0 "Q?" H 6610 2845 50  0000 L CNN
+F 0 "Q801" H 6610 2845 50  0000 L CNN
 F 1 "BSS214NW" H 6610 2770 50  0000 L CNN
 F 2 "Package_TO_SOT_SMD:SOT-323_SC-70" H 6610 2695 50  0001 L CIN
@@
 	1270 1990 2160 1990
 $Comp
-L Custom_Library:R_Custom R?
+L Custom_Library:R_Custom R803
 U 1 1 5EB9A4D9
 P 6860 2250
-F 0 "R?" V 6760 2250 50  0000 C CNN
+F 0 "R803" V 6760 2250 50  0000 C CNN
 F 1 "10" V 6860 2250 50  0000 C CNN
 F 2 "Resistors_SMD:R_0402" H 6860 2250 50  0001 C CNN
