File: hdw/Pulse_Oximeter/POS3P3_Power_Supply.sch (KiCad schematic (older format))
At the start: 18 parts

Commit message: Continued schematic development
Parts:
- added C?: 4.7uF, Capacitors_SMD:C_0402, symbol Custom_Library:C_Custom
- added D?: BAT48JFILM, Diode_SMD:D_SOD-323, symbol Diode:BAT48JFILM
- added Q?: ZXMS6004FFTA, Package_TO_SOT_SMD:SOT-23, symbol Custom_Library:ZXMS6004FFTA
- added Q?: BSS214NW, Package_TO_SOT_SMD:SOT-323_SC-70, symbol Transistor_FET:BSS214NW
- added R?: 10k, Resistors_SMD:R_0603, symbol Custom_Library:R_Custom
Connections:
- wire segments 47 -> 54
Changed lines of the file:
@@
 Text Notes -580 1620 0    250  ~ 50
 CONSIDER A SMALLER SOLUTION WITH LOWER OUTPUT CURRENT
+$Comp
+L Custom_Library:ZXMS6004FFTA Q?
+U 1 1 5EB3BE62
+P 5020 7210
+F 0 "Q?" H 5220 7285 50  0000 L CNN
+F 1 "ZXMS6004FFTA" H 5220 7210 50  0000 L CNN
+F 2 "Package_TO_SOT_SMD:SOT-23" H 5220 7135 50  0001 L CIN
+F 3 "https://www.diodes.com/assets/Datasheets/ZXMS6004FF.pdf" H 5020 7210 50  0001 L CNN
+F 4 "ZXMS6004FFCT-ND" H 5020 7210 50  0001 C CNN "Digi-Key PN"
+	1    5020 7210
+	1    0    0    -1
+$EndComp
+$Comp
+L power:GND #PWR?
+U 1 1 5EB3CD64
+P 5120 7410
+F 0 "#PWR?" H 5120 7160 50  0001 C CNN
+F 1 "GND" H 5120 7260 50  0000 C CNN
+F 2 "" H 5120 7410 50  0001 C CNN
+F 3 "" H 5120 7410 50  0001 C CNN
+	1    5120 7410
+	1    0    0    -1
+$EndComp
+$Comp
+L power:+3.3V #PWR?
+U 1 1 5EB3E1B6
+P 5120 7010
+F 0 "#PWR?" H 5120 6860 50  0001 C CNN
+F 1 "+3.3V" H 5120 7150 50  0000 C CNN
+F 2 "" H 5120 7010 50  0001 C CNN
+F 3 "" H 5120 7010 50  0001 C CNN
+	1    5120 7010
+	1    0    0    -1
+$EndComp
+$Comp
+L Transistor_FET:BSS214NW Q?
+U 1 1 5EB3F7A8
+P 4290 7490
+F 0 "Q?" H 4490 7565 50  0000 L CNN
+F 1 "BSS214NW" H 4490 7490 50  0000 L CNN
+F 2 "Package_TO_SOT_SMD:SOT-323_SC-70" H 4490 7415 50  0001 L CIN
+F 3 "https://www.infineon.com/dgdl/Infineon-BSS214NW-DS-v02_02-en.pdf?fileId=db3a30431b3e89eb011b695aebc01bde" H 4290 7490 50  0001 L CNN
+	1    4290 7490
+	1    0    0    -1
+$EndComp
+$Comp
+L power:GND #PWR?
+U 1 1 5EB40BA6
+P 4390 7690
+F 0 "#PWR?" H 4390 7440 50  0001 C CNN
+F 1 "GND" H 4390 7540 50  0000 C CNN
+F 2 "" H 4390 7690 50  0001 C CNN
+F 3 "" H 4390 7690 50  0001 C CNN
+	1    4390 7690
+	1    0    0    -1
+$EndComp
+Text GLabel 4090 7490 0    50   Input ~ 0
+POS3P3_RUN
+$Comp
+L Custom_Library:R_Custom R?
+U 1 1 5EB41C61
+P 4390 6980
+AR Path="/5BB27BA3/5EB41C61" Ref="R?"  Part="1"
+AR Path="/5BB27BF7/5EB41C61" Ref="R?"  Part="1"
+AR Path="/5C1DE17A/5EB41C61" Ref="R?"  Part="1"
+AR Path="/5C1E3A08/5EB41C61" Ref="R?"  Part="1"
+AR Path="/5D779AE1/5EB41C61" Ref="R?"  Part="1"
+AR Path="/5CB7718D/5EB41C61" Ref="R?"  Part="1"
+AR Path="/5E0DC082/5EB41C61" Ref="R?"  Part="1"
+AR Path="/5E0F263A/5EB41C61" Ref="R?"  Part="1"
+AR Path="/5EAE2D8A/5EB41C61" Ref="R?"  Part="1"
+F 0 "R?" H 4310 6980 50  0000 R CNN
+F 1 "10k" V 4390 6980 50  0000 C CNN
+F 2 "Resistors_SMD:R_0603" H 4390 6980 50  0001 C CNN
+F 3 "" H 4390 6980 50  0001 C CNN
+F 4 "0603" H 4490 7060 50  0000 L CNN "display_footprint"
+F 5 "1%" H 4490 6980 50  0000 L CNN "Tolerance"
+F 6 "1/10W" H 4500 6900 50  0000 L CNN "Wattage"
+F 7 "RHM10KADCT-ND" H 4690 7380 60  0001 C CNN "Digi-Key PN"
+	1    4390 6980
+	1    0    0    -1
+$EndComp
+Wire Wire Line
+	4390 7130 4390 7210
+Wire Wire Line
+	4820 7210 4390 7210
+Connection ~ 4390 7210
+Wire Wire Line
+	4390 7210 4390 7290
+$Comp
+L Custom_Library:C_Custom C?
+U 1 1 5EB46F8D
+P 3680 6980
+AR Path="/5EAE2F97/5EB46F8D" Ref="C?"  Part="1"
+AR Path="/5EAE2D8A/5EB46F8D" Ref="C?"  Part="1"
+F 0 "C?" H 3705 7080 50  0000 L CNN
+F 1 "4.7uF" H 3705 6880 50  0000 L CNN
+F 2 "Capacitors_SMD:C_0402" H 3718 6830 50  0001 C CNN
+F 3 "" H 3705 7080 50  0001 C CNN
+F 4 "0402" H 3530 7080 50  0000 R CNN "display_footprint"
+F 5 "6.3V" H 3530 6980 50  0000 R CNN "Voltage"
+F 6 "X7R" H 3530 6880 50  0000 R CNN "Dielectric"
+F 7 "1276-2972-1-ND" H 4105 7480 60  0001 C CNN "Digi-Key PN"
+	1    3680 6980
+	1    0    0    -1
+$EndComp
+$Comp
+L power:GND #PWR?
+U 1 1 5EB47981
+P 3680 7130
+F 0 "#PWR?" H 3680 6880 50  0001 C CNN
+F 1 "GND" H 3680 6980 50  0000 C CNN
+F 2 "" H 3680 7130 50  0001 C CNN
+F 3 "" H 3680 7130 50  0001 C CNN
+	1    3680 7130
+	1    0    0    -1
+$EndComp
+Wire Wire Line
+	4390 6830 4390 6750
+Wire Wire Line
+	4390 6750 3680 6750
+Wire Wire Line
+	3680 6750 3680 6830
+$Comp
+L Diode:BAT48JFILM D?
+U 1 1 5EB4A7A8
+P 3680 6520
+F 0 "D?" V 3750 6400 50  0000 R CNN
+F 1 "BAT48JFILM" V 3650 6400 50  0000 R CNN
+F 2 "Diode_SMD:D_SOD-323" H 3680 6345 50  0001 C CNN
+F 3 "www.st.com/resource/en/datasheet/bat48.pdf" H 3680 6520 50  0001 C CNN
+	1    3680 6520
+	0    -1   -1   0
+$EndComp
+Wire Wire Line
+	3680 6670 3680 6750
+Connection ~ 3680 6750
+$Comp
+L power:+3.3V #PWR?
+U 1 1 5EB4C2CE
+P 3680 6370
+F 0 "#PWR?" H 3680 6220 50  0001 C CNN
+F 1 "+3.3V" H 3680 6510 50  0000 C CNN
+F 2 "" H 3680 6370 50  0001 C CNN
+F 3 "" H 3680 6370 50  0001 C CNN
+	1    3680 6370
+	1    0    0    -1
+$EndComp
+Text GLabel 2280 6700 2    50   Output ~ 0
+POS3P3_RUN
 $EndSCHEMATC

Commit message: few sch additions
Parts:
- removed C?: 4.7uF, Capacitors_SMD:C_0402, symbol Custom_Library:C_Custom
- added C?: 10uF, Capacitors_SMD:C_0402, symbol Custom_Library:C_Custom
- added R?: 10, Resistors_SMD:R_0402, symbol Custom_Library:R_Custom
- Q?: Digi-Key PN (none) -> BSS214NWH6327XTSA1CT-ND
Connections:
- net labels added: POS12_PGOOD
Changed lines of the file:
@@
 F 2 "Package_TO_SOT_SMD:SOT-323_SC-70" H 4490 7415 50  0001 L CIN
 F 3 "https://www.infineon.com/dgdl/Infineon-BSS214NW-DS-v02_02-en.pdf?fileId=db3a30431b3e89eb011b695aebc01bde" H 4290 7490 50  0001 L CNN
+F 4 "BSS214NWH6327XTSA1CT-ND" H 4290 7490 50  0001 C CNN "Digi-Key PN"
 	1    4290 7490
 	1    0    0    -1
@@
 	4390 7210 4390 7290
 $Comp
-L Custom_Library:C_Custom C?
-U 1 1 5EB46F8D
-P 3680 6980
-AR Path="/5EAE2F97/5EB46F8D" Ref="C?"  Part="1"
-AR Path="/5EAE2D8A/5EB46F8D" Ref="C?"  Part="1"
-F 0 "C?" H 3705 7080 50  0000 L CNN
-F 1 "4.7uF" H 3705 6880 50  0000 L CNN
-F 2 "Capacitors_SMD:C_0402" H 3718 6830 50  0001 C CNN
-F 3 "" H 3705 7080 50  0001 C CNN
-F 4 "0402" H 3530 7080 50  0000 R CNN "display_footprint"
-F 5 "6.3V" H 3530 6980 50  0000 R CNN "Voltage"
-F 6 "X7R" H 3530 6880 50  0000 R CNN "Dielectric"
-F 7 "1276-2972-1-ND" H 4105 7480 60  0001 C CNN "Digi-Key PN"
-	1    3680 6980
-	1    0    0    -1
-$EndComp
-$Comp
 L power:GND #PWR?
 U 1 1 5EB47981
@@
 Text GLabel 2280 6700 2    50   Output ~ 0
 POS3P3_RUN
+$Comp
+L Custom_Library:R_Custom R?
+U 1 1 5EB895CA
+P 2130 6700
+AR Path="/5EAE2D66/5EB895CA" Ref="R?"  Part="1"
+AR Path="/5EAE2D8A/5EB895CA" Ref="R?"  Part="1"
+F 0 "R?" V 2030 6700 50  0000 C CNN
+F 1 "10" V 2130 6700 50  0000 C CNN
+F 2 "Resistors_SMD:R_0402" H 2130 6700 50  0001 C CNN
+F 3 "" H 2130 6700 50  0001 C CNN
+F 4 "" H 2430 7100 60  0001 C CNN "Digi-Key PN"
+F 5 "0402" V 2230 6700 50  0000 C CNN "display_footprint"
+F 6 "1%" V 2330 6700 50  0000 C CNN "Tolerance"
+F 7 "1/16W" V 2430 6700 50  0000 C CNN "Wattage"
+	1    2130 6700
+	0    1    1    0
+$EndComp
+Text GLabel 1980 6700 0    50   Input ~ 0
+POS12_PGOOD
+$Comp
+L Custom_Library:C_Custom C?
+U 1 1 5EBB9A75
+P 3680 6980
+AR Path="/5CB7718D/5EBB9A75" Ref="C?"  Part="1"
+AR Path="/5E0DC082/5EBB9A75" Ref="C?"  Part="1"
+AR Path="/5E0F9110/5EBB9A75" Ref="C?"  Part="1"
+AR Path="/5A557C58/5EBB9A75" Ref="C?"  Part="1"
+AR Path="/5CB25152/5EBB9A75" Ref="C?"  Part="1"
+AR Path="/5E697934/5EBB9A75" Ref="C?"  Part="1"
+AR Path="/5EAE2F02/5EBB9A75" Ref="C?"  Part="1"
+AR Path="/5EAE3021/5EBB9A75" Ref="C?"  Part="1"
+AR Path="/5EAE2D8A/5EBB9A75" Ref="C?"  Part="1"
+F 0 "C?" H 3705 7080 50  0000 L CNN
+F 1 "10uF" H 3705 6880 50  0000 L CNN
+F 2 "Capacitors_SMD:C_0402" H 3718 6830 50  0001 C CNN
+F 3 "" H 3705 7080 50  0001 C CNN
+F 4 "0402" H 3530 7080 50  0000 R CNN "display_footprint"
+F 5 "6.3V" H 3530 6980 50  0000 R CNN "Voltage"
+F 6 "X5R" H 3530 6880 50  0000 R CNN "Dielectric"
+F 7 "490-13211-1-ND" H 3680 6980 50  0001 C CNN "Digi-Key PN"
+	1    3680 6980
+	1    0    0    -1
+$EndComp
 $EndSCHEMATC

Commit message: Added more stuff to sch
Parts:
- removed C?: 22uF, Capacitors_SMD:C_1206, symbol Custom_Library:C_Custom
- removed U?: TPS62130, Housings_DFN_QFN:QFN-16-1EP_3x3mm_Pitch0.5mm, symbol Custom_Library:TPS62130
- added U?: TPS62150, Package_DFN_QFN:QFN-16-1EP_3x3mm_P0.5mm_EP1.8x1.8mm, symbol Custom_Library:TPS62150
- C?: value 22uF -> 100uF; Dielectric X7R -> X5R; Digi-Key PN 1276-3148-1-ND -> (none); Voltage 10V -> 6.3V
- C? (x2): footprint Capacitors_SMD:C_0603 -> Capacitors_SMD:C_0402; Digi-Key PN 490-8020-1-ND -> 490-10701-1-ND; display_footprint 0603 -> (none)
- C?: footprint Capacitors_SMD:C_0603 -> Capacitors_SMD:C_0402; Digi-Key PN 1276-1921-1-ND -> 490-13295-1-ND; display_footprint 0603 -> (none)
- L?: value 2.2u -> 3.3uH; footprint Inductors_SMD:L_Vishay_IHLP-2020 -> Inductors_SMD:L_Vishay_IHLP-1212; Ampacity 5.5A -> 2.7A; Digi-Key PN 541-1236-1-ND -> 541-2567-1-ND; display_footprint IHLP2020 -> IHLP1212
- R?: footprint Resistors_SMD:R_0603 -> Resistors_SMD:R_0402; Digi-Key PN 311-562KHRCT-ND -> (none); Wattage 1/10W -> 1/16W; display_footprint 0603 -> 0402
- R? (x2): footprint Resistors_SMD:R_0603 -> Resistors_SMD:R_0402; Digi-Key PN RHM10KADCT-ND -> RMCF0402FT10K0CT-ND; Wattage 1/10W -> 1/16W; display_footprint 0603 -> 0402
- R?: footprint Resistors_SMD:R_0603 -> Resistors_SMD:R_0402; Digi-Key PN 749-1763-1-ND -> (none); Wattage 1/10W -> 1/16W; display_footprint 0603 -> 0402
- R? (x4): footprint Resistors_SMD:R_0603 -> Resistors_SMD:R_0402; Digi-Key PN (none) -> 541-3964-1-ND; Wattage 1/10W -> 1/16W; display_footprint 0603 -> 0402
- R?: Digi-Key PN (none) -> 541-3964-1-ND
Connections:
- wire segments 54 -> 52
Other:
- note removed: "CONSIDER A SMALLER SOLUTION WITH LOWER OUTPUT CURRENT"
- moved on the sheet: C?, L?, R?, TP?

Commit message: Added digikey pn's, footprints
Parts:
- C405: renamed from C?; Digi-Key PN (none) -> 587-1963-1-ND
- D401: renamed from D?; Digi-Key PN (none) -> 497-5711-1-ND
- R410: renamed from R?; Digi-Key PN (none) -> 311-562KLRCT-ND
- R411: renamed from R?; Digi-Key PN (none) -> A129654CT-ND
- gave numbers to parts that had none: 19

Commit message: More part arrangements
Parts:
- removed R401, R404: 10, Resistors_SMD:R_0402, symbol Custom_Library:R_Custom
- removed R402: 0.02, Resistors_SMD:R_0612, symbol Custom_Library:R_Custom
Connections:
- net +12V: now also C401.1, C404.1, U401.10 (AVIN), U401.11 (PVIN), U401.12 (PVIN)
Changed lines of the file:
@@
 $Descr A 11000 8500
 encoding utf-8
-Sheet 4 23
+Sheet 4 21
 Title "Pulse Oximeter"
 Date "2019-01-03"
@@
 Wire Wire Line
 	2770 2570 2770 2640
-$Comp
-L power:PWR_FLAG #FLG0401
-U 1 1 5E4082E4
-P 2770 2570
-F 0 "#FLG0401" H 2770 2645 50  0001 C CNN
-F 1 "PWR_FLAG" H 2770 2720 50  0000 C CNN
-F 2 "" H 2770 2570 50  0001 C CNN
-F 3 "~" H 2770 2570 50  0001 C CNN
-	1    2770 2570
-	1    0    0    -1
-$EndComp
-$Comp
-L Custom_Library:R_Custom R?
-U 1 1 5E2B33E5
-P 2300 2950
-AR Path="/5CB0BC26/5E2B33E5" Ref="R?"  Part="1"
-AR Path="/5E1352F5/5E2B33E5" Ref="R?"  Part="1"
-AR Path="/5CB6F1ED/5E2B33E5" Ref="R?"  Part="1"
-AR Path="/5CB7718D/5E2B33E5" Ref="R?"  Part="1"
-AR Path="/5EAE2D8A/5E2B33E5" Ref="R404"  Part="1"
-F 0 "R404" V 2200 2950 50  0000 C CNN
-F 1 "10" V 2300 2950 50  0000 C CNN
-F 2 "Resistors_SMD:R_0402" H 2300 2950 50  0001 C CNN
-F 3 "" H 2300 2950 50  0001 C CNN
-F 4 "0402" V 2400 2950 50  0001 C CNN "display_footprint"
-F 5 "1%" V 2500 2950 50  0001 C CNN "Tolerance"
-F 6 "1/16W" V 2600 2950 50  0001 C CNN "Wattage"
-F 7 "541-3964-1-ND" H 2300 2950 50  0001 C CNN "Digi-Key PN"
-	1    2300 2950
-	-1   0    0    1
-$EndComp
-$Comp
-L Custom_Library:R_Custom R?
-U 1 1 5E2B33DB
-P 1840 2950
-AR Path="/5CB0BC26/5E2B33DB" Ref="R?"  Part="1"
-AR Path="/5E1352F5/5E2B33DB" Ref="R?"  Part="1"
-AR Path="/5CB6F1ED/5E2B33DB" Ref="R?"  Part="1"
-AR Path="/5CB7718D/5E2B33DB" Ref="R?"  Part="1"
-AR Path="/5EAE2D8A/5E2B33DB" Ref="R401"  Part="1"
-F 0 "R401" V 1740 2950 50  0000 C CNN
-F 1 "10" V 1840 2950 50  0000 C CNN
-F 2 "Resistors_SMD:R_0402" H 1840 2950 50  0001 C CNN
-F 3 "" H 1840 2950 50  0001 C CNN
-F 4 "0402" V 1940 2950 50  0001 C CNN "display_footprint"
-F 5 "1%" V 2040 2950 50  0001 C CNN "Tolerance"
-F 6 "1/16W" V 2140 2950 50  0001 C CNN "Wattage"
-F 7 "541-3964-1-ND" H 1840 2950 50  0001 C CNN "Digi-Key PN"
-	1    1840 2950
-	-1   0    0    1
-$EndComp
 Connection ~ 2770 2640
-Connection ~ 1840 2640
-Wire Wire Line
-	1840 2640 1920 2640
-Wire Wire Line
-	1840 2800 1840 2640
-Wire Wire Line
-	2300 2640 2770 2640
-Connection ~ 2300 2640
-Wire Wire Line
-	2300 2800 2300 2640
-Wire Wire Line
-	2220 2640 2300 2640
-Text GLabel 2300 3100 3    50   UnSpc ~ 0
-POS3P3_SNS_IN-
-Text GLabel 1840 3100 3    50   UnSpc ~ 0
-POS3P3_SNS_IN+
-$Comp
-L Custom_Library:R_Custom R?
-U 1 1 5E2AA992
-P 2070 2640
-AR Path="/5CB6F1ED/5E2AA992" Ref="R?"  Part="1"
-AR Path="/5CB7718D/5E2AA992" Ref="R?"  Part="1"
-AR Path="/5E0DC082/5E2AA992" Ref="R?"  Part="1"
-AR Path="/5E0F263A/5E2AA992" Ref="R?"  Part="1"
-AR Path="/5EAE2D8A/5E2AA992" Ref="R402"  Part="1"
-F 0 "R402" V 1970 2640 50  0000 C CNN
-F 1 "0.02" V 2070 2640 40  0000 C CNN
-F 2 "Resistors_SMD:R_0612" H 2070 2640 50  0001 C CNN
-F 3 "" H 2070 2640 50  0001 C CNN
-F 4 "P16010CT-ND" H 2370 3040 60  0001 C CNN "Digi-Key PN"
-F 5 "0612" V 2170 2640 50  0000 C CNN "display_footprint"
-F 6 "1%" V 2270 2640 50  0000 C CNN "Tolerance"
-F 7 "1W" V 2370 2640 50  0000 C CNN "Wattage"
-	1    2070 2640
-	0    -1   -1   0
-$EndComp
 $Comp
 L power:+3.3V #PWR?
@@
 	1    0    0    -1
 $EndComp
-Wire Wire Line
-	1840 2560 1840 2640
 $Comp
 L power:+12V #PWR?
 U 1 1 5E2AA972
-P 1840 2560
+P 2770 2570
 AR Path="/5CB7718D/5E2AA972" Ref="#PWR?"  Part="1"
 AR Path="/5E0DC082/5E2AA972" Ref="#PWR?"  Part="1"
 AR Path="/5E0F263A/5E2AA972" Ref="#PWR?"  Part="1"
 AR Path="/5EAE2D8A/5E2AA972" Ref="#PWR0401"  Part="1"
-F 0 "#PWR0401" H 1840 2410 50  0001 C CNN
-F 1 "+12V" H 1840 2700 50  0000 C CNN
-F 2 "" H 1840 2560 50  0001 C CNN
-F 3 "" H 1840 2560 50  0001 C CNN
-	1    1840 2560
-	1    0    0    -1
-$EndComp
+F 0 "#PWR0401" H 2770 2420 50  0001 C CNN
+F 1 "+12V" H 2770 2710 50  0000 C CNN
+F 2 "" H 2770 2570 50  0001 C CNN
+F 3 "" H 2770 2570 50  0001 C CNN
+	1    2770 2570
+	1    0    0    -1
+$EndComp
