File: hdw/Pulse_Oximeter/POS3P3_Telemetry.sch (KiCad schematic (older format))
At the start: 7 parts, among them U502 MCP9804, U503 INA219BxDCN

Commit message: Set TELEMETRY configs to visible in SCH
Changed lines of the file:
@@
 F 3 "http://ww1.microchip.com/downloads/en/DeviceDoc/22203b.pdf" H 5180 5290 50  0001 C CNN
 F 4 "MCP9804T-E/MCCT-ND" H 5430 4840 50  0001 C CNN "Digi-Key PN"
-F 5 "Telemetry" H 5430 4840 50  0001 C CNN "Configuration"
+F 5 "Telemetry" H 5830 5360 50  0000 C CNN "Configuration"
 	1    5430 4840
 	-1   0    0    -1
@@
 F 3 "http://www.ti.com/lit/ds/symlink/ina219.pdf" H 8530 2110 50  0001 C CNN
 F 4 "296-46420-1-ND" H 8180 2210 50  0001 C CNN "Digi-Key PN"
-F 5 "Telemetry" H 8180 2210 50  0001 C CNN "Configuration"
+F 5 "Telemetry" H 8440 2640 50  0000 C CNN "Configuration"
 	1    8180 2210
 	1    0    0    -1
