File: hdw/Pulse_Oximeter/USB_Telemetry.sch (KiCad schematic (older format))
At the start: 7 parts

Commit message: More sch work
Parts:
- DOC?: value 0x1E -> kjqw3rqwr
- DOC?: value 0x48 -> kjhewkljaefs
Connections:
- net labels added: +3.3V, GND, I2C_SCL, I2C_SDA
- net labels removed: +5V_USB, GND_USB, I2C_USB_SCL, I2C_USB_SDA
Changed lines of the file:
@@
 $EndComp
 Text GLabel 5510 4340 2    50   Input ~ 0
-I2C_USB_SCL
+I2C_SCL
 Text GLabel 5510 4240 2    50   BiDi ~ 0
-I2C_USB_SDA
+I2C_SDA
 NoConn ~ 4710 4540
 $Comp
@@
 AR Path="/5EAE2FAC/5E0CB7BC" Ref="DOC?"  Part="1"
 F 0 "DOC?" H 6010 5810 60  0001 C CNN
-F 1 "0x1E" H 5560 5560 60  0000 L CNN
+F 1 "kjqw3rqwr" H 5560 5560 60  0000 L CNN
 F 2 "" H 6010 5910 60  0001 C CNN
 F 3 "" H 6010 5910 60  0001 C CNN
 	1    6010 5560
-	1    0    0    -1
-$EndComp
-$Comp
-L Custom_Library:+5V_USB #PWR?
-U 1 1 5E0588FF
-P 5110 4040
-F 0 "#PWR?" H 5110 3890 50  0001 C CNN
-F 1 "+5V_USB" H 5110 4180 50  0000 C CNN
-F 2 "" H 5110 4040 50  0001 C CNN
-F 3 "" H 5110 4040 50  0001 C CNN
-	1    5110 4040
-	1    0    0    -1
-$EndComp
-$Comp
-L Custom_Library:+5V_USB #PWR?
-U 1 1 5E058F97
-P 5110 5540
-F 0 "#PWR?" H 5110 5390 50  0001 C CNN
-F 1 "+5V_USB" H 5110 5680 50  0000 C CNN
-F 2 "" H 5110 5540 50  0001 C CNN
-F 3 "" H 5110 5540 50  0001 C CNN
-	1    5110 5540
-	1    0    0    -1
-$EndComp
-$Comp
-L Custom_Library:GND_USB #PWR?
-U 1 1 5E05A2DA
-P 5110 5120
-F 0 "#PWR?" H 5110 4870 50  0001 C CNN
-F 1 "GND_USB" H 5110 4970 50  0000 C CNN
-F 2 "" H 5110 5120 50  0001 C CNN
-F 3 "" H 5110 5120 50  0001 C CNN
-	1    5110 5120
-	1    0    0    -1
-$EndComp
-$Comp
-L Custom_Library:GND_USB #PWR?
-U 1 1 5E05A9FB
-P 5110 5840
-F 0 "#PWR?" H 5110 5590 50  0001 C CNN
-F 1 "GND_USB" H 5110 5690 50  0000 C CNN
-F 2 "" H 5110 5840 50  0001 C CNN
-F 3 "" H 5110 5840 50  0001 C CNN
-	1    5110 5840
 	1    0    0    -1
 $EndComp
@@
 AR Path="/5EAE2FAC/5E200B2A" Ref="DOC?"  Part="1"
 F 0 "DOC?" H 6010 3190 60  0001 C CNN
-F 1 "0x48" H 5560 2940 60  0000 L CNN
+F 1 "kjhewkljaefs" H 5560 2940 60  0000 L CNN
 F 2 "" H 6010 3290 60  0001 C CNN
 F 3 "" H 6010 3290 60  0001 C CNN
@@
 Connection ~ 4230 2320
 Text GLabel 5510 2000 2    50   Input ~ 0
-I2C_USB_SCL
+I2C_SCL
 Text GLabel 5510 1900 2    50   BiDi ~ 0
-I2C_USB_SDA
-$Comp
-L Custom_Library:+5V_USB #PWR?
-U 1 1 5E42C648
-P 5110 1700
-F 0 "#PWR?" H 5110 1550 50  0001 C CNN
-F 1 "+5V_USB" H 5110 1840 50  0000 C CNN
-F 2 "" H 5110 1700 50  0001 C CNN
-F 3 "" H 5110 1700 50  0001 C CNN
-	1    5110 1700
-	1    0    0    -1
-$EndComp
-$Comp
-L Custom_Library:+5V_USB #PWR?
-U 1 1 5E42CB13
-P 5110 2920
-F 0 "#PWR?" H 5110 2770 50  0001 C CNN
-F 1 "+5V_USB" H 5110 3060 50  0000 C CNN
-F 2 "" H 5110 2920 50  0001 C CNN
-F 3 "" H 5110 2920 50  0001 C CNN
-	1    5110 2920
-	1    0    0    -1
-$EndComp
-Text GLabel 5510 2200 2    50   BiDi ~ 0
-I2C_USB_SDA
-$Comp
-L Custom_Library:GND_USB #PWR?
-U 1 1 5E42F98E
-P 5110 2500
-F 0 "#PWR?" H 5110 2250 50  0001 C CNN
-F 1 "GND_USB" H 5110 2350 50  0000 C CNN
-F 2 "" H 5110 2500 50  0001 C CNN
-F 3 "" H 5110 2500 50  0001 C CNN
-	1    5110 2500
-	1    0    0    -1
-$EndComp
-$Comp
-L Custom_Library:GND_USB #PWR?
-U 1 1 5E42FE27
-P 5110 3220
-F 0 "#PWR?" H 5110 2970 50  0001 C CNN
-F 1 "GND_USB" H 5110 3070 50  0000 C CNN
-F 2 "" H 5110 3220 50  0001 C CNN
-F 3 "" H 5110 3220 50  0001 C CNN
-	1    5110 3220
-	1    0    0    -1
-$EndComp
-$Comp
-L Custom_Library:GND_USB #PWR?
-U 1 1 5E4302E4
-P 5510 2300
-F 0 "#PWR?" H 5510 2050 50  0001 C CNN
-F 1 "GND_USB" V 5510 2150 50  0000 R CNN
-F 2 "" H 5510 2300 50  0001 C CNN
-F 3 "" H 5510 2300 50  0001 C CNN
-	1    5510 2300
-	0    -1   -1   0
-$EndComp
-$Comp
-L Custom_Library:GND_USB #PWR?
-U 1 1 5E43080C
-P 5510 4640
-F 0 "#PWR?" H 5510 4390 50  0001 C CNN
-F 1 "GND_USB" V 5510 4490 50  0000 R CNN
-F 2 "" H 5510 4640 50  0001 C CNN
-F 3 "" H 5510 4640 50  0001 C CNN
-	1    5510 4640
-	0    -1   -1   0
-$EndComp
-$Comp
-L Custom_Library:+5V_USB #PWR?
-U 1 1 5E431507
-P 5510 4740
-F 0 "#PWR?" H 5510 4590 50  0001 C CNN
-F 1 "+5V_USB" V 5510 4880 50  0000 L CNN
-F 2 "" H 5510 4740 50  0001 C CNN
-F 3 "" H 5510 4740 50  0001 C CNN
-	1    5510 4740
-	0    1    1    0
-$EndComp
-$Comp
-L Custom_Library:+5V_USB #PWR?
-U 1 1 5E431E8C
-P 5510 4840
-F 0 "#PWR?" H 5510 4690 50  0001 C CNN
-F 1 "+5V_USB" V 5510 4980 50  0000 L CNN
-F 2 "" H 5510 4840 50  0001 C CNN
-F 3 "" H 5510 4840 50  0001 C CNN
-	1    5510 4840
-	0    1    1    0
-$EndComp
+I2C_SDA
 Text GLabel 3790 2320 0    50   UnSpc ~ 0
 POS5_USB_SNS-
 Text GLabel 3790 1860 0    50   UnSpc ~ 0
 POS5_USB_SNS+
+$Comp
+L power:GND #PWR?
+U 1 1 5EB928E1
+P 5110 2500
+F 0 "#PWR?" H 5110 2250 50  0001 C CNN
+F 1 "GND" H 5110 2350 50  0000 C CNN
+F 2 "" H 5110 2500 50  0001 C CNN
+F 3 "" H 5110 2500 50  0001 C CNN
+	1    5110 2500
+	1    0    0    -1
+$EndComp
+$Comp
+L power:GND #PWR?
+U 1 1 5EB92D79
+P 5110 3220
+F 0 "#PWR?" H 5110 2970 50  0001 C CNN
+F 1 "GND" H 5110 3070 50  0000 C CNN
+F 2 "" H 5110 3220 50  0001 C CNN
+F 3 "" H 5110 3220 50  0001 C CNN
+	1    5110 3220
+	1    0    0    -1
+$EndComp
+$Comp
+L power:GND #PWR?
+U 1 1 5EB9320A
+P 5110 5120
+F 0 "#PWR?" H 5110 4870 50  0001 C CNN
+F 1 "GND" H 5110 4970 50  0000 C CNN
+F 2 "" H 5110 5120 50  0001 C CNN
+F 3 "" H 5110 5120 50  0001 C CNN
+	1    5110 5120
+	1    0    0    -1
+$EndComp
+$Comp
+L power:GND #PWR?
+U 1 1 5EB93821
+P 5110 5840
+F 0 "#PWR?" H 5110 5590 50  0001 C CNN
+F 1 "GND" H 5110 5690 50  0000 C CNN
+F 2 "" H 5110 5840 50  0001 C CNN
+F 3 "" H 5110 5840 50  0001 C CNN
+	1    5110 5840
+	1    0    0    -1
+$EndComp
+$Comp
+L power:+3.3V #PWR?
+U 1 1 5EB93D83
+P 5110 5540
+F 0 "#PWR?" H 5110 5390 50  0001 C CNN
+F 1 "+3.3V" H 5110 5680 50  0000 C CNN
+F 2 "" H 5110 5540 50  0001 C CNN
+F 3 "" H 5110 5540 50  0001 C CNN
+	1    5110 5540
+	1    0    0    -1
+$EndComp
+$Comp
+L power:+3.3V #PWR?
+U 1 1 5EB94277
+P 5110 4040
+F 0 "#PWR?" H 5110 3890 50  0001 C CNN
+F 1 "+3.3V" H 5110 4180 50  0000 C CNN
+F 2 "" H 5110 4040 50  0001 C CNN
+F 3 "" H 5110 4040 50  0001 C CNN
+	1    5110 4040
+	1    0    0    -1
+$EndComp
+$Comp
+L power:+3.3V #PWR?
+U 1 1 5EB94BE3
+P 5110 2920
+F 0 "#PWR?" H 5110 2770 50  0001 C CNN
+F 1 "+3.3V" H 5110 3060 50  0000 C CNN
+F 2 "" H 5110 2920 50  0001 C CNN
+F 3 "" H 5110 2920 50  0001 C CNN
+	1    5110 2920
+	1    0    0    -1
+$EndComp
+$Comp
+L power:+3.3V #PWR?
+U 1 1 5EB95503
+P 5110 1700
+F 0 "#PWR?" H 5110 1550 50  0001 C CNN
+F 1 "+3.3V" H 5110 1840 50  0000 C CNN
+F 2 "" H 5110 1700 50  0001 C CNN
+F 3 "" H 5110 1700 50  0001 C CNN
+	1    5110 1700
+	1    0    0    -1
+$EndComp
 $EndSCHEMATC

Commit message: Added more stuff to sch
Parts:
- removed DOC?: kjqw3rqwr, symbol Custom_Library:I2C_Address
- removed DOC?: kjhewkljaefs, symbol Custom_Library:I2C_Address
- added DOC?: 0x45, symbol Custom_Library:I2C_Address
- added DOC?: 0x1B, symbol Custom_Library:I2C_Address
- C? (x3): footprint Capacitors_SMD:C_0603 -> Capacitors_SMD:C_0402; Digi-Key PN 399-6856-1-ND -> 490-10701-1-ND; display_footprint 0603 -> (none)
Connections:
- net +3V3: now also U?.6 (A1), U?.7 (A0), U?.7 (A0), U?.8 (A1)
- net GND: now also U?.5 (A2)
Changed lines of the file:
@@
 $Descr A 11000 8500
 encoding utf-8
-Sheet 13 19
-Title ""
+Sheet 13 20
+Title "Pulse Oximeter"
 Date ""
-Rev ""
-Comp ""
+Rev "A"
+Comp "Drew Maatman"
 Comment1 ""
 Comment2 ""
@@
 F 0 "C?" H 5135 5790 50  0000 L CNN
 F 1 "0.1uF" H 5135 5590 50  0000 L CNN
-F 2 "Capacitors_SMD:C_0603" H 5148 5540 50  0001 C CNN
+F 2 "Capacitors_SMD:C_0402" H 5148 5540 50  0001 C CNN
 F 3 "" H 5135 5790 50  0001 C CNN
-F 4 "0603" H 4960 5790 50  0000 R CNN "display_footprint"
+F 4 "" H 4960 5790 50  0000 R CNN "display_footprint"
 F 5 "50V" H 4960 5690 50  0000 R CNN "Voltage"
 F 6 "X7R" H 4960 5590 50  0000 R CNN "Dielectric"
-F 7 "399-6856-1-ND" H 1200 -1190 50  0001 C CNN "Digi-Key PN"
+F 7 "490-10701-1-ND" H 1200 -1190 50  0001 C CNN "Digi-Key PN"
 	1    5110 5690
-	1    0    0    -1
-$EndComp
-$Comp
-L Custom_Library:I2C_Address DOC?
-U 1 1 5E0CB7BC
-P 6010 5560
-AR Path="/5E0652BA/5E0CB7BC" Ref="DOC?"  Part="1"
-AR Path="/5E0A0E29/5E0CB7BC" Ref="DOC?"  Part="1"
-AR Path="/5E052856/5E0CB7BC" Ref="DOC?"  Part="1"
-AR Path="/5EAE2FAC/5E0CB7BC" Ref="DOC?"  Part="1"
-F 0 "DOC?" H 6010 5810 60  0001 C CNN
-F 1 "kjqw3rqwr" H 5560 5560 60  0000 L CNN
-F 2 "" H 6010 5910 60  0001 C CNN
-F 3 "" H 6010 5910 60  0001 C CNN
-	1    6010 5560
 	1    0    0    -1
 $EndComp
@@
 F 0 "C?" H 5135 3170 50  0000 L CNN
 F 1 "0.1uF" H 5135 2970 50  0000 L CNN
-F 2 "Capacitors_SMD:C_0603" H 5148 2920 50  0001 C CNN
+F 2 "Capacitors_SMD:C_0402" H 5148 2920 50  0001 C CNN
 F 3 "" H 5135 3170 50  0001 C CNN
-F 4 "0603" H 4960 3170 50  0000 R CNN "display_footprint"
+F 4 "" H 4960 3170 50  0000 R CNN "display_footprint"
 F 5 "50V" H 4960 3070 50  0000 R CNN "Voltage"
 F 6 "X7R" H 4960 2970 50  0000 R CNN "Dielectric"
-F 7 "399-6856-1-ND" H 1200 -3810 50  0001 C CNN "Digi-Key PN"
+F 7 "490-10701-1-ND" H 1200 -3810 50  0001 C CNN "Digi-Key PN"
 	1    5110 3070
-	1    0    0    -1
-$EndComp
-$Comp
-L Custom_Library:I2C_Address DOC?
-U 1 1 5E200B2A
-P 6010 2940
-AR Path="/5E0652BA/5E200B2A" Ref="DOC?"  Part="1"
-AR Path="/5E0A0E29/5E200B2A" Ref="DOC?"  Part="1"
-AR Path="/5E052856/5E200B2A" Ref="DOC?"  Part="1"
-AR Path="/5EAE2FAC/5E200B2A" Ref="DOC?"  Part="1"
-F 0 "DOC?" H 6010 3190 60  0001 C CNN
-F 1 "kjhewkljaefs" H 5560 2940 60  0000 L CNN
-F 2 "" H 6010 3290 60  0001 C CNN
-F 3 "" H 6010 3290 60  0001 C CNN
-	1    6010 2940
 	1    0    0    -1
 $EndComp
@@
 F 0 "C?" H 4255 2190 50  0000 L CNN
 F 1 "0.1uF" H 4255 1990 50  0000 L CNN
-F 2 "Capacitors_SMD:C_0603" H 4268 1940 50  0001 C CNN
+F 2 "Capacitors_SMD:C_0402" H 4268 1940 50  0001 C CNN
 F 3 "" H 4255 2190 50  0001 C CNN
-F 4 "0603" H 4080 2190 50  0000 R CNN "display_footprint"
+F 4 "" H 4080 2190 50  0000 R CNN "display_footprint"
 F 5 "50V" H 4080 2090 50  0000 R CNN "Voltage"
 F 6 "X7R" H 4080 1990 50  0000 R CNN "Dielectric"
-F 7 "399-6856-1-ND" H 320 -4790 50  0001 C CNN "Digi-Key PN"
+F 7 "490-10701-1-ND" H 320 -4790 50  0001 C CNN "Digi-Key PN"
 	1    4230 2090
 	1    0    0    -1
@@
 	1    0    0    -1
 $EndComp
+$Comp
+L Custom_Library:I2C_Address DOC?
+U 1 1 5EC33AD2
+P 6010 2940
+AR Path="/5E0652BA/5EC33AD2" Ref="DOC?"  Part="1"
+AR Path="/5E0A0E29/5EC33AD2" Ref="DOC?"  Part="1"
+AR Path="/5E052856/5EC33AD2" Ref="DOC?"  Part="1"
+AR Path="/5EAE2DDC/5EC33AD2" Ref="DOC?"  Part="1"
+AR Path="/5EAE2E6F/5EC33AD2" Ref="DOC?"  Part="1"
+AR Path="/5EAE2FAC/5EC33AD2" Ref="DOC?"  Part="1"
+F 0 "DOC?" H 6010 3190 60  0001 C CNN
+F 1 "0x45" H 5560 2940 60  0000 L CNN
+F 2 "" H 6010 3290 60  0001 C CNN
+F 3 "" H 6010 3290 60  0001 C CNN
+	1    6010 2940
+	1    0    0    -1
+$EndComp
+$Comp
+L power:+3.3V #PWR?
+U 1 1 5EC33D87
+P 5510 2300
+F 0 "#PWR?" H 5510 2150 50  0001 C CNN
+F 1 "+3.3V" V 5510 2440 50  0000 L CNN
+F 2 "" H 5510 2300 50  0001 C CNN
+F 3 "" H 5510 2300 50  0001 C CNN
+	1    5510 2300
+	0    1    1    0
+$EndComp
+$Comp
+L power:+3.3V #PWR?
+U 1 1 5EC34469
+P 5510 2200
+F 0 "#PWR?" H 5510 2050 50  0001 C CNN
+F 1 "+3.3V" V 5510 2340 50  0000 L CNN
+F 2 "" H 5510 2200 50  0001 C CNN
+F 3 "" H 5510 2200 50  0001 C CNN
+	1    5510 2200
+	0    1    1    0
+$EndComp
+$Comp
+L Custom_Library:I2C_Address DOC?
+U 1 1 5EC3977D
+P 6010 5560
+AR Path="/5E0652BA/5EC3977D" Ref="DOC?"  Part="1"
+AR Path="/5E0A0E29/5EC3977D" Ref="DOC?"  Part="1"
+AR Path="/5E0DC084/5EC3977D" Ref="DOC?"  Part="1"
+AR Path="/5E0F263C/5EC3977D" Ref="DOC?"  Part="1"
+AR Path="/5EAE2DDC/5EC3977D" Ref="DOC?"  Part="1"
+AR Path="/5EAE2E6F/5EC3977D" Ref="DOC?"  Part="1"
+AR Path="/5EAE2FAC/5EC3977D" Ref="DOC?"  Part="1"
+F 0 "DOC?" H 6010 5810 60  0001 C CNN
+F 1 "0x1B" H 5560 5560 60  0000 L CNN
+F 2 "" H 6010 5910 60  0001 C CNN
+F 3 "" H 6010 5910 60  0001 C CNN
+	1    6010 5560
+	1    0    0    -1
+$EndComp
+$Comp
+L power:GND #PWR?
+U 1 1 5EC39789
+P 5510 4840
+AR Path="/5EAE2DDC/5EC39789" Ref="#PWR?"  Part="1"
+AR Path="/5EAE2FAC/5EC39789" Ref="#PWR?"  Part="1"
+F 0 "#PWR?" H 5510 4590 50  0001 C CNN
+F 1 "GND" V 5510 4690 50  0000 R CNN
+F 2 "" H 5510 4840 50  0001 C CNN
+F 3 "" H 5510 4840 50  0001 C CNN
+	1    5510 4840
+	0    -1   -1   0
+$EndComp
+$Comp
+L power:+3.3V #PWR?
+U 1 1 5EC3978F
+P 5510 4740
+AR Path="/5E0652BA/5EC3978F" Ref="#PWR?"  Part="1"
+AR Path="/5E0A0E29/5EC3978F" Ref="#PWR?"  Part="1"
+AR Path="/5E0DC084/5EC3978F" Ref="#PWR?"  Part="1"
+AR Path="/5E0F263C/5EC3978F" Ref="#PWR?"  Part="1"
+AR Path="/5EAE2DDC/5EC3978F" Ref="#PWR?"  Part="1"
+AR Path="/5EAE2E6F/5EC3978F" Ref="#PWR?"  Part="1"
+AR Path="/5EAE2FAC/5EC3978F" Ref="#PWR?"  Part="1"
+F 0 "#PWR?" H 5510 4590 50  0001 C CNN
+F 1 "+3.3V" V 5510 4880 50  0000 L CNN
+F 2 "" H 5510 4740 50  0001 C CNN
+F 3 "" H 5510 4740 50  0001 C CNN
+	1    5510 4740
+	0    1    -1   0
+$EndComp
+$Comp
+L power:+3.3V #PWR?
+U 1 1 5EC398CD
+P 5510 4640
+AR Path="/5E0652BA/5EC398CD" Ref="#PWR?"  Part="1"
+AR Path="/5E0A0E29/5EC398CD" Ref="#PWR?"  Part="1"
+AR Path="/5E0DC084/5EC398CD" Ref="#PWR?"  Part="1"
+AR Path="/5E0F263C/5EC398CD" Ref="#PWR?"  Part="1"
+AR Path="/5EAE2DDC/5EC398CD" Ref="#PWR?"  Part="1"
+AR Path="/5EAE2E6F/5EC398CD" Ref="#PWR?"  Part="1"
+AR Path="/5EAE2FAC/5EC398CD" Ref="#PWR?"  Part="1"
+F 0 "#PWR?" H 5510 4490 50  0001 C CNN
+F 1 "+3.3V" V 5510 4780 50  0000 L CNN
+F 2 "" H 5510 4640 50  0001 C CNN
+F 3 "" H 5510 4640 50  0001 C CNN
+	1    5510 4640
+	0    1    -1   0
+$EndComp
 $EndSCHEMATC

Commit message: Added mech sheet, more complicated bullshit you dont need
Parts:
- U? (x2): Configuration (none) -> Telemetry
Changed lines of the file:
@@
 $Descr A 11000 8500
 encoding utf-8
-Sheet 13 22
+Sheet 13 23
 Title "Pulse Oximeter"
 Date ""
@@
 F 3 "http://ww1.microchip.com/downloads/en/DeviceDoc/22203b.pdf" H 4860 4990 50  0001 C CNN
 F 4 "MCP9804T-E/MCCT-ND" H 5110 4540 50  0001 C CNN "Digi-Key PN"
+F 5 "Telemetry" H 5110 4540 50  0001 C CNN "Configuration"
 	1    5110 4540
 	-1   0    0    -1
@@
 F 3 "http://www.ti.com/lit/ds/symlink/ina219.pdf" H 5460 2000 50  0001 C CNN
 F 4 "296-46420-1-ND" H 5110 2100 50  0001 C CNN "Digi-Key PN"
+F 5 "Telemetry" H 5110 2100 50  0001 C CNN "Configuration"
 	1    5110 2100
 	1    0    0    -1
