File: hdw/Pulse_Oximeter/USB_UART_Bridge.sch (KiCad schematic (older format))
At the start: 26 parts

Commit message: Continued schematic development
Parts:
- removed C?: 0.1uF, Capacitors_SMD:C_0402, symbol Custom_Library:C_Custom
- removed R?: 10k, Resistors_SMD:R_0402, symbol Custom_Library:R_Custom
- added R?: 0.02, Resistors_SMD:R_0612, symbol Custom_Library:R_Custom
- added R? (x2): 10, Resistors_SMD:R_0603, symbol Custom_Library:R_Custom
Connections:
- net labels added: +3.3V, POS5_USB_SNS+, POS5_USB_SNS-
- net labels removed: GND_USB
- wire segments 45 -> 47
- no-connect marks 3 -> 4

Commit message: More sch work
Connections:
- net GND: now reaches J?.5 (GND)
- net GND: now also C?.2, C?.2, C?.2, C?.2, C?.2, C?.2, C?.2, C?.2, C?.2, L?.1, R?.2, U?.13 (GND), U?.2 (GND), U?.2 (GND), U?.5 (GND)
- net USB_UART_RX_ISO renamed USB_UART_RX
- net USB_UART_TX_ISO renamed USB_UART_TX
Other:
- note removed: "11. USB UART Bridge"
Changed lines of the file:
@@
 $EndComp
 Text GLabel 2870 3090 0    50   Output ~ 0
-USB_UART_RX_ISO
+USB_UART_RX
 Text GLabel 2870 3190 0    50   Input ~ 0
-USB_UART_TX_ISO
+USB_UART_TX
 NoConn ~ 2870 3290
 NoConn ~ 2870 3390
@@
 Wire Wire Line
 	3470 6590 3470 6390
-Text Notes 550  700  0    100  ~ 20
-11. USB UART Bridge
 $Comp
 L Custom_Library:C_Custom C?
@@
 	1    0    0    -1
 $EndComp
+$Comp
+L power:GND #PWR?
+U 1 1 5EBA2F52
+P 1840 7470
+F 0 "#PWR?" H 1840 7220 50  0001 C CNN
+F 1 "GND" H 1840 7320 50  0000 C CNN
+F 2 "" H 1840 7470 50  0001 C CNN
+F 3 "" H 1840 7470 50  0001 C CNN
+	1    1840 7470
+	1    0    0    -1
+$EndComp
+$Comp
+L power:GND #PWR?
+U 1 1 5EBA3918
+P 2790 7440
+F 0 "#PWR?" H 2790 7190 50  0001 C CNN
+F 1 "GND" H 2790 7290 50  0000 C CNN
+F 2 "" H 2790 7440 50  0001 C CNN
+F 3 "" H 2790 7440 50  0001 C CNN
+	1    2790 7440
+	1    0    0    -1
+$EndComp
+$Comp
+L power:GND #PWR?
+U 1 1 5EBA3F3A
+P 3540 7700
+F 0 "#PWR?" H 3540 7450 50  0001 C CNN
+F 1 "GND" H 3540 7550 50  0000 C CNN
+F 2 "" H 3540 7700 50  0001 C CNN
+F 3 "" H 3540 7700 50  0001 C CNN
+	1    3540 7700
+	1    0    0    -1
+$EndComp
+$Comp
+L power:GND #PWR?
+U 1 1 5EBA4505
+P 4650 4990
+F 0 "#PWR?" H 4650 4740 50  0001 C CNN
+F 1 "GND" H 4650 4840 50  0000 C CNN
+F 2 "" H 4650 4990 50  0001 C CNN
+F 3 "" H 4650 4990 50  0001 C CNN
+	1    4650 4990
+	1    0    0    -1
+$EndComp
+$Comp
+L power:GND #PWR?
+U 1 1 5EBA4B03
+P 3970 4990
+F 0 "#PWR?" H 3970 4740 50  0001 C CNN
+F 1 "GND" H 3970 4840 50  0000 C CNN
+F 2 "" H 3970 4990 50  0001 C CNN
+F 3 "" H 3970 4990 50  0001 C CNN
+	1    3970 4990
+	1    0    0    -1
+$EndComp
+$Comp
+L power:GND #PWR?
+U 1 1 5EBA4FE4
+P 3280 4990
+F 0 "#PWR?" H 3280 4740 50  0001 C CNN
+F 1 "GND" H 3280 4840 50  0000 C CNN
+F 2 "" H 3280 4990 50  0001 C CNN
+F 3 "" H 3280 4990 50  0001 C CNN
+	1    3280 4990
+	1    0    0    -1
+$EndComp
+$Comp
+L power:GND #PWR?
+U 1 1 5EBA52A1
+P 3420 3790
+F 0 "#PWR?" H 3420 3540 50  0001 C CNN
+F 1 "GND" H 3420 3640 50  0000 C CNN
+F 2 "" H 3420 3790 50  0001 C CNN
+F 3 "" H 3420 3790 50  0001 C CNN
+	1    3420 3790
+	1    0    0    -1
+$EndComp
+$Comp
+L power:GND #PWR?
+U 1 1 5EBA5919
+P 3620 3790
+F 0 "#PWR?" H 3620 3540 50  0001 C CNN
+F 1 "GND" H 3620 3640 50  0000 C CNN
+F 2 "" H 3620 3790 50  0001 C CNN
+F 3 "" H 3620 3790 50  0001 C CNN
+	1    3620 3790
+	1    0    0    -1
+$EndComp
+$Comp
+L power:GND #PWR?
+U 1 1 5EBA5C2E
+P 4880 4090
+F 0 "#PWR?" H 4880 3840 50  0001 C CNN
+F 1 "GND" H 4880 3940 50  0000 C CNN
+F 2 "" H 4880 4090 50  0001 C CNN
+F 3 "" H 4880 4090 50  0001 C CNN
+	1    4880 4090
+	1    0    0    -1
+$EndComp
+$Comp
+L power:GND #PWR?
+U 1 1 5EBA6333
+P 6150 3870
+F 0 "#PWR?" H 6150 3620 50  0001 C CNN
+F 1 "GND" H 6150 3720 50  0000 C CNN
+F 2 "" H 6150 3870 50  0001 C CNN
+F 3 "" H 6150 3870 50  0001 C CNN
+	1    6150 3870
+	1    0    0    -1
+$EndComp
+$Comp
+L power:GND #PWR?
+U 1 1 5EBA6B87
+P 6980 3870
+F 0 "#PWR?" H 6980 3620 50  0001 C CNN
+F 1 "GND" H 6980 3720 50  0000 C CNN
+F 2 "" H 6980 3870 50  0001 C CNN
+F 3 "" H 6980 3870 50  0001 C CNN
+	1    6980 3870
+	1    0    0    -1
+$EndComp
+$Comp
+L power:GND #PWR?
+U 1 1 5EBA703C
+P 8910 3690
+F 0 "#PWR?" H 8910 3440 50  0001 C CNN
+F 1 "GND" H 8910 3540 50  0000 C CNN
+F 2 "" H 8910 3690 50  0001 C CNN
+F 3 "" H 8910 3690 50  0001 C CNN
+	1    8910 3690
+	1    0    0    -1
+$EndComp
+$Comp
+L power:GND #PWR?
+U 1 1 5EBA769C
+P 9980 3830
+F 0 "#PWR?" H 9980 3580 50  0001 C CNN
+F 1 "GND" H 9980 3680 50  0000 C CNN
+F 2 "" H 9980 3830 50  0001 C CNN
+F 3 "" H 9980 3830 50  0001 C CNN
+	1    9980 3830
+	1    0    0    -1
+$EndComp
+$Comp
+L power:GND #PWR?
+U 1 1 5EBA7DC6
+P 7900 2600
+F 0 "#PWR?" H 7900 2350 50  0001 C CNN
+F 1 "GND" H 7900 2450 50  0000 C CNN
+F 2 "" H 7900 2600 50  0001 C CNN
+F 3 "" H 7900 2600 50  0001 C CNN
+	1    7900 2600
+	1    0    0    -1
+$EndComp
+$Comp
+L power:GND #PWR?
+U 1 1 5EBA839E
+P 6730 2620
+F 0 "#PWR?" H 6730 2370 50  0001 C CNN
+F 1 "GND" H 6730 2470 50  0000 C CNN
+F 2 "" H 6730 2620 50  0001 C CNN
+F 3 "" H 6730 2620 50  0001 C CNN
+	1    6730 2620
+	1    0    0    -1
+$EndComp
+$Comp
+L power:GND #PWR?
+U 1 1 5EBA85F5
+P 4830 2570
+F 0 "#PWR?" H 4830 2320 50  0001 C CNN
+F 1 "GND" H 4830 2420 50  0000 C CNN
+F 2 "" H 4830 2570 50  0001 C CNN
+F 3 "" H 4830 2570 50  0001 C CNN
+	1    4830 2570
+	1    0    0    -1
+$EndComp

Commit message: Added more stuff to sch
Parts:
- R? (x2): footprint Resistors_SMD:R_0603 -> Resistors_SMD:R_0402; Digi-Key PN (none) -> 541-3964-1-ND; Wattage 1/10W -> 1/16W; display_footprint 0603 -> 0402
Changed lines of the file:
@@
 $Descr A 11000 8500
 encoding utf-8
-Sheet 12 19
-Title "VFD Clock"
+Sheet 12 20
+Title "Pulse Oximeter"
 Date "2019-04-11"
 Rev "A"
@@
 F 0 "R?" V 5150 1890 50  0000 C CNN
 F 1 "10" V 5250 1890 50  0000 C CNN
-F 2 "Resistors_SMD:R_0603" H 5250 1890 50  0001 C CNN
+F 2 "Resistors_SMD:R_0402" H 5250 1890 50  0001 C CNN
 F 3 "" H 5250 1890 50  0001 C CNN
-F 4 "0603" V 5350 1890 50  0001 C CNN "display_footprint"
+F 4 "0402" V 5350 1890 50  0001 C CNN "display_footprint"
 F 5 "1%" V 5450 1890 50  0001 C CNN "Tolerance"
-F 6 "1/10W" V 5550 1890 50  0001 C CNN "Wattage"
+F 6 "1/16W" V 5550 1890 50  0001 C CNN "Wattage"
+F 7 "541-3964-1-ND" H 5250 1890 50  0001 C CNN "Digi-Key PN"
 	1    5250 1890
 	-1   0    0    -1
@@
 F 0 "R?" V 5610 1890 50  0000 C CNN
 F 1 "10" V 5710 1890 50  0000 C CNN
-F 2 "Resistors_SMD:R_0603" H 5710 1890 50  0001 C CNN
+F 2 "Resistors_SMD:R_0402" H 5710 1890 50  0001 C CNN
 F 3 "" H 5710 1890 50  0001 C CNN
-F 4 "0603" V 5810 1890 50  0001 C CNN "display_footprint"
+F 4 "0402" V 5810 1890 50  0001 C CNN "display_footprint"
 F 5 "1%" V 5910 1890 50  0001 C CNN "Tolerance"
-F 6 "1/10W" V 6010 1890 50  0001 C CNN "Wattage"
+F 6 "1/16W" V 6010 1890 50  0001 C CNN "Wattage"
+F 7 "541-3964-1-ND" H 5710 1890 50  0001 C CNN "Digi-Key PN"
 	1    5710 1890
 	-1   0    0    -1

Commit message: Added digikey pn's, footprints
Parts:
- gave numbers to parts that had none: 27

Commit message: More part arrangements
Parts:
- C1204: footprint Capacitors_SMD:C_0805 -> Capacitors_SMD:C_0402; Dielectric X7R -> X5R; Digi-Key PN 1276-2972-1-ND -> 490-14306-1-ND; display_footprint 0805 -> 0402
Changed lines of the file:
@@
 $Descr A 11000 8500
 encoding utf-8
-Sheet 12 23
+Sheet 12 21
 Title "Pulse Oximeter"
 Date "2019-01-03"
@@
 F 0 "C1204" H 4675 4940 50  0000 L CNN
 F 1 "4.7uF" H 4675 4740 50  0000 L CNN
-F 2 "Capacitors_SMD:C_0805" H 4688 4690 50  0001 C CNN
+F 2 "Capacitors_SMD:C_0402" H 4688 4690 50  0001 C CNN
 F 3 "" H 4675 4940 50  0001 C CNN
-F 4 "0805" H 4500 4940 50  0000 R CNN "display_footprint"
+F 4 "0402" H 4500 4940 50  0000 R CNN "display_footprint"
 F 5 "10V" H 4500 4840 50  0000 R CNN "Voltage"
-F 6 "X7R" H 4500 4740 50  0000 R CNN "Dielectric"
-F 7 "1276-2972-1-ND" H 5075 5340 60  0001 C CNN "Digi-Key PN"
+F 6 "X5R" H 4500 4740 50  0000 R CNN "Dielectric"
+F 7 "490-14306-1-ND" H 5075 5340 60  0001 C CNN "Digi-Key PN"
 	1    4650 4840
 	1    0    0    -1
