File: hdw/Pulse_Oximeter/Pushbuttons.sch (KiCad schematic (older format))
At the start: 0 parts

Commit message: Added more stuff to sch
Parts:
- added C601, C602, C609, C610: 0.1uF, Capacitors_SMD:C_0402, symbol Custom_Library:C_Custom
- added C603, C604: 10nF, Capacitors_SMD:C_0402, symbol Custom_Library:C_Custom
- added C? (x4): 10uF, Capacitors_SMD:C_0402, symbol Custom_Library:C_Custom
- added R601, R602: 499, Resistors_SMD:R_0402, symbol Custom_Library:R_Custom
- added R603, R604, R605, R606: 10k, Resistors_SMD:R_0402, symbol Custom_Library:R_Custom
- added SW601, SW602: Cap_Touch, Custom Footprints Library:Capacitive_Touch_Pad, symbol Custom_Library:Cap_Touch
- added U603, U604: AT42QT1010-TSHR, TO_SOT_Packages_SMD:SOT-23-6, symbol Sensor_Touch:AT42QT1010-TSHR
- added U? (x2): TPS71530, Package_TO_SOT_SMD:SOT-353_SC-70-5, symbol Regulator_Linear:TPS71530__SC70
- added U? (x2): 74LVC1G17, TO_SOT_Packages_SMD:SOT-353_SC-70-5, symbol Custom_Library:74LVC1G17_Power
Connections:
- new net: R604.1, R606.2, U604.1 (OUT)
- new net: C604.2, R602.2, U604.3 (SNSK)
- new net: C604.1, U604.4 (SNS)
- new net: C?.1, U604.5 (VDD), U604.6 (SYNC), U?.5 (OUT)
- new net: R602.1, SW602.1 (TP)
- new net: C?.1, R606.1, U?.2
- new net: R603.1, R605.2, U603.1 (OUT)
- new net: C603.2, R601.2, U603.3 (SNSK)
- new net: C603.1, U603.4 (SNS)
- new net: C?.1, U603.5 (VDD), U603.6 (SYNC), U?.5 (OUT)
- new net: R601.1, SW601.1 (TP)
- new net: C?.1, R605.1, U?.2
- new net +3V3: C601.1, C602.1, C609.1, C610.1, U?.4 (IN), U?.4 (IN), U?.5 (VCC), U?.5 (VCC)
- new net Cap_Touch_Power: U?.4
- new net Cap_Touch_Start_Stop: U?.4
- new net GND: C601.2, C602.2, C609.2, C610.2, C?.2, C?.2, C?.2, C?.2, R603.2, R604.2, U603.2 (VSS), U604.2 (VSS), U?.2 (GND), U?.2 (GND), U?.3 (GND), U?.3 (GND)
Other:
- note added: "Consider removing this and making POX sensor automatically start scanning"

Commit message: Added mech sheet, more complicated bullshit you dont need
Parts:
- renumbered C609 to C?, C604 to C?, C610 to C?, C602 to C?, C603 to C?, C601 to C?, R602 to R?, R606 to R?, R601 to R?, R604 to R?, R603 to R?, R605 to R?, SW602 to SW?, SW601 to SW?, U604 to U?, U603 to U?

Commit message: Added digikey pn's, footprints
Parts:
- R1701, R1702: renamed from R?; Digi-Key PN (none) -> RMCF0402FT499RCT-ND
- U1701, U1702: renamed from U?; Digi-Key PN (none) -> 296-15045-1-ND
- gave numbers to parts that had none: 20

Commit message: a few sch tweaks
Parts:
- removed C1701, C1709: 0.1uF, Capacitors_SMD:C_0402, symbol Custom_Library:C_Custom
- removed C1703: 10nF, Capacitors_SMD:C_0402, symbol Custom_Library:C_Custom
- removed C1705, C1707: 10uF, Capacitors_SMD:C_0402, symbol Custom_Library:C_Custom
- removed R1701: 499, Resistors_SMD:R_0402, symbol Custom_Library:R_Custom
- removed R1703, R1705: 10k, Resistors_SMD:R_0402, symbol Custom_Library:R_Custom
- removed SW1701: Cap_Touch, Custom Footprints Library:Capacitive_Touch_Pad, symbol Custom_Library:Cap_Touch
- removed U1701: TPS71530, Package_TO_SOT_SMD:SOT-353_SC-70-5, symbol Regulator_Linear:TPS71530__SC70
- removed U1703: AT42QT1010-TSHR, TO_SOT_Packages_SMD:SOT-23-6, symbol Sensor_Touch:AT42QT1010-TSHR
- removed U1705: 74LVC1G17, TO_SOT_Packages_SMD:SOT-353_SC-70-5, symbol Custom_Library:74LVC1G17_Power
Other:
- note removed: "Consider removing this and making POX sensor automatically start scanning"

Commit message: More part arranging
Parts:
- C1704: display_footprint (none) -> 0402
Changed lines of the file:
@@
 F 3 "" H 4025 2560 50  0001 C CNN
 F 4 "490-13295-1-ND" H -790 240 50  0001 C CNN "Digi-Key PN"
-F 5 "" V 3658 2460 50  0000 C CNN "display_footprint"
+F 5 "0402" V 3658 2460 50  0000 C CNN "display_footprint"
 F 6 "50V" V 3749 2460 50  0000 C CNN "Voltage"
 F 7 "X7R" V 3840 2460 50  0000 C CNN "Dielectric"
