File: hdw/Pulse_Oximeter/Pulse_Oximeter.kicad_pcb (KiCad board)
At the start: 4 copper layers, 314 parts, among them J1201 USB_B_Mini, J2001 I2C, J2002 USB UART, J201 +12V IN, J2101 CR2032 socket, J2201 Micro_SD_Card_Det, J801 PICKIT3, Q201 Si4946BEY, Q2101 BSS214NW, Q401 BSS214NW, Q402 ZXMS6004FFTA, Q801 BSS214NW, SW1701 Cap_Touch, SW1702 Cap_Touch, SW801 MRST, U1101 PIC32MZ0512EFE064T-I_PT, U1201 TLV6700, U1202 FT234XD, U1203 TPD3S014DBVR, U1301 INA219BxDCN, U1302 MCP9804, U1401 DS1683, U1501 TPS22929D, U1502 TCA9803, U1503 MAX30102, U1601 74LVC1G17, U1602 NHD-0420H1Z, U1701 TPS71530, U1702 TPS71530, U1703 AT42QT1010-TSHR, U1704 AT42QT1010-TSHR, U1705 74LVC1G17, U1706 74LVC1G17, U1801 TPS71530, U1802 74LVC1G06, U1803 74LVC1G06, U1804 74LVC1G06, U1805 74LVC1G06, U1806 74LVC1G06, U1901 74LVC1G06, U1902 74LVC1G06, U1903 74LVC1G06, U1904 74LVC1G06, U2001 MCP9804, U201 LTC4365DDB, U2101 DS3231MZ, U301 INA219BxDCN, U302 MCP9804, U401 TPS62150, U501 INA219BxDCN, U502 MCP9804, U503 INA219BxDCN, U601 TPS7A91, U701 INA219BxDCN, U702 MCP9804, U703 INA219BxDCN, X1001 ASE-8.000MHz, X1002 ECS-327KE

Commit message: few sch additions
Parts:
- removed C1701, C1709, C1804: 0.1uF, Capacitors_SMD:C_0402
- removed C1703: 10nF, Capacitors_SMD:C_0402
- removed C1705, C1707: 10uF, Capacitors_SMD:C_0402
- removed D1803: Green, LEDs:LED_0402
- removed R1701: 499, Resistors_SMD:R_0402
- removed R1703, R1705: 10k, Resistors_SMD:R_0402
- removed R1803: 1k, Resistors_SMD:R_0402
- removed RN1601: 10k, Resistors_SMD:R_Array_Convex_8x0602
- removed SW1701: Cap_Touch, Custom Footprints Library:Capacitive_Touch_Pad
- removed U1701: TPS71530, Package_TO_SOT_SMD:SOT-353_SC-70-5
- removed U1703: AT42QT1010-TSHR, TO_SOT_Packages_SMD:SOT-23-6
- removed U1705: 74LVC1G17, TO_SOT_Packages_SMD:SOT-353_SC-70-5
- removed U1804: 74LVC1G06, TO_SOT_Packages_SMD:SOT-353_SC-70-5
- added R1006: 10k, Resistors_SMD:R_0402, F.Cu at (263.6, 95.0)
- added R1606: 10k, Resistors_SMD:R_0402, F.Cu at (132.2, 68.2)
- added R1607: 10k, Resistors_SMD:R_0402, F.Cu at (132.2, 70.4)
- added R1608: 10k, Resistors_SMD:R_0402, F.Cu at (134.9, 68.2)
- added R1609: 10k, Resistors_SMD:R_0402, F.Cu at (134.9, 70.4)
- added R1610: 10k, Resistors_SMD:R_0402, F.Cu at (137.5, 68.2)
- added R1611: 10k, Resistors_SMD:R_0402, F.Cu at (137.5, 70.4)
- added R1612: 10k, Resistors_SMD:R_0402, F.Cu at (140.2, 68.2)
- added R1613: 10k, Resistors_SMD:R_0402, F.Cu at (140.2, 70.4)
- added TP1001: TP, Custom Footprints Library:Test_Point, F.Cu at (260.7, 95.5)
- added TP2101: TP, Custom Footprints Library:Test_Point, F.Cu at (155.6, 98.4)
Connections:
- U1101 pad 10: Net-(U1101-Pad10) -> SD_Logging_Config
- U1101 pad 13: Net-(U1101-Pad13) -> Cap_Touch_Power
- U1101 pad 14: Net-(U1101-Pad14) -> ~POX_INT
- U1101 pad 15: Net-(U1101-Pad15) -> POS3P3_POX_Enable
- U1101 pad 16: Net-(U1101-Pad16) -> POX_I2C_Enable
- U1101 pad 21: Net-(U1101-Pad21) -> SD_SPI_CS
- U1101 pad 22: Net-(U1101-Pad22) -> SD_SPI_MOSI
- U1101 pad 23: Net-(U1101-Pad23) -> SD_SPI_MISO
- U1101 pad 28: Net-(U1101-Pad28) -> ~SD_CARD_DETECT
- U1101 pad 29: Net-(U1101-Pad29) -> SD_SPI_SCLK
- U1101 pad 4: Net-(U1101-Pad4) -> VBAT_ADC
- U1101 pad 43: Net-(U1101-Pad43) -> Error_LED
- U1101 pad 44: Net-(U1101-Pad44) -> CPU_Trap_LED
- U1101 pad 45: Net-(U1101-Pad45) -> Telemetry_Config
- U1101 pad 46: Net-(U1101-Pad46) -> POS1P8_PGOOD
- U1101 pad 47: PIC32MZ_REFCLK -> PIC32MZ_REFCLK1
- U1101 pad 49: Net-(U1101-Pad49) -> POS1P8_RUN
- U1101 pad 5: PIC32MZ_REFCLK1 -> POS3P3_POX_ADC
- U1101 pad 56: Net-(U1101-Pad56) -> Reset_LED
- U1101 pad 57: Net-(U1101-Pad57) -> Heartbeat_LED
- U1101 pad 59: (no net) -> GND
- U1101 pad 60: GND -> +3V3

Commit message: arranged some parts in PCB
Parts:
- R1001, R1004, R1005, R1101, R1102: moved to B.Cu
- moved R2102 419.3 mm to (575.8, 103.2)
- moved C2101 419.3 mm to (568.5, 106.8)
- moved C2102 419.3 mm to (573.0, 103.1)
- moved C2103 419.3 mm to (568.5, 108.8)
- moved J2101 419.3 mm to (550.0, 108.0)
- moved Q2101 419.3 mm to (569.2, 103.9)
- moved R2101 419.3 mm to (571.4, 106.8)
- moved TP2101 419.3 mm to (574.9, 107.6)
- moved U2101 419.3 mm to (571.2, 98.9)
- moved R1601 362.2 mm to (518.9, 45.1)
- moved C1601 362.2 mm to (505.5, 45.0)
- moved C1602 362.2 mm to (493.3, 45.0)
- moved C1603 362.2 mm to (496.3, 45.0)
- moved C1604 362.2 mm to (499.4, 45.0)
- moved C1605 362.2 mm to (502.4, 45.0)
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
Commit message: More part arrangements
Parts:
- removed C2101, C2103, C2202, C501, C502, C701, C702: 0.1uF, Capacitors_SMD:C_0402
- removed C2102, C2203: 10nF, Capacitors_SMD:C_0402
- removed C2201: 10uF, Capacitors_SMD:C_0402
- removed C2204: 1nF, Capacitors_SMD:C_0402
- removed D2201: PESD3V3L5UY, Package_TO_SOT_SMD:SOT-363_SC-70-6
- removed J2101: CR2032 socket, Battery_Holders:Keystone_1058_1x2032-CoinCell
- removed J2201: Micro_SD_Card_Det, Connector_Card:microSD_HC_Molex_104031-0811
- removed Q2101: BSS214NW, Package_TO_SOT_SMD:SOT-323_SC-70
- removed R2101, R2102, R2206, R2207, R2208, R2209, R2210: 10k, Resistors_SMD:R_0402
- removed R2201, R2202, R2203, R2204, R2205, R401, R404, R603, R605: 10, Resistors_SMD:R_0402
- removed R402, R604: 0.02, Resistors_SMD:R_0612
- removed TP2101: TP, Custom Footprints Library:Test_Point
- removed U2101: DS3231MZ, Package_SO:SOIC-8_3.9x4.9mm_P1.27mm
- removed U501, U701: INA219BxDCN, Package_TO_SOT_SMD:SOT-23-8
- added REF**: Symbol_Barrel_Polarity, Symbol:Symbol_Barrel_Polarity, F.Cu at (28.1, 112.3)
- C1201, C1202, C1203, C1206, C1207, C1208, C1401, C1402, C1403, C1404, C301, C302, C303, C503, C504, C505, C703, C704, C705, D1401, D201, R1207, R1208, R205, R206, R208, R601, R602, U1202, U301, U302, U502, U503, U702, U703: moved to B.Cu
- C1204: footprint Capacitors_SMD:C_0805 -> Capacitors_SMD:C_0402; moved to B.Cu
- moved D1401 446.2 mm to (23.2, 69.1), turned to 180 degrees
- moved C1403 442.2 mm to (26.4, 69.5), turned to 270 degrees
- moved C1401 440.1 mm to (25.5, 69.5), turned to 270 degrees
- moved U1401 437.8 mm to (25.4, 70.8)
- moved C1404 434.5 mm to (28.1, 69.5), turned to 270 degrees
- moved C1402 432.3 mm to (27.2, 69.5), turned to 270 degrees
- moved R203 371.5 mm to (36.5, 105.5)
- moved C303 371.0 mm to (35.4, 98.1)
- moved R208 370.5 mm to (35.1, 110.2), turned to 270 degrees
- moved R202 370.0 mm to (34.9, 105.5)
- moved U302 369.7 mm to (36.2, 99.9), turned to 180 degrees
- moved C301 369.2 mm to (41.1, 101.5), turned to 90 degrees
- moved R211 369.0 mm to (34.1, 110.2), turned to 270 degrees
- moved R206 368.9 mm to (38.1, 103.8), turned to 270 degrees
- moved U301 367.6 mm to (43.5, 100.8)
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Connections:
- C401 pad 1: Net-(C401-Pad1) -> +12V
- C404 pad 1: Net-(C401-Pad1) -> +12V
- C601 pad 1: Net-(C601-Pad1) -> +3V3
- U401 pad 10: Net-(C401-Pad1) -> +12V
- U401 pad 11: Net-(C401-Pad1) -> +12V
- U401 pad 12: Net-(C401-Pad1) -> +12V
- U601 pad 10: Net-(C601-Pad1) -> +3V3
- U601 pad 9: Net-(C601-Pad1) -> +3V3
Other:
- board text added: "+"
- board text added: "+1.8V"
- board text added: "+12V"
- board text added: "+12VIN"
- board text added: "-"

Commit message: More part arranging
Parts:
- removed R2003: 10k, Resistors_SMD:R_0402
- removed R2004: 10, Resistors_SMD:R_0402
- added TP1201: TP, Custom Footprints Library:Test_Point, F.Cu at (40.8, 137.6)
- C1301, C1302, C1303, C1708, C1710, C1801, C1802, C1803, C1805, C1806, C1901, C1902, C1903, C1904, C802, Q801, R1706, R1901, R1902, R1905, R1906, R801, R802, R803, R804, R805, U1301, U1302, U1706, U1801: moved to B.Cu
- moved C1303 524.4 mm to (35.6, 142.9), turned to 270 degrees
- moved U1302 521.9 mm to (33.7, 143.9), turned to 90 degrees
- moved U1301 520.6 mm to (39.8, 142.0), turned to 270 degrees
- moved C1302 514.9 mm to (42.0, 142.0), turned to 270 degrees
- moved C1301 514.6 mm to (39.1, 139.6)
- moved R803 357.3 mm to (119.1, 24.0), turned to 180 degrees
- moved C802 357.2 mm to (116.7, 21.8), turned to 90 degrees
- moved R804 356.3 mm to (117.3, 24.0)
- moved R801 351.8 mm to (117.2, 19.6)
- moved R805 350.4 mm to (118.2, 25.1)
- moved R802 347.6 mm to (118.9, 19.6)
- moved Q801 347.3 mm to (118.6, 21.8), turned to 270 degrees
- moved SW801 342.5 mm to (121.3, 23.8), turned to 180 degrees
- moved R1702 338.8 mm to (107.6, 49.6), turned to 90 degrees
- moved C1704 338.5 mm to (110.0, 50.0), turned to 180 degrees
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Other:
- board text added: "+3.3V"
- board text added: "+5V USB"
- board text added: "CPU Trap"
- board text added: "Error"
- board text added: "Heart Beat"
- board text added: "MRST"
- board text added: "PGOOD:"
- board text added: "Power"
- board text added: "Reset/ Prog"
- board text added: "TX/RX"

Commit message: more part groupings
Parts:
- C1502, C1503, C1504, C1505, C1507, C1508, C1509, C1510, C1511, C1512, C1513, C1514, C1601, C1602, C1603, C1604, C1605, R1505, R1506, R1507, R1601, R1602, R1603, R1604, R1605, R1606, R1607, R1608, R1609, R1610, R1611, R1612, R1613, RV1601, U1501, U1601: moved to B.Cu
- moved R1504 394.6 mm to (18.7, 23.2), turned to 180 degrees
- moved C1506 391.5 mm to (18.7, 24.2), turned to 180 degrees
- moved R2001 280.0 mm to (56.4, 154.3)
- moved R2002 280.0 mm to (56.8, 152.1)
- moved C1502 265.3 mm to (129.5, 104.6), turned to 270 degrees
- moved R1505 265.1 mm to (133.8, 104.2)
- moved C1505 264.7 mm to (131.3, 104.6), turned to 270 degrees
- moved H2301 263.8 mm to (60.0, 76.9)
- moved H2302 263.8 mm to (60.0, 84.4)
- moved H2303 263.8 mm to (67.5, 76.9)
- moved H2304 263.8 mm to (67.5, 84.4)
- moved R1506 263.8 mm to (133.8, 105.2)
- moved C1503 261.9 mm to (130.4, 104.6), turned to 270 degrees
- moved R1502 261.3 mm to (130.8, 106.9), turned to 180 degrees
- moved C1504 257.6 mm to (132.1, 104.6), turned to 270 degrees
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Other:
- board text added: "GND"
- board text added: "I2C"
- board text added: "RX"
- board text added: "SCL"
- board text added: "SDA"
- board text added: "TX"
- board text added: "USB UART"

Commit message: Finished grouping parts within PCB outline:
Parts:
- C1201, C1202, C1203, C1204, C1206, C1207, C1208, C1301, C1302, C1303, C1401, C1402, C1403, C1404, C1502, C1503, C1504, C1505, C1507, C1508, C1509, C1510, C1511, C1512, C1513, C1514, C1601, C1602, C1603, C1604, C1605, C1708, C1710, C1801, C504, C505, C703, C704, C705, C802, D1401, D201, Q801, R1207, R1208, R1505, R1506, R1507, R1601, R1602, R1603, R1604, R1605, R1606, R1607, R1608, R1609, R1610, R1611, R1612, R1613, R1706, R601, R602, R801, R802, R803, R804, R805, RV1601, U1202, U1301, U1302, U1501, U1601, U1706, U1801, U503, U702, U703: moved to F.Cu
- C1205, C1209, C1501, C1702, C1704, C1706, C601, C602, C603, C604, C605, J1201, J201, L1201, L1202, R1201, R1202, R1203, R1204, R1205, R1206, R1209, R1501, R1502, R1503, R1702, R1704, R606, R607, R608, R609, R610, REF**, SW1702, U1201, U1203, U1502, U1503, U1602, U1702, U1704, U601: moved to B.Cu
- moved C1801 192.8 mm to (185.4, 67.0), turned to 0 degrees
- moved U1801 192.8 mm to (185.4, 68.9), turned to 180 degrees
- moved C1802 180.4 mm to (169.0, 68.8)
- moved C1803 180.4 mm to (169.0, 81.2)
- moved C1805 180.4 mm to (169.0, 77.1)
- moved C1806 180.4 mm to (169.0, 73.0)
- moved D1801 180.4 mm to (171.7, 69.4)
- moved D1802 180.4 mm to (171.7, 81.7)
- moved D1804 180.4 mm to (171.7, 77.6)
- moved D1805 180.4 mm to (171.7, 73.5)
- moved R1801 180.4 mm to (171.7, 68.3)
- moved R1802 180.4 mm to (171.7, 80.7)
- moved R1804 180.4 mm to (171.7, 76.6)
- moved R1805 180.4 mm to (171.7, 72.5)
- moved U1802 180.4 mm to (169.0, 68.8)
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Other:
- board outline added: 100 x 50 mm
- board text added: "REFCLK1"

Commit message: removed SOSC, started routing
Parts:
- removed C1002: 0.1uF, Capacitors_SMD:C_0402
- removed C1004: 10nF, Capacitors_SMD:C_0402
- removed C1006: 1nF, Capacitors_SMD:C_0402
- removed L1002: 600R 0.5A, Inductors_SMD:L_0402
- removed R1003: 100, Resistors_SMD:R_0402
- removed R1005: 10k, Resistors_SMD:R_0402
- removed X1002: ECS-327KE, Custom Footprints Library:ECS-327KE
- moved C1401 27.5 mm to (126.0, 73.8)
- moved D1401 27.5 mm to (123.8, 73.9)
- moved C1402 27.5 mm to (127.8, 73.8)
- moved C1404 27.5 mm to (128.7, 73.8)
- moved U1401 27.5 mm to (126.2, 77.7)
- moved C1403 27.5 mm to (126.9, 73.8)
- moved C909 1.54 mm to (150.9, 72.8)
Connections:
- U1101 pad 48: PIC32MZ_SOSC -> Net-(U1101-Pad48)
Routing:
- net GND: track 0.00 -> 57.2 mm, vias 0 -> 26
- net +3V3: track 0.00 -> 31.4 mm, vias 0 -> 8
- net PIC32MZ_POSC_EC_Enable: track 0.00 -> 12.4 mm, vias 0 -> 1
- net Net-(R801-Pad1): track 0.00 -> 9.47 mm
- net PIC32MZ_REFCLK1: track 0.00 -> 7.85 mm
- net Telemetry_Config: track 0.00 -> 6.28 mm
- net Net-(C1001-Pad1): track 0.00 -> 4.92 mm
- net GNDA_MZ: track 0.00 -> 4.75 mm
- net +3.3VA_MZ: track 0.00 -> 4.73 mm
- net +12Vin: track 0.00 -> 4.52 mm
- net Net-(C802-Pad1): track 0.00 -> 4.44 mm
- net PIC32MZ_POSC_EC: track 0.00 -> 3.30 mm, vias 0 -> 1
- net POS3P3_POX_ADC: track 0.00 -> 3.19 mm
- net Net-(C1802-Pad1): track 0.00 -> 2.89 mm, vias 0 -> 1
- net LCD_BACKLIGHT: track 0.00 -> 2.30 mm
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- added copper zone on PWR, net +3V3
- added copper zone on GND, net GND

Commit message: More routing
Parts:
- moved C503 4.13 mm to (173.8, 102.0), turned to 180 degrees
- moved U502 1.24 mm to (172.8, 100.2), turned to 0 degrees
- moved C1401 1.14 mm to (126.0, 72.6)
- moved C1402 1.14 mm to (127.8, 72.6)
- moved C1403 1.14 mm to (126.9, 72.6)
- moved C1404 1.14 mm to (128.7, 72.6)
- moved D1401 1.14 mm to (123.8, 72.7)
- moved U1401 1.14 mm to (126.2, 76.6)
- moved C908 0.25 mm to (153.5, 73.5)
- moved C909 0.25 mm to (150.9, 72.6)
- moved C912 0.25 mm to (150.9, 73.5)
- moved C910 0.25 mm to (153.5, 74.4)
- moved C911 0.25 mm to (153.5, 75.2)
- moved C914 0.25 mm to (150.9, 74.4)
- moved C915 0.25 mm to (150.9, 75.2)
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Routing:
- net GND: track 57.2 -> 187.4 mm, vias 26 -> 60
- net LCD_PMP_DB1: track 1.57 -> 67.2 mm
- net LCD_PMP_DB0: track 1.57 -> 60.0 mm, vias 0 -> 1
- net +3V3: track 31.4 -> 87.1 mm, vias 8 -> 25
- net LCD_PMP_E: track 1.57 -> 54.3 mm, vias 0 -> 1
- net LCD_PMP_R_W: track 1.57 -> 52.8 mm, vias 0 -> 1
- net LCD_PMP_DB2: track 1.55 -> 44.1 mm
- net LCD_PMP_DB3: track 1.55 -> 42.5 mm
- net LCD_BACKLIGHT_PWM: track 1.26 -> 41.9 mm, vias 0 -> 2
- net LCD_PMP_RS: track 1.57 -> 41.6 mm, vias 0 -> 1
- net LCD_PMP_DB4: track 1.55 -> 40.8 mm
- net LCD_PMP_DB7: track 1.55 -> 38.3 mm
- net LCD_PMP_DB6: track 1.55 -> 38.2 mm
- net LCD_PMP_DB5: track 1.55 -> 37.3 mm
- net PIC32MZ_ICSPDAT: track 0.00 -> 30.4 mm
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