File: hdw/Pulse_Oximeter/Pulse_Oximeter.kicad_pcb (KiCad board)
At the start: 4 copper layers, 100 x 50 mm, 264 parts, among them J1201 USB_B_Mini, J2001 I2C, J2002 USB UART, J201 +12V IN, J801 PICKIT3, Q201 Si4946BEY, Q401 BSS214NW, Q402 ZXMS6004FFTA, Q801 BSS214NW, SW1702 Cap_Touch, SW801 MRST, U1101 PIC32MZ0512EFE064T-I_PT, U1201 TLV6700, U1202 FT234XD, U1203 TPD3S014DBVR, U1301 INA219BxDCN, U1302 MCP9804, U1401 DS1683, U1501 TPS22929D, U1502 TCA9803, U1503 MAX30102, U1601 74LVC1G17, U1602 NHD-0420H1Z, U1702 TPS71530, U1704 AT42QT1010-TSHR, U1706 74LVC1G17, U1801 TPS71530, U1802 74LVC1G06, U1803 74LVC1G06, U1805 74LVC1G06, U1806 74LVC1G06, U1901 74LVC1G06, U1902 74LVC1G06, U1903 74LVC1G06, U1904 74LVC1G06, U2001 MCP9804, U201 LTC4365DDB, U301 INA219BxDCN, U302 MCP9804, U401 TPS62150, U502 MCP9804, U503 INA219BxDCN, U601 TPS7A91, U702 MCP9804, U703 INA219BxDCN, X1001 ASE-8.000MHz

Commit message: More routing
Parts:
- moved R403 0.80 mm to (176.0, 91.2), turned to 90 degrees
Routing:
- net ~PIC32MZ_MCLR: track 0.00 -> 58.9 mm, vias 0 -> 2
- net USB_UART_TX: track 5.62 -> 62.0 mm, vias 0 -> 2
- net GND: track 187.4 -> 243.6 mm, vias 60 -> 95
- net +12V: track 9.43 -> 49.2 mm, vias 0 -> 2
- net +3V3: track 87.1 -> 124.7 mm, vias 25 -> 53
- net USB_UART_RX: track 5.56 -> 36.7 mm, vias 0 -> 4
- net +5V_USB: track 5.05 -> 28.3 mm, vias 0 -> 2
- net Net-(R205-Pad1): track 3.84 -> 17.9 mm, vias 0 -> 1
- net +12Vin: track 32.9 -> 45.9 mm
- net +1.8V: track 19.9 -> 25.8 mm, vias 2 -> 3
- net Net-(R1505-Pad2): track 0.00 -> 5.45 mm, vias 0 -> 1
- net Net-(R1506-Pad2): track 0.00 -> 5.26 mm, vias 0 -> 1
- net Net-(Q201-Pad1): track 0.00 -> 5.24 mm
- net POS12_PGOOD: track 2.03 -> 7.26 mm, vias 1 -> 2
- net POS1P8_SNS_OUT+: track 0.00 -> 4.58 mm, vias 0 -> 1
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- added copper zone on F.Cu, net +12V
- added copper zone on F.Cu, net +12Vin
- added copper zone on B.Cu, net +3V3
- added copper zone on F.Cu, net +3V3
- added copper zone on F.Cu, net Net-(C405-Pad1)
- added copper zone on B.Cu, net Net-(C603-Pad1)
- added copper zone on F.Cu, net Net-(L401-Pad1)
- added copper zone on F.Cu, net Net-(Q201-Pad5)

Commit message: Mcu hmore routing, ran autorouter
Connections:
- net SD_Logging_Config renamed Net-(U1101-Pad10)
- net SD_SPI_CS renamed Net-(U1101-Pad21)
- net SD_SPI_MISO renamed Net-(U1101-Pad23)
- net SD_SPI_MOSI renamed Net-(U1101-Pad22)
- net SD_SPI_SCLK renamed Net-(U1101-Pad29)
- net VBAT_ADC renamed Net-(U1101-Pad4)
- net ~SD_CARD_DETECT renamed Net-(U1101-Pad28)
Routing:
- net I2C_SCL: track 5.23 -> 249.5 mm, vias 1 -> 10
- net I2C_SDA: track 3.95 -> 238.5 mm, vias 1 -> 7
- net POS1P8_PGOOD: track 1.88 -> 83.4 mm, vias 1 -> 2
- net POS1P8_RUN: track 3.62 -> 71.3 mm, vias 1 -> 2
- net USB_UART_TX: track 62.0 -> 120.0 mm, vias 2 -> 3
- net POS3P3_POX_ADC: track 3.19 -> 57.6 mm, vias 0 -> 1
- net USB_UART_RX: track 36.7 -> 87.7 mm, vias 4 -> 6
- net Cap_Touch_Power: track 0.00 -> 49.3 mm, vias 0 -> 7
- net POS3P3_POX_Enable: track 1.34 -> 46.7 mm, vias 1 -> 2
- net CPU_Trap_LED: track 2.42 -> 38.1 mm, vias 1 -> 2
- net POS3P3_PGOOD: track 2.15 -> 37.3 mm, vias 0 -> 2
- net ~POX_INT: track 0.00 -> 34.7 mm, vias 0 -> 3
- net POS5_USB_PGOOD: track 3.54 -> 36.2 mm, vias 0 -> 1
- net Error_LED: track 2.30 -> 33.0 mm, vias 1 -> 2
- net POX_I2C_Enable: track 2.81 -> 32.7 mm, vias 0 -> 1
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
Commit message: More PCB work, generated BOM
Parts:
- added G***: Microchip_Logo, Custom Footprints Library:Microchip_Logo, F.Cu at (152.5, 82.8)
- added G***: PIC32_Logo, Custom Footprints Library:PIC32_Logo, F.Cu at (152.5, 96.7)
- added G***: Owl_1_Logo, Custom Footprints Library:Owl_1_Logo, F.Cu at (124.8, 94.0)
Other:
- board text added: "1"
- board text added: "2"
- board text added: "3"
- board text added: "4"
- board text added: "JLCJLCJLCJLC"
- board text added: "Layer:"
- board text added: "Pulse Oximeter REV A June 2020"
- board text added: "Track Segments: 1787 Nets: 160 Vias: 256 Components: 276"
- board text added: "USB COM Port: Baud: 115.2kbps Data Bits: 8 Stop Bits: 1 Parity: None Flow Control: None"
