File: hdw/Pulse_Oximeter/Mechanical.sch (KiCad schematic (older format))
At the start: 12 parts

Commit message: Added digikey pn's, footprints
Parts:
- gave numbers to parts that had none: 12
Changed lines of the file:
@@
 encoding utf-8
 Sheet 23 23
-Title "VFD Clock"
-Date "2019-04-11"
+Title "Pulse Oximeter"
+Date "2019-01-03"
 Rev "A"
 Comp "Drew Maatman"
@@
 $EndDescr
 $Comp
-L Mechanical:MountingHole H?
+L Mechanical:MountingHole H2301
 U 1 1 5CC525BF
 P 4070 1580
-F 0 "H?" H 4070 1780 50  0000 C CNN
+F 0 "H2301" H 4070 1780 50  0000 C CNN
 F 1 "MountingHole" H 4070 1705 50  0000 C CNN
 F 2 "MountingHole:MountingHole_3mm" H 4070 1580 50  0001 C CNN
@@
 $EndComp
 $Comp
-L Mechanical:MountingHole H?
+L Mechanical:MountingHole H2303
 U 1 1 5CC5295F
 P 4820 1580
-F 0 "H?" H 4820 1780 50  0000 C CNN
+F 0 "H2303" H 4820 1780 50  0000 C CNN
 F 1 "MountingHole" H 4820 1705 50  0000 C CNN
 F 2 "MountingHole:MountingHole_3mm" H 4820 1580 50  0001 C CNN
@@
 $EndComp
 $Comp
-L Mechanical:MountingHole H?
+L Mechanical:MountingHole H2302
 U 1 1 5CC53950
 P 4070 2080
-F 0 "H?" H 4070 2280 50  0000 C CNN
+F 0 "H2302" H 4070 2280 50  0000 C CNN
 F 1 "MountingHole" H 4070 2205 50  0000 C CNN
 F 2 "MountingHole:MountingHole_3mm" H 4070 2080 50  0001 C CNN
@@
 $EndComp
 $Comp
-L Mechanical:MountingHole H?
+L Mechanical:MountingHole H2304
 U 1 1 5CC5395A
 P 4820 2080
-F 0 "H?" H 4820 2280 50  0000 C CNN
+F 0 "H2304" H 4820 2280 50  0000 C CNN
 F 1 "MountingHole" H 4820 2205 50  0000 C CNN
 F 2 "MountingHole:MountingHole_3mm" H 4820 2080 50  0001 C CNN
@@
 $EndComp
 $Comp
-L Custom_Library:Standoff MK?
+L Custom_Library:Standoff MK2301
 U 1 1 5CC60957
 P 4070 3560
-F 0 "MK?" H 4070 3710 50  0000 C CNN
+F 0 "MK2301" H 4070 3710 50  0000 C CNN
 F 1 "Standoff" H 4070 3810 50  0000 C CNN
 F 2 "" H 4070 3910 50  0001 C CNN
@@
 $EndComp
 $Comp
-L Custom_Library:Standoff MK?
+L Custom_Library:Standoff MK2305
 U 1 1 5CC60961
 P 4820 3560
-F 0 "MK?" H 4820 3710 50  0000 C CNN
+F 0 "MK2305" H 4820 3710 50  0000 C CNN
 F 1 "Standoff" H 4820 3810 50  0000 C CNN
 F 2 "" H 4820 3910 50  0001 C CNN
@@
 $EndComp
 $Comp
-L Custom_Library:Standoff MK?
+L Custom_Library:Standoff MK2302
 U 1 1 5CC6097F
 P 4070 4060
-F 0 "MK?" H 4070 4210 50  0000 C CNN
+F 0 "MK2302" H 4070 4210 50  0000 C CNN
 F 1 "Standoff" H 4070 4310 50  0000 C CNN
 F 2 "" H 4070 4410 50  0001 C CNN
@@
 $EndComp
 $Comp
-L Custom_Library:Standoff MK?
+L Custom_Library:Standoff MK2306
 U 1 1 5CC60989
 P 4820 4060
-F 0 "MK?" H 4820 4210 50  0000 C CNN
+F 0 "MK2306" H 4820 4210 50  0000 C CNN
 F 1 "Standoff" H 4820 4310 50  0000 C CNN
 F 2 "" H 4820 4410 50  0001 C CNN
@@
 $EndComp
 $Comp
-L Custom_Library:Screw MK?
+L Custom_Library:Screw MK2303
 U 1 1 5CC6CBF3
 P 4070 5670
-F 0 "MK?" H 4070 5770 50  0000 C CNN
+F 0 "MK2303" H 4070 5770 50  0000 C CNN
 F 1 "Screw" H 4070 5870 50  0000 C CNN
 F 2 "" H 4070 5920 50  0001 C CNN
@@
 $EndComp
 $Comp
-L Custom_Library:Screw MK?
+L Custom_Library:Screw MK2307
 U 1 1 5CC6D1A5
 P 4820 5670
-F 0 "MK?" H 4820 5770 50  0000 C CNN
+F 0 "MK2307" H 4820 5770 50  0000 C CNN
 F 1 "Screw" H 4820 5870 50  0000 C CNN
 F 2 "" H 4820 5920 50  0001 C CNN
@@
 $EndComp
 $Comp
-L Custom_Library:Screw MK?
+L Custom_Library:Screw MK2304
 U 1 1 5CC70A99
 P 4070 6170
-F 0 "MK?" H 4070 6270 50  0000 C CNN
+F 0 "MK2304" H 4070 6270 50  0000 C CNN
 F 1 "Screw" H 4070 6370 50  0000 C CNN
 F 2 "" H 4070 6420 50  0001 C CNN
@@
 $EndComp
 $Comp
-L Custom_Library:Screw MK?
+L Custom_Library:Screw MK2308
 U 1 1 5CC70AA3
 P 4820 6170
-F 0 "MK?" H 4820 6270 50  0000 C CNN
+F 0 "MK2308" H 4820 6270 50  0000 C CNN
 F 1 "Screw" H 4820 6370 50  0000 C CNN
 F 2 "" H 4820 6420 50  0001 C CNN
