File: hdw/Pulse_Oximeter/PIC32MZ_Bypass.sch (KiCad schematic (older format))
At the start: 31 parts

Commit message: Continued schematic development
Parts:
- removed C? (x2): 0.1uF, Capacitors_SMD:C_0402, symbol Custom_Library:C_Custom
- removed C? (x2): 1nF, Capacitors_SMD:C_0402, symbol Custom_Library:C_Custom
- removed C? (x2): 10nF, Capacitors_SMD:C_0402, symbol Custom_Library:C_Custom
- removed C?: 10uF, Capacitors_SMD:C_0402, symbol Custom_Library:C_Custom
- removed C?: 22uF, Capacitors_SMD:C_1206, symbol Custom_Library:C_Custom

Commit message: Added digikey pn's, footprints
Parts:
- gave numbers to parts that had none: 23
