File: hdw/Pulse_Oximeter/POS12_Input.sch (KiCad schematic (older format))
At the start: 24 parts

Commit message: few sch additions
Parts:
- removed R?: 100k, Resistors_SMD:R_0402, symbol Custom_Library:R_Custom
- removed R?: 5.1k, Resistors_SMD:R_0402, symbol Custom_Library:R_Custom
- added R? (x2): 5.23k, Resistors_SMD:R_0402, symbol Custom_Library:R_Custom
- added R?: 13.7k, Resistors_SMD:R_0402, symbol Custom_Library:R_Custom
- added R?: 243k, Resistors_SMD:R_0402, symbol Custom_Library:R_Custom
Connections:
- wire segments 71 -> 70
Other:
- moved on the sheet: C?, D?, J?, Q?A, Q?B, R?, TP?, U?

Commit message: Added more stuff to sch
Parts:
- R? (x4): Digi-Key PN (none) -> 541-3964-1-ND
Changed lines of the file:
@@
 $Descr A 11000 8500
 encoding utf-8
-Sheet 2 19
-Title "QI Charger"
+Sheet 2 20
+Title "Pulse Oximeter"
 Date "2019-01-03"
 Rev "A"
-Comp ""
+Comp "Drew Maatman"
 Comment1 ""
 Comment2 ""
@@
 F 2 "Resistors_SMD:R_0402" H 4490 2660 50  0001 C CNN
 F 3 "" H 4490 2660 50  0001 C CNN
-F 4 "" H 4790 3060 60  0001 C CNN "Digi-Key PN"
+F 4 "541-3964-1-ND" H 4790 3060 60  0001 C CNN "Digi-Key PN"
 F 5 "0402" V 4590 2660 50  0000 C CNN "display_footprint"
 F 6 "1%" V 4690 2660 50  0000 C CNN "Tolerance"
@@
 F 2 "Resistors_SMD:R_0402" H 5360 2660 50  0001 C CNN
 F 3 "" H 5360 2660 50  0001 C CNN
-F 4 "" H 5660 3060 60  0001 C CNN "Digi-Key PN"
+F 4 "541-3964-1-ND" H 5660 3060 60  0001 C CNN "Digi-Key PN"
 F 5 "0402" V 5460 2660 50  0000 C CNN "display_footprint"
 F 6 "1%" V 5560 2660 50  0000 C CNN "Tolerance"
@@
 F 5 "1%" V 6330 2040 50  0001 C CNN "Tolerance"
 F 6 "1/16W" V 6430 2040 50  0001 C CNN "Wattage"
+F 7 "541-3964-1-ND" H 6130 2040 50  0001 C CNN "Digi-Key PN"
 	1    6130 2040
 	-1   0    0    -1
@@
 F 5 "1%" V 6790 2040 50  0001 C CNN "Tolerance"
 F 6 "1/16W" V 6890 2040 50  0001 C CNN "Wattage"
+F 7 "541-3964-1-ND" H 6590 2040 50  0001 C CNN "Digi-Key PN"
 	1    6590 2040
 	-1   0    0    -1

Commit message: Added digikey pn's, footprints
Parts:
- R201: renamed from R?; Digi-Key PN (none) -> 541-CRCW04026M04FKEDCT-ND
- R202: renamed from R?; Digi-Key PN (none) -> 541-86.6KLCT-ND
- R203, R204: renamed from R?; Digi-Key PN (none) -> YAG3070CT-ND
- R207: renamed from R?; Digi-Key PN (none) -> RMCF0402FT13K7CT-ND
- R208, R211: renamed from R?; Digi-Key PN (none) -> RMCF0402FT5K23CT-ND
- R213: renamed from R?; Digi-Key PN (none) -> RMCF0402FT10K0CT-ND
- gave numbers to parts that had none: 17
