File: hdw/Pulse_Oximeter/Pulse_Oximeter.sch (KiCad schematic (older format))
At the start: 0 parts

Commit message: Added more stuff to sch
Changed lines of the file:
@@
 $Descr A 11000 8500
 encoding utf-8
-Sheet 1 19
-Title ""
-Date "2020-05-02"
-Rev ""
-Comp ""
+Sheet 1 20
+Title "Pulse Oximeter"
+Date "2020-05-10"
+Rev "A"
+Comp "Drew Maatman"
 Comment1 ""
 Comment2 ""
@@
 F1 "Status_LEDs.sch" 50
 $EndSheet
+$Sheet
+S 5320 2020 500  150
+U 5EBEB0C5
+F0 "Misc Circuits" 50
+F1 "Misc_Circuits.sch" 50
+$EndSheet
 $EndSCHEMATC

Commit message: Added SD card slot and backup RTC
Changed lines of the file:
@@
 $Descr A 11000 8500
 encoding utf-8
-Sheet 1 20
+Sheet 1 22
 Title "Pulse Oximeter"
 Date "2020-05-10"
@@
 F1 "Misc_Circuits.sch" 50
 $EndSheet
+$Sheet
+S 5320 2370 500  150
+U 5EB8C603
+F0 "Backup RTC" 50
+F1 "Backup_RTC.sch" 50
+$EndSheet
+$Sheet
+S 5320 2720 500  150
+U 5EB8D6D6
+F0 "SD Card Slot" 50
+F1 "SD_Card_Slot.sch" 50
+$EndSheet
 $EndSCHEMATC

Commit message: Added mech sheet, more complicated bullshit you dont need
Changed lines of the file:
@@
 $Descr A 11000 8500
 encoding utf-8
-Sheet 1 22
+Sheet 1 23
 Title "Pulse Oximeter"
 Date "2020-05-10"
@@
 F1 "SD_Card_Slot.sch" 50
 $EndSheet
+$Sheet
+S 5320 3070 500  150
+U 5EC12282
+F0 "Mechanical" 50
+F1 "Mechanical.sch" 50
+$EndSheet
 $EndSCHEMATC

Commit message: More part arrangements
Changed lines of the file:
@@
 $Descr A 11000 8500
 encoding utf-8
-Sheet 1 23
+Sheet 1 21
 Title "Pulse Oximeter"
 Date "2019-01-03"
@@
 $EndSheet
 $Sheet
-S 5320 3070 500  150
+S 5320 2370 500  150
 U 5EC12282
 F0 "Mechanical" 50
 F1 "Mechanical.sch" 50
 $EndSheet
-$Sheet
-S 5320 2720 500  150
-U 5EB8D6D6
-F0 "SD Card Slot" 50
-F1 "SD_Card_Slot.sch" 50
-$EndSheet
-$Sheet
-S 5320 2370 500  150
-U 5EB8C603
-F0 "Backup RTC" 50
-F1 "Backup_RTC.sch" 50
-$EndSheet
 $EndSCHEMATC

Commit message: Cleaned up schematic, generated PCB renders
Other:
- note added: "01. Table of Contents"
- note added: "02. +12V Input"
- note added: "03. +12V Telemetry"
- note added: "04. +3.3V Power Supply"
- note added: "05. +3.3V Telemetry"
- note added: "06. +1.8V Power Supply"
- note added: "07. +1.8V Telemetry"
- note added: "08. PIC32MZ Programming"
- note added: "09. PIC32MZ Bypass"
- note added: "10. PIC32MZ Clocking"
- note added: "11. PIC32MZ"
- note added: "12. USB UART Bridge"
- note added: "13. USB Telemetry"
- note added: "14. Time of Flight"
- note added: "15. POX Sensor"
- note added: "16. Display"
- note added: "17. Pushbuttons"
- note added: "18. PGOOD LEDs"
- note added: "19. Status LEDs"
- note added: "20. Misc Circuits"
- note added: "21. Mechanical"
- note added: "Pulse Oximeter"
Changed lines of the file:
@@
 Sheet 1 21
 Title "Pulse Oximeter"
-Date "2019-01-03"
+Date "2020-08-01"
 Rev "A"
 Comp "Drew Maatman"
@@
 $EndDescr
 $Sheet
-S 2470 1320 500  150
+S 4320 1730 500  150
 U 5EAE2D66
 F0 "+12V Input" 50
@@
 $EndSheet
 $Sheet
-S 2470 1670 500  150
+S 4320 2080 500  150
 U 5EAE2D84
 F0 "+12V Telemetry" 50
@@
 $EndSheet
 $Sheet
-S 2470 2020 500  150
+S 4320 2430 500  150
 U 5EAE2D8A
 F0 "+3.3V Power Supply" 50
@@
 $EndSheet
 $Sheet
-S 2470 2370 500  150
+S 4320 2780 500  150
 U 5EAE2DDC
 F0 "+3.3V Telemetry" 50
@@
 $EndSheet
 $Sheet
-S 2470 2720 500  150
+S 4320 3130 500  150
 U 5EAE2E5F
 F0 "+1.8V Power Supply" 50
@@
 $EndSheet
 $Sheet
-S 2470 3070 500  160
+S 4320 3480 500  160
 U 5EAE2E6F
 F0 "+1.8V Telemetry" 50
@@
 $EndSheet
 $Sheet
-S 2470 3420 500  150
+S 4320 3830 500  150
 U 5EAE2EF2
 F0 "PIC32MZ Programming" 50
@@
 $EndSheet
 $Sheet
-S 2470 3770 500  150
+S 4320 4180 500  150
 U 5EAE2F02
 F0 "PIC32MZ Bypass" 50
@@
 $EndSheet
 $Sheet
-S 2470 4120 500  150
+S 4320 4530 500  150
 U 5EAE2F15
 F0 "PIC32MZ Clocking" 50
@@
 $EndSheet
 $Sheet
-S 2470 4470 500  150
+S 4320 4880 500  150
 U 5EAE2F23
 F0 "PIC32MZ" 50
@@
 $EndSheet
 $Sheet
-S 2470 4820 500  150
+S 4320 5230 500  150
 U 5EAE2F97
 F0 "USB UART Bridge" 50
@@
 $EndSheet
 $Sheet
-S 2470 5170 500  150
+S 4320 5580 500  150
 U 5EAE2FAC
 F0 "USB Telemetry" 50
@@
 $EndSheet
 $Sheet
-S 2470 5520 500  150
+S 4320 5930 500  150
 U 5EAE3021
 F0 "Time of Flight" 50
@@
 $EndSheet
 $Sheet
-S 2470 5870 500  150
+S 4320 6280 500  150
 U 5EAE30C7
 F0 "POX Sensor" 50
@@
 $EndSheet
 $Sheet
-S 2470 6220 500  150
+S 4320 6630 500  150
 U 5EAE4A89
 F0 "Display" 50
@@
 $EndSheet
 $Sheet
-S 2470 6570 500  150
+S 4320 6980 500  150
 U 5EAE4AB6
 F0 "Pushbuttons" 50
@@
 $EndSheet
 $Sheet
-S 5320 1320 500  150
+S 7570 1730 500  150
 U 5EAE4ADE
 F0 "PGOOD LEDs" 50
@@
 $EndSheet
 $Sheet
-S 5320 1670 500  150
+S 7570 2080 500  150
 U 5EAE4AE4
 F0 "Status LEDs" 50
@@
 $EndSheet
 $Sheet
-S 5320 2020 500  150
+S 7570 2430 500  150
 U 5EBEB0C5
 F0 "Misc Circuits" 50
@@
 $EndSheet
 $Sheet
-S 5320 2370 500  150
+S 7570 2780 500  150
 U 5EC12282
 F0 "Mechanical" 50
 F1 "Mechanical.sch" 50
 $EndSheet
+Text Notes 4120 950  0    250  ~ 50
+Pulse Oximeter
+Text Notes 2160 1880 0    100  ~ 20
+02. +12V Input
+Text Notes 2160 2230 0    100  ~ 20
+03. +12V Telemetry
+Text Notes 2160 2580 0    100  ~ 20
+04. +3.3V Power Supply
+Text Notes 2160 2930 0    100  ~ 20
+05. +3.3V Telemetry
+Text Notes 2160 3280 0    100  ~ 20
+06. +1.8V Power Supply
+Text Notes 2160 3640 0    100  ~ 20
+07. +1.8V Telemetry
+Text Notes 2160 3980 0    100  ~ 20
+08. PIC32MZ Programming
+Text Notes 2160 4330 0    100  ~ 20
+09. PIC32MZ Bypass
+Text Notes 2160 4680 0    100  ~ 20
+10. PIC32MZ Clocking
+Text Notes 2160 5030 0    100  ~ 20
+11. PIC32MZ
+Text Notes 2160 5380 0    100  ~ 20
+12. USB UART Bridge
+Text Notes 2160 5730 0    100  ~ 20
+13. USB Telemetry
+Text Notes 2160 6080 0    100  ~ 20
+14. Time of Flight
+Text Notes 2160 6430 0    100  ~ 20
+15. POX Sensor
+Text Notes 2160 6780 0    100  ~ 20
+16. Display
+Text Notes 2160 7130 0    100  ~ 20
+17. Pushbuttons
+Text Notes 2160 1530 0    100  ~ 20
+01. Table of Contents
+Text Notes 5810 1880 0    100  ~ 20
+18. PGOOD LEDs
+Text Notes 5810 2230 0    100  ~ 20
+19. Status LEDs
+Text Notes 5810 2580 0    100  ~ 20
+20. Misc Circuits
+Text Notes 5810 2930 0    100  ~ 20
+21. Mechanical
 $EndSCHEMATC
