File: hdw/Pulse_Oximeter/Misc_Circuits.sch (KiCad schematic (older format))
At the start: 7 parts

Commit message: Added mech sheet, more complicated bullshit you dont need
Parts:
- added R?: 10k, Resistors_SMD:R_0402, symbol Custom_Library:R_Custom
- added R?: 10, Resistors_SMD:R_0402, symbol Custom_Library:R_Custom
- U?: Configuration (none) -> Telemetry
Connections:
- net +3V3: now also R?.1
- net GND: now also R?.2
- new net SD_Logging_Config: R?.1, R?.2
Changed lines of the file:
@@
 $Descr A 11000 8500
 encoding utf-8
-Sheet 20 22
+Sheet 20 23
 Title "Pulse Oximeter"
 Date ""
@@
 F 3 "http://ww1.microchip.com/downloads/en/DeviceDoc/22203b.pdf" H 4950 2690 50  0001 C CNN
 F 4 "MCP9804T-E/MCCT-ND" H 5200 2240 50  0001 C CNN "Digi-Key PN"
+F 5 "Telemetry" H 5200 2240 50  0001 C CNN "Configuration"
 	1    5200 2240
 	-1   0    0    -1
@@
 	0    -1   -1   0
 $EndComp
+$Comp
+L Custom_Library:R_Custom R?
+U 1 1 5EC05B32
+P 7050 4930
+AR Path="/5BB27BA3/5EC05B32" Ref="R?"  Part="1"
+AR Path="/5BB27BF7/5EC05B32" Ref="R?"  Part="1"
+AR Path="/5C1DE17A/5EC05B32" Ref="R?"  Part="1"
+AR Path="/5C1E3A08/5EC05B32" Ref="R?"  Part="1"
+AR Path="/5D779AE1/5EC05B32" Ref="R?"  Part="1"
+AR Path="/5CB7718D/5EC05B32" Ref="R?"  Part="1"
+AR Path="/5E0DC082/5EC05B32" Ref="R?"  Part="1"
+AR Path="/5E0F9110/5EC05B32" Ref="R?"  Part="1"
+AR Path="/5E9E0EA5/5EC05B32" Ref="R?"  Part="1"
+AR Path="/5E9E0E87/5EC05B32" Ref="R?"  Part="1"
+AR Path="/5EAE2D66/5EC05B32" Ref="R?"  Part="1"
+AR Path="/5EAE4A89/5EC05B32" Ref="R?"  Part="1"
+AR Path="/5EAE2F23/5EC05B32" Ref="R?"  Part="1"
+AR Path="/5EBEB0C5/5EC05B32" Ref="R?"  Part="1"
+F 0 "R?" H 6970 4930 50  0000 R CNN
+F 1 "10k" V 7050 4930 50  0000 C CNN
+F 2 "Resistors_SMD:R_0402" H 7050 4930 50  0001 C CNN
+F 3 "" H 7050 4930 50  0001 C CNN
+F 4 "0402" H 7150 5010 50  0000 L CNN "display_footprint"
+F 5 "1%" H 7150 4930 50  0000 L CNN "Tolerance"
+F 6 "1/16W" H 7160 4850 50  0000 L CNN "Wattage"
+	1    7050 4930
+	1    0    0    -1
+$EndComp
+$Comp
+L power:+3.3V #PWR?
+U 1 1 5EC05B3C
+P 7050 4780
+F 0 "#PWR?" H 7050 4630 50  0001 C CNN
+F 1 "+3.3V" H 7050 4920 50  0000 C CNN
+F 2 "" H 7050 4780 50  0001 C CNN
+F 3 "" H 7050 4780 50  0001 C CNN
+	1    7050 4780
+	1    0    0    -1
+$EndComp
+$Comp
+L power:GND #PWR?
+U 1 1 5EC05B46
+P 7050 5540
+F 0 "#PWR?" H 7050 5290 50  0001 C CNN
+F 1 "GND" H 7050 5390 50  0000 C CNN
+F 2 "" H 7050 5540 50  0001 C CNN
+F 3 "" H 7050 5540 50  0001 C CNN
+	1    7050 5540
+	1    0    0    -1
+$EndComp
+$Comp
+L Custom_Library:R_Custom R?
+U 1 1 5EC05B55
+P 7050 5390
+AR Path="/5BB27BA3/5EC05B55" Ref="R?"  Part="1"
+AR Path="/5BB27BF7/5EC05B55" Ref="R?"  Part="1"
+AR Path="/5C1DE17A/5EC05B55" Ref="R?"  Part="1"
+AR Path="/5C1E3A08/5EC05B55" Ref="R?"  Part="1"
+AR Path="/5D779AE1/5EC05B55" Ref="R?"  Part="1"
+AR Path="/5CB7718D/5EC05B55" Ref="R?"  Part="1"
+AR Path="/5E0DC082/5EC05B55" Ref="R?"  Part="1"
+AR Path="/5E0F9110/5EC05B55" Ref="R?"  Part="1"
+AR Path="/5E9E0EA5/5EC05B55" Ref="R?"  Part="1"
+AR Path="/5E9E0E87/5EC05B55" Ref="R?"  Part="1"
+AR Path="/5EAE2D66/5EC05B55" Ref="R?"  Part="1"
+AR Path="/5EAE4A89/5EC05B55" Ref="R?"  Part="1"
+AR Path="/5EAE2F23/5EC05B55" Ref="R?"  Part="1"
+AR Path="/5EBEB0C5/5EC05B55" Ref="R?"  Part="1"
+F 0 "R?" H 6970 5390 50  0000 R CNN
+F 1 "10" V 7050 5390 50  0000 C CNN
+F 2 "Resistors_SMD:R_0402" H 7050 5390 50  0001 C CNN
+F 3 "" H 7050 5390 50  0001 C CNN
+F 4 "0402" H 7150 5470 50  0000 L CNN "display_footprint"
+F 5 "1%" H 7150 5390 50  0000 L CNN "Tolerance"
+F 6 "1/16W" H 7160 5310 50  0000 L CNN "Wattage"
+F 7 "SD Logging" H 7160 5230 50  0000 L CNN "Configuration"
+F 8 "541-3964-1-ND" H 7050 5390 50  0001 C CNN "Digi-Key PN"
+	1    7050 5390
+	1    0    0    -1
+$EndComp
+Wire Wire Line
+	7050 5240 7050 5160
+Text GLabel 7130 5160 2    50   UnSpc ~ 0
+SD_Logging_Config
+Wire Wire Line
+	7130 5160 7050 5160
+Connection ~ 7050 5160
+Wire Wire Line
+	7050 5160 7050 5080
 $EndSCHEMATC

Commit message: Added digikey pn's, footprints
Parts:
- J2001, J2002: renamed from J?; footprint (none) -> Connector_PinHeader_2.54mm:PinHeader_1x03_P2.54mm_Vertical
- R2001, R2003: renamed from R?; Digi-Key PN (none) -> RMCF0402FT10K0CT-ND
- gave numbers to parts that had none: 5
Changed lines of the file:
@@
 Sheet 20 23
 Title "Pulse Oximeter"
-Date ""
+Date "2019-01-03"
 Rev "A"
 Comp "Drew Maatman"
@@
 AR Path="/5E0F263C/5EBEF913" Ref="#PWR?"  Part="1"
 AR Path="/5EAE2E6F/5EBEF913" Ref="#PWR?"  Part="1"
-AR Path="/5EBEB0C5/5EBEF913" Ref="#PWR?"  Part="1"
-F 0 "#PWR?" H 5200 2570 50  0001 C CNN
+AR Path="/5EBEB0C5/5EBEF913" Ref="#PWR02004"  Part="1"
+F 0 "#PWR02004" H 5200 2570 50  0001 C CNN
 F 1 "GND" H 5200 2670 50  0000 C CNN
 F 2 "" H 5200 2820 50  0001 C CNN
@@
 AR Path="/5E0F263C/5EBEF91E" Ref="#PWR?"  Part="1"
 AR Path="/5EAE2E6F/5EBEF91E" Ref="#PWR?"  Part="1"
-AR Path="/5EBEB0C5/5EBEF91E" Ref="#PWR?"  Part="1"
-F 0 "#PWR?" H 5200 1590 50  0001 C CNN
+AR Path="/5EBEB0C5/5EBEF91E" Ref="#PWR02003"  Part="1"
+F 0 "#PWR02003" H 5200 1590 50  0001 C CNN
 F 1 "+3.3V" H 5200 1880 50  0000 C CNN
 F 2 "" H 5200 1740 50  0001 C CNN
@@
 AR Path="/5E0F263C/5EBEF925" Ref="U?"  Part="1"
 AR Path="/5EAE2E6F/5EBEF925" Ref="U?"  Part="1"
-AR Path="/5EBEB0C5/5EBEF925" Ref="U?"  Part="1"
-F 0 "U?" H 4950 2690 50  0000 C CNN
+AR Path="/5EBEB0C5/5EBEF925" Ref="U2001"  Part="1"
+F 0 "U2001" H 4950 2690 50  0000 C CNN
 F 1 "MCP9804" H 5600 2690 50  0000 C CNN
 F 2 "Package_DFN_QFN:DFN-8-1EP_3x2mm_P0.5mm_EP1.3x1.5mm" H 4100 1740 50  0001 C CNN
@@
 AR Path="/5E0F263C/5EBEF932" Ref="C?"  Part="1"
 AR Path="/5EAE2E6F/5EBEF932" Ref="C?"  Part="1"
-AR Path="/5EBEB0C5/5EBEF932" Ref="C?"  Part="1"
-F 0 "C?" H 5225 3490 50  0000 L CNN
+AR Path="/5EBEB0C5/5EBEF932" Ref="C2001"  Part="1"
+F 0 "C2001" H 5225 3490 50  0000 L CNN
 F 1 "0.1uF" H 5225 3290 50  0000 L CNN
 F 2 "Capacitors_SMD:C_0402" H 5238 3240 50  0001 C CNN
@@
 AR Path="/5E0F263C/5EBEF938" Ref="#PWR?"  Part="1"
 AR Path="/5EAE2E6F/5EBEF938" Ref="#PWR?"  Part="1"
-AR Path="/5EBEB0C5/5EBEF938" Ref="#PWR?"  Part="1"
-F 0 "#PWR?" H 5200 3090 50  0001 C CNN
+AR Path="/5EBEB0C5/5EBEF938" Ref="#PWR02005"  Part="1"
+F 0 "#PWR02005" H 5200 3090 50  0001 C CNN
 F 1 "+3.3V" H 5200 3380 50  0000 C CNN
 F 2 "" H 5200 3240 50  0001 C CNN
@@
 AR Path="/5E0F263C/5EBEF93E" Ref="#PWR?"  Part="1"
 AR Path="/5EAE2E6F/5EBEF93E" Ref="#PWR?"  Part="1"
-AR Path="/5EBEB0C5/5EBEF93E" Ref="#PWR?"  Part="1"
-F 0 "#PWR?" H 5200 3290 50  0001 C CNN
+AR Path="/5EBEB0C5/5EBEF93E" Ref="#PWR02006"  Part="1"
+F 0 "#PWR02006" H 5200 3290 50  0001 C CNN
 F 1 "GND" H 5200 3390 50  0000 C CNN
 F 2 "" H 5200 3540 50  0001 C CNN
@@
 $EndComp
 $Comp
-L Connector_Generic:Conn_01x03 J?
+L Connector_Generic:Conn_01x03 J2001
 U 1 1 5EBF5609
 P 3850 5190
-F 0 "J?" H 3850 5390 50  0000 C CNN
+F 0 "J2001" H 3850 5390 50  0000 C CNN
 F 1 "I2C" H 3850 4990 50  0000 C CNN
-F 2 "" H 3850 5190 50  0001 C CNN
+F 2 "Connector_PinHeader_2.54mm:PinHeader_1x03_P2.54mm_Vertical" H 3850 5190 50  0001 C CNN
 F 3 "~" H 3850 5190 50  0001 C CNN
 	1    3850 5190
@@
 $EndComp
 $Comp
-L power:GND #PWR?
+L power:GND #PWR02001
 U 1 1 5EBF560F
 P 3570 5370
-F 0 "#PWR?" H 3570 5120 50  0001 C CNN
+F 0 "#PWR02001" H 3570 5120 50  0001 C CNN
 F 1 "GND" H 3570 5220 50  0000 C CNN
 F 2 "" H 3570 5370 50  0001 C CNN
@@
 	3570 5290 3650 5290
 $Comp
-L Connector_Generic:Conn_01x03 J?
+L Connector_Generic:Conn_01x03 J2002
 U 1 1 5EBF5617
 P 5000 5190
-F 0 "J?" H 5000 5390 50  0000 C CNN
+F 0 "J2002" H 5000 5390 50  0000 C CNN
 F 1 "USB UART" H 5000 4990 50  0000 C CNN
-F 2 "" H 5000 5190 50  0001 C CNN
+F 2 "Connector_PinHeader_2.54mm:PinHeader_1x03_P2.54mm_Vertical" H 5000 5190 50  0001 C CNN
 F 3 "~" H 5000 5190 50  0001 C CNN
 	1    5000 5190
@@
 $EndComp
 $Comp
-L power:GND #PWR?
+L power:GND #PWR02002
 U 1 1 5EBF561D
 P 4720 5370
-F 0 "#PWR?" H 4720 5120 50  0001 C CNN
+F 0 "#PWR02002" H 4720 5120 50  0001 C CNN
 F 1 "GND" H 4720 5220 50  0000 C CNN
 F 2 "" H 4720 5370 50  0001 C CNN
@@
 AR Path="/5EAE4A89/5EBF562C" Ref="R?"  Part="1"
 AR Path="/5EAE2F23/5EBF562C" Ref="R?"  Part="1"
-AR Path="/5EBEB0C5/5EBF562C" Ref="R?"  Part="1"
-F 0 "R?" H 5490 4930 50  0000 R CNN
+AR Path="/5EBEB0C5/5EBF562C" Ref="R2001"  Part="1"
+F 0 "R2001" H 5490 4930 50  0000 R CNN
 F 1 "10k" V 5570 4930 50  0000 C CNN
 F 2 "Resistors_SMD:R_0402" H 5570 4930 50  0001 C CNN
@@
 F 5 "1%" H 5670 4930 50  0000 L CNN "Tolerance"
 F 6 "1/16W" H 5680 4850 50  0000 L CNN "Wattage"
+F 7 "RMCF0402FT10K0CT-ND" H 5570 4930 50  0001 C CNN "Digi-Key PN"
 	1    5570 4930
 	1    0    0    -1
 $EndComp
 $Comp
-L power:+3.3V #PWR?
+L power:+3.3V #PWR02007
 U 1 1 5EBF5632
 P 5570 4780
-F 0 "#PWR?" H 5570 4630 50  0001 C CNN
+F 0 "#PWR02007" H 5570 4630 50  0001 C CNN
 F 1 "+3.3V" H 5570 4920 50  0000 C CNN
 F 2 "" H 5570 4780 50  0001 C CNN
@@
 $EndComp
 $Comp
-L power:GND #PWR?
+L power:GND #PWR02008
 U 1 1 5EBF5638
 P 5570 5540
-F 0 "#PWR?" H 5570 5290 50  0001 C CNN
+F 0 "#PWR02008" H 5570 5290 50  0001 C CNN
 F 1 "GND" H 5570 5390 50  0000 C CNN
 F 2 "" H 5570 5540 50  0001 C CNN
@@
 AR Path="/5EAE4A89/5EBF5642" Ref="R?"  Part="1"
 AR Path="/5EAE2F23/5EBF5642" Ref="R?"  Part="1"
-AR Path="/5EBEB0C5/5EBF5642" Ref="R?"  Part="1"
-F 0 "R?" H 5490 5390 50  0000 R CNN
+AR Path="/5EBEB0C5/5EBF5642" Ref="R2002"  Part="1"
+F 0 "R2002" H 5490 5390 50  0000 R CNN
 F 1 "10" V 5570 5390 50  0000 C CNN
 F 2 "Resistors_SMD:R_0402" H 5570 5390 50  0001 C CNN
@@
 AR Path="/5EAE2E6F/5EC3C1C7" Ref="DOC?"  Part="1"
 AR Path="/5EAE2FAC/5EC3C1C7" Ref="DOC?"  Part="1"
-AR Path="/5EBEB0C5/5EC3C1C7" Ref="DOC?"  Part="1"
-F 0 "DOC?" H 6100 3510 60  0001 C CNN
+AR Path="/5EBEB0C5/5EC3C1C7" Ref="DOC2001"  Part="1"
+F 0 "DOC2001" H 6100 3510 60  0001 C CNN
 F 1 "0x1C" H 5650 3260 60  0000 L CNN
 F 2 "" H 6100 3610 60  0001 C CNN
@@
 P 5600 2440
 AR Path="/5EAE2DDC/5EC3C1CD" Ref="#PWR?"  Part="1"
-AR Path="/5EBEB0C5/5EC3C1CD" Ref="#PWR?"  Part="1"
-F 0 "#PWR?" H 5600 2190 50  0001 C CNN
+AR Path="/5EBEB0C5/5EC3C1CD" Ref="#PWR02010"  Part="1"
+F 0 "#PWR02010" H 5600 2190 50  0001 C CNN
 F 1 "GND" V 5600 2290 50  0000 R CNN
 F 2 "" H 5600 2440 50  0001 C CNN
@@
 AR Path="/5EAE2E6F/5EC3C1D3" Ref="#PWR?"  Part="1"
 AR Path="/5EAE2FAC/5EC3C1D3" Ref="#PWR?"  Part="1"
-AR Path="/5EBEB0C5/5EC3C1D3" Ref="#PWR?"  Part="1"
-F 0 "#PWR?" H 5600 2390 50  0001 C CNN
+AR Path="/5EBEB0C5/5EC3C1D3" Ref="#PWR02011"  Part="1"
+F 0 "#PWR02011" H 5600 2390 50  0001 C CNN
 F 1 "+3.3V" V 5600 2680 50  0000 L CNN
 F 2 "" H 5600 2540 50  0001 C CNN
@@
 P 5600 2340
 AR Path="/5EAE2DDC/5EC3C90F" Ref="#PWR?"  Part="1"
-AR Path="/5EBEB0C5/5EC3C90F" Ref="#PWR?"  Part="1"
-F 0 "#PWR?" H 5600 2090 50  0001 C CNN
+AR Path="/5EBEB0C5/5EC3C90F" Ref="#PWR02009"  Part="1"
+F 0 "#PWR02009" H 5600 2090 50  0001 C CNN
 F 1 "GND" V 5600 2190 50  0000 R CNN
 F 2 "" H 5600 2340 50  0001 C CNN
@@
 AR Path="/5EAE4A89/5EC05B32" Ref="R?"  Part="1"
 AR Path="/5EAE2F23/5EC05B32" Ref="R?"  Part="1"
-AR Path="/5EBEB0C5/5EC05B32" Ref="R?"  Part="1"
-F 0 "R?" H 6970 4930 50  0000 R CNN
+AR Path="/5EBEB0C5/5EC05B32" Ref="R2003"  Part="1"
+F 0 "R2003" H 6970 4930 50  0000 R CNN
 F 1 "10k" V 7050 4930 50  0000 C CNN
 F 2 "Resistors_SMD:R_0402" H 7050 4930 50  0001 C CNN
@@
 F 5 "1%" H 7150 4930 50  0000 L CNN "Tolerance"
 F 6 "1/16W" H 7160 4850 50  0000 L CNN "Wattage"
+F 7 "RMCF0402FT10K0CT-ND" H 7050 4930 50  0001 C CNN "Digi-Key PN"
 	1    7050 4930
 	1    0    0    -1
 $EndComp
 $Comp
-L power:+3.3V #PWR?
+L power:+3.3V #PWR02012
 U 1 1 5EC05B3C
 P 7050 4780
-F 0 "#PWR?" H 7050 4630 50  0001 C CNN
+F 0 "#PWR02012" H 7050 4630 50  0001 C CNN
 F 1 "+3.3V" H 7050 4920 50  0000 C CNN
 F 2 "" H 7050 4780 50  0001 C CNN
@@
 $EndComp
 $Comp
-L power:GND #PWR?
+L power:GND #PWR02013
 U 1 1 5EC05B46
 P 7050 5540
-F 0 "#PWR?" H 7050 5290 50  0001 C CNN
+F 0 "#PWR02013" H 7050 5290 50  0001 C CNN
 F 1 "GND" H 7050 5390 50  0000 C CNN
 F 2 "" H 7050 5540 50  0001 C CNN
@@
 AR Path="/5EAE4A89/5EC05B55" Ref="R?"  Part="1"
 AR Path="/5EAE2F23/5EC05B55" Ref="R?"  Part="1"
-AR Path="/5EBEB0C5/5EC05B55" Ref="R?"  Part="1"
-F 0 "R?" H 6970 5390 50  0000 R CNN
+AR Path="/5EBEB0C5/5EC05B55" Ref="R2004"  Part="1"
+F 0 "R2004" H 6970 5390 50  0000 R CNN
 F 1 "10" V 7050 5390 50  0000 C CNN
 F 2 "Resistors_SMD:R_0402" H 7050 5390 50  0001 C CNN

Commit message: More part arranging
Parts:
- removed R2003: 10k, Resistors_SMD:R_0402, symbol Custom_Library:R_Custom
- removed R2004: 10, Resistors_SMD:R_0402, symbol Custom_Library:R_Custom
Changed lines of the file:
@@
 	0    -1   -1   0
 $EndComp
-$Comp
-L Custom_Library:R_Custom R?
-U 1 1 5EC05B32
-P 7050 4930
-AR Path="/5BB27BA3/5EC05B32" Ref="R?"  Part="1"
-AR Path="/5BB27BF7/5EC05B32" Ref="R?"  Part="1"
-AR Path="/5C1DE17A/5EC05B32" Ref="R?"  Part="1"
-AR Path="/5C1E3A08/5EC05B32" Ref="R?"  Part="1"
-AR Path="/5D779AE1/5EC05B32" Ref="R?"  Part="1"
-AR Path="/5CB7718D/5EC05B32" Ref="R?"  Part="1"
-AR Path="/5E0DC082/5EC05B32" Ref="R?"  Part="1"
-AR Path="/5E0F9110/5EC05B32" Ref="R?"  Part="1"
-AR Path="/5E9E0EA5/5EC05B32" Ref="R?"  Part="1"
-AR Path="/5E9E0E87/5EC05B32" Ref="R?"  Part="1"
-AR Path="/5EAE2D66/5EC05B32" Ref="R?"  Part="1"
-AR Path="/5EAE4A89/5EC05B32" Ref="R?"  Part="1"
-AR Path="/5EAE2F23/5EC05B32" Ref="R?"  Part="1"
-AR Path="/5EBEB0C5/5EC05B32" Ref="R2003"  Part="1"
-F 0 "R2003" H 6970 4930 50  0000 R CNN
-F 1 "10k" V 7050 4930 50  0000 C CNN
-F 2 "Resistors_SMD:R_0402" H 7050 4930 50  0001 C CNN
-F 3 "" H 7050 4930 50  0001 C CNN
-F 4 "0402" H 7150 5010 50  0000 L CNN "display_footprint"
-F 5 "1%" H 7150 4930 50  0000 L CNN "Tolerance"
-F 6 "1/16W" H 7160 4850 50  0000 L CNN "Wattage"
-F 7 "RMCF0402FT10K0CT-ND" H 7050 4930 50  0001 C CNN "Digi-Key PN"
-	1    7050 4930
-	1    0    0    -1
-$EndComp
-$Comp
-L power:+3.3V #PWR02012
-U 1 1 5EC05B3C
-P 7050 4780
-F 0 "#PWR02012" H 7050 4630 50  0001 C CNN
-F 1 "+3.3V" H 7050 4920 50  0000 C CNN
-F 2 "" H 7050 4780 50  0001 C CNN
-F 3 "" H 7050 4780 50  0001 C CNN
-	1    7050 4780
-	1    0    0    -1
-$EndComp
-$Comp
-L power:GND #PWR02013
-U 1 1 5EC05B46
-P 7050 5540
-F 0 "#PWR02013" H 7050 5290 50  0001 C CNN
-F 1 "GND" H 7050 5390 50  0000 C CNN
-F 2 "" H 7050 5540 50  0001 C CNN
-F 3 "" H 7050 5540 50  0001 C CNN
-	1    7050 5540
-	1    0    0    -1
-$EndComp
-$Comp
-L Custom_Library:R_Custom R?
-U 1 1 5EC05B55
-P 7050 5390
-AR Path="/5BB27BA3/5EC05B55" Ref="R?"  Part="1"
-AR Path="/5BB27BF7/5EC05B55" Ref="R?"  Part="1"
-AR Path="/5C1DE17A/5EC05B55" Ref="R?"  Part="1"
-AR Path="/5C1E3A08/5EC05B55" Ref="R?"  Part="1"
-AR Path="/5D779AE1/5EC05B55" Ref="R?"  Part="1"
-AR Path="/5CB7718D/5EC05B55" Ref="R?"  Part="1"
-AR Path="/5E0DC082/5EC05B55" Ref="R?"  Part="1"
-AR Path="/5E0F9110/5EC05B55" Ref="R?"  Part="1"
-AR Path="/5E9E0EA5/5EC05B55" Ref="R?"  Part="1"
-AR Path="/5E9E0E87/5EC05B55" Ref="R?"  Part="1"
-AR Path="/5EAE2D66/5EC05B55" Ref="R?"  Part="1"
-AR Path="/5EAE4A89/5EC05B55" Ref="R?"  Part="1"
-AR Path="/5EAE2F23/5EC05B55" Ref="R?"  Part="1"
-AR Path="/5EBEB0C5/5EC05B55" Ref="R2004"  Part="1"
-F 0 "R2004" H 6970 5390 50  0000 R CNN
-F 1 "10" V 7050 5390 50  0000 C CNN
-F 2 "Resistors_SMD:R_0402" H 7050 5390 50  0001 C CNN
-F 3 "" H 7050 5390 50  0001 C CNN
-F 4 "0402" H 7150 5470 50  0000 L CNN "display_footprint"
-F 5 "1%" H 7150 5390 50  0000 L CNN "Tolerance"
-F 6 "1/16W" H 7160 5310 50  0000 L CNN "Wattage"
-F 7 "SD Logging" H 7160 5230 50  0000 L CNN "Configuration"
-F 8 "541-3964-1-ND" H 7050 5390 50  0001 C CNN "Digi-Key PN"
-	1    7050 5390
-	1    0    0    -1
-$EndComp
-Wire Wire Line
-	7050 5240 7050 5160
-Text GLabel 7130 5160 2    50   UnSpc ~ 0
-SD_Logging_Config
-Wire Wire Line
-	7130 5160 7050 5160
-Connection ~ 7050 5160
-Wire Wire Line
-	7050 5160 7050 5080
 $EndSCHEMATC

Commit message: Set TELEMETRY configs to visible in SCH
Changed lines of the file:
@@
 F 3 "http://ww1.microchip.com/downloads/en/DeviceDoc/22203b.pdf" H 4950 2690 50  0001 C CNN
 F 4 "MCP9804T-E/MCCT-ND" H 5200 2240 50  0001 C CNN "Digi-Key PN"
-F 5 "Telemetry" H 5200 2240 50  0001 C CNN "Configuration"
+F 5 "Telemetry" H 5600 2770 50  0000 C CNN "Configuration"
 	1    5200 2240
 	-1   0    0    -1
