File: hdw/Pulse_Oximeter/POS12_Telemetry.sch (KiCad schematic (older format))
At the start: 7 parts

Commit message: Added more stuff to sch
Parts:
- C? (x3): footprint Capacitors_SMD:C_0603 -> Capacitors_SMD:C_0402; Digi-Key PN 399-6856-1-ND -> 490-10701-1-ND; display_footprint 0603 -> (none)
Changed lines of the file:
@@
 $Descr A 11000 8500
 encoding utf-8
-Sheet 3 19
-Title ""
+Sheet 3 20
+Title "Pulse Oximeter"
 Date ""
-Rev ""
-Comp ""
+Rev "A"
+Comp "Drew Maatman"
 Comment1 ""
 Comment2 ""
@@
 F 0 "C?" H 5135 3110 50  0000 L CNN
 F 1 "0.1uF" H 5135 2910 50  0000 L CNN
-F 2 "Capacitors_SMD:C_0603" H 5148 2860 50  0001 C CNN
+F 2 "Capacitors_SMD:C_0402" H 5148 2860 50  0001 C CNN
 F 3 "" H 5135 3110 50  0001 C CNN
-F 4 "0603" H 4960 3110 50  0000 R CNN "display_footprint"
+F 4 "" H 4960 3110 50  0000 R CNN "display_footprint"
 F 5 "50V" H 4960 3010 50  0000 R CNN "Voltage"
 F 6 "X7R" H 4960 2910 50  0000 R CNN "Dielectric"
-F 7 "399-6856-1-ND" H 1200 -3870 50  0001 C CNN "Digi-Key PN"
+F 7 "490-10701-1-ND" H 1200 -3870 50  0001 C CNN "Digi-Key PN"
 	1    5110 3010
 	1    0    0    -1
@@
 F 0 "C?" H 5135 5790 50  0000 L CNN
 F 1 "0.1uF" H 5135 5590 50  0000 L CNN
-F 2 "Capacitors_SMD:C_0603" H 5148 5540 50  0001 C CNN
+F 2 "Capacitors_SMD:C_0402" H 5148 5540 50  0001 C CNN
 F 3 "" H 5135 5790 50  0001 C CNN
-F 4 "0603" H 4960 5790 50  0000 R CNN "display_footprint"
+F 4 "" H 4960 5790 50  0000 R CNN "display_footprint"
 F 5 "50V" H 4960 5690 50  0000 R CNN "Voltage"
 F 6 "X7R" H 4960 5590 50  0000 R CNN "Dielectric"
-F 7 "399-6856-1-ND" H 1200 -1190 50  0001 C CNN "Digi-Key PN"
+F 7 "490-10701-1-ND" H 1200 -1190 50  0001 C CNN "Digi-Key PN"
 	1    5110 5690
 	1    0    0    -1
@@
 F 0 "C?" H 4255 2130 50  0000 L CNN
 F 1 "0.1uF" H 4255 1930 50  0000 L CNN
-F 2 "Capacitors_SMD:C_0603" H 4268 1880 50  0001 C CNN
+F 2 "Capacitors_SMD:C_0402" H 4268 1880 50  0001 C CNN
 F 3 "" H 4255 2130 50  0001 C CNN
-F 4 "0603" H 4080 2130 50  0000 R CNN "display_footprint"
+F 4 "" H 4080 2130 50  0000 R CNN "display_footprint"
 F 5 "50V" H 4080 2030 50  0000 R CNN "Voltage"
 F 6 "X7R" H 4080 1930 50  0000 R CNN "Dielectric"
-F 7 "399-6856-1-ND" H 320 -4850 50  0001 C CNN "Digi-Key PN"
+F 7 "490-10701-1-ND" H 320 -4850 50  0001 C CNN "Digi-Key PN"
 	1    4230 2030
 	1    0    0    -1

Commit message: Added mech sheet, more complicated bullshit you dont need
Parts:
- U? (x2): Configuration (none) -> Telemetry
Changed lines of the file:
@@
 $Descr A 11000 8500
 encoding utf-8
-Sheet 3 22
+Sheet 3 23
 Title "Pulse Oximeter"
 Date ""
@@
 F 3 "http://ww1.microchip.com/downloads/en/DeviceDoc/22203b.pdf" H 4860 4990 50  0001 C CNN
 F 4 "MCP9804T-E/MCCT-ND" H 5110 4540 50  0001 C CNN "Digi-Key PN"
+F 5 "Telemetry" H 5110 4540 50  0001 C CNN "Configuration"
 	1    5110 4540
 	-1   0    0    -1
@@
 F 3 "http://www.ti.com/lit/ds/symlink/ina219.pdf" H 5460 1940 50  0001 C CNN
 F 4 "296-46420-1-ND" H 5110 2040 50  0001 C CNN "Digi-Key PN"
+F 5 "Telemetry" H 5110 2040 50  0001 C CNN "Configuration"
 	1    5110 2040
 	1    0    0    -1

Commit message: Added digikey pn's, footprints
Parts:
- gave numbers to parts that had none: 7
Changed lines of the file:
@@
 Sheet 3 23
 Title "Pulse Oximeter"
-Date ""
+Date "2019-01-03"
 Rev "A"
 Comp "Drew Maatman"
@@
 AR Path="/5E0A0E29/5E0ACFF2" Ref="#PWR?"  Part="1"
 AR Path="/5E052856/5E0ACFF2" Ref="#PWR?"  Part="1"
-AR Path="/5EAE2D84/5E0ACFF2" Ref="#PWR?"  Part="1"
-F 0 "#PWR?" H 5110 2190 50  0001 C CNN
+AR Path="/5EAE2D84/5E0ACFF2" Ref="#PWR0302"  Part="1"
+F 0 "#PWR0302" H 5110 2190 50  0001 C CNN
 F 1 "GND" H 5110 2290 50  0000 C CNN
 F 2 "" H 5110 2440 50  0001 C CNN
@@
 AR Path="/5E0A0E29/5E0AD665" Ref="#PWR?"  Part="1"
 AR Path="/5E052856/5E0AD665" Ref="#PWR?"  Part="1"
-AR Path="/5EAE2D84/5E0AD665" Ref="#PWR?"  Part="1"
-F 0 "#PWR?" H 5110 1490 50  0001 C CNN
+AR Path="/5EAE2D84/5E0AD665" Ref="#PWR0301"  Part="1"
+F 0 "#PWR0301" H 5110 1490 50  0001 C CNN
 F 1 "+3.3V" H 5110 1780 50  0000 C CNN
 F 2 "" H 5110 1640 50  0001 C CNN
@@
 AR Path="/5E0A0E29/5E0B2427" Ref="C?"  Part="1"
 AR Path="/5E052856/5E0B2427" Ref="C?"  Part="1"
-AR Path="/5EAE2D84/5E0B2427" Ref="C?"  Part="1"
-F 0 "C?" H 5135 3110 50  0000 L CNN
+AR Path="/5EAE2D84/5E0B2427" Ref="C302"  Part="1"
+F 0 "C302" H 5135 3110 50  0000 L CNN
 F 1 "0.1uF" H 5135 2910 50  0000 L CNN
 F 2 "Capacitors_SMD:C_0402" H 5148 2860 50  0001 C CNN
@@
 AR Path="/5E0A0E29/5E0B535B" Ref="#PWR?"  Part="1"
 AR Path="/5E052856/5E0B535B" Ref="#PWR?"  Part="1"
-AR Path="/5EAE2D84/5E0B535B" Ref="#PWR?"  Part="1"
-F 0 "#PWR?" H 5110 2710 50  0001 C CNN
+AR Path="/5EAE2D84/5E0B535B" Ref="#PWR0303"  Part="1"
+F 0 "#PWR0303" H 5110 2710 50  0001 C CNN
 F 1 "+3.3V" H 5110 3000 50  0000 C CNN
 F 2 "" H 5110 2860 50  0001 C CNN
@@
 AR Path="/5E0A0E29/5E0B592B" Ref="#PWR?"  Part="1"
 AR Path="/5E052856/5E0B592B" Ref="#PWR?"  Part="1"
-AR Path="/5EAE2D84/5E0B592B" Ref="#PWR?"  Part="1"
-F 0 "#PWR?" H 5110 2910 50  0001 C CNN
+AR Path="/5EAE2D84/5E0B592B" Ref="#PWR0304"  Part="1"
+F 0 "#PWR0304" H 5110 2910 50  0001 C CNN
 F 1 "GND" H 5110 3010 50  0000 C CNN
 F 2 "" H 5110 3160 50  0001 C CNN
@@
 AR Path="/5E0A0E29/5E0B8BC8" Ref="DOC?"  Part="1"
 AR Path="/5E052856/5E0B8BC8" Ref="DOC?"  Part="1"
-AR Path="/5EAE2D84/5E0B8BC8" Ref="DOC?"  Part="1"
-F 0 "DOC?" H 6010 3130 60  0001 C CNN
+AR Path="/5EAE2D84/5E0B8BC8" Ref="DOC301"  Part="1"
+F 0 "DOC301" H 6010 3130 60  0001 C CNN
 F 1 "0x40" H 5560 2880 60  0000 L CNN
 F 2 "" H 6010 3230 60  0001 C CNN
@@
 AR Path="/5E0A0E29/5E2AA995" Ref="#PWR?"  Part="1"
 AR Path="/5E052856/5E2AA995" Ref="#PWR?"  Part="1"
-AR Path="/5EAE2D84/5E2AA995" Ref="#PWR?"  Part="1"
-F 0 "#PWR?" H 5110 4870 50  0001 C CNN
+AR Path="/5EAE2D84/5E2AA995" Ref="#PWR0306"  Part="1"
+F 0 "#PWR0306" H 5110 4870 50  0001 C CNN
 F 1 "GND" H 5110 4970 50  0000 C CNN
 F 2 "" H 5110 5120 50  0001 C CNN
@@
 AR Path="/5E0A0E29/5E2AA99A" Ref="#PWR?"  Part="1"
 AR Path="/5E052856/5E2AA99A" Ref="#PWR?"  Part="1"
-AR Path="/5EAE2D84/5E2AA99A" Ref="#PWR?"  Part="1"
-F 0 "#PWR?" H 5110 3890 50  0001 C CNN
+AR Path="/5EAE2D84/5E2AA99A" Ref="#PWR0305"  Part="1"
+F 0 "#PWR0305" H 5110 3890 50  0001 C CNN
 F 1 "+3.3V" H 5110 4180 50  0000 C CNN
 F 2 "" H 5110 4040 50  0001 C CNN
@@
 AR Path="/5E0A0E29/5E2AA99D" Ref="U?"  Part="1"
 AR Path="/5E052856/5E2AA99D" Ref="U?"  Part="1"
-AR Path="/5EAE2D84/5E2AA99D" Ref="U?"  Part="1"
-F 0 "U?" H 4860 4990 50  0000 C CNN
+AR Path="/5EAE2D84/5E2AA99D" Ref="U302"  Part="1"
+F 0 "U302" H 4860 4990 50  0000 C CNN
 F 1 "MCP9804" H 5510 4990 50  0000 C CNN
 F 2 "Package_DFN_QFN:DFN-8-1EP_3x2mm_P0.5mm_EP1.3x1.5mm" H 4010 4040 50  0001 C CNN
@@
 AR Path="/5E0A0E29/5E2AA9A1" Ref="C?"  Part="1"
 AR Path="/5E052856/5E2AA9A1" Ref="C?"  Part="1"
-AR Path="/5EAE2D84/5E2AA9A1" Ref="C?"  Part="1"
-F 0 "C?" H 5135 5790 50  0000 L CNN
+AR Path="/5EAE2D84/5E2AA9A1" Ref="C303"  Part="1"
+F 0 "C303" H 5135 5790 50  0000 L CNN
 F 1 "0.1uF" H 5135 5590 50  0000 L CNN
 F 2 "Capacitors_SMD:C_0402" H 5148 5540 50  0001 C CNN
@@
 AR Path="/5E0A0E29/5E2AA9A6" Ref="#PWR?"  Part="1"
 AR Path="/5E052856/5E2AA9A6" Ref="#PWR?"  Part="1"
-AR Path="/5EAE2D84/5E2AA9A6" Ref="#PWR?"  Part="1"
-F 0 "#PWR?" H 5110 5390 50  0001 C CNN
+AR Path="/5EAE2D84/5E2AA9A6" Ref="#PWR0307"  Part="1"
+F 0 "#PWR0307" H 5110 5390 50  0001 C CNN
 F 1 "+3.3V" H 5110 5680 50  0000 C CNN
 F 2 "" H 5110 5540 50  0001 C CNN
@@
 AR Path="/5E0A0E29/5E2AA9AD" Ref="#PWR?"  Part="1"
 AR Path="/5E052856/5E2AA9AD" Ref="#PWR?"  Part="1"
-AR Path="/5EAE2D84/5E2AA9AD" Ref="#PWR?"  Part="1"
-F 0 "#PWR?" H 5110 5590 50  0001 C CNN
+AR Path="/5EAE2D84/5E2AA9AD" Ref="#PWR0308"  Part="1"
+F 0 "#PWR0308" H 5110 5590 50  0001 C CNN
 F 1 "GND" H 5110 5690 50  0000 C CNN
 F 2 "" H 5110 5840 50  0001 C CNN
@@
 AR Path="/5E0A0E29/5E2AA9AF" Ref="DOC?"  Part="1"
 AR Path="/5E052856/5E2AA9AF" Ref="DOC?"  Part="1"
-AR Path="/5EAE2D84/5E2AA9AF" Ref="DOC?"  Part="1"
-F 0 "DOC?" H 6010 5810 60  0001 C CNN
+AR Path="/5EAE2D84/5E2AA9AF" Ref="DOC302"  Part="1"
+F 0 "DOC302" H 6010 5810 60  0001 C CNN
 F 1 "0x18" H 5560 5560 60  0000 L CNN
 F 2 "" H 6010 5910 60  0001 C CNN
@@
 AR Path="/5E0A0E29/5E07E0FD" Ref="C?"  Part="1"
 AR Path="/5E052856/5E07E0FD" Ref="C?"  Part="1"
-AR Path="/5EAE2D84/5E07E0FD" Ref="C?"  Part="1"
-F 0 "C?" H 4255 2130 50  0000 L CNN
+AR Path="/5EAE2D84/5E07E0FD" Ref="C301"  Part="1"
+F 0 "C301" H 4255 2130 50  0000 L CNN
 F 1 "0.1uF" H 4255 1930 50  0000 L CNN
 F 2 "Capacitors_SMD:C_0402" H 4268 1880 50  0001 C CNN
@@
 	3790 1800 4230 1800
 $Comp
-L Analog_ADC:INA219BxDCN U?
+L Analog_ADC:INA219BxDCN U301
 U 1 1 5E1AAC3C
 P 5110 2040
-F 0 "U?" H 4860 2390 50  0000 C CNN
+F 0 "U301" H 4860 2390 50  0000 C CNN
 F 1 "INA219BxDCN" H 5360 2390 50  0000 C CNN
 F 2 "Package_TO_SOT_SMD:SOT-23-8" H 5760 1690 50  0001 C CNN
@@
 AR Path="/5E0A0E29/5E320C53" Ref="#PWR?"  Part="1"
 AR Path="/5E052856/5E320C53" Ref="#PWR?"  Part="1"
-AR Path="/5EAE2D84/5E320C53" Ref="#PWR?"  Part="1"
-F 0 "#PWR?" H 5510 1890 50  0001 C CNN
+AR Path="/5EAE2D84/5E320C53" Ref="#PWR0309"  Part="1"
+F 0 "#PWR0309" H 5510 1890 50  0001 C CNN
 F 1 "GND" V 5510 1990 50  0000 R CNN
 F 2 "" H 5510 2140 50  0001 C CNN
@@
 AR Path="/5E0A0E29/5E321138" Ref="#PWR?"  Part="1"
 AR Path="/5E052856/5E321138" Ref="#PWR?"  Part="1"
-AR Path="/5EAE2D84/5E321138" Ref="#PWR?"  Part="1"
-F 0 "#PWR?" H 5510 1990 50  0001 C CNN
+AR Path="/5EAE2D84/5E321138" Ref="#PWR0310"  Part="1"
+F 0 "#PWR0310" H 5510 1990 50  0001 C CNN
 F 1 "GND" V 5510 2090 50  0000 R CNN
 F 2 "" H 5510 2240 50  0001 C CNN
@@
 AR Path="/5E0A0E29/5E35CA2A" Ref="#PWR?"  Part="1"
 AR Path="/5E052856/5E35CA2A" Ref="#PWR?"  Part="1"
-AR Path="/5EAE2D84/5E35CA2A" Ref="#PWR?"  Part="1"
-F 0 "#PWR?" H 5510 4590 50  0001 C CNN
+AR Path="/5EAE2D84/5E35CA2A" Ref="#PWR0313"  Part="1"
+F 0 "#PWR0313" H 5510 4590 50  0001 C CNN
 F 1 "GND" V 5510 4690 50  0000 R CNN
 F 2 "" H 5510 4840 50  0001 C CNN
@@
 AR Path="/5E0A0E29/5E35C74D" Ref="#PWR?"  Part="1"
 AR Path="/5E052856/5E35C74D" Ref="#PWR?"  Part="1"
-AR Path="/5EAE2D84/5E35C74D" Ref="#PWR?"  Part="1"
-F 0 "#PWR?" H 5510 4490 50  0001 C CNN
+AR Path="/5EAE2D84/5E35C74D" Ref="#PWR0312"  Part="1"
+F 0 "#PWR0312" H 5510 4490 50  0001 C CNN
 F 1 "GND" V 5510 4590 50  0000 R CNN
 F 2 "" H 5510 4740 50  0001 C CNN
@@
 AR Path="/5E0A0E29/5E35BF65" Ref="#PWR?"  Part="1"
 AR Path="/5E052856/5E35BF65" Ref="#PWR?"  Part="1"
-AR Path="/5EAE2D84/5E35BF65" Ref="#PWR?"  Part="1"
-F 0 "#PWR?" H 5510 4390 50  0001 C CNN
+AR Path="/5EAE2D84/5E35BF65" Ref="#PWR0311"  Part="1"
+F 0 "#PWR0311" H 5510 4390 50  0001 C CNN
 F 1 "GND" V 5510 4490 50  0000 R CNN
 F 2 "" H 5510 4640 50  0001 C CNN

Commit message: Set TELEMETRY configs to visible in SCH
Changed lines of the file:
@@
 F 3 "http://ww1.microchip.com/downloads/en/DeviceDoc/22203b.pdf" H 4860 4990 50  0001 C CNN
 F 4 "MCP9804T-E/MCCT-ND" H 5110 4540 50  0001 C CNN "Digi-Key PN"
-F 5 "Telemetry" H 5110 4540 50  0001 C CNN "Configuration"
+F 5 "Telemetry" H 5510 5070 50  0000 C CNN "Configuration"
 	1    5110 4540
 	-1   0    0    -1
@@
 F 3 "http://www.ti.com/lit/ds/symlink/ina219.pdf" H 5460 1940 50  0001 C CNN
 F 4 "296-46420-1-ND" H 5110 2040 50  0001 C CNN "Digi-Key PN"
-F 5 "Telemetry" H 5110 2040 50  0001 C CNN "Configuration"
+F 5 "Telemetry" H 5370 2470 50  0000 C CNN "Configuration"
 	1    5110 2040
 	1    0    0    -1
