File: hdw/rev_b/Pulse_Oximeter/POS12_Input.sch (KiCad schematic (older format))
At the start: 25 parts, among them J201 +12V IN, Q201 Si4946BEY, U201 LTC4365DDB

Commit message: lots of rev B sch progress
Parts:
- removed C204: 0.1uF, Capacitors_SMD:C_0402, symbol Custom_Library:C_Custom
- removed Q201: Si4946BEY, Package_SO:SOIC-8_3.9x4.9mm_P1.27mm, symbol Custom_Library:Si4946BEY
- removed R212: 10, Resistors_SMD:R_0402, symbol Custom_Library:R_Custom
- removed R213: 10k, Resistors_SMD:R_0402, symbol Custom_Library:R_Custom
- removed TP202, TP203: TP, Custom Footprints Library:Test_Point, symbol Custom_Library:TP
- removed U201: LTC4365DDB, Housings_DFN_QFN:DFN-8-1EP_2x3mm_Pitch0.5mm, symbol Custom_Library:LTC4365DDB
- added C201: 10nF, Capacitors_SMD:C_0603, symbol Custom_Library:C_Custom
- added N201: +12V 1A Power Supply, symbol Mechanical:Housing
- added TP202, TP203: TP_Pad, Custom Footprints Library:Test_Point, symbol Custom_Library:TP_Pad
- added U201: TPS26600RHFT, Housings_DFN_QFN:QFN-24-1EP_4x5mm_Pitch0.5mm, symbol Custom_Library:TPS26600RHFT
- C202: renamed from C201; footprint Capacitors_SMD:C_0402 -> Capacitors_SMD:C_0603; Digi-Key PN 490-10701-1-ND -> 399-7845-1-ND; display_footprint 0402 -> 0603
- C203: renamed from C202; footprint Capacitors_SMD:C_0402 -> Capacitors_SMD:C_0603; Digi-Key PN 490-13295-1-ND -> 399-7842-1-ND; display_footprint 0402 -> 0603
- C204: renamed from C203; footprint Capacitors_SMD:C_0402 -> Capacitors_SMD:C_0603; Digi-Key PN 399-1032-1-ND -> 399-1083-1-ND; display_footprint 0402 -> 0603
- D201: Configuration (none) -> DNP
- J201: Digi-Key PN CP-202BH-ND -> (none)
- R201: value 6.04M -> 51.1k; footprint Resistors_SMD:R_0402 -> Resistors_SMD:R_0603; Digi-Key PN 541-CRCW04026M04FKEDCT-ND -> RMCF0603FT51K1TR-ND; Wattage 1/16W -> 1/10W; display_footprint 0402 -> 0603
- R202: value 86.6k -> 1.15k; footprint Resistors_SMD:R_0402 -> Resistors_SMD:R_0603; Digi-Key PN 541-86.6KLCT-ND -> RMCF0603FT1K15CT-ND; Wattage 1/16W -> 1/10W; display_footprint 0402 -> 0603
- R203: value 243k -> 5.11k; footprint Resistors_SMD:R_0402 -> Resistors_SMD:R_0603; Digi-Key PN YAG3070CT-ND -> CR0603-FX-5111ELFCT-ND; Wattage 1/16W -> 1/10W; display_footprint 0402 -> 0603
- R204: value 243k -> 10k; footprint Resistors_SMD:R_0402 -> Resistors_SMD:R_0603; Digi-Key PN YAG3070CT-ND -> YAG2321CT-ND; Wattage 1/16W -> 1/10W; display_footprint 0402 -> 0603
- R205: footprint Resistors_SMD:R_0402 -> Resistors_SMD:R_0603; Digi-Key PN 541-3964-1-ND -> YAG2321CT-ND; Wattage 1/16W -> 1/10W; display_footprint 0402 -> 0603
- R206: value 10 -> 0.02; footprint Resistors_SMD:R_0402 -> Resistors_SMD:R_0612; Digi-Key PN 541-3964-1-ND -> P16010CT-ND; Wattage 1/16W -> 1W; display_footprint 0402 -> 0612
- R207: value 13.7k -> 10k; footprint Resistors_SMD:R_0402 -> Resistors_SMD:R_0603; Digi-Key PN RMCF0402FT13K7CT-ND -> YAG2321CT-ND; Wattage 1/16W -> 1/10W; display_footprint 0402 -> 0603
- R208: value 5.23k -> 13k; footprint Resistors_SMD:R_0402 -> Resistors_SMD:R_0603; Digi-Key PN RMCF0402FT5K23CT-ND -> 311-13.0KHRCT-ND; Wattage 1/16W -> 1/10W; display_footprint 0402 -> 0603
- R209: value 10 -> 5.11k; footprint Resistors_SMD:R_0402 -> Resistors_SMD:R_0603; Digi-Key PN 541-3964-1-ND -> CR0603-FX-5111ELFCT-ND; Wattage 1/16W -> 1/10W; display_footprint 0402 -> 0603
- R210: value 0.02 -> 10; footprint Resistors_SMD:R_0612 -> Resistors_SMD:R_0603; Digi-Key PN P16010CT-ND -> YAG2321CT-ND; Wattage 1W -> 1/10W; display_footprint 0612 -> 0603
- R211: value 5.23k -> 10k; footprint Resistors_SMD:R_0402 -> Resistors_SMD:R_0603; Digi-Key PN RMCF0402FT5K23CT-ND -> YAG2321CT-ND; Wattage 1/16W -> 1/10W; display_footprint 0402 -> 0603
Connections:
- wire segments 70 -> 74
- no-connect marks 0 -> 1
Other:
- note added: "+3.3V Logic Level"
- note added: "UVLO threshold set to 10.8V\nOVLO threshold set to 13.2V\n\nMODE set to Circuit Breaker with Auto-Retry\n\nOutput Current Limit set to 1.2A"
- note removed: "3.3V Logic Level"
- note removed: "UVLO threshold set to 10V\nOVLO threshold set to 14V"
- moved on the sheet: C202, C203, C204, C205, D201, J201

Commit message: lots of rev b changes
Parts:
- removed C203: 10nF, Capacitors_SMD:C_0603, symbol Custom_Library:C_Custom
- removed C204: 1nF, Capacitors_SMD:C_0603, symbol Custom_Library:C_Custom
- removed R201: 51.1k, Resistors_SMD:R_0603, symbol Custom_Library:R_Custom
- removed R202: 1.15k, Resistors_SMD:R_0603, symbol Custom_Library:R_Custom
- removed R203, R209: 5.11k, Resistors_SMD:R_0603, symbol Custom_Library:R_Custom
- removed R208: 13k, Resistors_SMD:R_0603, symbol Custom_Library:R_Custom
- added R? (x4): 1k, Resistors_SMD:R_0603, symbol Custom_Library:R_Custom
- added R? (x5): 10k, Resistors_SMD:R_0603, symbol Custom_Library:R_Custom
- added R? (x2): 100k, Resistors_SMD:R_0603, symbol Custom_Library:R_Custom
Connections:
- net +12V: now also R?.1
- net +12Vin: now also R?.1, R?.1
- net GND: now also R?.2, R?.2
- net POS12_PGOOD: now also R?.1, R?.1, R?.2
- net at U201.10 (UVLO): now also R?.1, R?.2, R?.2
- net at U201.12 (OVP): now also R?.1, R?.1, R?.2
- net at C201.2, R207.2, R211.2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: now also R?.2, R?.2
- new net: R?.1, R?.2 (x3)
Other:
- note added: "UVLO threshold set to TBD\nOVLO threshold set to TBD\n\nMODE set to Circuit Breaker with Auto-Retry\n\nOutput Current Limit set to 1.2A"
- note removed: "UVLO threshold set to 10.8V\nOVLO threshold set to 13.2V\n\nMODE set to Circuit Breaker with Auto-Retry\n\nOutput Current Limit set to 1.2A"
- moved on the sheet: D201, J201

Commit message: merged, more cleanups
Parts:
- R205, R210: Configuration (none) -> Telemetry
Other:
- moved on the sheet: C202
Changed lines of the file:
@@
 L Custom_Library:+12Vin #PWR0206
 U 1 1 5BB6907F
-P 5300 5960
-F 0 "#PWR0206" H 5300 5810 50  0001 C CNN
-F 1 "+12Vin" H 5300 6110 50  0000 C CNN
-F 2 "" H 5300 5960 50  0000 C CNN
-F 3 "" H 5300 5960 50  0000 C CNN
-	1    5300 5960
+P 5600 5960
+F 0 "#PWR0206" H 5600 5810 50  0001 C CNN
+F 1 "+12Vin" H 5600 6110 50  0000 C CNN
+F 2 "" H 5600 5960 50  0000 C CNN
+F 3 "" H 5600 5960 50  0000 C CNN
+	1    5600 5960
 	1    0    0    -1
 $EndComp
@@
 L power:GND #PWR0207
 U 1 1 5BB5EFF4
-P 5300 6260
-F 0 "#PWR0207" H 5300 6010 50  0001 C CNN
-F 1 "GND" H 5300 6110 50  0000 C CNN
-F 2 "" H 5300 6260 50  0001 C CNN
-F 3 "" H 5300 6260 50  0001 C CNN
-	1    5300 6260
+P 5600 6260
+F 0 "#PWR0207" H 5600 6010 50  0001 C CNN
+F 1 "GND" H 5600 6110 50  0000 C CNN
+F 2 "" H 5600 6260 50  0001 C CNN
+F 3 "" H 5600 6260 50  0001 C CNN
+	1    5600 6260
 	1    0    0    -1
 $EndComp
@@
 L Custom_Library:C_Custom C?
 U 1 1 5BB576FA
-P 5300 6110
+P 5600 6110
 AR Path="/5BAAE16C/5BB576FA" Ref="C?"  Part="1"
 AR Path="/5BB181D8/5BB576FA" Ref="C?"  Part="1"
@@
 AR Path="/5E939CFF/5BB576FA" Ref="C202"  Part="1"
 AR Path="/5EAE2D66/5BB576FA" Ref="C202"  Part="1"
-F 0 "C202" H 5325 6210 50  0000 L CNN
-F 1 "0.1uF" H 5325 6010 50  0000 L CNN
-F 2 "Capacitors_SMD:C_0603" H 5338 5960 50  0001 C CNN
-F 3 "" H 5325 6210 50  0001 C CNN
-F 4 "0603" H 5150 6210 50  0000 R CNN "display_footprint"
-F 5 "50V" H 5150 6110 50  0000 R CNN "Voltage"
-F 6 "X7R" H 5150 6010 50  0000 R CNN "Dielectric"
-F 7 "399-7845-1-ND" H 5725 6610 60  0001 C CNN "Digi-Key PN"
-	1    5300 6110
+F 0 "C202" H 5625 6210 50  0000 L CNN
+F 1 "0.1uF" H 5625 6010 50  0000 L CNN
+F 2 "Capacitors_SMD:C_0603" H 5638 5960 50  0001 C CNN
+F 3 "" H 5625 6210 50  0001 C CNN
+F 4 "0603" H 5450 6210 50  0000 R CNN "display_footprint"
+F 5 "50V" H 5450 6110 50  0000 R CNN "Voltage"
+F 6 "X7R" H 5450 6010 50  0000 R CNN "Dielectric"
+F 7 "399-7845-1-ND" H 6025 6610 60  0001 C CNN "Digi-Key PN"
+	1    5600 6110
 	1    0    0    -1
 $EndComp
@@
 F 6 "1/10W" V 6580 1910 50  0001 C CNN "Wattage"
 F 7 "YAG2321CT-ND" H 6280 1910 50  0001 C CNN "Digi-Key PN"
+F 8 "Telemetry" V 6370 1910 50  0000 C CNN "Configuration"
 	1    6280 1910
 	-1   0    0    -1
@@
 F 6 "1/10W" V 7040 1910 50  0001 C CNN "Wattage"
 F 7 "YAG2321CT-ND" H 6740 1910 50  0001 C CNN "Digi-Key PN"
+F 8 "Telemetry" V 6830 1910 50  0000 C CNN "Configuration"
 	1    6740 1910
 	-1   0    0    -1

Commit message: changed all passives to 0402, cleared digikey pns
Parts:
- removed N201: +12V 1A Power Supply, symbol Mechanical:Housing
- C201: footprint Capacitors_SMD:C_0603 -> Capacitors_SMD:C_0402; Digi-Key PN 399-7842-1-ND -> (none); display_footprint 0603 -> 0402
- C202: footprint Capacitors_SMD:C_0603 -> Capacitors_SMD:C_0402; Digi-Key PN 399-7845-1-ND -> (none); display_footprint 0603 -> 0402
- R204, R205, R207, R210, R211, R? (x5): footprint Resistors_SMD:R_0603 -> Resistors_SMD:R_0402; Digi-Key PN YAG2321CT-ND -> (none); Wattage 1/10W -> 1/16W; display_footprint 0603 -> 0402
- R? (x4): footprint Resistors_SMD:R_0603 -> Resistors_SMD:R_0402; Digi-Key PN 311-1.00KHRCT-ND -> (none); Wattage 1/10W -> 1/16W; display_footprint 0603 -> 0402
- R? (x2): footprint Resistors_SMD:R_0603 -> Resistors_SMD:R_0402; Digi-Key PN RMCF0603FT100KCT-ND -> (none); Wattage 1/10W -> 1/16W; display_footprint 0603 -> 0402
Other:
- moved on the sheet: C201, C202, C205, D201, J201, R204, R205, R206, R207, R210, R211, R?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

Commit message: removed more unique components, cleaned up SCH
Parts:
- added R? (x3): 0, Resistors_SMD:R_0402, symbol Custom_Library:R_Custom
- R206: Configuration (none) -> Telemetry
Connections:
- net +12V: now also R?.2, R?.2, R?.2
- net at R205.2, R206.1, U201.23 (OUT)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: now also R?.1, R?.1, R?.1
Other:
- note added: "UVLO threshold set to 11.12V\nOVLO threshold set to 13.33V\n\nMODE set to Circuit Breaker with Auto-Retry\n\nOutput Current Limit set to 1.2A\n\nOutput ramp rate = 12.5V/ms"
- note removed: "UVLO threshold set to TBD\nOVLO threshold set to TBD\n\nMODE set to Circuit Breaker with Auto-Retry\n\nOutput Current Limit set to 1.2A"
- moved on the sheet: R?

Commit message: annotated schematic
Parts:
- gave numbers to parts that had none: 14
- renumbered C205 to C203, R204 to R206, R205 to R207, R206 to R208, R207 to R212, R210 to R213, R211 to R214
