File: hdw/rev_b/Pulse_Oximeter/POS3P3_Power_Supply.sch (KiCad schematic (older format))
At the start: 20 parts, among them Q401 BSS214NW, Q402 ZXMS6004FFTA, U401 TPS62150

Commit message: merged, more cleanups
Parts:
- Q401: footprint Package_TO_SOT_SMD:SOT-323_SC-70 -> TO_SOT_Packages_SMD:SOT-323_SC-70
- R403: value 10 -> 0; Digi-Key PN 541-3964-1-ND -> (none)
- R407, R409: Configuration (none) -> Telemetry
Connections:
- net POS12_PGOOD: now also R403.1; no longer R403.2
- net POS3P3_RUN: now also R403.2; no longer R403.1
Changed lines of the file:
@@
 F 6 "1/16W" V 7590 2710 50  0001 C CNN "Wattage"
 F 7 "541-3964-1-ND" H 7290 2710 50  0001 C CNN "Digi-Key PN"
+F 8 "Telemetry" V 7390 2710 50  0000 C CNN "Configuration"
 	1    7290 2710
 	-1   0    0    -1
@@
 F 6 "1/16W" V 8050 2710 50  0001 C CNN "Wattage"
 F 7 "541-3964-1-ND" H 7750 2710 50  0001 C CNN "Digi-Key PN"
+F 8 "Telemetry" V 7850 2710 50  0000 C CNN "Configuration"
 	1    7750 2710
 	-1   0    0    -1
@@
 F 0 "Q401" H 4490 7565 50  0000 L CNN
 F 1 "BSS214NW" H 4490 7490 50  0000 L CNN
-F 2 "Package_TO_SOT_SMD:SOT-323_SC-70" H 4490 7415 50  0001 L CIN
+F 2 "TO_SOT_Packages_SMD:SOT-323_SC-70" H 4490 7415 50  0001 L CIN
 F 3 "https://www.infineon.com/dgdl/Infineon-BSS214NW-DS-v02_02-en.pdf?fileId=db3a30431b3e89eb011b695aebc01bde" H 4290 7490 50  0001 L CNN
 F 4 "BSS214NWH6327XTSA1CT-ND" H 4290 7490 50  0001 C CNN "Digi-Key PN"
@@
 Text GLabel 2280 6700 2    50   Output ~ 0
 POS3P3_RUN
-$Comp
-L Custom_Library:R_Custom R?
-U 1 1 5EB895CA
-P 2130 6700
-AR Path="/5EAE2D66/5EB895CA" Ref="R?"  Part="1"
-AR Path="/5EAE2D8A/5EB895CA" Ref="R403"  Part="1"
-F 0 "R403" V 2030 6700 50  0000 C CNN
-F 1 "10" V 2130 6700 50  0000 C CNN
-F 2 "Resistors_SMD:R_0402" H 2130 6700 50  0001 C CNN
-F 3 "" H 2130 6700 50  0001 C CNN
-F 4 "541-3964-1-ND" H 2430 7100 60  0001 C CNN "Digi-Key PN"
-F 5 "0402" V 2230 6700 50  0000 C CNN "display_footprint"
-F 6 "1%" V 2330 6700 50  0000 C CNN "Tolerance"
-F 7 "1/16W" V 2430 6700 50  0000 C CNN "Wattage"
-	1    2130 6700
-	0    1    1    0
-$EndComp
 Text GLabel 1980 6700 0    50   Input ~ 0
 POS12_PGOOD
@@
 Text GLabel 4090 7490 0    50   Input ~ 0
 POS3P3_RUN
+$Comp
+L Custom_Library:R_Custom R?
+U 1 1 5FE28635
+P 2130 6700
+AR Path="/5EAE2EF2/5FE28635" Ref="R?"  Part="1"
+AR Path="/5EAE30C7/5FE28635" Ref="R?"  Part="1"
+AR Path="/5EAE2D8A/5FE28635" Ref="R403"  Part="1"
+F 0 "R403" V 2030 6700 50  0000 C CNN
+F 1 "0" V 2130 6700 50  0000 C CNN
+F 2 "Resistors_SMD:R_0402" H 2130 6700 50  0001 C CNN
+F 3 "" H 2130 6700 50  0001 C CNN
+F 4 "0402" V 2230 6700 50  0000 C CNN "display_footprint"
+F 5 "1%" V 2330 6700 50  0000 C CNN "Tolerance"
+F 6 "1/16W" V 2430 6700 50  0000 C CNN "Wattage"
+	1    2130 6700
+	0    -1   1    0
+$EndComp
 $EndSCHEMATC

Commit message: changed all passives to 0402, cleared digikey pns
Parts:
- C402: Digi-Key PN 490-13211-1-ND -> (none)
- C403: Digi-Key PN 490-13295-1-ND -> (none)
- C404, C406: Digi-Key PN 490-10701-1-ND -> (none)
- R405, R406: Digi-Key PN RMCF0402FT10K0CT-ND -> (none)
- R407, R409: Digi-Key PN 541-3964-1-ND -> (none)
- R410: Digi-Key PN 311-562KLRCT-ND -> (none)
- R411: Digi-Key PN A129654CT-ND -> (none)
Changed lines of the file:
@@
 F 5 "50V" H 4400 2970 50  0000 R CNN "Voltage"
 F 6 "X7R" H 4400 2870 50  0000 R CNN "Dielectric"
-F 7 "490-10701-1-ND" H 4975 3470 60  0001 C CNN "Digi-Key PN"
+F 7 "" H 4975 3470 60  0001 C CNN "Digi-Key PN"
 	1    4550 2970
 	1    0    0    -1
@@
 $EndComp
 $Comp
-L Custom_Library:C_Custom C?
-U 1 1 5E2AA97D
-P 4190 4770
-AR Path="/5C1D5CD8/5E2AA97D" Ref="C?"  Part="1"
-AR Path="/5C1D5CCA/5E2AA97D" Ref="C?"  Part="1"
-AR Path="/5C1E3A0B/5E2AA97D" Ref="C?"  Part="1"
-AR Path="/5C1E3A08/5E2AA97D" Ref="C?"  Part="1"
-AR Path="/5D779AE1/5E2AA97D" Ref="C?"  Part="1"
-AR Path="/5CB7718D/5E2AA97D" Ref="C?"  Part="1"
-AR Path="/5E0DC082/5E2AA97D" Ref="C?"  Part="1"
-AR Path="/5E0F263A/5E2AA97D" Ref="C?"  Part="1"
-AR Path="/5EAE2D8A/5E2AA97D" Ref="C403"  Part="1"
-F 0 "C403" H 4215 4870 50  0000 L CNN
-F 1 "10nF" H 4215 4670 50  0000 L CNN
-F 2 "Capacitors_SMD:C_0402" H 4228 4620 50  0001 C CNN
-F 3 "" H 4215 4870 50  0001 C CNN
-F 4 "" H 4040 4870 50  0000 R CNN "display_footprint"
-F 5 "50V" H 4040 4770 50  0000 R CNN "Voltage"
-F 6 "X7R" H 4040 4670 50  0000 R CNN "Dielectric"
-F 7 "490-13295-1-ND" H 270 550 50  0001 C CNN "Digi-Key PN"
-	1    4190 4770
-	1    0    0    -1
-$EndComp
-$Comp
 L power:GND #PWR?
 U 1 1 5C294444
@@
 F 5 "1%" H 8320 3810 50  0000 L CNN "Tolerance"
 F 6 "1/16W" H 8330 3730 50  0000 L CNN "Wattage"
-F 7 "311-562KLRCT-ND" H 8220 3810 50  0001 C CNN "Digi-Key PN"
+F 7 "" H 8220 3810 50  0001 C CNN "Digi-Key PN"
 	1    8220 3810
 	1    0    0    -1
@@
 F 5 "1%" H 8320 4720 50  0000 L CNN "Tolerance"
 F 6 "1/16W" H 8330 4640 50  0000 L CNN "Wattage"
-F 7 "A129654CT-ND" H 8220 4720 50  0001 C CNN "Digi-Key PN"
+F 7 "" H 8220 4720 50  0001 C CNN "Digi-Key PN"
 	1    8220 4720
 	1    0    0    -1
@@
 F 5 "50V" H 8520 3270 50  0000 R CNN "Voltage"
 F 6 "X7R" H 8520 3170 50  0000 R CNN "Dielectric"
-F 7 "490-10701-1-ND" H 9095 3770 60  0001 C CNN "Digi-Key PN"
+F 7 "" H 9095 3770 60  0001 C CNN "Digi-Key PN"
 	1    8670 3270
 	1    0    0    -1
@@
 F 5 "1%" V 7490 2710 50  0001 C CNN "Tolerance"
 F 6 "1/16W" V 7590 2710 50  0001 C CNN "Wattage"
-F 7 "541-3964-1-ND" H 7290 2710 50  0001 C CNN "Digi-Key PN"
+F 7 "" H 7290 2710 50  0001 C CNN "Digi-Key PN"
 F 8 "Telemetry" V 7390 2710 50  0000 C CNN "Configuration"
 	1    7290 2710
@@
 F 5 "1%" V 7950 2710 50  0001 C CNN "Tolerance"
 F 6 "1/16W" V 8050 2710 50  0001 C CNN "Wattage"
-F 7 "541-3964-1-ND" H 7750 2710 50  0001 C CNN "Digi-Key PN"
+F 7 "" H 7750 2710 50  0001 C CNN "Digi-Key PN"
 F 8 "Telemetry" V 7850 2710 50  0000 C CNN "Configuration"
 	1    7750 2710
@@
 F 5 "1%" H 4490 6980 50  0000 L CNN "Tolerance"
 F 6 "1/16W" H 4500 6900 50  0000 L CNN "Wattage"
-F 7 "RMCF0402FT10K0CT-ND" H 4690 7380 60  0001 C CNN "Digi-Key PN"
+F 7 "" H 4690 7380 60  0001 C CNN "Digi-Key PN"
 	1    4390 6980
 	1    0    0    -1
@@
 F 5 "6.3V" H 3530 6980 50  0000 R CNN "Voltage"
 F 6 "X5R" H 3530 6880 50  0000 R CNN "Dielectric"
-F 7 "490-13211-1-ND" H 3680 6980 50  0001 C CNN "Digi-Key PN"
+F 7 "" H 3680 6980 50  0001 C CNN "Digi-Key PN"
 	1    3680 6980
 	1    0    0    -1
@@
 F 5 "1%" H 2870 3810 50  0000 L CNN "Tolerance"
 F 6 "1/16W" H 2880 3730 50  0000 L CNN "Wattage"
-F 7 "RMCF0402FT10K0CT-ND" H 3070 4210 60  0001 C CNN "Digi-Key PN"
+F 7 "" H 3070 4210 60  0001 C CNN "Digi-Key PN"
 	1    2770 3810
 	1    0    0    -1
@@
 	0    -1   1    0
 $EndComp
+$Comp
+L Custom_Library:C_Custom C?
+U 1 1 5E2AA97D
+P 4190 4770
+AR Path="/5C1D5CD8/5E2AA97D" Ref="C?"  Part="1"
+AR Path="/5C1D5CCA/5E2AA97D" Ref="C?"  Part="1"
+AR Path="/5C1E3A0B/5E2AA97D" Ref="C?"  Part="1"
+AR Path="/5C1E3A08/5E2AA97D" Ref="C?"  Part="1"
+AR Path="/5D779AE1/5E2AA97D" Ref="C?"  Part="1"
+AR Path="/5CB7718D/5E2AA97D" Ref="C?"  Part="1"
+AR Path="/5E0DC082/5E2AA97D" Ref="C?"  Part="1"
+AR Path="/5E0F263A/5E2AA97D" Ref="C?"  Part="1"
+AR Path="/5EAE2D8A/5E2AA97D" Ref="C403"  Part="1"
+F 0 "C403" H 4215 4870 50  0000 L CNN
+F 1 "10nF" H 4215 4670 50  0000 L CNN
+F 2 "Capacitors_SMD:C_0402" H 4228 4620 50  0001 C CNN
+F 3 "" H 4215 4870 50  0001 C CNN
+F 4 "" H 4040 4870 50  0000 R CNN "display_footprint"
+F 5 "50V" H 4040 4770 50  0000 R CNN "Voltage"
+F 6 "X7R" H 4040 4670 50  0000 R CNN "Dielectric"
+F 7 "" H 270 550 50  0001 C CNN "Digi-Key PN"
+	1    4190 4770
+	1    0    0    -1
+$EndComp
 $EndSCHEMATC

Commit message: few little tweaks
Parts:
- removed C406: 0.1uF, Capacitors_SMD:C_0402, symbol Custom_Library:C_Custom
- added C?: 0.1uF, Capacitors_SMD:C_0402, symbol Custom_Library:C_Custom
- added R?: 10k, Resistors_SMD:R_0402, symbol Custom_Library:R_Custom
- added R?: 0, Resistors_SMD:R_0402, symbol Custom_Library:R_Custom
- added U?: 74LVC1G97, Package_TO_SOT_SMD:SOT-363_SC-70-6, symbol Custom_Library:74LVC1G97_Power_AND
- C403, C404: display_footprint (none) -> 0402
- R410, R411: Configuration (none) -> DNP
- U401: value TPS62150 -> TPS62152; Digi-Key PN 296-41757-1-ND -> (none)
Connections:
- net +3V3: now also C?.1, U?.5 (VCC)
- net GND: now also C?.2, R?.2, R?.2, U?.1 (GND), U?.2 (GND)
- net POS3P3_PGOOD: now also R?.1, U?.4; no longer R405.2, U401.4 (PG)
- net POS3P3_RUN: now also U?.3
- net at R410.2, R411.1, U401.5 (FB): now also R?.1
- new net: R405.2, U401.4 (PG), U?.6
Other:
- note added: "Fixed VOUT = +3.3V"

Commit message: removed more unique components, cleaned up SCH
Parts:
- removed Q402: ZXMS6004FFTA, Package_TO_SOT_SMD:SOT-23, symbol Custom_Library:ZXMS6004FFTA
- added C?: 10uF, Capacitors_SMD:C_1206, symbol Custom_Library:C_Custom
- added Q?: BSS214NW, TO_SOT_Packages_SMD:SOT-323_SC-70, symbol Transistor_FET:BSS214NW
- added R? (x3): 0, Resistors_SMD:R_0402, symbol Custom_Library:R_Custom
- added R?: 100, Resistors_SMD:R_0402, symbol Custom_Library:R_Custom
- C401: Dielectric X7R -> X5R; Digi-Key PN 1276-7031-1-ND -> 1276-1075-1-ND
- C405: value 100uF -> 10uF; Digi-Key PN 587-1963-1-ND -> 1276-1075-1-ND; Voltage 6.3V -> 25V
- R408: Configuration (none) -> Telemetry
- U401: Digi-Key PN (none) -> 296-43621-1-ND
Connections:
- net +3V3: now also R?.1
- net GND: now also C?.2, Q?.2 (S)
- net at C405.1, L401.2, R407.2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: now also C?.1, R?.1, R?.1, R?.1
- net at Q401.3 (D), R406.2: now also Q?.1 (G)
- new net: R?.2, R?.2, R?.2
- new net: Q?.3 (D), R?.2
Other:
- moved on the sheet: R407, R408, R409, R410, R411, R?, TP401

Commit message: reworked +3.3V discharge holdup circuit
Parts:
- removed D401: BAT48JFILM, Diode_SMD:D_SOD-323, symbol Diode:BAT48JFILM
- added D?: Red, LEDs:LED_0402, symbol Device:LED
- added R? (x2): 10k, Resistors_SMD:R_0402, symbol Custom_Library:R_Custom
Connections:
- net +12V: now also R?.1
- net GND: now also R?.2
- net at C402.1, R406.1: now also D?.1 (K), R?.1
- new net: D?.2 (A), R?.2
Other:
- moved on the sheet: R403
Changed lines of the file:
@@
 Wire Wire Line
 	3680 6750 3680 6830
-$Comp
-L Diode:BAT48JFILM D401
-U 1 1 5EB4A7A8
-P 3680 6520
-F 0 "D401" V 3750 6400 50  0000 R CNN
-F 1 "BAT48JFILM" V 3650 6400 50  0000 R CNN
-F 2 "Diode_SMD:D_SOD-323" H 3680 6345 50  0001 C CNN
-F 3 "www.st.com/resource/en/datasheet/bat48.pdf" H 3680 6520 50  0001 C CNN
-F 4 "497-5711-1-ND" H 3680 6520 50  0001 C CNN "Digi-Key PN"
-	1    3680 6520
-	0    -1   -1   0
-$EndComp
 Wire Wire Line
 	3680 6670 3680 6750
 Connection ~ 3680 6750
-$Comp
-L power:+3.3V #PWR0404
-U 1 1 5EB4C2CE
-P 3680 6370
-F 0 "#PWR0404" H 3680 6220 50  0001 C CNN
-F 1 "+3.3V" H 3680 6510 50  0000 C CNN
-F 2 "" H 3680 6370 50  0001 C CNN
-F 3 "" H 3680 6370 50  0001 C CNN
-	1    3680 6370
-	1    0    0    -1
-$EndComp
-Text GLabel 2280 6700 2    50   Output ~ 0
+Text GLabel 1990 6470 2    50   Output ~ 0
 POS3P3_RUN
-Text GLabel 1980 6700 0    50   Input ~ 0
+Text GLabel 1690 6470 0    50   Input ~ 0
 POS12_PGOOD
 $Comp
@@
 L Custom_Library:R_Custom R?
 U 1 1 5FE28635
-P 2130 6700
+P 1840 6470
 AR Path="/5EAE2EF2/5FE28635" Ref="R?"  Part="1"
 AR Path="/5EAE30C7/5FE28635" Ref="R?"  Part="1"
 AR Path="/5EAE2D8A/5FE28635" Ref="R403"  Part="1"
-F 0 "R403" V 2030 6700 50  0000 C CNN
-F 1 "0" V 2130 6700 50  0000 C CNN
-F 2 "Resistors_SMD:R_0402" H 2130 6700 50  0001 C CNN
-F 3 "" H 2130 6700 50  0001 C CNN
-F 4 "0402" V 2230 6700 50  0000 C CNN "display_footprint"
-F 5 "1%" V 2330 6700 50  0000 C CNN "Tolerance"
-F 6 "1/16W" V 2430 6700 50  0000 C CNN "Wattage"
-	1    2130 6700
+F 0 "R403" V 1740 6470 50  0000 C CNN
+F 1 "0" V 1840 6470 50  0000 C CNN
+F 2 "Resistors_SMD:R_0402" H 1840 6470 50  0001 C CNN
+F 3 "" H 1840 6470 50  0001 C CNN
+F 4 "0402" V 1940 6470 50  0000 C CNN "display_footprint"
+F 5 "1%" V 2040 6470 50  0000 C CNN "Tolerance"
+F 6 "1/16W" V 2140 6470 50  0000 C CNN "Wattage"
+	1    1840 6470
 	0    -1   1    0
 $EndComp
@@
 Wire Wire Line
 	6820 3040 7410 3040
+$Comp
+L Custom_Library:R_Custom R?
+U 1 1 5FEC8503
+P 2890 6980
+AR Path="/5BB27BA3/5FEC8503" Ref="R?"  Part="1"
+AR Path="/5BB27BF7/5FEC8503" Ref="R?"  Part="1"
+AR Path="/5C1DE17A/5FEC8503" Ref="R?"  Part="1"
+AR Path="/5C1E3A08/5FEC8503" Ref="R?"  Part="1"
+AR Path="/5D779AE1/5FEC8503" Ref="R?"  Part="1"
+AR Path="/5CB7718D/5FEC8503" Ref="R?"  Part="1"
+AR Path="/5E0DC082/5FEC8503" Ref="R?"  Part="1"
+AR Path="/5E0F263A/5FEC8503" Ref="R?"  Part="1"
+AR Path="/5EAE2D8A/5FEC8503" Ref="R?"  Part="1"
+F 0 "R?" H 2810 6980 50  0000 R CNN
+F 1 "10k" V 2890 6980 50  0000 C CNN
+F 2 "Resistors_SMD:R_0402" H 2890 6980 50  0001 C CNN
+F 3 "" H 2890 6980 50  0001 C CNN
+F 4 "0402" H 2990 7060 50  0000 L CNN "display_footprint"
+F 5 "1%" H 2990 6980 50  0000 L CNN "Tolerance"
+F 6 "1/16W" H 3000 6900 50  0000 L CNN "Wattage"
+F 7 "" H 3190 7380 60  0001 C CNN "Digi-Key PN"
+	1    2890 6980
+	1    0    0    -1
+$EndComp
+$Comp
+L power:GND #PWR?
+U 1 1 5FEC96FB
+P 2890 7130
+F 0 "#PWR?" H 2890 6880 50  0001 C CNN
+F 1 "GND" H 2890 6980 50  0000 C CNN
+F 2 "" H 2890 7130 50  0001 C CNN
+F 3 "" H 2890 7130 50  0001 C CNN
+	1    2890 7130
+	1    0    0    -1
+$EndComp
+Wire Wire Line
+	3680 6750 2890 6750
+Wire Wire Line
+	2890 6750 2890 6830
+$Comp
+L Device:LED D?
+U 1 1 5FECDEC8
+P 3680 6520
+AR Path="/5BB844FD/5FECDEC8" Ref="D?"  Part="1"
+AR Path="/5BF346B3/5FECDEC8" Ref="D?"  Part="1"
+AR Path="/5BAAE1F3/5FECDEC8" Ref="D?"  Part="1"
+AR Path="/5CAD2D97/5FECDEC8" Ref="D?"  Part="1"
+AR Path="/5CB7A8BC/5FECDEC8" Ref="D?"  Part="1"
+AR Path="/5E6AF016/5FECDEC8" Ref="D?"  Part="1"
+AR Path="/5EAE4AE4/5FECDEC8" Ref="D?"  Part="1"
+F 0 "D?" V 3719 6403 50  0000 R CNN
+F 1 "Red" V 3628 6403 50  0000 R CNN
+F 2 "LEDs:LED_0402" H 3680 6520 50  0001 C CNN
+F 3 "~" H 3680 6520 50  0001 C CNN
+F 4 "1497-1174-1-ND" H 3680 6520 50  0001 C CNN "Digi-Key PN"
+	1    3680 6520
+	0    -1   -1   0
+$EndComp
+$Comp
+L Custom_Library:R_Custom R?
+U 1 1 5FECF137
+P 3680 6220
+AR Path="/5BB27BA3/5FECF137" Ref="R?"  Part="1"
+AR Path="/5BB27BF7/5FECF137" Ref="R?"  Part="1"
+AR Path="/5C1DE17A/5FECF137" Ref="R?"  Part="1"
+AR Path="/5C1E3A08/5FECF137" Ref="R?"  Part="1"
+AR Path="/5D779AE1/5FECF137" Ref="R?"  Part="1"
+AR Path="/5CB7718D/5FECF137" Ref="R?"  Part="1"
+AR Path="/5E0DC082/5FECF137" Ref="R?"  Part="1"
+AR Path="/5E0F263A/5FECF137" Ref="R?"  Part="1"
+AR Path="/5EAE2D8A/5FECF137" Ref="R?"  Part="1"
+F 0 "R?" H 3600 6220 50  0000 R CNN
+F 1 "10k" V 3680 6220 50  0000 C CNN
+F 2 "Resistors_SMD:R_0402" H 3680 6220 50  0001 C CNN
+F 3 "" H 3680 6220 50  0001 C CNN
+F 4 "0402" H 3780 6300 50  0000 L CNN "display_footprint"
+F 5 "1%" H 3780 6220 50  0000 L CNN "Tolerance"
+F 6 "1/16W" H 3790 6140 50  0000 L CNN "Wattage"
+F 7 "" H 3980 6620 60  0001 C CNN "Digi-Key PN"
+	1    3680 6220
+	1    0    0    -1
+$EndComp
+$Comp
+L power:+12V #PWR?
+U 1 1 5FECF71F
+P 3680 6070
+AR Path="/5CB7718D/5FECF71F" Ref="#PWR?"  Part="1"
+AR Path="/5E0DC082/5FECF71F" Ref="#PWR?"  Part="1"
+AR Path="/5E0F263A/5FECF71F" Ref="#PWR?"  Part="1"
+AR Path="/5EAE2D8A/5FECF71F" Ref="#PWR?"  Part="1"
+F 0 "#PWR?" H 3680 5920 50  0001 C CNN
+F 1 "+12V" H 3680 6210 50  0000 C CNN
+F 2 "" H 3680 6070 50  0001 C CNN
+F 3 "" H 3680 6070 50  0001 C CNN
+	1    3680 6070
+	1    0    0    -1
+$EndComp
 $EndSCHEMATC

Commit message: annotated schematic
Parts:
- U401: renamed from U?; Digi-Key PN (none) -> 296-SN74LVC1G97DCK3CT-ND
- gave numbers to parts that had none: 12
- renumbered C401 to C402, C402 to C403, C403 to C404, C404 to C405, C405 to C407, R403 to R402, R405 to R403, R407 to R409, R408 to R410, R409 to R414, R410 to R415, R411 to R416, U401 to U402
