File: hdw/rev_b/Pulse_Oximeter/PIC32MZ_Programming.sch (KiCad schematic (older format))
At the start: 10 parts, among them J801 PICKIT3, Q801 BSS214NW, SW801 MRST

Commit message: changed POX filtering and level shifting
Parts:
- R801: value 10 -> 0; Digi-Key PN 541-3964-1-ND -> (none)
Changed lines of the file:
@@
 P 5470 2770
 F 0 "R801" V 5370 2770 50  0000 C CNN
-F 1 "10" V 5470 2770 50  0000 C CNN
+F 1 "0" V 5470 2770 50  0000 C CNN
 F 2 "Resistors_SMD:R_0402" H 5470 2770 50  0001 C CNN
 F 3 "" H 5470 2770 50  0001 C CNN
@@
 F 5 "1%" V 5670 2770 50  0000 C CNN "Tolerance"
 F 6 "1/16W" V 5770 2770 50  0000 C CNN "Wattage"
-F 7 "541-3964-1-ND" H 5770 3170 60  0001 C CNN "Digi-Key PN"
 	1    5470 2770
 	0    -1   -1   0

Commit message: lots of rev b changes
Parts:
- removed J801: PICKIT3, Custom Footprints Library:PICKIT3_Header, symbol Connector_Generic:Conn_01x06
- removed Q801: BSS214NW, Package_TO_SOT_SMD:SOT-323_SC-70, symbol Transistor_FET:BSS214NW
- removed R803: 10, Resistors_SMD:R_0402, symbol Custom_Library:R_Custom
- added J1501: PICKIT4, Custom Footprints Library:PICKIT4_Header, symbol Connector_Generic:Conn_01x08
- added Q1501: BSS214NW, TO_SOT_Packages_SMD:SOT-323_SC-70, symbol Transistor_FET:BSS214NW
- added R1503: 100, Resistors_SMD:R_0603, symbol Custom_Library:R_Custom
- C1501: renamed from C801; footprint Capacitors_SMD:C_0402 -> Capacitors_SMD:C_0603; Digi-Key PN 490-10701-1-ND -> 311-1344-1-ND; display_footprint 0402 -> 0603
- C1502: renamed from C802; footprint Capacitors_SMD:C_0402 -> Capacitors_SMD:C_0603; Digi-Key PN 490-10701-1-ND -> 311-1344-1-ND; display_footprint 0402 -> 0603
- R1501: renamed from R801; value 0 -> 10; footprint Resistors_SMD:R_0402 -> Resistors_SMD:R_0603; Digi-Key PN (none) -> YAG3351CT-ND; Wattage 1/16W -> 1/10W; display_footprint 0402 -> 0603
- R1502: renamed from R802; footprint Resistors_SMD:R_0402 -> Resistors_SMD:R_0603; Digi-Key PN RMCF0402FT10K0CT-ND -> RMCF0603FT10K0CT-ND; Wattage 1/16W -> 1/10W; display_footprint 0402 -> 0603
- R1504: renamed from R804; footprint Resistors_SMD:R_0402 -> Resistors_SMD:R_0603; Digi-Key PN RMCF0402FT10K0CT-ND -> RMCF0603FT10K0CT-ND; Wattage 1/16W -> 1/10W; display_footprint 0402 -> 0603
- R1505: renamed from R805; footprint Resistors_SMD:R_0402 -> Resistors_SMD:R_0603; Digi-Key PN 541-1.00KLCT-ND -> RMCF0603FT1K00CT-ND; Wattage 1/16W -> 1/10W; display_footprint 0402 -> 0603
- renumbered SW801 to SW1501
Connections:
- net labels added: ~MCLR
- no-connect marks 1 -> 3
Other:
- moved on the sheet: C1501

Commit message: changed all passives to 0402, cleared digikey pns
Parts:
- C1501, C1502: footprint Capacitors_SMD:C_0603 -> Capacitors_SMD:C_0402; Digi-Key PN 311-1344-1-ND -> (none); display_footprint 0603 -> 0402
- R1501: footprint Resistors_SMD:R_0603 -> Resistors_SMD:R_0402; Digi-Key PN YAG3351CT-ND -> (none); Wattage 1/10W -> 1/16W; display_footprint 0603 -> 0402
- R1502, R1504: footprint Resistors_SMD:R_0603 -> Resistors_SMD:R_0402; Digi-Key PN RMCF0603FT10K0CT-ND -> (none); Wattage 1/10W -> 1/16W; display_footprint 0603 -> 0402
- R1503: footprint Resistors_SMD:R_0603 -> Resistors_SMD:R_0402; Digi-Key PN A106047CT-ND -> (none); Wattage 1/10W -> 1/16W; display_footprint 0603 -> 0402
- R1505: footprint Resistors_SMD:R_0603 -> Resistors_SMD:R_0402; Digi-Key PN RMCF0603FT1K00CT-ND -> (none); Wattage 1/10W -> 1/16W; display_footprint 0603 -> 0402
Changed lines of the file:
@@
 F 0 "C1501" H 3015 2130 50  0000 L CNN
 F 1 "0.1uF" H 3015 1930 50  0000 L CNN
-F 2 "Capacitors_SMD:C_0603" H 3028 1880 50  0001 C CNN
+F 2 "Capacitors_SMD:C_0402" H 3028 1880 50  0001 C CNN
 F 3 "" H 3015 2130 50  0001 C CNN
-F 4 "0603" H 2840 2130 50  0000 R CNN "display_footprint"
+F 4 "0402" H 2840 2130 50  0000 R CNN "display_footprint"
 F 5 "50V" H 2840 2030 50  0000 R CNN "Voltage"
 F 6 "X7R" H 2840 1930 50  0000 R CNN "Dielectric"
-F 7 "311-1344-1-ND" H 3415 2530 60  0001 C CNN "Digi-Key PN"
+F 7 "" H 3415 2530 60  0001 C CNN "Digi-Key PN"
 	1    2990 2030
 	1    0    0    -1
@@
 F 0 "R1504" H 7490 2020 50  0000 R CNN
 F 1 "10k" V 7550 2020 50  0000 C CNN
-F 2 "Resistors_SMD:R_0603" H 7550 2020 50  0001 C CNN
+F 2 "Resistors_SMD:R_0402" H 7550 2020 50  0001 C CNN
 F 3 "" H 7550 2020 50  0001 C CNN
-F 4 "0603" H 7740 2100 50  0000 C CNN "display_footprint"
+F 4 "0402" H 7740 2100 50  0000 C CNN "display_footprint"
 F 5 "1%" H 7730 2020 50  0000 C CNN "Tolerance"
-F 6 "1/10W" H 7760 1950 50  0000 C CNN "Wattage"
-F 7 "RMCF0603FT10K0CT-ND" H 7850 2420 60  0001 C CNN "Digi-Key PN"
+F 6 "1/16W" H 7760 1950 50  0000 C CNN "Wattage"
+F 7 "" H 7850 2420 60  0001 C CNN "Digi-Key PN"
 	1    7550 2020
 	-1   0    0    -1
@@
 F 0 "C1502" H 7575 2930 50  0000 L CNN
 F 1 "0.1uF" H 7575 2730 50  0000 L CNN
-F 2 "Capacitors_SMD:C_0603" H 7588 2680 50  0001 C CNN
+F 2 "Capacitors_SMD:C_0402" H 7588 2680 50  0001 C CNN
 F 3 "" H 7575 2930 50  0001 C CNN
-F 4 "0603" H 7400 2930 50  0000 R CNN "display_footprint"
+F 4 "0402" H 7400 2930 50  0000 R CNN "display_footprint"
 F 5 "50V" H 7400 2830 50  0000 R CNN "Voltage"
 F 6 "X7R" H 7400 2730 50  0000 R CNN "Dielectric"
-F 7 "311-1344-1-ND" H 7975 3330 60  0001 C CNN "Digi-Key PN"
+F 7 "" H 7975 3330 60  0001 C CNN "Digi-Key PN"
 	1    7550 2830
 	1    0    0    -1
@@
 F 0 "R1505" V 7980 2250 50  0000 C CNN
 F 1 "1k" V 8080 2250 50  0000 C CNN
-F 2 "Resistors_SMD:R_0603" H 8080 2250 50  0001 C CNN
+F 2 "Resistors_SMD:R_0402" H 8080 2250 50  0001 C CNN
 F 3 "" H 8080 2250 50  0001 C CNN
-F 4 "0603" V 8180 2250 50  0000 C CNN "display_footprint"
+F 4 "0402" V 8180 2250 50  0000 C CNN "display_footprint"
 F 5 "1%" V 8280 2250 50  0000 C CNN "Tolerance"
-F 6 "1/10W" V 8380 2250 50  0000 C CNN "Wattage"
-F 7 "RMCF0603FT1K00CT-ND" H 8380 2650 60  0001 C CNN "Digi-Key PN"
+F 6 "1/16W" V 8380 2250 50  0000 C CNN "Wattage"
+F 7 "" H 8380 2650 60  0001 C CNN "Digi-Key PN"
 	1    8080 2250
 	0    1    1    0
@@
 F 0 "R1503" V 6760 2250 50  0000 C CNN
 F 1 "100" V 6860 2250 50  0000 C CNN
-F 2 "Resistors_SMD:R_0603" H 6860 2250 50  0001 C CNN
+F 2 "Resistors_SMD:R_0402" H 6860 2250 50  0001 C CNN
 F 3 "" H 6860 2250 50  0001 C CNN
-F 4 "0603" V 6960 2250 50  0000 C CNN "display_footprint"
+F 4 "0402" V 6960 2250 50  0000 C CNN "display_footprint"
 F 5 "1%" V 7060 2250 50  0000 C CNN "Tolerance"
-F 6 "1/10W" V 7160 2250 50  0000 C CNN "Wattage"
-F 7 "A106047CT-ND" H 7160 2650 60  0001 C CNN "Digi-Key PN"
+F 6 "1/16W" V 7160 2250 50  0000 C CNN "Wattage"
+F 7 "" H 7160 2650 60  0001 C CNN "Digi-Key PN"
 	1    6860 2250
 	0    1    1    0
@@
 F 0 "R1501" V 5370 2770 50  0000 C CNN
 F 1 "10" V 5470 2770 50  0000 C CNN
-F 2 "Resistors_SMD:R_0603" H 5470 2770 50  0001 C CNN
+F 2 "Resistors_SMD:R_0402" H 5470 2770 50  0001 C CNN
 F 3 "" H 5470 2770 50  0001 C CNN
-F 4 "0603" V 5570 2770 50  0000 C CNN "display_footprint"
+F 4 "0402" V 5570 2770 50  0000 C CNN "display_footprint"
 F 5 "1%" V 5670 2770 50  0000 C CNN "Tolerance"
-F 6 "1/10W" V 5770 2770 50  0000 C CNN "Wattage"
-F 7 "YAG3351CT-ND" H 5770 3170 60  0001 C CNN "Digi-Key PN"
+F 6 "1/16W" V 5770 2770 50  0000 C CNN "Wattage"
+F 7 "" H 5770 3170 60  0001 C CNN "Digi-Key PN"
 	1    5470 2770
 	0    -1   -1   0
@@
 F 0 "R1502" H 5860 3000 50  0000 R CNN
 F 1 "10k" V 5920 3000 50  0000 C CNN
-F 2 "Resistors_SMD:R_0603" H 5920 3000 50  0001 C CNN
+F 2 "Resistors_SMD:R_0402" H 5920 3000 50  0001 C CNN
 F 3 "" H 5920 3000 50  0001 C CNN
-F 4 "0603" H 6110 3080 50  0000 C CNN "display_footprint"
+F 4 "0402" H 6110 3080 50  0000 C CNN "display_footprint"
 F 5 "1%" H 6100 3000 50  0000 C CNN "Tolerance"
-F 6 "1/10W" H 6130 2930 50  0000 C CNN "Wattage"
-F 7 "RMCF0603FT10K0CT-ND" H 6220 3400 60  0001 C CNN "Digi-Key PN"
+F 6 "1/16W" H 6130 2930 50  0000 C CNN "Wattage"
+F 7 "" H 6220 3400 60  0001 C CNN "Digi-Key PN"
 	1    5920 3000
 	1    0    0    -1

Commit message: few little tweaks
Parts:
- R1501: value 10 -> 100
Connections:
- net at SW1501.2: now also R1501.2; no longer R1501.1
- net at Q1501.1 (G), R1502.1: now also R1501.1; no longer R1501.2
Changed lines of the file:
@@
-$EndComp
-$Comp
-L Custom_Library:R_Custom R1501
-U 1 1 5BE087CB
-P 5470 2770
-F 0 "R1501" V 5370 2770 50  0000 C CNN
-F 1 "10" V 5470 2770 50  0000 C CNN
-F 2 "Resistors_SMD:R_0402" H 5470 2770 50  0001 C CNN
-F 3 "" H 5470 2770 50  0001 C CNN
-F 4 "0402" V 5570 2770 50  0000 C CNN "display_footprint"
-F 5 "1%" V 5670 2770 50  0000 C CNN "Tolerance"
-F 6 "1/16W" V 5770 2770 50  0000 C CNN "Wattage"
-F 7 "" H 5770 3170 60  0001 C CNN "Digi-Key PN"
-	1    5470 2770
-	0    -1   -1   0
 $EndComp
 $Comp
@@
 Wire Wire Line
 	1270 1990 2320 1990
+$Comp
+L Custom_Library:R_Custom R1501
+U 1 1 5FE81E3C
+P 5470 2770
+F 0 "R1501" V 5370 2770 50  0000 C CNN
+F 1 "100" V 5470 2770 50  0000 C CNN
+F 2 "Resistors_SMD:R_0402" H 5470 2770 50  0001 C CNN
+F 3 "" H 5470 2770 50  0001 C CNN
+F 4 "0402" V 5570 2770 50  0000 C CNN "display_footprint"
+F 5 "1%" V 5670 2770 50  0000 C CNN "Tolerance"
+F 6 "1/16W" V 5770 2770 50  0000 C CNN "Wattage"
+F 7 "" H 5770 3170 60  0001 C CNN "Digi-Key PN"
+	1    5470 2770
+	0    1    -1   0
+$EndComp
 $EndSCHEMATC

Commit message: annotated schematic
Parts:
- renumbered C1501 to C801, C1502 to C802, J1501 to J801, Q1501 to Q801, R1501 to R801, R1502 to R802, R1503 to R803, R1504 to R804, R1505 to R805, SW1501 to SW801
Changed lines of the file:
@@
 PIC32MZ_ICSPCLK
 $Comp
-L power:GND #PWR01502
+L power:GND #PWR0802
 U 1 1 5BB4A7C4
 P 2320 2040
-F 0 "#PWR01502" H 2320 1790 50  0001 C CNN
+F 0 "#PWR0802" H 2320 1790 50  0001 C CNN
 F 1 "GND" H 2320 1890 50  0000 C CNN
 F 2 "" H 2320 2040 50  0001 C CNN
@@
 NoConn ~ 1270 2290
 $Comp
-L Custom_Library:C_Custom C1501
+L Custom_Library:C_Custom C801
 U 1 1 5BC13497
 P 2990 2030
-F 0 "C1501" H 3015 2130 50  0000 L CNN
+F 0 "C801" H 3015 2130 50  0000 L CNN
 F 1 "0.1uF" H 3015 1930 50  0000 L CNN
 F 2 "Capacitors_SMD:C_0402" H 3028 1880 50  0001 C CNN
@@
 $EndComp
 $Comp
-L power:GND #PWR01504
+L power:GND #PWR0804
 U 1 1 5BC1349E
 P 2990 2180
-F 0 "#PWR01504" H 2990 1930 50  0001 C CNN
+F 0 "#PWR0804" H 2990 1930 50  0001 C CNN
 F 1 "GND" H 2990 2030 50  0000 C CNN
 F 2 "" H 2990 2180 50  0001 C CNN
@@
 AR Path="/5BAAE16C/5BC152E5" Ref="R?"  Part="1"
 AR Path="/5C1D5CB6/5BC152E5" Ref="R?"  Part="1"
-AR Path="/5CB0BC26/5BC152E5" Ref="R1504"  Part="1"
-AR Path="/5EAE2EF2/5BC152E5" Ref="R1504"  Part="1"
-F 0 "R1504" H 7490 2020 50  0000 R CNN
+AR Path="/5CB0BC26/5BC152E5" Ref="R?"  Part="1"
+AR Path="/5EAE2EF2/5BC152E5" Ref="R804"  Part="1"
+F 0 "R804" H 7490 2020 50  0000 R CNN
 F 1 "10k" V 7550 2020 50  0000 C CNN
 F 2 "Resistors_SMD:R_0402" H 7550 2020 50  0001 C CNN
@@
 $EndComp
 $Comp
-L Custom_Library:C_Custom C1502
+L Custom_Library:C_Custom C802
 U 1 1 5BC1574E
 P 7550 2830
-F 0 "C1502" H 7575 2930 50  0000 L CNN
+F 0 "C802" H 7575 2930 50  0000 L CNN
 F 1 "0.1uF" H 7575 2730 50  0000 L CNN
 F 2 "Capacitors_SMD:C_0402" H 7588 2680 50  0001 C CNN
@@
 $EndComp
 $Comp
-L power:GND #PWR01509
+L power:GND #PWR0809
 U 1 1 5BC15E18
 P 7550 2980
-F 0 "#PWR01509" H 7550 2730 50  0001 C CNN
+F 0 "#PWR0809" H 7550 2730 50  0001 C CNN
 F 1 "GND" H 7550 2830 50  0000 C CNN
 F 2 "" H 7550 2980 50  0001 C CNN
@@
 $EndComp
 $Comp
-L Custom_Library:R_Custom R1505
+L Custom_Library:R_Custom R805
 U 1 1 5BC16316
 P 8080 2250
-F 0 "R1505" V 7980 2250 50  0000 C CNN
+F 0 "R805" V 7980 2250 50  0000 C CNN
 F 1 "1k" V 8080 2250 50  0000 C CNN
 F 2 "Resistors_SMD:R_0402" H 8080 2250 50  0001 C CNN
@@
 ~MCLR
 $Comp
-L Switch:SW_Push SW1501
+L Switch:SW_Push SW801
 U 1 1 5BC17B44
 P 5020 2770
-F 0 "SW1501" H 5020 3055 50  0000 C CNN
+F 0 "SW801" H 5020 3055 50  0000 C CNN
 F 1 "MRST" H 5020 2964 50  0000 C CNN
 F 2 "Buttons_Switches_THT:SW_PUSH_6mm" H 5020 2970 50  0001 C CNN
@@
 $EndComp
 $Comp
-L Custom_Library:R_Custom R1503
+L Custom_Library:R_Custom R803
 U 1 1 5BC190FF
 P 6860 2250
-F 0 "R1503" V 6760 2250 50  0000 C CNN
+F 0 "R803" V 6760 2250 50  0000 C CNN
 F 1 "100" V 6860 2250 50  0000 C CNN
 F 2 "Resistors_SMD:R_0402" H 6860 2250 50  0001 C CNN
@@
 AR Path="/5BB844FD/5BE087BA" Ref="Q?"  Part="1"
 AR Path="/5C1D5CB6/5BE087BA" Ref="Q?"  Part="1"
-AR Path="/5CB0BC26/5BE087BA" Ref="Q1501"  Part="1"
-AR Path="/5EAE2EF2/5BE087BA" Ref="Q1501"  Part="1"
-F 0 "Q1501" H 6610 2845 50  0000 L CNN
+AR Path="/5CB0BC26/5BE087BA" Ref="Q?"  Part="1"
+AR Path="/5EAE2EF2/5BE087BA" Ref="Q801"  Part="1"
+F 0 "Q801" H 6610 2845 50  0000 L CNN
 F 1 "BSS214NW" H 6610 2770 50  0000 L CNN
 F 2 "TO_SOT_Packages_SMD:SOT-323_SC-70" H 6610 2695 50  0001 L CIN
@@
 $EndComp
 $Comp
-L power:GND #PWR01507
+L power:GND #PWR0807
 U 1 1 5BE087C1
 P 6510 2970
-F 0 "#PWR01507" H 6510 2720 50  0001 C CNN
+F 0 "#PWR0807" H 6510 2720 50  0001 C CNN
 F 1 "GND" H 6510 2820 50  0000 C CNN
 F 2 "" H 6510 2970 50  0001 C CNN
@@
 AR Path="/5BB844FD/5BE087D6" Ref="R?"  Part="1"
 AR Path="/5C1D5CB6/5BE087D6" Ref="R?"  Part="1"
-AR Path="/5CB0BC26/5BE087D6" Ref="R1502"  Part="1"
-AR Path="/5EAE2EF2/5BE087D6" Ref="R1502"  Part="1"
-F 0 "R1502" H 5860 3000 50  0000 R CNN
+AR Path="/5CB0BC26/5BE087D6" Ref="R?"  Part="1"
+AR Path="/5EAE2EF2/5BE087D6" Ref="R802"  Part="1"
+F 0 "R802" H 5860 3000 50  0000 R CNN
 F 1 "10k" V 5920 3000 50  0000 C CNN
 F 2 "Resistors_SMD:R_0402" H 5920 3000 50  0001 C CNN
@@
 $EndComp
 $Comp
-L power:GND #PWR01506
+L power:GND #PWR0806
 U 1 1 5BE087DD
 P 5920 3150
-F 0 "#PWR01506" H 5920 2900 50  0001 C CNN
+F 0 "#PWR0806" H 5920 2900 50  0001 C CNN
 F 1 "GND" H 5920 3000 50  0000 C CNN
 F 2 "" H 5920 3150 50  0001 C CNN
@@
 	7550 2680 7550 2250
 $Comp
-L Connector_Generic:Conn_01x08 J1501
+L Connector_Generic:Conn_01x08 J801
 U 1 1 5F816A14
 P 1070 2090
-F 0 "J1501" H 940 2650 50  0000 C CNN
+F 0 "J801" H 940 2650 50  0000 C CNN
 F 1 "PICKIT4" H 940 2550 50  0000 C CNN
 F 2 "Custom Footprints Library:PICKIT4_Header" H 1070 2090 50  0001 C CNN
@@
 NoConn ~ 1270 2490
 $Comp
-L power:+3.3V #PWR01501
+L power:+3.3V #PWR0801
 U 1 1 5F81A9D9
 P 2320 1820
-F 0 "#PWR01501" H 2320 1670 50  0001 C CNN
+F 0 "#PWR0801" H 2320 1670 50  0001 C CNN
 F 1 "+3.3V" H 2320 1960 50  0000 C CNN
 F 2 "" H 2320 1820 50  0001 C CNN
@@
 $EndComp
 $Comp
-L power:+3.3V #PWR01503
+L power:+3.3V #PWR0803
 U 1 1 5F81AC2F
 P 2990 1880
-F 0 "#PWR01503" H 2990 1730 50  0001 C CNN
+F 0 "#PWR0803" H 2990 1730 50  0001 C CNN
 F 1 "+3.3V" H 2990 2020 50  0000 C CNN
 F 2 "" H 2990 1880 50  0001 C CNN
@@
 $EndComp
 $Comp
-L power:+3.3V #PWR01505
+L power:+3.3V #PWR0805
 U 1 1 5F81B753
 P 4670 2720
-F 0 "#PWR01505" H 4670 2570 50  0001 C CNN
+F 0 "#PWR0805" H 4670 2570 50  0001 C CNN
 F 1 "+3.3V" H 4670 2860 50  0000 C CNN
 F 2 "" H 4670 2720 50  0001 C CNN
@@
 $EndComp
 $Comp
-L power:+3.3V #PWR01508
+L power:+3.3V #PWR0808
 U 1 1 5F81BC42
 P 7550 1870
-F 0 "#PWR01508" H 7550 1720 50  0001 C CNN
+F 0 "#PWR0808" H 7550 1720 50  0001 C CNN
 F 1 "+3.3V" H 7550 2010 50  0000 C CNN
 F 2 "" H 7550 1870 50  0001 C CNN
@@
 	1270 1990 2320 1990
 $Comp
-L Custom_Library:R_Custom R1501
+L Custom_Library:R_Custom R801
 U 1 1 5FE81E3C
 P 5470 2770
-F 0 "R1501" V 5370 2770 50  0000 C CNN
+F 0 "R801" V 5370 2770 50  0000 C CNN
 F 1 "100" V 5470 2770 50  0000 C CNN
 F 2 "Resistors_SMD:R_0402" H 5470 2770 50  0001 C CNN

Commit message: passed ERC
Connections:
- net ~MCLR is gone; now on net ~PIC32MZ_MCLR: R805.1
Changed lines of the file:
@@
 Connection ~ 7550 2250
 Text GLabel 8230 2250 2    50   UnSpc ~ 0
-~MCLR
+~PIC32MZ_MCLR
 $Comp
 L Switch:SW_Push SW801
