File: hdw/rev_b/Pulse_Oximeter/PIC32MZ_Programming.sch (KiCad schematic (older format))
At the start: 10 parts, among them J801 PICKIT4, Q801 BSS214NW, SW801 MRST

Commit message: assigned digikey PNs
Parts:
- C801, C802: Digi-Key PN (none) -> 490-10698-1-ND; Voltage 50V -> 25V
- R801, R803: Digi-Key PN (none) -> RMCF0402FT100RCT-ND
- R802, R804: Digi-Key PN (none) -> RMCF0402FT10K0CT-ND
- R805: Digi-Key PN (none) -> RMCF0402FT1K00CT-ND
Changed lines of the file:
@@
 F 3 "" H 3015 2130 50  0001 C CNN
 F 4 "0402" H 2840 2130 50  0000 R CNN "display_footprint"
-F 5 "50V" H 2840 2030 50  0000 R CNN "Voltage"
+F 5 "25V" H 2840 2030 50  0000 R CNN "Voltage"
 F 6 "X7R" H 2840 1930 50  0000 R CNN "Dielectric"
-F 7 "" H 3415 2530 60  0001 C CNN "Digi-Key PN"
+F 7 "490-10698-1-ND" H 3415 2530 60  0001 C CNN "Digi-Key PN"
 	1    2990 2030
 	1    0    0    -1
@@
 F 5 "1%" H 7730 2020 50  0000 C CNN "Tolerance"
 F 6 "1/16W" H 7760 1950 50  0000 C CNN "Wattage"
-F 7 "" H 7850 2420 60  0001 C CNN "Digi-Key PN"
+F 7 "RMCF0402FT10K0CT-ND" H 7850 2420 60  0001 C CNN "Digi-Key PN"
 	1    7550 2020
 	-1   0    0    -1
@@
 F 3 "" H 7575 2930 50  0001 C CNN
 F 4 "0402" H 7400 2930 50  0000 R CNN "display_footprint"
-F 5 "50V" H 7400 2830 50  0000 R CNN "Voltage"
+F 5 "25V" H 7400 2830 50  0000 R CNN "Voltage"
 F 6 "X7R" H 7400 2730 50  0000 R CNN "Dielectric"
-F 7 "" H 7975 3330 60  0001 C CNN "Digi-Key PN"
+F 7 "490-10698-1-ND" H 7975 3330 60  0001 C CNN "Digi-Key PN"
 	1    7550 2830
 	1    0    0    -1
@@
 F 5 "1%" V 8280 2250 50  0000 C CNN "Tolerance"
 F 6 "1/16W" V 8380 2250 50  0000 C CNN "Wattage"
-F 7 "" H 8380 2650 60  0001 C CNN "Digi-Key PN"
+F 7 "RMCF0402FT1K00CT-ND" H 8380 2650 60  0001 C CNN "Digi-Key PN"
 	1    8080 2250
 	0    1    1    0
@@
 F 5 "1%" V 7060 2250 50  0000 C CNN "Tolerance"
 F 6 "1/16W" V 7160 2250 50  0000 C CNN "Wattage"
-F 7 "" H 7160 2650 60  0001 C CNN "Digi-Key PN"
+F 7 "RMCF0402FT100RCT-ND" H 7160 2650 60  0001 C CNN "Digi-Key PN"
 	1    6860 2250
 	0    1    1    0
@@
 F 5 "1%" H 6100 3000 50  0000 C CNN "Tolerance"
 F 6 "1/16W" H 6130 2930 50  0000 C CNN "Wattage"
-F 7 "" H 6220 3400 60  0001 C CNN "Digi-Key PN"
+F 7 "RMCF0402FT10K0CT-ND" H 6220 3400 60  0001 C CNN "Digi-Key PN"
 	1    5920 3000
 	1    0    0    -1
@@
 F 5 "1%" V 5670 2770 50  0000 C CNN "Tolerance"
 F 6 "1/16W" V 5770 2770 50  0000 C CNN "Wattage"
-F 7 "" H 5770 3170 60  0001 C CNN "Digi-Key PN"
+F 7 "RMCF0402FT100RCT-ND" H 5770 3170 60  0001 C CNN "Digi-Key PN"
 	1    5470 2770
 	0    1    -1   0
