File: hdw/rev_b/Pulse_Oximeter/PGOOD_LEDs.sch (KiCad schematic (older format))
At the start: 18 parts, among them U1801 TPS71530, U1802 74LVC1G06, U1803 74LVC1G06, U1805 74LVC1G06, U1806 74LVC1G06

Commit message: changed PGOOD LED drivers
Parts:
- removed C1801: 0.1uF, Capacitors_SMD:C_0402, symbol Custom_Library:C_Custom
- removed C1802: 10uF, Capacitors_SMD:C_0402, symbol Custom_Library:C_Custom
- removed U1801: TPS71530, Package_TO_SOT_SMD:SOT-353_SC-70-5, symbol Regulator_Linear:TPS71530__SC70
- removed U1802, U1803, U1805, U1806: 74LVC1G06, TO_SOT_Packages_SMD:SOT-353_SC-70-5, symbol Custom_Library:74LVC1G06_Power
- added R?: 10k, Resistors_SMD:R_0402, symbol Custom_Library:R_Custom
- added U? (x4): 74LVC1G97, Package_TO_SOT_SMD:SOT-363_SC-70-6, symbol Custom_Library:74LVC1G97_Power_AND
Connections:
- net labels added: PGOOD_LED_EN
- net labels removed: +12V
- wire segments 17 -> 11

Commit message: changed all passives to 0402, cleared digikey pns
Parts:
- C1803: footprint Capacitors_SMD:C_0402 -> (none); Configuration (none) -> USB; Digi-Key PN 490-10701-1-ND -> (none); display_footprint (none) -> 0402
- C1805, C1806: Digi-Key PN 490-10701-1-ND -> (none)
- D1802, U?: Configuration (none) -> USB
- R1801, R1804, R1805: Digi-Key PN 541-1.00KLCT-ND -> (none)
- R1802: Configuration (none) -> USB; Digi-Key PN 541-1.00KLCT-ND -> (none)
- R?: Digi-Key PN RMCF0402FT10K0CT-ND -> (none)
Other:
- moved on the sheet: C1803, C1805, C1806, D1801, D1802, D1804, D1805, R1801, R1802, R1804, R1805, R?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

Commit message: removed more unique components, cleaned up SCH
Parts:
- C1803: footprint (none) -> Capacitors_SMD:C_0402
- C1805, C1806: display_footprint (none) -> 0402
Changed lines of the file:
@@
 F 3 "" H 6565 3150 50  0001 C CNN
 F 4 "" H 6965 3550 60  0001 C CNN "Digi-Key PN"
-F 5 "" H 6390 3150 50  0000 R CNN "display_footprint"
+F 5 "0402" H 6390 3150 50  0000 R CNN "display_footprint"
 F 6 "50V" H 6390 3050 50  0000 R CNN "Voltage"
 F 7 "X7R" H 6390 2950 50  0000 R CNN "Dielectric"
@@
 F 3 "" H 8565 3150 50  0001 C CNN
 F 4 "" H 8965 3550 60  0001 C CNN "Digi-Key PN"
-F 5 "" H 8390 3150 50  0000 R CNN "display_footprint"
+F 5 "0402" H 8390 3150 50  0000 R CNN "display_footprint"
 F 6 "50V" H 8390 3050 50  0000 R CNN "Voltage"
 F 7 "X7R" H 8390 2950 50  0000 R CNN "Dielectric"
@@
 F 0 "C1803" H 4565 3150 50  0000 L CNN
 F 1 "0.1uF" H 4565 2950 50  0000 L CNN
-F 2 "" H 4578 2900 50  0001 C CNN
+F 2 "Capacitors_SMD:C_0402" H 4578 2900 50  0001 C CNN
 F 3 "" H 4565 3150 50  0001 C CNN
 F 4 "0402" H 4390 3150 50  0000 R CNN "display_footprint"

Commit message: annotated schematic
Parts:
- U1801, U1802, U1803, U1804: renamed from U?; Digi-Key PN (none) -> 296-SN74LVC1G97DCK3CT-ND
- gave numbers to parts that had none: 1
- renumbered C1803 to C1801, C1805 to C1802, C1806 to C1803, D1804 to D1803, D1805 to D1804, R1801 to R1802, R1802 to R1803

Commit message: fixed PGOOD LED drivers
Parts:
- removed U1801, U1802, U1803, U1804: 74LVC1G97, Package_TO_SOT_SMD:SOT-363_SC-70-6, symbol Custom_Library:74LVC1G97_Power_AND
- added U1801, U1802, U1803, U1804: 74LVC1G97, Package_TO_SOT_SMD:SOT-363_SC-70-6, symbol Custom_Library:74LVC1G97_Power_NAND_INV
Connections:
- net +3V3: now also U1801.1 (VCC), U1801.5 (VCC), U1802.1 (VCC), U1802.5 (VCC), U1803.1 (VCC), U1803.5 (VCC), U1804.1 (VCC), U1804.5 (VCC)
- net GND: now also U1801.2 (GND), U1802.2 (GND), U1803.2 (GND), U1804.2 (GND)
- net POS12_PGOOD: now also U1801.6
- net POS1P8_PGOOD: now also U1803.6
- net POS3P3_PGOOD: now also U1804.6
- net POS5_USB_PGOOD: now also U1802.6
- net at D1801.1 (K): now also U1801.4
- net at D1803.1 (K): now also U1803.4
- net at D1804.1 (K): now also U1804.4
- net at D1802.1 (K): now also U1802.4
- net PGOOD_LED_EN renamed PGOOD_LED_SHDN
- net PGOOD_LED_SHDN: now also U1801.3, U1802.3, U1803.3, U1804.3
Changed lines of the file:
@@
 POS5_USB_PGOOD
-$Comp
-L Custom_Library:74LVC1G97_Power_AND U1803
-U 1 1 5FDA165A
-P 6650 3740
-F 0 "U1803" H 6710 3890 50  0000 L CNN
-F 1 "74LVC1G97" H 6710 3590 50  0000 L CNN
-F 2 "Package_TO_SOT_SMD:SOT-363_SC-70-6" H 6700 3740 50  0001 C CNN
-F 3 "http://www.ti.com/lit/ds/symlink/sn74lvc1g97.pdf" H 6700 3740 50  0001 C CNN
-F 4 "296-SN74LVC1G97DCK3CT-ND" H 6650 3740 50  0001 C CNN "Digi-Key PN"
-	1    6650 3740
-	1    0    0    -1
-$EndComp
-$Comp
-L Custom_Library:74LVC1G97_Power_AND U1801
-U 1 1 5FDA52FA
-P 2650 3740
-F 0 "U1801" H 2710 3890 50  0000 L CNN
-F 1 "74LVC1G97" H 2710 3590 50  0000 L CNN
-F 2 "Package_TO_SOT_SMD:SOT-363_SC-70-6" H 2700 3740 50  0001 C CNN
-F 3 "http://www.ti.com/lit/ds/symlink/sn74lvc1g97.pdf" H 2700 3740 50  0001 C CNN
-F 4 "296-SN74LVC1G97DCK3CT-ND" H 2650 3740 50  0001 C CNN "Digi-Key PN"
-	1    2650 3740
-	1    0    0    -1
-$EndComp
-$Comp
-L Custom_Library:74LVC1G97_Power_AND U1802
-U 1 1 5FDA580E
-P 4650 3740
-F 0 "U1802" H 4710 3890 50  0000 L CNN
-F 1 "74LVC1G97" H 4710 3590 50  0000 L CNN
-F 2 "Package_TO_SOT_SMD:SOT-363_SC-70-6" H 4700 3740 50  0001 C CNN
-F 3 "http://www.ti.com/lit/ds/symlink/sn74lvc1g97.pdf" H 4700 3740 50  0001 C CNN
-F 4 "USB" H 4870 3490 50  0000 C CNN "Configuration"
-F 5 "296-SN74LVC1G97DCK3CT-ND" H 4650 3740 50  0001 C CNN "Digi-Key PN"
-	1    4650 3740
-	1    0    0    -1
-$EndComp
-$Comp
-L Custom_Library:74LVC1G97_Power_AND U1804
-U 1 1 5FDA5C2B
-P 8650 3740
-F 0 "U1804" H 8710 3890 50  0000 L CNN
-F 1 "74LVC1G97" H 8710 3590 50  0000 L CNN
-F 2 "Package_TO_SOT_SMD:SOT-363_SC-70-6" H 8700 3740 50  0001 C CNN
-F 3 "http://www.ti.com/lit/ds/symlink/sn74lvc1g97.pdf" H 8700 3740 50  0001 C CNN
-F 4 "296-SN74LVC1G97DCK3CT-ND" H 8650 3740 50  0001 C CNN "Digi-Key PN"
-	1    8650 3740
-	1    0    0    -1
-$EndComp
 $Comp
 L power:+3.3V #PWR01804
@@
 $EndComp
 Text GLabel 2190 3790 0    50   Input ~ 0
-PGOOD_LED_EN
-Text GLabel 4350 3790 0    50   Input ~ 0
-PGOOD_LED_EN
-Text GLabel 6350 3790 0    50   Input ~ 0
-PGOOD_LED_EN
-Text GLabel 8350 3790 0    50   Input ~ 0
-PGOOD_LED_EN
+PGOOD_LED_SHDN
 $Comp
 L Custom_Library:R_Custom R?
@@
 	1    0    0    -1
 $EndComp
+$Comp
+L Custom_Library:74LVC1G97_Power_NAND_INV U1801
+U 1 1 5FE744B0
+P 2650 3740
+F 0 "U1801" H 2710 3890 50  0000 L CNN
+F 1 "74LVC1G97" H 2710 3590 50  0000 L CNN
+F 2 "Package_TO_SOT_SMD:SOT-363_SC-70-6" H 2700 3740 50  0001 C CNN
+F 3 "http://www.ti.com/lit/ds/symlink/sn74lvc1g97.pdf" H 2700 3740 50  0001 C CNN
+	1    2650 3740
+	1    0    0    -1
+$EndComp
+Text GLabel 4350 3790 0    50   Input ~ 0
+PGOOD_LED_SHDN
+Text GLabel 6350 3790 0    50   Input ~ 0
+PGOOD_LED_SHDN
+Text GLabel 8350 3790 0    50   Input ~ 0
+PGOOD_LED_SHDN
+$Comp
+L Custom_Library:74LVC1G97_Power_NAND_INV U1802
+U 1 1 5FE78E95
+P 4650 3740
+F 0 "U1802" H 4710 3890 50  0000 L CNN
+F 1 "74LVC1G97" H 4710 3590 50  0000 L CNN
+F 2 "Package_TO_SOT_SMD:SOT-363_SC-70-6" H 4700 3740 50  0001 C CNN
+F 3 "http://www.ti.com/lit/ds/symlink/sn74lvc1g97.pdf" H 4700 3740 50  0001 C CNN
+F 4 "USB" H 4650 3410 50  0000 C CNN "Configuration"
+	1    4650 3740
+	1    0    0    -1
+$EndComp
+$Comp
+L Custom_Library:74LVC1G97_Power_NAND_INV U1803
+U 1 1 5FE79518
+P 6650 3740
+F 0 "U1803" H 6710 3890 50  0000 L CNN
+F 1 "74LVC1G97" H 6710 3590 50  0000 L CNN
+F 2 "Package_TO_SOT_SMD:SOT-363_SC-70-6" H 6700 3740 50  0001 C CNN
+F 3 "http://www.ti.com/lit/ds/symlink/sn74lvc1g97.pdf" H 6700 3740 50  0001 C CNN
+	1    6650 3740
+	1    0    0    -1
+$EndComp
+$Comp
+L Custom_Library:74LVC1G97_Power_NAND_INV U1804
+U 1 1 5FE79BFE
+P 8650 3740
+F 0 "U1804" H 8710 3890 50  0000 L CNN
+F 1 "74LVC1G97" H 8710 3590 50  0000 L CNN
+F 2 "Package_TO_SOT_SMD:SOT-363_SC-70-6" H 8700 3740 50  0001 C CNN
+F 3 "http://www.ti.com/lit/ds/symlink/sn74lvc1g97.pdf" H 8700 3740 50  0001 C CNN
+	1    8650 3740
+	1    0    0    -1
+$EndComp

Commit message: USB circuit adjustments, add UART dongle header, resolve some open rev B SCH issues
Parts:
- C1801, D1802, R1803, U1802: Configuration USB -> (none)
Changed lines of the file:
@@
 Sheet 18 21
 Title "Pulse Oximeter"
-Date "2020-12-09"
+Date "2020-12-31"
 Rev "B"
-Comp "Drew Maatman"
+Comp "Drew Maatman, Nick Mussoline"
 Comment1 ""
 Comment2 ""
@@
 F 5 "50V" H 4390 3050 50  0000 R CNN "Voltage"
 F 6 "X7R" H 4390 2950 50  0000 R CNN "Dielectric"
-F 7 "USB" H 4730 3050 50  0000 C CNN "Configuration"
 	1    4540 3050
 	-1   0    0    -1
@@
 F 3 "~" H 5220 3470 50  0001 C CNN
 F 4 "1497-1219-1-ND" H 60  -2850 50  0001 C CNN "Digi-Key PN"
-F 5 "USB" V 5220 3630 50  0000 C CNN "Configuration"
 	1    5220 3470
 	0    -1   -1   0
@@
 F 5 "1%" H 5290 3170 50  0000 L CNN "Tolerance"
 F 6 "1/16W" H 5290 3100 50  0000 L CNN "Wattage"
-F 7 "" H 5520 3570 60  0001 C CNN "Digi-Key PN"
-F 8 "USB" H 5080 3260 50  0000 C CNN "Configuration"
 	1    5220 3170
 	-1   0    0    -1
@@
 F 2 "Package_TO_SOT_SMD:SOT-363_SC-70-6" H 4700 3740 50  0001 C CNN
 F 3 "http://www.ti.com/lit/ds/symlink/sn74lvc1g97.pdf" H 4700 3740 50  0001 C CNN
-F 4 "USB" H 4650 3410 50  0000 C CNN "Configuration"
 	1    4650 3740
 	1    0    0    -1
