File: hdw/rev_b/Pulse_Oximeter/POS1P8_Power_Supply.sch (KiCad schematic (older format))
At the start: 14 parts, among them U601 TPS7A91

Commit message: lots of rev b changes
Parts:
- removed C604: 10uF, Capacitors_SMD:C_0402, symbol Custom_Library:C_Custom
- removed C605: 0.1uF, Capacitors_SMD:C_0402, symbol Custom_Library:C_Custom
- removed R609: 1.87k, Resistors_SMD:R_0402, symbol Custom_Library:R_Custom
- removed R610: 1.5k, Resistors_SMD:R_0402, symbol Custom_Library:R_Custom
- removed U601: TPS7A91, Package_DFN_QFN:Texas_S-PDSO-N10_EP1.2x2mm, symbol Custom_Library:TPS7A91
- added R? (x2): 100, Resistors_SMD:R_0402, symbol Custom_Library:R_Custom
- added U?: TPS7A7200RGTR, Package_DFN_QFN:QFN-16-1EP_3x3mm_P0.5mm_EP1.75x1.75mm, symbol Custom_Library:TPS7A7200RGTR
Connections:
- wire segments 27 -> 31
- no-connect marks 0 -> 4
Other:
- moved on the sheet: C601, C602, C603, R601, R602, R606, R607, R608, TP601

Commit message: merged, more cleanups
Parts:
- R606, R608: Configuration (none) -> Telemetry
Other:
- moved on the sheet: C601, C602, C603, R601, R602, R606, R607, R608, R?, TP601, U?

Commit message: changed all passives to 0402, cleared digikey pns
Parts:
- C601, C603: Digi-Key PN 490-13211-1-ND -> (none)
- C602: Digi-Key PN 490-10701-1-ND -> (none)
- R601, R602: Digi-Key PN RMCF0402FT10K0CT-ND -> (none)
- R606, R608: Digi-Key PN 541-3964-1-ND -> (none)
Changed lines of the file:
@@
 F 5 "50V" H 3760 4740 50  0000 R CNN "Voltage"
 F 6 "X7R" H 3760 4640 50  0000 R CNN "Dielectric"
-F 7 "490-10701-1-ND" H 4335 5240 60  0001 C CNN "Digi-Key PN"
+F 7 "" H 4335 5240 60  0001 C CNN "Digi-Key PN"
 	1    3910 4740
 	1    0    0    -1
@@
 F 5 "1%" H 2360 3490 50  0000 L CNN "Tolerance"
 F 6 "1/16W" H 2370 3410 50  0000 L CNN "Wattage"
-F 7 "RMCF0402FT10K0CT-ND" H 2260 3490 50  0001 C CNN "Digi-Key PN"
+F 7 "" H 2260 3490 50  0001 C CNN "Digi-Key PN"
 	1    2260 3490
 	1    0    0    -1
@@
 F 5 "1%" H 2360 4190 50  0000 L CNN "Tolerance"
 F 6 "1/16W" H 2370 4110 50  0000 L CNN "Wattage"
-F 7 "RMCF0402FT10K0CT-ND" H 2260 4190 50  0001 C CNN "Digi-Key PN"
+F 7 "" H 2260 4190 50  0001 C CNN "Digi-Key PN"
 	1    2260 4190
 	1    0    0    -1
@@
 F 5 "1%" V 6740 2930 50  0001 C CNN "Tolerance"
 F 6 "1/16W" V 6840 2930 50  0001 C CNN "Wattage"
-F 7 "541-3964-1-ND" H 6540 2930 50  0001 C CNN "Digi-Key PN"
+F 7 "" H 6540 2930 50  0001 C CNN "Digi-Key PN"
 F 8 "Telemetry" V 6360 2930 50  0000 C CNN "Configuration"
 	1    6540 2930
@@
 F 5 "1%" V 7200 2930 50  0001 C CNN "Tolerance"
 F 6 "1/16W" V 7300 2930 50  0001 C CNN "Wattage"
-F 7 "541-3964-1-ND" H 7000 2930 50  0001 C CNN "Digi-Key PN"
+F 7 "" H 7000 2930 50  0001 C CNN "Digi-Key PN"
 F 8 "Telemetry" V 7100 2930 50  0000 C CNN "Configuration"
 	1    7000 2930
@@
 F 5 "6.3V" H 3430 3490 50  0000 R CNN "Voltage"
 F 6 "X5R" H 3430 3390 50  0000 R CNN "Dielectric"
-F 7 "490-13211-1-ND" H 3580 3490 50  0001 C CNN "Digi-Key PN"
+F 7 "" H 3580 3490 50  0001 C CNN "Digi-Key PN"
 	1    3580 3490
 	1    0    0    -1
@@
 F 5 "6.3V" H 5330 3670 50  0000 R CNN "Voltage"
 F 6 "X5R" H 5330 3570 50  0000 R CNN "Dielectric"
-F 7 "490-13211-1-ND" H 5480 3670 50  0001 C CNN "Digi-Key PN"
+F 7 "" H 5480 3670 50  0001 C CNN "Digi-Key PN"
 	1    5480 3670
 	1    0    0    -1

Commit message: removed more unique components, cleaned up SCH
Parts:
- added R? (x3): 0, Resistors_SMD:R_0402, symbol Custom_Library:R_Custom
- R607: Configuration (none) -> Telemetry
Connections:
- net +1.8V: now also R?.2, R?.2, R?.2
- net at C603.1, R606.2, R607.1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: now also R?.1, R?.1, R?.1
Other:
- moved on the sheet: R606, R607, R608, TP601

Commit message: annotated schematic
Parts:
- C602: value 0.1uF -> 10nF
- gave numbers to parts that had none: 6
- renumbered R606 to R605, R607 to R606, R608 to R610
Changed lines of the file:
@@
 $EndDescr
 $Comp
-L power:GND #PWR0607
+L power:GND #PWR0606
 U 1 1 5EBAD848
 P 4590 4710
-F 0 "#PWR0607" H 4590 4460 50  0001 C CNN
+F 0 "#PWR0606" H 4590 4460 50  0001 C CNN
 F 1 "GND" H 4590 4560 50  0000 C CNN
 F 2 "" H 4590 4710 50  0001 C CNN
 F 3 "" H 4590 4710 50  0001 C CNN
 	1    4590 4710
-	1    0    0    -1
-$EndComp
-$Comp
-L Custom_Library:C_Custom C?
-U 1 1 5EBB0D1E
-P 3910 4740
-AR Path="/5BAAE16C/5EBB0D1E" Ref="C?"  Part="1"
-AR Path="/5BB181D8/5EBB0D1E" Ref="C?"  Part="1"
-AR Path="/5BB2595E/5EBB0D1E" Ref="C?"  Part="1"
-AR Path="/5BAAE0FA/5EBB0D1E" Ref="C?"  Part="1"
-AR Path="/5BB86F23/5EBB0D1E" Ref="C?"  Part="1"
-AR Path="/5C1D5C9E/5EBB0D1E" Ref="C?"  Part="1"
-AR Path="/5CB6F1ED/5EBB0D1E" Ref="C?"  Part="1"
-AR Path="/5E939CFF/5EBB0D1E" Ref="C?"  Part="1"
-AR Path="/5E9E0E87/5EBB0D1E" Ref="C?"  Part="1"
-AR Path="/5EAE2D66/5EBB0D1E" Ref="C?"  Part="1"
-AR Path="/5EAE2E5F/5EBB0D1E" Ref="C602"  Part="1"
-F 0 "C602" H 3935 4840 50  0000 L CNN
-F 1 "0.1uF" H 3935 4640 50  0000 L CNN
-F 2 "Capacitors_SMD:C_0402" H 3948 4590 50  0001 C CNN
-F 3 "" H 3935 4840 50  0001 C CNN
-F 4 "0402" H 3760 4840 50  0000 R CNN "display_footprint"
-F 5 "50V" H 3760 4740 50  0000 R CNN "Voltage"
-F 6 "X7R" H 3760 4640 50  0000 R CNN "Dielectric"
-F 7 "" H 4335 5240 60  0001 C CNN "Digi-Key PN"
-	1    3910 4740
 	1    0    0    -1
 $EndComp
@@
 AR Path="/5CB7718D/5EBE152B" Ref="R?"  Part="1"
 AR Path="/5EAE2D8A/5EBE152B" Ref="R?"  Part="1"
-AR Path="/5EAE2E5F/5EBE152B" Ref="R606"  Part="1"
-F 0 "R606" V 7130 2930 50  0000 C CNN
+AR Path="/5EAE2E5F/5EBE152B" Ref="R605"  Part="1"
+F 0 "R605" V 7130 2930 50  0000 C CNN
 F 1 "10" V 7230 2930 50  0000 C CNN
 F 2 "Resistors_SMD:R_0402" H 7230 2930 50  0001 C CNN
@@
 AR Path="/5CB7718D/5EBE1534" Ref="R?"  Part="1"
 AR Path="/5EAE2D8A/5EBE1534" Ref="R?"  Part="1"
-AR Path="/5EAE2E5F/5EBE1534" Ref="R608"  Part="1"
-F 0 "R608" V 7590 2930 50  0000 C CNN
+AR Path="/5EAE2E5F/5EBE1534" Ref="R610"  Part="1"
+F 0 "R610" V 7590 2930 50  0000 C CNN
 F 1 "10" V 7690 2930 50  0000 C CNN
 F 2 "Resistors_SMD:R_0402" H 7690 2930 50  0001 C CNN
@@
 $EndComp
 $Comp
-L Custom_Library:+1.8V #PWR0613
+L Custom_Library:+1.8V #PWR0612
 U 1 1 5EBF6C95
 P 9050 3190
-F 0 "#PWR0613" H 9050 3040 50  0001 C CNN
+F 0 "#PWR0612" H 9050 3040 50  0001 C CNN
 F 1 "+1.8V" H 9050 3330 50  0000 C CNN
 F 2 "" H 9050 3190 50  0000 C CNN
@@
 $EndComp
 $Comp
-L Custom_Library:+1.8V #PWR0614
+L Custom_Library:+1.8V #PWR0613
 U 1 1 5EBF722E
 P 9560 3190
-F 0 "#PWR0614" H 9560 3040 50  0001 C CNN
+F 0 "#PWR0613" H 9560 3040 50  0001 C CNN
 F 1 "+1.8V" H 9560 3330 50  0000 C CNN
 F 2 "" H 9560 3190 50  0000 C CNN
@@
 Connection ~ 3580 3260
 $Comp
-L Custom_Library:TPS7A7200RGTR U?
+L Custom_Library:TPS7A7200RGTR U601
 U 1 1 5FE64715
 P 4590 3910
-F 0 "U?" H 4340 4710 50  0000 C CNN
+F 0 "U601" H 4340 4710 50  0000 C CNN
 F 1 "TPS7A7200RGTR" H 4740 4710 50  0000 C CNN
 F 2 "Package_DFN_QFN:QFN-16-1EP_3x3mm_P0.5mm_EP1.75x1.75mm" H 4640 4810 50  0001 C CNN
@@
 AR Path="/5E0F263A/5EBE1520" Ref="R?"  Part="1"
 AR Path="/5EAE2D8A/5EBE1520" Ref="R?"  Part="1"
-AR Path="/5EAE2E5F/5EBE1520" Ref="R607"  Part="1"
-F 0 "R607" V 7830 3260 50  0000 C CNN
+AR Path="/5EAE2E5F/5EBE1520" Ref="R606"  Part="1"
+F 0 "R606" V 7830 3260 50  0000 C CNN
 F 1 "0.02" V 7460 3260 40  0000 C CNN
 F 2 "Resistors_SMD:R_0612" H 7460 3260 50  0001 C CNN
@@
 AR Path="/5E9E0E87/5FE7BF72" Ref="R?"  Part="1"
 AR Path="/5EAE2D66/5FE7BF72" Ref="R?"  Part="1"
-AR Path="/5EAE2E5F/5FE7BF72" Ref="R?"  Part="1"
-F 0 "R?" H 6080 3670 50  0000 R CNN
+AR Path="/5EAE2E5F/5FE7BF72" Ref="R603"  Part="1"
+F 0 "R603" H 6080 3670 50  0000 R CNN
 F 1 "100" V 6160 3670 50  0000 C CNN
 F 2 "Resistors_SMD:R_0402" H 6160 3670 50  0001 C CNN
@@
 AR Path="/5E9E0E87/5FE7E11C" Ref="R?"  Part="1"
 AR Path="/5EAE2D66/5FE7E11C" Ref="R?"  Part="1"
-AR Path="/5EAE2E5F/5FE7E11C" Ref="R?"  Part="1"
-F 0 "R?" H 6460 3670 50  0000 R CNN
+AR Path="/5EAE2E5F/5FE7E11C" Ref="R604"  Part="1"
+F 0 "R604" H 6460 3670 50  0000 R CNN
 F 1 "100" V 6540 3670 50  0000 C CNN
 F 2 "Resistors_SMD:R_0402" H 6540 3670 50  0001 C CNN
@@
 $EndComp
 $Comp
-L power:GND #PWR?
+L power:GND #PWR0609
 U 1 1 5FE7E82D
 P 6160 3820
-F 0 "#PWR?" H 6160 3570 50  0001 C CNN
+F 0 "#PWR0609" H 6160 3570 50  0001 C CNN
 F 1 "GND" H 6160 3670 50  0000 C CNN
 F 2 "" H 6160 3820 50  0001 C CNN
@@
 $EndComp
 $Comp
-L power:GND #PWR?
+L power:GND #PWR0610
 U 1 1 5FE7EA6D
 P 6540 3820
-F 0 "#PWR?" H 6540 3570 50  0001 C CNN
+F 0 "#PWR0610" H 6540 3570 50  0001 C CNN
 F 1 "GND" H 6540 3670 50  0000 C CNN
 F 2 "" H 6540 3820 50  0001 C CNN
@@
 NoConn ~ 4990 3910
 $Comp
-L power:GND #PWR?
+L power:GND #PWR0607
 U 1 1 5FE82A1F
 P 5070 4710
-F 0 "#PWR?" H 5070 4460 50  0001 C CNN
+F 0 "#PWR0607" H 5070 4460 50  0001 C CNN
 F 1 "GND" H 5070 4560 50  0000 C CNN
 F 2 "" H 5070 4710 50  0001 C CNN
@@
 AR Path="/5EAE2D8A/5FE71F02" Ref="R?"  Part="1"
 AR Path="/5EAE2D66/5FE71F02" Ref="R?"  Part="1"
-AR Path="/5EAE2E5F/5FE71F02" Ref="R?"  Part="1"
-F 0 "R?" V 7360 3670 50  0000 C CNN
+AR Path="/5EAE2E5F/5FE71F02" Ref="R607"  Part="1"
+F 0 "R607" V 7360 3670 50  0000 C CNN
 F 1 "0" V 7460 3670 50  0000 C CNN
 F 2 "Resistors_SMD:R_0402" H 7460 3670 50  0001 C CNN
@@
 AR Path="/5EAE2D8A/5FE71F0C" Ref="R?"  Part="1"
 AR Path="/5EAE2D66/5FE71F0C" Ref="R?"  Part="1"
-AR Path="/5EAE2E5F/5FE71F0C" Ref="R?"  Part="1"
-F 0 "R?" V 7360 3970 50  0000 C CNN
+AR Path="/5EAE2E5F/5FE71F0C" Ref="R608"  Part="1"
+F 0 "R608" V 7360 3970 50  0000 C CNN
 F 1 "0" V 7460 3970 50  0000 C CNN
 F 2 "Resistors_SMD:R_0402" H 7460 3970 50  0001 C CNN
@@
 AR Path="/5EAE2D8A/5FE71F16" Ref="R?"  Part="1"
 AR Path="/5EAE2D66/5FE71F16" Ref="R?"  Part="1"
-AR Path="/5EAE2E5F/5FE71F16" Ref="R?"  Part="1"
-F 0 "R?" V 7360 4270 50  0000 C CNN
+AR Path="/5EAE2E5F/5FE71F16" Ref="R609"  Part="1"
+F 0 "R609" V 7360 4270 50  0000 C CNN
 F 1 "0" V 7460 4270 50  0000 C CNN
 F 2 "Resistors_SMD:R_0402" H 7460 4270 50  0001 C CNN
@@
 	7690 3260 8400 3260
 Connection ~ 7690 3360
+$Comp
+L Custom_Library:C_Custom C?
+U 1 1 5FEE01A3
+P 3910 4740
+AR Path="/5BAAE16C/5FEE01A3" Ref="C?"  Part="1"
+AR Path="/5BB181D8/5FEE01A3" Ref="C?"  Part="1"
+AR Path="/5BB2595E/5FEE01A3" Ref="C?"  Part="1"
+AR Path="/5BAAE0FA/5FEE01A3" Ref="C?"  Part="1"
+AR Path="/5BB86F23/5FEE01A3" Ref="C?"  Part="1"
+AR Path="/5D77A516/5FEE01A3" Ref="C?"  Part="1"
+AR Path="/5E939CFF/5FEE01A3" Ref="C?"  Part="1"
+AR Path="/5EAE2D66/5FEE01A3" Ref="C?"  Part="1"
+AR Path="/5EAE2E5F/5FEE01A3" Ref="C602"  Part="1"
+F 0 "C602" H 3935 4840 50  0000 L CNN
+F 1 "10nF" H 3935 4640 50  0000 L CNN
+F 2 "Capacitors_SMD:C_0402" H 3948 4590 50  0001 C CNN
+F 3 "" H 3935 4840 50  0001 C CNN
+F 4 "0402" H 3760 4840 50  0000 R CNN "display_footprint"
+F 5 "50V" H 3760 4740 50  0000 R CNN "Voltage"
+F 6 "X7R" H 3760 4640 50  0000 R CNN "Dielectric"
+F 7 "" H 4335 5240 60  0001 C CNN "Digi-Key PN"
+	1    3910 4740
+	1    0    0    -1
+$EndComp
 $EndSCHEMATC

Commit message: USB circuit adjustments, add UART dongle header, resolve some open rev B SCH issues
Parts:
- R607, R608, R609: Configuration !Telemetry -> ~Telemetry
Changed lines of the file:
@@
 Sheet 6 21
 Title "Pulse Oximeter"
-Date "2020-12-09"
+Date "2020-12-31"
 Rev "B"
-Comp "Drew Maatman"
+Comp "Drew Maatman, Nick Mussoline"
 Comment1 ""
 Comment2 ""
@@
 F 5 "1%" V 7660 3670 50  0001 C CNN "Tolerance"
 F 6 "1/16W" V 7760 3670 50  0001 C CNN "Wattage"
-F 7 "!Telemetry" V 7560 3670 50  0000 C CNN "Configuration"
+F 7 "~Telemetry" V 7560 3670 50  0000 C CNN "Configuration"
 	1    7460 3670
 	0    -1   1    0
@@
 F 5 "1%" V 7660 3970 50  0001 C CNN "Tolerance"
 F 6 "1/16W" V 7760 3970 50  0001 C CNN "Wattage"
-F 7 "!Telemetry" V 7560 3970 50  0000 C CNN "Configuration"
+F 7 "~Telemetry" V 7560 3970 50  0000 C CNN "Configuration"
 	1    7460 3970
 	0    -1   1    0
@@
 F 5 "1%" V 7660 4270 50  0001 C CNN "Tolerance"
 F 6 "1/16W" V 7760 4270 50  0001 C CNN "Wattage"
-F 7 "!Telemetry" V 7560 4270 50  0000 C CNN "Configuration"
+F 7 "~Telemetry" V 7560 4270 50  0000 C CNN "Configuration"
 	1    7460 4270
 	0    -1   1    0
