File: hdw/rev_b/Pulse_Oximeter/POS1P8_Power_Supply.sch (KiCad schematic (older format))
At the start: 15 parts, among them U601 TPS7A7200RGTR

Commit message: assigned digikey PNs
Parts:
- C601, C603: Digi-Key PN (none) -> 1276-6830-1-ND; Voltage 6.3V -> 10V
- C602: Digi-Key PN (none) -> 399-3066-1-ND
- R601, R602: Digi-Key PN (none) -> RMCF0402FT10K0CT-ND
- R603, R604: Digi-Key PN (none) -> RMCF0402FT100RCT-ND
- R605, R610: Digi-Key PN (none) -> RMCF0402FT10R0CT-ND
- R607, R608, R609: Digi-Key PN (none) -> 2019-RK73Z1ETTPCT-ND
Changed lines of the file:
@@
 F 5 "1%" H 2360 3490 50  0000 L CNN "Tolerance"
 F 6 "1/16W" H 2370 3410 50  0000 L CNN "Wattage"
-F 7 "" H 2260 3490 50  0001 C CNN "Digi-Key PN"
+F 7 "RMCF0402FT10K0CT-ND" H 2260 3490 50  0001 C CNN "Digi-Key PN"
 	1    2260 3490
 	1    0    0    -1
@@
 F 5 "1%" H 2360 4190 50  0000 L CNN "Tolerance"
 F 6 "1/16W" H 2370 4110 50  0000 L CNN "Wattage"
-F 7 "" H 2260 4190 50  0001 C CNN "Digi-Key PN"
+F 7 "RMCF0402FT10K0CT-ND" H 2260 4190 50  0001 C CNN "Digi-Key PN"
 	1    2260 4190
 	1    0    0    -1
@@
 F 5 "1%" V 7430 2930 50  0001 C CNN "Tolerance"
 F 6 "1/16W" V 7530 2930 50  0001 C CNN "Wattage"
-F 7 "" H 7230 2930 50  0001 C CNN "Digi-Key PN"
+F 7 "RMCF0402FT10R0CT-ND" H 7230 2930 50  0001 C CNN "Digi-Key PN"
 F 8 "Telemetry" V 7050 2930 50  0000 C CNN "Configuration"
 	1    7230 2930
@@
 F 5 "1%" V 7890 2930 50  0001 C CNN "Tolerance"
 F 6 "1/16W" V 7990 2930 50  0001 C CNN "Wattage"
-F 7 "" H 7690 2930 50  0001 C CNN "Digi-Key PN"
+F 7 "RMCF0402FT10R0CT-ND" H 7690 2930 50  0001 C CNN "Digi-Key PN"
 F 8 "Telemetry" V 7510 2930 50  0000 C CNN "Configuration"
 	1    7690 2930
@@
 F 3 "" H 3605 3590 50  0001 C CNN
 F 4 "0402" H 3430 3590 50  0000 R CNN "display_footprint"
-F 5 "6.3V" H 3430 3490 50  0000 R CNN "Voltage"
+F 5 "10V" H 3430 3490 50  0000 R CNN "Voltage"
 F 6 "X5R" H 3430 3390 50  0000 R CNN "Dielectric"
-F 7 "" H 3580 3490 50  0001 C CNN "Digi-Key PN"
+F 7 "1276-6830-1-ND" H 3580 3490 50  0001 C CNN "Digi-Key PN"
 	1    3580 3490
 	1    0    0    -1
@@
 F 3 "" H 5505 3770 50  0001 C CNN
 F 4 "0402" H 5330 3770 50  0000 R CNN "display_footprint"
-F 5 "6.3V" H 5330 3670 50  0000 R CNN "Voltage"
+F 5 "10V" H 5330 3670 50  0000 R CNN "Voltage"
 F 6 "X5R" H 5330 3570 50  0000 R CNN "Dielectric"
-F 7 "" H 5480 3670 50  0001 C CNN "Digi-Key PN"
+F 7 "1276-6830-1-ND" H 5480 3670 50  0001 C CNN "Digi-Key PN"
 	1    5480 3670
 	1    0    0    -1
@@
 F 5 "1%" H 6260 3670 50  0000 L CNN "Tolerance"
 F 6 "1/16W" H 6270 3590 50  0000 L CNN "Wattage"
+F 7 "RMCF0402FT100RCT-ND" H 6160 3670 50  0001 C CNN "Digi-Key PN"
 	1    6160 3670
 	-1   0    0    -1
@@
 F 5 "1%" H 6640 3670 50  0001 L CNN "Tolerance"
 F 6 "1/16W" H 6650 3590 50  0001 L CNN "Wattage"
+F 7 "RMCF0402FT100RCT-ND" H 6540 3670 50  0001 C CNN "Digi-Key PN"
 	1    6540 3670
 	-1   0    0    -1
@@
 F 6 "1/16W" V 7760 3670 50  0001 C CNN "Wattage"
 F 7 "~Telemetry" V 7560 3670 50  0000 C CNN "Configuration"
+F 8 "2019-RK73Z1ETTPCT-ND" H 7460 3670 50  0001 C CNN "Digi-Key PN"
 	1    7460 3670
 	0    -1   1    0
@@
 F 6 "1/16W" V 7760 3970 50  0001 C CNN "Wattage"
 F 7 "~Telemetry" V 7560 3970 50  0000 C CNN "Configuration"
+F 8 "2019-RK73Z1ETTPCT-ND" H 7460 3970 50  0001 C CNN "Digi-Key PN"
 	1    7460 3970
 	0    -1   1    0
@@
 F 6 "1/16W" V 7760 4270 50  0001 C CNN "Wattage"
 F 7 "~Telemetry" V 7560 4270 50  0000 C CNN "Configuration"
+F 8 "2019-RK73Z1ETTPCT-ND" H 7460 4270 50  0001 C CNN "Digi-Key PN"
 	1    7460 4270
 	0    -1   1    0
@@
 F 5 "50V" H 3760 4740 50  0000 R CNN "Voltage"
 F 6 "X7R" H 3760 4640 50  0000 R CNN "Dielectric"
-F 7 "" H 4335 5240 60  0001 C CNN "Digi-Key PN"
+F 7 "399-3066-1-ND" H 4335 5240 60  0001 C CNN "Digi-Key PN"
 	1    3910 4740
 	1    0    0    -1
