File: hdw/rev_b/Pulse_Oximeter/POX_Sensor.sch (KiCad schematic (older format))
At the start: 25 parts, among them U1501 TPS22929D, U1502 TCA9803, U1503 MAX30102

Commit message: changed POX filtering and level shifting
Parts:
- removed C1509, C1512: 10nF, Capacitors_SMD:C_0402, symbol Custom_Library:C_Custom
- removed C1510, C1513: 1nF, Capacitors_SMD:C_0402, symbol Custom_Library:C_Custom
- removed C1511: 0.1uF, Capacitors_SMD:C_0402, symbol Custom_Library:C_Custom
- removed R1505, R1506: 10k, Resistors_SMD:R_0402, symbol Custom_Library:R_Custom
- added C?: 0.1uF, Capacitors_SMD:C_0402, symbol Custom_Library:C_Custom
- added C? (x2): 10uF, Capacitors_SMD:C_0402, symbol Custom_Library:C_Custom
- added L? (x2): 600R 0.5A, Inductors_SMD:L_0402, symbol Device:Ferrite_Bead
- added R? (x2): 0, Resistors_SMD:R_0402, symbol Custom_Library:R_Custom
- U1502: Configuration (none) -> POX_LV_SHIFT
Connections:
- net +1.8V: now also L?.2; no longer C1507.1, C1508.1, U1503.11 (VDD)
- net +3.3V_POX: now also L?.2; no longer C1514.1, U1503.10 (VLED+), U1503.9 (VLED+)
- net GND: now also C?.2, C?.2, C?.2
- net I2C_SCL: now also R?.1
- net I2C_SDA: now also R?.1
- net at U1502.7 (SCLB), U1503.2 (SCL): now also R?.2
- net at U1502.6 (SDAB), U1503.3 (SDA): now also R?.2
- new net: C1514.1, C?.1, C?.1, L?.1, U1503.10 (VLED+), U1503.9 (VLED+)
- new net: C1507.1, C1508.1, C?.1, L?.1, U1503.11 (VDD)
Other:
- moved on the sheet: C1502, C1503, C1504, C1505, C1507, C1508, C1514, R1502, U1502

Commit message: merged, more cleanups
Parts:
- C1506: value 10nF -> 0.1uF; Digi-Key PN 490-13295-1-ND -> 490-10701-1-ND
Changed lines of the file:
@@
 	4490 6440 4490 6360
-$Comp
-L Custom_Library:C_Custom C?
-U 1 1 5EC2763B
-P 5190 6590
-AR Path="/5BAAE16C/5EC2763B" Ref="C?"  Part="1"
-AR Path="/5BB181D8/5EC2763B" Ref="C?"  Part="1"
-AR Path="/5BB2595E/5EC2763B" Ref="C?"  Part="1"
-AR Path="/5BAAE0FA/5EC2763B" Ref="C?"  Part="1"
-AR Path="/5BB86F23/5EC2763B" Ref="C?"  Part="1"
-AR Path="/5C1D5C9E/5EC2763B" Ref="C?"  Part="1"
-AR Path="/5CB6F1ED/5EC2763B" Ref="C?"  Part="1"
-AR Path="/5E939CFF/5EC2763B" Ref="C?"  Part="1"
-AR Path="/5E9E0E87/5EC2763B" Ref="C?"  Part="1"
-AR Path="/5EAE2D66/5EC2763B" Ref="C?"  Part="1"
-AR Path="/5EAE30C7/5EC2763B" Ref="C1506"  Part="1"
-F 0 "C1506" H 5215 6690 50  0000 L CNN
-F 1 "10nF" H 5215 6490 50  0000 L CNN
-F 2 "Capacitors_SMD:C_0402" H 5228 6440 50  0001 C CNN
-F 3 "" H 5215 6690 50  0001 C CNN
-F 4 "0402" H 5040 6690 50  0000 R CNN "display_footprint"
-F 5 "50V" H 5040 6590 50  0000 R CNN "Voltage"
-F 6 "X7R" H 5040 6490 50  0000 R CNN "Dielectric"
-F 7 "490-13295-1-ND" H 5615 7090 60  0001 C CNN "Digi-Key PN"
-	1    5190 6590
-	-1   0    0    -1
-$EndComp
 $Comp
 L power:GND #PWR01521
@@
 Wire Wire Line
 	4480 4040 6430 4040
+$Comp
+L Custom_Library:C_Custom C?
+U 1 1 5FE1722F
+P 5190 6590
+AR Path="/5BAAE16C/5FE1722F" Ref="C?"  Part="1"
+AR Path="/5BB181D8/5FE1722F" Ref="C?"  Part="1"
+AR Path="/5BB2595E/5FE1722F" Ref="C?"  Part="1"
+AR Path="/5BAAE0FA/5FE1722F" Ref="C?"  Part="1"
+AR Path="/5BB86F23/5FE1722F" Ref="C?"  Part="1"
+AR Path="/5C1D5C9E/5FE1722F" Ref="C?"  Part="1"
+AR Path="/5CB6F1ED/5FE1722F" Ref="C?"  Part="1"
+AR Path="/5E939CFF/5FE1722F" Ref="C?"  Part="1"
+AR Path="/5E9E0E87/5FE1722F" Ref="C?"  Part="1"
+AR Path="/5EAE2D66/5FE1722F" Ref="C?"  Part="1"
+AR Path="/5EAE30C7/5FE1722F" Ref="C1506"  Part="1"
+F 0 "C1506" H 5215 6690 50  0000 L CNN
+F 1 "0.1uF" H 5215 6490 50  0000 L CNN
+F 2 "Capacitors_SMD:C_0402" H 5228 6440 50  0001 C CNN
+F 3 "" H 5215 6690 50  0001 C CNN
+F 4 "0402" H 5040 6690 50  0000 R CNN "display_footprint"
+F 5 "50V" H 5040 6590 50  0000 R CNN "Voltage"
+F 6 "X7R" H 5040 6490 50  0000 R CNN "Dielectric"
+F 7 "490-10701-1-ND" H 5615 7090 60  0001 C CNN "Digi-Key PN"
+	1    5190 6590
+	1    0    0    -1
+$EndComp
 $EndSCHEMATC

Commit message: changed all passives to 0402, cleared digikey pns
Parts:
- C1501, C1503, C1505, C1507, C1514, C? (x2): Digi-Key PN 490-13211-1-ND -> (none)
- C1502, C1504, C1506, C1508, C?: Digi-Key PN 490-10701-1-ND -> (none)
- R1501, R1502, R1503, R1504, R1507: Digi-Key PN RMCF0402FT10K0CT-ND -> (none)
Changed lines of the file:
@@
 F 5 "1%" H 8050 3810 50  0000 L CNN "Tolerance"
 F 6 "1/16W" H 8060 3730 50  0000 L CNN "Wattage"
-F 7 "RMCF0402FT10K0CT-ND" H 7950 3810 50  0001 C CNN "Digi-Key PN"
+F 7 "" H 7950 3810 50  0001 C CNN "Digi-Key PN"
 	1    7950 3810
 	1    0    0    -1
@@
 F 5 "50V" H 6240 2670 50  0000 R CNN "Voltage"
 F 6 "X7R" H 6240 2570 50  0000 R CNN "Dielectric"
-F 7 "490-10701-1-ND" H 6815 3170 60  0001 C CNN "Digi-Key PN"
+F 7 "" H 6815 3170 60  0001 C CNN "Digi-Key PN"
 	1    6390 2670
 	1    0    0    -1
@@
 F 5 "6.3V" H 4930 2670 50  0000 R CNN "Voltage"
 F 6 "X5R" H 4930 2570 50  0000 R CNN "Dielectric"
-F 7 "490-13211-1-ND" H 5080 2670 50  0001 C CNN "Digi-Key PN"
+F 7 "" H 5080 2670 50  0001 C CNN "Digi-Key PN"
 	1    5080 2670
 	1    0    0    -1
@@
 F 5 "6.3V" H 4930 1770 50  0000 R CNN "Voltage"
 F 6 "X5R" H 4930 1670 50  0000 R CNN "Dielectric"
-F 7 "490-13211-1-ND" H 5080 1770 50  0001 C CNN "Digi-Key PN"
+F 7 "" H 5080 1770 50  0001 C CNN "Digi-Key PN"
 	1    5080 1770
 	1    0    0    -1
@@
 F 5 "1%" H 2710 6410 50  0000 L CNN "Tolerance"
 F 6 "1/16W" H 2720 6330 50  0000 L CNN "Wattage"
-F 7 "RMCF0402FT10K0CT-ND" H 2610 6410 50  0001 C CNN "Digi-Key PN"
+F 7 "" H 2610 6410 50  0001 C CNN "Digi-Key PN"
 	1    2610 6410
 	1    0    0    -1
@@
 F 5 "6.3V" H 1260 6110 50  0000 R CNN "Voltage"
 F 6 "X5R" H 1260 6010 50  0000 R CNN "Dielectric"
-F 7 "490-13211-1-ND" H 1410 6110 50  0001 C CNN "Digi-Key PN"
+F 7 "" H 1410 6110 50  0001 C CNN "Digi-Key PN"
 	1    1410 6110
 	1    0    0    -1
@@
 F 5 "1%" H 2880 4370 50  0000 L CNN "Tolerance"
 F 6 "1/16W" H 2890 4290 50  0000 L CNN "Wattage"
-F 7 "RMCF0402FT10K0CT-ND" H 2780 4370 50  0001 C CNN "Digi-Key PN"
+F 7 "" H 2780 4370 50  0001 C CNN "Digi-Key PN"
 	1    2780 4370
 	1    0    0    -1
@@
 F 5 "6.3V" H 2830 2420 50  0000 R CNN "Voltage"
 F 6 "X5R" H 2830 2320 50  0000 R CNN "Dielectric"
-F 7 "490-13211-1-ND" H 2980 2420 50  0001 C CNN "Digi-Key PN"
+F 7 "" H 2980 2420 50  0001 C CNN "Digi-Key PN"
 	1    2980 2420
 	1    0    0    -1
@@
 F 5 "50V" H 2230 2420 50  0000 R CNN "Voltage"
 F 6 "X7R" H 2230 2320 50  0000 R CNN "Dielectric"
-F 7 "490-10701-1-ND" H 2805 2920 60  0001 C CNN "Digi-Key PN"
+F 7 "" H 2805 2920 60  0001 C CNN "Digi-Key PN"
 	1    2380 2420
 	1    0    0    -1
@@
 F 5 "6.3V" H 1460 2420 50  0000 R CNN "Voltage"
 F 6 "X5R" H 1460 2320 50  0000 R CNN "Dielectric"
-F 7 "490-13211-1-ND" H 1610 2420 50  0001 C CNN "Digi-Key PN"
+F 7 "" H 1610 2420 50  0001 C CNN "Digi-Key PN"
 	1    1610 2420
 	1    0    0    -1
@@
 F 5 "50V" H 860 2420 50  0000 R CNN "Voltage"
 F 6 "X7R" H 860 2320 50  0000 R CNN "Dielectric"
-F 7 "490-10701-1-ND" H 1435 2920 60  0001 C CNN "Digi-Key PN"
+F 7 "" H 1435 2920 60  0001 C CNN "Digi-Key PN"
 	1    1010 2420
 	1    0    0    -1
@@
 F 5 "1%" H 4590 6130 50  0000 L CNN "Tolerance"
 F 6 "1/16W" H 4600 6050 50  0000 L CNN "Wattage"
-F 7 "RMCF0402FT10K0CT-ND" H 4490 6130 50  0001 C CNN "Digi-Key PN"
+F 7 "" H 4490 6130 50  0001 C CNN "Digi-Key PN"
 	1    4490 6130
 	1    0    0    -1
@@
 F 5 "1%" H 4590 6590 50  0000 L CNN "Tolerance"
 F 6 "1/16W" H 4600 6510 50  0000 L CNN "Wattage"
-F 7 "RMCF0402FT10K0CT-ND" H 4490 6590 50  0001 C CNN "Digi-Key PN"
+F 7 "" H 4490 6590 50  0001 C CNN "Digi-Key PN"
 	1    4490 6590
 	1    0    0    -1
@@
 F 5 "50V" H 6240 1770 50  0000 R CNN "Voltage"
 F 6 "X7R" H 6240 1670 50  0000 R CNN "Dielectric"
-F 7 "490-10701-1-ND" H 6815 2270 60  0001 C CNN "Digi-Key PN"
+F 7 "" H 6815 2270 60  0001 C CNN "Digi-Key PN"
 	1    6390 1770
 	1    0    0    -1
@@
 F 5 "6.3V" H 5640 1770 50  0000 R CNN "Voltage"
 F 6 "X5R" H 5640 1670 50  0000 R CNN "Dielectric"
-F 7 "490-13211-1-ND" H 5790 1770 50  0001 C CNN "Digi-Key PN"
+F 7 "" H 5790 1770 50  0001 C CNN "Digi-Key PN"
 	1    5790 1770
 	1    0    0    -1
@@
 F 5 "6.3V" H 5640 2670 50  0000 R CNN "Voltage"
 F 6 "X5R" H 5640 2570 50  0000 R CNN "Dielectric"
-F 7 "490-13211-1-ND" H 5790 2670 50  0001 C CNN "Digi-Key PN"
+F 7 "" H 5790 2670 50  0001 C CNN "Digi-Key PN"
 	1    5790 2670
 	1    0    0    -1
@@
 F 5 "50V" H 5040 6590 50  0000 R CNN "Voltage"
 F 6 "X7R" H 5040 6490 50  0000 R CNN "Dielectric"
-F 7 "490-10701-1-ND" H 5615 7090 60  0001 C CNN "Digi-Key PN"
+F 7 "" H 5615 7090 60  0001 C CNN "Digi-Key PN"
 	1    5190 6590
 	1    0    0    -1

Commit message: annotated schematic
Parts:
- U1502: Configuration POX_LV_SHIFT -> DNP
- gave numbers to parts that had none: 7
- renumbered C1502 to C1501, C1501 to C1502, C1514 to C1506, C1506 to C1508, C1508 to C1512, R1503 to R1505, R1504 to R1506

Commit message: passed ERC
Other:
- moved on the sheet: C1503, C1504, C1505
Changed lines of the file:
@@
 L Custom_Library:C_Custom C?
 U 1 1 5EBE16BC
-P 2980 2420
+P 3200 2420
 AR Path="/5CB7718D/5EBE16BC" Ref="C?"  Part="1"
 AR Path="/5E0DC082/5EBE16BC" Ref="C?"  Part="1"
@@
 AR Path="/5EAE3021/5EBE16BC" Ref="C?"  Part="1"
 AR Path="/5EAE30C7/5EBE16BC" Ref="C1505"  Part="1"
-F 0 "C1505" H 3005 2520 50  0000 L CNN
-F 1 "10uF" H 3005 2320 50  0000 L CNN
-F 2 "Capacitors_SMD:C_0402" H 3018 2270 50  0001 C CNN
-F 3 "" H 3005 2520 50  0001 C CNN
-F 4 "0402" H 2830 2520 50  0000 R CNN "display_footprint"
-F 5 "6.3V" H 2830 2420 50  0000 R CNN "Voltage"
-F 6 "X5R" H 2830 2320 50  0000 R CNN "Dielectric"
-F 7 "" H 2980 2420 50  0001 C CNN "Digi-Key PN"
-	1    2980 2420
+F 0 "C1505" H 3225 2520 50  0000 L CNN
+F 1 "10uF" H 3225 2320 50  0000 L CNN
+F 2 "Capacitors_SMD:C_0402" H 3238 2270 50  0001 C CNN
+F 3 "" H 3225 2520 50  0001 C CNN
+F 4 "0402" H 3050 2520 50  0000 R CNN "display_footprint"
+F 5 "6.3V" H 3050 2420 50  0000 R CNN "Voltage"
+F 6 "X5R" H 3050 2320 50  0000 R CNN "Dielectric"
+F 7 "" H 3200 2420 50  0001 C CNN "Digi-Key PN"
+	1    3200 2420
 	1    0    0    -1
 $EndComp
@@
 L power:GND #PWR01512
 U 1 1 5EBE16C2
-P 2980 2570
-F 0 "#PWR01512" H 2980 2320 50  0001 C CNN
-F 1 "GND" H 2980 2420 50  0000 C CNN
-F 2 "" H 2980 2570 50  0001 C CNN
-F 3 "" H 2980 2570 50  0001 C CNN
-	1    2980 2570
+P 3200 2570
+F 0 "#PWR01512" H 3200 2320 50  0001 C CNN
+F 1 "GND" H 3200 2420 50  0000 C CNN
+F 2 "" H 3200 2570 50  0001 C CNN
+F 3 "" H 3200 2570 50  0001 C CNN
+	1    3200 2570
 	1    0    0    -1
 $EndComp
@@
 L Custom_Library:+1.8V #PWR01511
 U 1 1 5EBE16C8
-P 2980 2270
-F 0 "#PWR01511" H 2980 2120 50  0001 C CNN
-F 1 "+1.8V" H 2980 2410 50  0000 C CNN
-F 2 "" H 2980 2270 50  0000 C CNN
-F 3 "" H 2980 2270 50  0000 C CNN
-	1    2980 2270
+P 3200 2270
+F 0 "#PWR01511" H 3200 2120 50  0001 C CNN
+F 1 "+1.8V" H 3200 2410 50  0000 C CNN
+F 2 "" H 3200 2270 50  0000 C CNN
+F 3 "" H 3200 2270 50  0000 C CNN
+	1    3200 2270
 	1    0    0    -1
 $EndComp
@@
 L Custom_Library:C_Custom C?
 U 1 1 5EBE24C0
-P 2380 2420
+P 2460 2420
 AR Path="/5BAAE16C/5EBE24C0" Ref="C?"  Part="1"
 AR Path="/5BB181D8/5EBE24C0" Ref="C?"  Part="1"
@@
 AR Path="/5EAE2D66/5EBE24C0" Ref="C?"  Part="1"
 AR Path="/5EAE30C7/5EBE24C0" Ref="C1504"  Part="1"
-F 0 "C1504" H 2405 2520 50  0000 L CNN
-F 1 "0.1uF" H 2405 2320 50  0000 L CNN
-F 2 "Capacitors_SMD:C_0402" H 2418 2270 50  0001 C CNN
-F 3 "" H 2405 2520 50  0001 C CNN
-F 4 "0402" H 2230 2520 50  0000 R CNN "display_footprint"
-F 5 "50V" H 2230 2420 50  0000 R CNN "Voltage"
-F 6 "X7R" H 2230 2320 50  0000 R CNN "Dielectric"
-F 7 "" H 2805 2920 60  0001 C CNN "Digi-Key PN"
-	1    2380 2420
+F 0 "C1504" H 2485 2520 50  0000 L CNN
+F 1 "0.1uF" H 2485 2320 50  0000 L CNN
+F 2 "Capacitors_SMD:C_0402" H 2498 2270 50  0001 C CNN
+F 3 "" H 2485 2520 50  0001 C CNN
+F 4 "0402" H 2310 2520 50  0000 R CNN "display_footprint"
+F 5 "50V" H 2310 2420 50  0000 R CNN "Voltage"
+F 6 "X7R" H 2310 2320 50  0000 R CNN "Dielectric"
+F 7 "" H 2885 2920 60  0001 C CNN "Digi-Key PN"
+	1    2460 2420
 	1    0    0    -1
 $EndComp
@@
 L power:GND #PWR01508
 U 1 1 5EBE367E
-P 2380 2570
-F 0 "#PWR01508" H 2380 2320 50  0001 C CNN
-F 1 "GND" H 2380 2420 50  0000 C CNN
-F 2 "" H 2380 2570 50  0001 C CNN
-F 3 "" H 2380 2570 50  0001 C CNN
-	1    2380 2570
+P 2460 2570
+F 0 "#PWR01508" H 2460 2320 50  0001 C CNN
+F 1 "GND" H 2460 2420 50  0000 C CNN
+F 2 "" H 2460 2570 50  0001 C CNN
+F 3 "" H 2460 2570 50  0001 C CNN
+	1    2460 2570
 	1    0    0    -1
 $EndComp
@@
 L Custom_Library:+1.8V #PWR01507
 U 1 1 5EBE3A80
-P 2380 2270
-F 0 "#PWR01507" H 2380 2120 50  0001 C CNN
-F 1 "+1.8V" H 2380 2410 50  0000 C CNN
-F 2 "" H 2380 2270 50  0000 C CNN
-F 3 "" H 2380 2270 50  0000 C CNN
-	1    2380 2270
+P 2460 2270
+F 0 "#PWR01507" H 2460 2120 50  0001 C CNN
+F 1 "+1.8V" H 2460 2410 50  0000 C CNN
+F 2 "" H 2460 2270 50  0000 C CNN
+F 3 "" H 2460 2270 50  0000 C CNN
+	1    2460 2270
 	1    0    0    -1
 $EndComp
@@
 L Custom_Library:C_Custom C?
 U 1 1 5EBE4148
-P 1610 2420
+P 1690 2420
 AR Path="/5CB7718D/5EBE4148" Ref="C?"  Part="1"
 AR Path="/5E0DC082/5EBE4148" Ref="C?"  Part="1"
@@
 AR Path="/5EAE3021/5EBE4148" Ref="C?"  Part="1"
 AR Path="/5EAE30C7/5EBE4148" Ref="C1503"  Part="1"
-F 0 "C1503" H 1635 2520 50  0000 L CNN
-F 1 "10uF" H 1635 2320 50  0000 L CNN
-F 2 "Capacitors_SMD:C_0402" H 1648 2270 50  0001 C CNN
-F 3 "" H 1635 2520 50  0001 C CNN
-F 4 "0402" H 1460 2520 50  0000 R CNN "display_footprint"
-F 5 "6.3V" H 1460 2420 50  0000 R CNN "Voltage"
-F 6 "X5R" H 1460 2320 50  0000 R CNN "Dielectric"
-F 7 "" H 1610 2420 50  0001 C CNN "Digi-Key PN"
-	1    1610 2420
+F 0 "C1503" H 1715 2520 50  0000 L CNN
+F 1 "10uF" H 1715 2320 50  0000 L CNN
+F 2 "Capacitors_SMD:C_0402" H 1728 2270 50  0001 C CNN
+F 3 "" H 1715 2520 50  0001 C CNN
+F 4 "0402" H 1540 2520 50  0000 R CNN "display_footprint"
+F 5 "6.3V" H 1540 2420 50  0000 R CNN "Voltage"
+F 6 "X5R" H 1540 2320 50  0000 R CNN "Dielectric"
+F 7 "" H 1690 2420 50  0001 C CNN "Digi-Key PN"
+	1    1690 2420
 	1    0    0    -1
 $EndComp
@@
 L power:GND #PWR01506
 U 1 1 5EBE4152
-P 1610 2570
-F 0 "#PWR01506" H 1610 2320 50  0001 C CNN
-F 1 "GND" H 1610 2420 50  0000 C CNN
-F 2 "" H 1610 2570 50  0001 C CNN
-F 3 "" H 1610 2570 50  0001 C CNN
-	1    1610 2570
+P 1690 2570
+F 0 "#PWR01506" H 1690 2320 50  0001 C CNN
+F 1 "GND" H 1690 2420 50  0000 C CNN
+F 2 "" H 1690 2570 50  0001 C CNN
+F 3 "" H 1690 2570 50  0001 C CNN
+	1    1690 2570
 	1    0    0    -1
 $EndComp
@@
 L power:+3.3V #PWR01505
 U 1 1 5EBEBB9E
-P 1610 2270
-F 0 "#PWR01505" H 1610 2120 50  0001 C CNN
-F 1 "+3.3V" H 1610 2410 50  0000 C CNN
-F 2 "" H 1610 2270 50  0001 C CNN
-F 3 "" H 1610 2270 50  0001 C CNN
-	1    1610 2270
+P 1690 2270
+F 0 "#PWR01505" H 1690 2120 50  0001 C CNN
+F 1 "+3.3V" H 1690 2410 50  0000 C CNN
+F 2 "" H 1690 2270 50  0001 C CNN
+F 3 "" H 1690 2270 50  0001 C CNN
+	1    1690 2270
 	1    0    0    -1
 $EndComp
@@
 	1    0    0    -1
 $EndComp
+$Comp
+L power:PWR_FLAG #FLG0101
+U 1 1 5FEFC9CB
+P 5080 2360
+F 0 "#FLG0101" H 5080 2435 50  0001 C CNN
+F 1 "PWR_FLAG" H 5080 2510 50  0000 C CNN
+F 2 "" H 5080 2360 50  0001 C CNN
+F 3 "~" H 5080 2360 50  0001 C CNN
+	1    5080 2360
+	1    0    0    -1
+$EndComp
+Wire Wire Line
+	5080 2360 5080 2440
+$Comp
+L power:PWR_FLAG #FLG0102
+U 1 1 5FEFE52E
+P 5080 1460
+F 0 "#FLG0102" H 5080 1535 50  0001 C CNN
+F 1 "PWR_FLAG" H 5080 1610 50  0000 C CNN
+F 2 "" H 5080 1460 50  0001 C CNN
+F 3 "~" H 5080 1460 50  0001 C CNN
+	1    5080 1460
+	1    0    0    -1
+$EndComp
+Wire Wire Line
+	5080 1460 5080 1540
 $EndSCHEMATC
