File: hdw/rev_b/Pulse_Oximeter/POX_Sensor.sch (KiCad schematic (older format))
At the start: 25 parts, among them U1501 TPS22929D, U1502 TCA9803, U1503 MAX30102

Commit message: assigned digikey PNs
Parts:
- C1501, C1504, C1508, C1511, C1512: Digi-Key PN (none) -> 490-10698-1-ND; Voltage 50V -> 25V
- C1502, C1503, C1505, C1506, C1507, C1509, C1510: Digi-Key PN (none) -> 1276-6830-1-ND; Voltage 6.3V -> 10V
- R1501, R1502, R1505, R1506, R1507: Digi-Key PN (none) -> RMCF0402FT10K0CT-ND
- R1503, R1504: Digi-Key PN (none) -> 2019-RK73Z1ETTPCT-ND
Changed lines of the file:
@@
 F 5 "1%" H 8050 3810 50  0000 L CNN "Tolerance"
 F 6 "1/16W" H 8060 3730 50  0000 L CNN "Wattage"
-F 7 "" H 7950 3810 50  0001 C CNN "Digi-Key PN"
+F 7 "RMCF0402FT10K0CT-ND" H 7950 3810 50  0001 C CNN "Digi-Key PN"
 	1    7950 3810
 	1    0    0    -1
@@
 F 3 "" H 6415 2770 50  0001 C CNN
 F 4 "0402" H 6240 2770 50  0000 R CNN "display_footprint"
-F 5 "50V" H 6240 2670 50  0000 R CNN "Voltage"
+F 5 "25V" H 6240 2670 50  0000 R CNN "Voltage"
 F 6 "X7R" H 6240 2570 50  0000 R CNN "Dielectric"
-F 7 "" H 6815 3170 60  0001 C CNN "Digi-Key PN"
+F 7 "490-10698-1-ND" H 6815 3170 60  0001 C CNN "Digi-Key PN"
 	1    6390 2670
 	1    0    0    -1
@@
 F 3 "" H 5105 2770 50  0001 C CNN
 F 4 "0402" H 4930 2770 50  0000 R CNN "display_footprint"
-F 5 "6.3V" H 4930 2670 50  0000 R CNN "Voltage"
+F 5 "10V" H 4930 2670 50  0000 R CNN "Voltage"
 F 6 "X5R" H 4930 2570 50  0000 R CNN "Dielectric"
-F 7 "" H 5080 2670 50  0001 C CNN "Digi-Key PN"
+F 7 "1276-6830-1-ND" H 5080 2670 50  0001 C CNN "Digi-Key PN"
 	1    5080 2670
 	1    0    0    -1
@@
 F 3 "" H 5105 1870 50  0001 C CNN
 F 4 "0402" H 4930 1870 50  0000 R CNN "display_footprint"
-F 5 "6.3V" H 4930 1770 50  0000 R CNN "Voltage"
+F 5 "10V" H 4930 1770 50  0000 R CNN "Voltage"
 F 6 "X5R" H 4930 1670 50  0000 R CNN "Dielectric"
-F 7 "" H 5080 1770 50  0001 C CNN "Digi-Key PN"
+F 7 "1276-6830-1-ND" H 5080 1770 50  0001 C CNN "Digi-Key PN"
 	1    5080 1770
 	1    0    0    -1
@@
 F 5 "1%" H 2710 6410 50  0000 L CNN "Tolerance"
 F 6 "1/16W" H 2720 6330 50  0000 L CNN "Wattage"
-F 7 "" H 2610 6410 50  0001 C CNN "Digi-Key PN"
+F 7 "RMCF0402FT10K0CT-ND" H 2610 6410 50  0001 C CNN "Digi-Key PN"
 	1    2610 6410
 	1    0    0    -1
@@
 F 3 "" H 1435 6210 50  0001 C CNN
 F 4 "0402" H 1260 6210 50  0000 R CNN "display_footprint"
-F 5 "6.3V" H 1260 6110 50  0000 R CNN "Voltage"
+F 5 "10V" H 1260 6110 50  0000 R CNN "Voltage"
 F 6 "X5R" H 1260 6010 50  0000 R CNN "Dielectric"
-F 7 "" H 1410 6110 50  0001 C CNN "Digi-Key PN"
+F 7 "1276-6830-1-ND" H 1410 6110 50  0001 C CNN "Digi-Key PN"
 	1    1410 6110
 	1    0    0    -1
@@
 F 5 "1%" H 2880 4370 50  0000 L CNN "Tolerance"
 F 6 "1/16W" H 2890 4290 50  0000 L CNN "Wattage"
-F 7 "" H 2780 4370 50  0001 C CNN "Digi-Key PN"
+F 7 "RMCF0402FT10K0CT-ND" H 2780 4370 50  0001 C CNN "Digi-Key PN"
 	1    2780 4370
 	1    0    0    -1
@@
 F 3 "" H 3225 2520 50  0001 C CNN
 F 4 "0402" H 3050 2520 50  0000 R CNN "display_footprint"
-F 5 "6.3V" H 3050 2420 50  0000 R CNN "Voltage"
+F 5 "10V" H 3050 2420 50  0000 R CNN "Voltage"
 F 6 "X5R" H 3050 2320 50  0000 R CNN "Dielectric"
-F 7 "" H 3200 2420 50  0001 C CNN "Digi-Key PN"
+F 7 "1276-6830-1-ND" H 3200 2420 50  0001 C CNN "Digi-Key PN"
 	1    3200 2420
 	1    0    0    -1
@@
 F 3 "" H 2485 2520 50  0001 C CNN
 F 4 "0402" H 2310 2520 50  0000 R CNN "display_footprint"
-F 5 "50V" H 2310 2420 50  0000 R CNN "Voltage"
+F 5 "25V" H 2310 2420 50  0000 R CNN "Voltage"
 F 6 "X7R" H 2310 2320 50  0000 R CNN "Dielectric"
-F 7 "" H 2885 2920 60  0001 C CNN "Digi-Key PN"
+F 7 "490-10698-1-ND" H 2885 2920 60  0001 C CNN "Digi-Key PN"
 	1    2460 2420
 	1    0    0    -1
@@
 F 3 "" H 1715 2520 50  0001 C CNN
 F 4 "0402" H 1540 2520 50  0000 R CNN "display_footprint"
-F 5 "6.3V" H 1540 2420 50  0000 R CNN "Voltage"
+F 5 "10V" H 1540 2420 50  0000 R CNN "Voltage"
 F 6 "X5R" H 1540 2320 50  0000 R CNN "Dielectric"
-F 7 "" H 1690 2420 50  0001 C CNN "Digi-Key PN"
+F 7 "1276-6830-1-ND" H 1690 2420 50  0001 C CNN "Digi-Key PN"
 	1    1690 2420
 	1    0    0    -1
@@
 F 3 "" H 1035 2520 50  0001 C CNN
 F 4 "0402" H 860 2520 50  0000 R CNN "display_footprint"
-F 5 "50V" H 860 2420 50  0000 R CNN "Voltage"
+F 5 "25V" H 860 2420 50  0000 R CNN "Voltage"
 F 6 "X7R" H 860 2320 50  0000 R CNN "Dielectric"
-F 7 "" H 1435 2920 60  0001 C CNN "Digi-Key PN"
+F 7 "490-10698-1-ND" H 1435 2920 60  0001 C CNN "Digi-Key PN"
 	1    1010 2420
 	1    0    0    -1
@@
 F 5 "1%" H 4590 6130 50  0000 L CNN "Tolerance"
 F 6 "1/16W" H 4600 6050 50  0000 L CNN "Wattage"
-F 7 "" H 4490 6130 50  0001 C CNN "Digi-Key PN"
+F 7 "RMCF0402FT10K0CT-ND" H 4490 6130 50  0001 C CNN "Digi-Key PN"
 	1    4490 6130
 	1    0    0    -1
@@
 F 5 "1%" H 4590 6590 50  0000 L CNN "Tolerance"
 F 6 "1/16W" H 4600 6510 50  0000 L CNN "Wattage"
-F 7 "" H 4490 6590 50  0001 C CNN "Digi-Key PN"
+F 7 "RMCF0402FT10K0CT-ND" H 4490 6590 50  0001 C CNN "Digi-Key PN"
 	1    4490 6590
 	1    0    0    -1
@@
 F 3 "" H 6415 1870 50  0001 C CNN
 F 4 "0402" H 6240 1870 50  0000 R CNN "display_footprint"
-F 5 "50V" H 6240 1770 50  0000 R CNN "Voltage"
+F 5 "25V" H 6240 1770 50  0000 R CNN "Voltage"
 F 6 "X7R" H 6240 1670 50  0000 R CNN "Dielectric"
-F 7 "" H 6815 2270 60  0001 C CNN "Digi-Key PN"
+F 7 "490-10698-1-ND" H 6815 2270 60  0001 C CNN "Digi-Key PN"
 	1    6390 1770
 	1    0    0    -1
@@
 F 3 "" H 5815 1870 50  0001 C CNN
 F 4 "0402" H 5640 1870 50  0000 R CNN "display_footprint"
-F 5 "6.3V" H 5640 1770 50  0000 R CNN "Voltage"
+F 5 "10V" H 5640 1770 50  0000 R CNN "Voltage"
 F 6 "X5R" H 5640 1670 50  0000 R CNN "Dielectric"
-F 7 "" H 5790 1770 50  0001 C CNN "Digi-Key PN"
+F 7 "1276-6830-1-ND" H 5790 1770 50  0001 C CNN "Digi-Key PN"
 	1    5790 1770
 	1    0    0    -1
@@
 F 3 "" H 5815 2770 50  0001 C CNN
 F 4 "0402" H 5640 2770 50  0000 R CNN "display_footprint"
-F 5 "6.3V" H 5640 2670 50  0000 R CNN "Voltage"
+F 5 "10V" H 5640 2670 50  0000 R CNN "Voltage"
 F 6 "X5R" H 5640 2570 50  0000 R CNN "Dielectric"
-F 7 "" H 5790 2670 50  0001 C CNN "Digi-Key PN"
+F 7 "1276-6830-1-ND" H 5790 2670 50  0001 C CNN "Digi-Key PN"
 	1    5790 2670
 	1    0    0    -1
@@
 F 5 "1%" V 3360 5010 50  0001 C CNN "Tolerance"
 F 6 "1/16W" V 3460 5010 50  0001 C CNN "Wattage"
+F 7 "2019-RK73Z1ETTPCT-ND" H 3160 5010 50  0001 C CNN "Digi-Key PN"
 	1    3160 5010
 	0    -1   -1   0
@@
 F 5 "1%" V 3360 3110 50  0001 C CNN "Tolerance"
 F 6 "1/16W" V 3460 3110 50  0001 C CNN "Wattage"
+F 7 "2019-RK73Z1ETTPCT-ND" H 3160 3110 50  0001 C CNN "Digi-Key PN"
 	1    3160 3110
 	0    -1   -1   0
@@
 F 3 "" H 5215 6690 50  0001 C CNN
 F 4 "0402" H 5040 6690 50  0000 R CNN "display_footprint"
-F 5 "50V" H 5040 6590 50  0000 R CNN "Voltage"
+F 5 "25V" H 5040 6590 50  0000 R CNN "Voltage"
 F 6 "X7R" H 5040 6490 50  0000 R CNN "Dielectric"
-F 7 "" H 5615 7090 60  0001 C CNN "Digi-Key PN"
+F 7 "490-10698-1-ND" H 5615 7090 60  0001 C CNN "Digi-Key PN"
 	1    5190 6590
 	1    0    0    -1

Commit message: added POX LED, much more routing
Parts:
- added C1513: 0.1uF, Capacitors_SMD:C_0402, symbol Custom_Library:C_Custom
- added D1501: Green, LEDs:LED_0402, symbol Device:LED
- added R1508: 1k, Resistors_SMD:R_0402, symbol Custom_Library:R_Custom
- added U1504: 74LVC1G97, Package_TO_SOT_SMD:SOT-363_SC-70-6, symbol Custom_Library:74LVC1G97_Power_NAND_INV
Connections:
- net +3V3: now also C1513.1, R1508.1, U1504.1 (VCC), U1504.5 (VCC)
- net GND: now also C1513.2, U1504.2 (GND)
- net POS3P3_POX_Enable: now also U1504.6
- net ~POX_INT: now also U1504.3
- new net: D1501.1 (K), U1504.4
- new net: D1501.2 (A), R1508.2
Other:
- note added: "LED flickers when POX data is ready"
Changed lines of the file:
@@
 Wire Wire Line
 	5080 1460 5080 1540
+$Comp
+L power:GND #PWR?
+U 1 1 6005778D
+P 8300 5990
+AR Path="/5CB7A8BC/6005778D" Ref="#PWR?"  Part="1"
+AR Path="/5CB7A8C3/6005778D" Ref="#PWR?"  Part="1"
+AR Path="/5EAE4ADE/6005778D" Ref="#PWR?"  Part="1"
+AR Path="/5EAE30C7/6005778D" Ref="#PWR0106"  Part="1"
+F 0 "#PWR0106" H 8300 5740 50  0001 C CNN
+F 1 "GND" H 8300 5840 50  0000 C CNN
+F 2 "" H 8300 5990 50  0001 C CNN
+F 3 "" H 8300 5990 50  0001 C CNN
+	1    8300 5990
+	1    0    0    -1
+$EndComp
+$Comp
+L power:+3.3V #PWR?
+U 1 1 60057793
+P 8300 5790
+AR Path="/5CB7A8BC/60057793" Ref="#PWR?"  Part="1"
+AR Path="/5CB7A8C3/60057793" Ref="#PWR?"  Part="1"
+AR Path="/5EAE4ADE/60057793" Ref="#PWR?"  Part="1"
+AR Path="/5EAE30C7/60057793" Ref="#PWR0107"  Part="1"
+F 0 "#PWR0107" H 8300 5640 50  0001 C CNN
+F 1 "+3.3V" H 8300 5930 50  0000 C CNN
+F 2 "" H 8300 5790 50  0001 C CNN
+F 3 "" H 8300 5790 50  0001 C CNN
+	1    8300 5790
+	1    0    0    -1
+$EndComp
+$Comp
+L Custom_Library:74LVC1G97_Power_NAND_INV U?
+U 1 1 6005779A
+P 8300 5890
+AR Path="/5EAE4ADE/6005779A" Ref="U?"  Part="1"
+AR Path="/5EAE30C7/6005779A" Ref="U1504"  Part="1"
+F 0 "U1504" H 8360 6040 50  0000 L CNN
+F 1 "74LVC1G97" H 8360 5740 50  0000 L CNN
+F 2 "Package_TO_SOT_SMD:SOT-363_SC-70-6" H 8350 5890 50  0001 C CNN
+F 3 "http://www.ti.com/lit/ds/symlink/sn74lvc1g97.pdf" H 8350 5890 50  0001 C CNN
+F 4 "296-SN74LVC1G97DCK3CT-ND" H 8300 5890 50  0001 C CNN "Digi-Key PN"
+	1    8300 5890
+	1    0    0    -1
+$EndComp
+$Comp
+L Custom_Library:C_Custom C?
+U 1 1 600577A4
+P 8190 5200
+AR Path="/5BAAE1F3/600577A4" Ref="C?"  Part="1"
+AR Path="/5BAAE1CB/600577A4" Ref="C?"  Part="1"
+AR Path="/5BE48F98/600577A4" Ref="C?"  Part="1"
+AR Path="/5CAD2D97/600577A4" Ref="C?"  Part="1"
+AR Path="/5CB7A8BC/600577A4" Ref="C?"  Part="1"
+AR Path="/5CB7A8C3/600577A4" Ref="C?"  Part="1"
+AR Path="/5EAE4ADE/600577A4" Ref="C?"  Part="1"
+AR Path="/5EAE30C7/600577A4" Ref="C1513"  Part="1"
+F 0 "C1513" H 8215 5300 50  0000 L CNN
+F 1 "0.1uF" H 8215 5100 50  0000 L CNN
+F 2 "Capacitors_SMD:C_0402" H 8228 5050 50  0001 C CNN
+F 3 "" H 8215 5300 50  0001 C CNN
+F 4 "0402" H 8040 5300 50  0000 R CNN "display_footprint"
+F 5 "25V" H 8040 5200 50  0000 R CNN "Voltage"
+F 6 "X7R" H 8040 5100 50  0000 R CNN "Dielectric"
+F 7 "490-10698-1-ND" H 8190 5200 50  0001 C CNN "Digi-Key PN"
+	1    8190 5200
+	-1   0    0    -1
+$EndComp
+$Comp
+L power:+3.3V #PWR?
+U 1 1 600577AA
+P 8190 5050
+AR Path="/5CB7A8BC/600577AA" Ref="#PWR?"  Part="1"
+AR Path="/5CB7A8C3/600577AA" Ref="#PWR?"  Part="1"
+AR Path="/5EAE4ADE/600577AA" Ref="#PWR?"  Part="1"
+AR Path="/5EAE30C7/600577AA" Ref="#PWR0108"  Part="1"
+F 0 "#PWR0108" H 8190 4900 50  0001 C CNN
+F 1 "+3.3V" H 8190 5190 50  0000 C CNN
+F 2 "" H 8190 5050 50  0001 C CNN
+F 3 "" H 8190 5050 50  0001 C CNN
+	1    8190 5050
+	1    0    0    -1
+$EndComp
+$Comp
+L power:GND #PWR?
+U 1 1 600577B0
+P 8190 5350
+AR Path="/5CB7A8BC/600577B0" Ref="#PWR?"  Part="1"
+AR Path="/5CB7A8C3/600577B0" Ref="#PWR?"  Part="1"
+AR Path="/5EAE4ADE/600577B0" Ref="#PWR?"  Part="1"
+AR Path="/5EAE30C7/600577B0" Ref="#PWR0109"  Part="1"
+F 0 "#PWR0109" H 8190 5100 50  0001 C CNN
+F 1 "GND" H 8190 5200 50  0000 C CNN
+F 2 "" H 8190 5350 50  0001 C CNN
+F 3 "" H 8190 5350 50  0001 C CNN
+	1    8190 5350
+	1    0    0    -1
+$EndComp
+Text GLabel 8000 5940 0    40   Input ~ 0
+~POX_INT
+Text GLabel 8000 5840 0    50   Input ~ 0
+POS3P3_POX_Enable
+$Comp
+L Device:LED D?
+U 1 1 6005EAFD
+P 8870 5620
+AR Path="/5BB844FD/6005EAFD" Ref="D?"  Part="1"
+AR Path="/5BF346B3/6005EAFD" Ref="D?"  Part="1"
+AR Path="/5BAAE1F3/6005EAFD" Ref="D?"  Part="1"
+AR Path="/5CAD2D97/6005EAFD" Ref="D?"  Part="1"
+AR Path="/5CB7A8BC/6005EAFD" Ref="D?"  Part="1"
+AR Path="/5CB7A8C3/6005EAFD" Ref="D?"  Part="1"
+AR Path="/5EAE4ADE/6005EAFD" Ref="D?"  Part="1"
+AR Path="/5EAE30C7/6005EAFD" Ref="D1501"  Part="1"
+F 0 "D1501" V 8909 5503 50  0000 R CNN
+F 1 "Green" V 8818 5503 50  0000 R CNN
+F 2 "LEDs:LED_0402" H 8870 5620 50  0001 C CNN
+F 3 "~" H 8870 5620 50  0001 C CNN
+F 4 "1497-1219-1-ND" H 3710 -700 50  0001 C CNN "Digi-Key PN"
+	1    8870 5620
+	0    -1   -1   0
+$EndComp
+Wire Wire Line
+	8550 5890 8870 5890
+Wire Wire Line
+	8870 5890 8870 5770
+$Comp
+L Custom_Library:R_Custom R?
+U 1 1 6005EB09
+P 8870 5320
+AR Path="/5BAAE1F3/6005EB09" Ref="R?"  Part="1"
+AR Path="/5BAAE1DC/6005EB09" Ref="R?"  Part="1"
+AR Path="/5BAAE16C/6005EB09" Ref="R?"  Part="1"
+AR Path="/5BB844FD/6005EB09" Ref="R?"  Part="1"
+AR Path="/5BF346B3/6005EB09" Ref="R?"  Part="1"
+AR Path="/5CAD2D97/6005EB09" Ref="R?"  Part="1"
+AR Path="/5CB7A8BC/6005EB09" Ref="R?"  Part="1"
+AR Path="/5CB7A8C3/6005EB09" Ref="R?"  Part="1"
+AR Path="/5EAE4ADE/6005EB09" Ref="R?"  Part="1"
+AR Path="/5EAE30C7/6005EB09" Ref="R1508"  Part="1"
+F 0 "R1508" H 8810 5320 50  0000 R CNN
+F 1 "1k" V 8870 5320 50  0000 C CNN
+F 2 "Resistors_SMD:R_0402" H 8870 5320 50  0001 C CNN
+F 3 "" H 8870 5320 50  0001 C CNN
+F 4 "0402" H 8940 5400 50  0000 L CNN "display_footprint"
+F 5 "1%" H 8940 5320 50  0000 L CNN "Tolerance"
+F 6 "1/16W" H 8940 5250 50  0000 L CNN "Wattage"
+F 7 "RMCF0402FT1K00CT-ND" H 8870 5320 50  0001 C CNN "Digi-Key PN"
+	1    8870 5320
+	-1   0    0    -1
+$EndComp
+$Comp
+L power:+3.3V #PWR?
+U 1 1 6005EB0F
+P 8870 5170
+AR Path="/5CB7A8BC/6005EB0F" Ref="#PWR?"  Part="1"
+AR Path="/5CB7A8C3/6005EB0F" Ref="#PWR?"  Part="1"
+AR Path="/5EAE4ADE/6005EB0F" Ref="#PWR?"  Part="1"
+AR Path="/5EAE30C7/6005EB0F" Ref="#PWR0110"  Part="1"
+F 0 "#PWR0110" H 8870 5020 50  0001 C CNN
+F 1 "+3.3V" H 8870 5310 50  0000 C CNN
+F 2 "" H 8870 5170 50  0001 C CNN
+F 3 "" H 8870 5170 50  0001 C CNN
+	1    8870 5170
+	1    0    0    -1
+$EndComp
+Text Notes 8700 6280 0    50   ~ 0
+LED flickers when POX data is ready
 $EndSCHEMATC
