File: hdw/rev_b/Pulse_Oximeter/Pulse_Oximeter.sch (KiCad schematic (older format))
At the start: 0 parts

Commit message: removed rev a output files, renamed Time of Flight to Platform_ETC
Other:
- note added: "14. Platform ETC"
- note removed: "14. Time of Flight"
Changed lines of the file:
@@
 EESchema Schematic File Version 4
-LIBS:Pulse_Oximeter-cache
 EELAYER 30 0
 EELAYER END
@@
 S 4320 5930 500  150
 U 5EAE3021
-F0 "Time of Flight" 50
-F1 "Time_of_Flight.sch" 50
+F0 "Platform ETC" 50
+F1 "Platform_ETC.sch" 50
 $EndSheet
 $Sheet
@@
 13. USB Telemetry
 Text Notes 2160 6080 0    100  ~ 20
-14. Time of Flight
+14. Platform ETC
 Text Notes 2160 6430 0    100  ~ 20
 15. POX Sensor
