File: hdw/rev_b/Pulse_Oximeter/USB_UART_Bridge.sch (KiCad schematic (older format))
At the start: 28 parts, among them J1201 USB_B_Mini, U1201 TLV6700, U1202 FT234XD, U1203 TPD3S014DBVR

Commit message: lots of rev b changes
Parts:
- removed C1204: 4.7uF, Capacitors_SMD:C_0402, symbol Custom_Library:C_Custom
- removed C1209: 0.1uF, Capacitors_SMD:C_0402, symbol Custom_Library:C_Custom
- removed R1205, R1209: 10, Resistors_SMD:R_0402, symbol Custom_Library:R_Custom
- removed R1206: 0.02, Resistors_SMD:R_0612, symbol Custom_Library:R_Custom
- removed TP1201: TP, Custom Footprints Library:Test_Point, symbol Custom_Library:TP
- added C1303: 10uF, Capacitors_SMD:C_0603, symbol Custom_Library:C_Custom
- added C1310, C1312: 0.1uF, Capacitors_SMD:C_0603, symbol Custom_Library:C_Custom
- added R1306, R1308, R1314, R1315: 100k, Resistors_SMD:R_0603, symbol Custom_Library:R_Custom
- added R1309, R1313: 10, Resistors_SMD:R_0603, symbol Custom_Library:R_Custom
- added R1310: 0.02, Resistors_SMD:R_0612, symbol Custom_Library:R_Custom
- added TP1301: TP, Custom Footprints Library:Test_Point, symbol Custom_Library:TP
- added U1304: TXB0102DCU, Package_SO:VSSOP-8_2.4x2.1mm_P0.5mm, symbol Logic_LevelTranslator:TXB0102DCU
- C1301: renamed from C1201; footprint Capacitors_SMD:C_0402 -> Capacitors_SMD:C_0603; Digi-Key PN 490-10701-1-ND -> 399-7845-1-ND; display_footprint 0402 -> 0603
- C1302: renamed from C1203; footprint Capacitors_SMD:C_0402 -> Capacitors_SMD:C_0603; Digi-Key PN 490-10701-1-ND -> 399-7845-1-ND; display_footprint 0402 -> 0603
- C1304: renamed from C1202; footprint Capacitors_SMD:C_0402 -> Capacitors_SMD:C_0603; Digi-Key PN 490-10701-1-ND -> 399-7845-1-ND; display_footprint 0402 -> 0603
- C1306: renamed from C1205; footprint Capacitors_SMD:C_0402 -> Capacitors_SMD:C_0603; Digi-Key PN 490-10701-1-ND -> 399-7845-1-ND; display_footprint 0402 -> 0603
- C1307: renamed from C1206; footprint Capacitors_SMD:C_0402 -> Capacitors_SMD:C_0603; Digi-Key PN 490-10701-1-ND -> 399-7845-1-ND; display_footprint 0402 -> 0603
- C1309: renamed from C1207; footprint Capacitors_SMD:C_0402 -> Capacitors_SMD:C_0603; Digi-Key PN 399-17558-1-ND -> 399-7918-1-ND; display_footprint 0402 -> 0603
- C1311: renamed from C1208; footprint Capacitors_SMD:C_0402 -> Capacitors_SMD:C_0603; Digi-Key PN 399-17558-1-ND -> 399-7918-1-ND; display_footprint 0402 -> 0603
- D1301: renamed from D1201; footprint LEDs:LED_0402 -> LEDs:LED_0603; Digi-Key PN 1497-1389-1-ND -> (none)
- L1301: renamed from L1201; value DNP -> 600R 0.5A; footprint Inductors_SMD:L_0402 -> Inductors_SMD:L_0603; Configuration DNP -> (none); Digi-Key PN DNP -> 732-1593-1-ND
- L1302: renamed from L1202; footprint Inductors_SMD:L_0402 -> Inductors_SMD:L_0603; Digi-Key PN 490-5441-1-ND -> 732-1593-1-ND
- R1301: renamed from R1210; footprint Resistors_SMD:R_0402 -> Resistors_SMD:R_0603; Digi-Key PN 541-1.00KLCT-ND -> 311-1.00KHRCT-ND; Wattage 1/16W -> 1/10W; display_footprint 0402 -> 0603
- R1302: renamed from R1201; footprint Resistors_SMD:R_0402 -> Resistors_SMD:R_0603; Digi-Key PN RMCF0402FT487KCT-ND -> 311-487KHRCT-ND; Wattage 1/16W -> 1/10W; display_footprint 0402 -> 0603
- R1303: renamed from R1202; footprint Resistors_SMD:R_0402 -> Resistors_SMD:R_0603; Digi-Key PN 541-4067-1-ND -> RMCF0603FT6K04CT-ND; Wattage 1/16W -> 1/10W; display_footprint 0402 -> 0603
- R1304: renamed from R1203; footprint Resistors_SMD:R_0402 -> Resistors_SMD:R_0603; Digi-Key PN 541-4097-1-ND -> RMCF0603FT40K2CT-ND; Wattage 1/16W -> 1/10W; display_footprint 0402 -> 0603
- R1305: renamed from R1204; footprint Resistors_SMD:R_0402 -> Resistors_SMD:R_0603; Digi-Key PN RMCF0402FT10K0CT-ND -> YAG2321CT-ND; Wattage 1/16W -> 1/10W; display_footprint 0402 -> 0603
- R1311: renamed from R1207; footprint Resistors_SMD:R_0402 -> Resistors_SMD:R_0603; Digi-Key PN 541-4082-1-ND -> 311-27.0HRCT-ND; Wattage 1/16W -> 1/10W; display_footprint 0402 -> 0603
- R1312: renamed from R1208; footprint Resistors_SMD:R_0402 -> Resistors_SMD:R_0603; Digi-Key PN 541-4082-1-ND -> 311-27.0HRCT-ND; Wattage 1/16W -> 1/10W; display_footprint 0402 -> 0603
- renumbered DOC1201 to DOC1301, J1201 to J1301, U1201 to U1301, U1202 to U1302, U1203 to U1305
Connections:
- net +3V3: now also C1310.1, R1306.1, R1308.1, U1304.3 (VCCA); no longer C1301.1, U1302.9 (VCCIO)
- net +5V_USB: now also C1303.1, R1309.2, R1310.1, TP1301.1 (TP)
- net GND: now also C1303.2, C1310.2, C1312.2, U1304.2 (GND)
- net POS5_USB_PGOOD: now also U1304.6 (OE)
- net POS5_USB_SNS+: now also R1313.1
- net POS5_USB_SNS-: now also R1309.1
- net USB_UART_RX: now also R1308.2, U1304.5 (A1); no longer U1302.7 (TXD)
- net USB_UART_TX: now also R1306.2, U1304.4 (A2); no longer U1302.10 (RXD)
- net +3.3V_USB: now reaches C1307.1, U1302.3 (3V3OUT)
- net +3.3V_USB: now also C1301.1, U1302.9 (VCCIO), C1312.1, R1314.1, R1315.1, U1304.7 (VCCB)
- net at U1305.4 (OUT): now also R1310.2, R1313.2
- new net USB_UART_RX_BUF: R1314.2, U1302.7 (TXD), U1304.8 (B1)
- new net USB_UART_TX_BUF: R1315.2, U1302.10 (RXD), U1304.1 (B2)
Other:
- note added: "TODO: Add FTDI Header (un-buffered)"
- note removed: "ECO: Run a modwire from +3.3V to +5V_USB somewhere, and ensure L1201 is non-popped"
- note removed: "ECR: Add pullups on RX and TX"
- note removed: "ECR: Change VCCIO from global +3.3V! This creates sequencing issues!\nPick something else, or do it the old way"
- moved on the sheet: C1301, C1302, C1304, C1306, C1307, C1309, C1311, D1301, J1301, L1301, L1302, R1301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

Commit message: merged, more cleanups
Parts:
- R1309, R1313: Configuration (none) -> Telemetry
- renumbered C1309 to C?, C1302 to C?, C1311 to C?, C1301 to C?, C1307 to C?, C1306 to C?, C1310 to C?, C1312 to C?, D1301 to D?, DOC1301 to DOC?, J1301 to J?, L1301 to L?, L1302 to L?, R1301 to R?, R1311 to R?, R1303 to R?, R1304 to R?, R1302 to R?, R1305 to R?, R1312 to R?, U1302 to U?, U1305 to U?, U1301 to U?, U1304 to U?

Commit message: changed all passives to 0402, cleared digikey pns
Parts:
- C1201, C1202, C1205, C1206, C1208, C1210: renamed from C?; footprint Capacitors_SMD:C_0603 -> Capacitors_SMD:C_0402; Configuration (none) -> USB; Digi-Key PN 399-7845-1-ND -> (none); display_footprint 0603 -> 0402
- C1207, C1209: renamed from C?; footprint Capacitors_SMD:C_0603 -> Capacitors_SMD:C_0402; Configuration (none) -> USB; display_footprint 0603 -> 0402
- C1303: footprint Capacitors_SMD:C_0603 -> Capacitors_SMD:C_0402; Configuration (none) -> USB; Digi-Key PN 490-10474-1-ND -> (none); display_footprint 0603 -> 0402
- C1304: footprint Capacitors_SMD:C_0603 -> Capacitors_SMD:C_0402; Configuration (none) -> USB; Digi-Key PN 399-7845-1-ND -> (none); display_footprint 0603 -> 0402
- D1201: renamed from D?; footprint LEDs:LED_0603 -> LEDs:LED_0402; Configuration (none) -> USB
- J1201: renamed from J?; Configuration (none) -> USB
- L1201, L1202: renamed from L?; footprint Inductors_SMD:L_0603 -> Inductors_SMD:L_0402; Configuration (none) -> USB; Digi-Key PN 732-1593-1-ND -> (none)
- R1201: renamed from R?; footprint Resistors_SMD:R_0603 -> Resistors_SMD:R_0402; Configuration (none) -> USB; Digi-Key PN 311-1.00KHRCT-ND -> (none); Wattage 1/10W -> 1/16W; display_footprint 0603 -> 0402
- R1202: renamed from R?; footprint Resistors_SMD:R_0603 -> Resistors_SMD:R_0402; Configuration (none) -> USB; Digi-Key PN 311-487KHRCT-ND -> (none); Wattage 1/10W -> 1/16W; display_footprint 0603 -> 0402
- R1203: renamed from R?; footprint Resistors_SMD:R_0603 -> Resistors_SMD:R_0402; Configuration (none) -> USB; Digi-Key PN RMCF0603FT6K04CT-ND -> (none); Wattage 1/10W -> 1/16W; display_footprint 0603 -> 0402
- R1204: renamed from R?; footprint Resistors_SMD:R_0603 -> Resistors_SMD:R_0402; Configuration (none) -> USB; Digi-Key PN RMCF0603FT40K2CT-ND -> (none); Wattage 1/10W -> 1/16W; display_footprint 0603 -> 0402
- R1205: renamed from R?; footprint Resistors_SMD:R_0603 -> Resistors_SMD:R_0402; Configuration (none) -> USB; Digi-Key PN YAG2321CT-ND -> (none); Wattage 1/10W -> 1/16W; display_footprint 0603 -> 0402
- R1210, R1211: renamed from R?; footprint Resistors_SMD:R_0603 -> Resistors_SMD:R_0402; Configuration (none) -> USB; Digi-Key PN 311-27.0HRCT-ND -> (none); Wattage 1/10W -> 1/16W; display_footprint 0603 -> 0402
- R1306, R1308, R1314, R1315: footprint Resistors_SMD:R_0603 -> Resistors_SMD:R_0402; Configuration (none) -> USB; Digi-Key PN RMCF0603FT100KCT-ND -> (none); Wattage 1/10W -> 1/16W; display_footprint 0603 -> 0402
- R1309, R1313: footprint Resistors_SMD:R_0603 -> Resistors_SMD:R_0402; Digi-Key PN YAG2321CT-ND -> (none); Wattage 1/10W -> 1/16W; display_footprint 0603 -> 0402
- R1310: Configuration (none) -> USB
- U1201, U1202, U1203, U1204: renamed from U?; Configuration (none) -> USB
- gave numbers to parts that had none: 1
Other:
- note added: "Note: All components on this sheet have "Configuration" field set to "USB", unless otherwise noted"

Commit message: removed more unique components, cleaned up SCH
Parts:
- added R? (x3): 0, Resistors_SMD:R_0402, symbol Custom_Library:R_Custom
- R1310: Configuration USB -> Telemetry
Connections:
- net +5V_USB: now also R?.1, R?.1, R?.1
- net at R1310.2, R1313.2, U1204.4 (OUT): now also R?.2, R?.2, R?.2
Other:
- note added: "TODO: Add FTDI Header (buffered)"
- note removed: "TODO: Add FTDI Header (un-buffered)"
- moved on the sheet: C1205, R1208, R1209, R1212, TP1201, U1204

Commit message: annotated schematic
Parts:
- L1201, L1202: Digi-Key PN (none) -> 490-5441-1-ND
- gave numbers to parts that had none: 3
- renumbered C1303 to C1203, C1304 to C1204, R1306 to R1206, R1308 to R1207, R1309 to R1208, R1310 to R1209, R1210 to R1213, R1211 to R1214, R1313 to R1215, R1314 to R1216, R1315 to R1217, TP1301 to TP1201
Changed lines of the file:
@@
 F 2 "Inductors_SMD:L_0402" V 7650 4500 50  0001 C CNN
 F 3 "~" H 7720 4500 50  0001 C CNN
-F 4 "" H -470 1410 50  0001 C CNN "Digi-Key PN"
+F 4 "490-5441-1-ND" H -470 1410 50  0001 C CNN "Digi-Key PN"
 F 5 "USB" H 7720 4500 50  0001 C CNN "Configuration"
 	1    7720 4500
@@
 $EndComp
 $Comp
-L Custom_Library:R_Custom R1210
+L Custom_Library:R_Custom R1213
 U 1 1 5BBF0F91
 P 5110 4700
-F 0 "R1210" V 5200 4700 50  0000 C CNN
+F 0 "R1213" V 5200 4700 50  0000 C CNN
 F 1 "27" V 5110 4700 50  0000 C CNN
 F 2 "Resistors_SMD:R_0402" H 5110 4700 50  0001 C CNN
@@
 F 2 "Inductors_SMD:L_0402" V 8990 5170 50  0001 C CNN
 F 3 "~" H 9060 5170 50  0001 C CNN
-F 4 "" H -470 1410 50  0001 C CNN "Digi-Key PN"
+F 4 "490-5441-1-ND" H -470 1410 50  0001 C CNN "Digi-Key PN"
 F 5 "USB" H 9060 5170 50  0001 C CNN "Configuration"
 	1    9060 5170
@@
 AR Path="/5BE48F98/5C037C42" Ref="C?"  Part="1"
 AR Path="/5CAD2D97/5C037C42" Ref="C?"  Part="1"
-AR Path="/5E939F76/5C037C42" Ref="C1304"  Part="1"
+AR Path="/5E939F76/5C037C42" Ref="C?"  Part="1"
 AR Path="/5EAE2F97/5C037C42" Ref="C1204"  Part="1"
 F 0 "C1204" H 3505 7700 50  0000 L CNN
@@
 	5260 4800 6510 4800
 $Comp
-L Custom_Library:R_Custom R1211
+L Custom_Library:R_Custom R1214
 U 1 1 5C04BC29
 P 5110 4800
-F 0 "R1211" V 5490 4800 50  0000 C CNN
+F 0 "R1214" V 5490 4800 50  0000 C CNN
 F 1 "27" V 5110 4800 50  0000 C CNN
 F 2 "Resistors_SMD:R_0402" H 5110 4800 50  0001 C CNN
@@
 AR Path="/5A0BC776/5E3059D8" Ref="TP?"  Part="1"
 AR Path="/5CAD2D97/5E3059D8" Ref="TP?"  Part="1"
-AR Path="/5E939F76/5E3059D8" Ref="TP1301"  Part="1"
+AR Path="/5E939F76/5E3059D8" Ref="TP?"  Part="1"
 AR Path="/5EAE2F97/5E3059D8" Ref="TP1201"  Part="1"
 F 0 "TP1201" H 4050 3550 50  0000 C CNN
@@
 AR Path="/5CB6F1ED/5E954115" Ref="R?"  Part="1"
 AR Path="/5E939CFF/5E954115" Ref="R?"  Part="1"
-AR Path="/5E939F76/5E954115" Ref="R1313"  Part="1"
-AR Path="/5EAE2F97/5E954115" Ref="R1212"  Part="1"
-F 0 "R1212" V 5140 3240 50  0000 C CNN
+AR Path="/5E939F76/5E954115" Ref="R?"  Part="1"
+AR Path="/5EAE2F97/5E954115" Ref="R1215"  Part="1"
+F 0 "R1215" V 5140 3240 50  0000 C CNN
 F 1 "10" V 5240 3240 50  0000 C CNN
 F 2 "Resistors_SMD:R_0402" H 5240 3240 50  0001 C CNN
@@
 AR Path="/5CB6F1ED/5E95410C" Ref="R?"  Part="1"
 AR Path="/5E939CFF/5E95410C" Ref="R?"  Part="1"
-AR Path="/5E939F76/5E95410C" Ref="R1309"  Part="1"
+AR Path="/5E939F76/5E95410C" Ref="R?"  Part="1"
 AR Path="/5EAE2F97/5E95410C" Ref="R1208"  Part="1"
 F 0 "R1208" V 4680 3240 50  0000 C CNN
@@
 P 6220 1130
 AR Path="/5E939D51/5F3B373F" Ref="R?"  Part="1"
-AR Path="/5E939F76/5F3B373F" Ref="R1314"  Part="1"
-AR Path="/5EAE2F97/5F3B373F" Ref="R1213"  Part="1"
-F 0 "R1213" H 6290 1260 50  0000 L CNN
+AR Path="/5E939F76/5F3B373F" Ref="R?"  Part="1"
+AR Path="/5EAE2F97/5F3B373F" Ref="R1216"  Part="1"
+F 0 "R1216" H 6290 1260 50  0000 L CNN
 F 1 "100k" V 6220 1130 40  0000 C CNN
 F 2 "Resistors_SMD:R_0402" H 6220 1130 50  0001 C CNN
@@
 P 6730 1130
 AR Path="/5E939D51/5F3B4F3C" Ref="R?"  Part="1"
-AR Path="/5E939F76/5F3B4F3C" Ref="R1315"  Part="1"
-AR Path="/5EAE2F97/5F3B4F3C" Ref="R1214"  Part="1"
-F 0 "R1214" H 6800 1260 50  0000 L CNN
+AR Path="/5E939F76/5F3B4F3C" Ref="R?"  Part="1"
+AR Path="/5EAE2F97/5F3B4F3C" Ref="R1217"  Part="1"
+F 0 "R1217" H 6800 1260 50  0000 L CNN
 F 1 "100k" V 6730 1130 40  0000 C CNN
 F 2 "Resistors_SMD:R_0402" H 6730 1130 50  0001 C CNN
@@
 AR Path="/5EAE2D8A/5F6EB551" Ref="C?"  Part="1"
 AR Path="/5E939D31/5F6EB551" Ref="C?"  Part="1"
-AR Path="/5E939F76/5F6EB551" Ref="C1303"  Part="1"
+AR Path="/5E939F76/5F6EB551" Ref="C?"  Part="1"
 AR Path="/5EAE2F97/5F6EB551" Ref="C1203"  Part="1"
 F 0 "C1203" H 3065 3780 50  0000 L CNN
@@
 P 3970 1130
 AR Path="/5E939D51/5F3C147E" Ref="R?"  Part="1"
-AR Path="/5E939F76/5F3C147E" Ref="R1306"  Part="1"
+AR Path="/5E939F76/5F3C147E" Ref="R?"  Part="1"
 AR Path="/5EAE2F97/5F3C147E" Ref="R1206"  Part="1"
 F 0 "R1206" H 4040 1260 50  0000 L CNN
@@
 P 4480 1130
 AR Path="/5E939D51/5F3C1475" Ref="R?"  Part="1"
-AR Path="/5E939F76/5F3C1475" Ref="R1308"  Part="1"
+AR Path="/5E939F76/5F3C1475" Ref="R?"  Part="1"
 AR Path="/5EAE2F97/5F3C1475" Ref="R1207"  Part="1"
 F 0 "R1207" H 4550 1260 50  0000 L CNN
@@
 AR Path="/5A0BC776/5E0650D5" Ref="R?"  Part="1"
 AR Path="/5CAD2D97/5E0650D5" Ref="R?"  Part="1"
-AR Path="/5E939F76/5E0650D5" Ref="R1310"  Part="1"
+AR Path="/5E939F76/5E0650D5" Ref="R?"  Part="1"
 AR Path="/5EAE2F97/5E0650D5" Ref="R1209"  Part="1"
 F 0 "R1209" V 4910 3470 50  0000 C CNN
@@
 AR Path="/5EAE2D8A/5FE7820C" Ref="R?"  Part="1"
 AR Path="/5EAE2D66/5FE7820C" Ref="R?"  Part="1"
-AR Path="/5EAE2F97/5FE7820C" Ref="R?"  Part="1"
-F 0 "R?" V 4910 3820 50  0000 C CNN
+AR Path="/5EAE2F97/5FE7820C" Ref="R1210"  Part="1"
+F 0 "R1210" V 4910 3820 50  0000 C CNN
 F 1 "0" V 5010 3820 50  0000 C CNN
 F 2 "Resistors_SMD:R_0402" H 5010 3820 50  0001 C CNN
@@
 AR Path="/5EAE2D8A/5FE78216" Ref="R?"  Part="1"
 AR Path="/5EAE2D66/5FE78216" Ref="R?"  Part="1"
-AR Path="/5EAE2F97/5FE78216" Ref="R?"  Part="1"
-F 0 "R?" V 4910 4090 50  0000 C CNN
+AR Path="/5EAE2F97/5FE78216" Ref="R1211"  Part="1"
+F 0 "R1211" V 4910 4090 50  0000 C CNN
 F 1 "0" V 5010 4090 50  0000 C CNN
 F 2 "Resistors_SMD:R_0402" H 5010 4090 50  0001 C CNN
@@
 AR Path="/5EAE2D8A/5FE78220" Ref="R?"  Part="1"
 AR Path="/5EAE2D66/5FE78220" Ref="R?"  Part="1"
-AR Path="/5EAE2F97/5FE78220" Ref="R?"  Part="1"
-F 0 "R?" V 4910 4360 50  0000 C CNN
+AR Path="/5EAE2F97/5FE78220" Ref="R1212"  Part="1"
+F 0 "R1212" V 4910 4360 50  0000 C CNN
 F 1 "0" V 5010 4360 50  0000 C CNN
 F 2 "Resistors_SMD:R_0402" H 5010 4360 50  0001 C CNN

Commit message: USB circuit adjustments, add UART dongle header, resolve some open rev B SCH issues
Parts:
- added C?: 0.1uF, Capacitors_SMD:C_0402, symbol Custom_Library:C_Custom
- added J?: OSEPP_FTDI_01, symbol Connector_Generic:Conn_01x06
- added R?: 0, Resistors_SMD:R_0402, symbol Custom_Library:R_Custom
- C1208, C1210, R1206, R1207, R1216, R1217, U1203: Configuration USB -> (none)
- R1210, R1211, R1212: Configuration !Telemetry -> ~Telemetry
Connections:
- net +3.3V_USB: now also C?.1, J?.4 (Pin_4), R?.2
- net GND: now also C?.2, J?.6 (Pin_6)
- net POS5_USB_PGOOD: now also R?.1
- net USB_UART_RX_BUF: now also J?.3 (Pin_3)
- net USB_UART_TX_BUF: now also J?.2 (Pin_2)
- no-connect marks 4 -> 6
Other:
- note added: "Note: All components within box appear on all configurations"
- note added: "Note: Plugging in an OSEPP FTDI_01 module\non non-USB configs will drive +3.3V onto \n+3.3V_USB net, and force POS5_USB_PGOOD\nhigh in order to enable UART buffer. Module\nVCCIO must be set to +3.3V. This allows a serial\nconnection without any USB components placed\nin the design."
- note removed: "TODO: Add FTDI Header (buffered)"
- moved on the sheet: C1208, C1210, R1206, R1207, R1216, R1217, U1203
