File: hdw/rev_b/Pulse_Oximeter/USB_UART_Bridge.sch (KiCad schematic (older format))
At the start: 40 parts, among them J1201 USB_B_Mini, U1201 TLV6700, U1202 FT234XD, U1203 TXB0102DCU, U1204 TPD3S014DBVR

Commit message: assigned digikey PNs
Parts:
- C1201, C1202, C1204, C1205, C1206, C1208, C1210, C?: Digi-Key PN (none) -> 490-10698-1-ND; Voltage 50V -> 25V
- C1203: Digi-Key PN (none) -> 1276-6830-1-ND
- C1207, C1209: Digi-Key PN 399-7918-1-ND -> 311-3783-1-ND
- D1201: Digi-Key PN (none) -> 1497-1198-1-ND
- J?: footprint (none) -> Connector_PinHeader_2.54mm:PinHeader_1x06_P2.54mm_Vertical
- R1201: Digi-Key PN (none) -> RMCF0402FT1K00CT-ND
- R1202: Digi-Key PN (none) -> RMCF0402FT487KCT-ND
- R1203: Digi-Key PN (none) -> RMCF0402FT6K04CT-ND
- R1204: Digi-Key PN (none) -> 311-40.2KLRCT-ND
- R1205: Digi-Key PN (none) -> RMCF0402FT10K0CT-ND
- R1206, R1207, R1216, R1217: Digi-Key PN (none) -> RMCF0402FT100KCT-ND
- R1208, R1215: Digi-Key PN (none) -> RMCF0402FT10R0CT-ND
- R1210, R1211, R1212, R?: Digi-Key PN (none) -> 2019-RK73Z1ETTPCT-ND
- R1213, R1214: Digi-Key PN (none) -> RMCF0402FT27R0CT-ND
Changed lines of the file:
@@
 F 5 "50V" H 5530 5130 50  0000 R CNN "Voltage"
 F 6 "NP0" H 5530 5030 50  0000 R CNN "Dielectric"
-F 7 "399-7918-1-ND" H 5680 5130 50  0001 C CNN "Digi-Key PN"
+F 7 "311-3783-1-ND" H 5680 5130 50  0001 C CNN "Digi-Key PN"
 F 8 "USB" H 5680 5130 50  0001 C CNN "Configuration"
 	1    5680 5130
@@
 F 3 "" H 2385 3780 50  0001 C CNN
 F 4 "0402" H 2210 3780 50  0000 R CNN "display_footprint"
-F 5 "50V" H 2210 3680 50  0000 R CNN "Voltage"
+F 5 "25V" H 2210 3680 50  0000 R CNN "Voltage"
 F 6 "X7R" H 2210 3580 50  0000 R CNN "Dielectric"
-F 7 "" H 2785 4180 60  0001 C CNN "Digi-Key PN"
+F 7 "490-10698-1-ND" H 2785 4180 60  0001 C CNN "Digi-Key PN"
 F 8 "USB" H 2360 3680 50  0001 C CNN "Configuration"
 	1    2360 3680
@@
 F 5 "50V" H 6360 5130 50  0000 R CNN "Voltage"
 F 6 "NP0" H 6360 5030 50  0000 R CNN "Dielectric"
-F 7 "399-7918-1-ND" H 6510 5130 50  0001 C CNN "Digi-Key PN"
+F 7 "311-3783-1-ND" H 6510 5130 50  0001 C CNN "Digi-Key PN"
 F 8 "USB" H 6510 5130 50  0001 C CNN "Configuration"
 	1    6510 5130
@@
 F 3 "" H 1695 3780 50  0001 C CNN
 F 4 "0402" H 1520 3780 50  0000 R CNN "display_footprint"
-F 5 "50V" H 1520 3680 50  0000 R CNN "Voltage"
+F 5 "25V" H 1520 3680 50  0000 R CNN "Voltage"
 F 6 "X7R" H 1520 3580 50  0000 R CNN "Dielectric"
-F 7 "" H 2095 4180 60  0001 C CNN "Digi-Key PN"
+F 7 "490-10698-1-ND" H 2095 4180 60  0001 C CNN "Digi-Key PN"
 F 8 "USB" H 1670 3680 50  0001 C CNN "Configuration"
 	1    1670 3680
@@
 F 3 "" H 4435 5450 50  0001 C CNN
 F 4 "0402" H 4260 5450 50  0000 R CNN "display_footprint"
-F 5 "50V" H 4260 5350 50  0000 R CNN "Voltage"
+F 5 "25V" H 4260 5350 50  0000 R CNN "Voltage"
 F 6 "X7R" H 4260 5250 50  0000 R CNN "Dielectric"
-F 7 "" H 4835 5850 60  0001 C CNN "Digi-Key PN"
+F 7 "490-10698-1-ND" H 4835 5850 60  0001 C CNN "Digi-Key PN"
 F 8 "USB" H 4410 5350 50  0001 C CNN "Configuration"
 	1    4410 5350
@@
 F 5 "1%" H 1010 4480 50  0000 L CNN "Tolerance"
 F 6 "1/16W" H 1010 4410 50  0000 L CNN "Wattage"
-F 7 "" H 1240 4880 60  0001 C CNN "Digi-Key PN"
+F 7 "RMCF0402FT1K00CT-ND" H 1240 4880 60  0001 C CNN "Digi-Key PN"
 F 8 "USB" H 940 4480 50  0001 C CNN "Configuration"
 	1    940  4480
@@
 F 6 "1/16W" V 5225 4700 50  0001 C CNN "Wattage"
 F 7 "USB" H 5110 4700 50  0001 C CNN "Configuration"
+F 8 "RMCF0402FT27R0CT-ND" H 5110 4700 50  0001 C CNN "Digi-Key PN"
 	1    5110 4700
 	0    1    -1   0
@@
 F 3 "~" H 940 4780 50  0001 C CNN
 F 4 "USB" H 940 4780 50  0001 C CNN "Configuration"
+F 5 "1497-1198-1-ND" H 940 4780 50  0001 C CNN "Digi-Key PN"
 	1    940  4780
 	0    -1   -1   0
@@
 F 5 "1%" H 1880 6880 50  0000 L CNN "Tolerance"
 F 6 "1/16W" H 1890 6800 50  0000 L CNN "Wattage"
-F 7 "" H 2080 7280 60  0001 C CNN "Digi-Key PN"
+F 7 "RMCF0402FT6K04CT-ND" H 2080 7280 60  0001 C CNN "Digi-Key PN"
 F 8 "USB" H 1780 6880 50  0001 C CNN "Configuration"
 	1    1780 6880
@@
 F 5 "1%" H 1880 7370 50  0000 L CNN "Tolerance"
 F 6 "1/16W" H 1890 7290 50  0000 L CNN "Wattage"
-F 7 "" H 2080 7770 60  0001 C CNN "Digi-Key PN"
+F 7 "311-40.2KLRCT-ND" H 2080 7770 60  0001 C CNN "Digi-Key PN"
 F 8 "USB" H 1780 7370 50  0001 C CNN "Configuration"
 	1    1780 7370
@@
 F 5 "1%" H 1880 6340 50  0000 L CNN "Tolerance"
 F 6 "1/16W" H 1890 6260 50  0000 L CNN "Wattage"
-F 7 "" H 2080 6740 60  0001 C CNN "Digi-Key PN"
+F 7 "RMCF0402FT487KCT-ND" H 2080 6740 60  0001 C CNN "Digi-Key PN"
 F 8 "USB" H 1780 6340 50  0001 C CNN "Configuration"
 	1    1780 6340
@@
 F 5 "1%" H 3510 6290 50  0000 L CNN "Tolerance"
 F 6 "1/16W" H 3520 6210 50  0000 L CNN "Wattage"
-F 7 "" H 3710 6690 60  0001 C CNN "Digi-Key PN"
+F 7 "RMCF0402FT10K0CT-ND" H 3710 6690 60  0001 C CNN "Digi-Key PN"
 F 8 "USB" H 3410 6290 50  0001 C CNN "Configuration"
 	1    3410 6290
@@
 F 2 "Capacitors_SMD:C_0402" H 3518 7450 50  0001 C CNN
 F 3 "" H 3505 7700 50  0001 C CNN
-F 4 "" H 3905 8100 60  0001 C CNN "Digi-Key PN"
+F 4 "490-10698-1-ND" H 3905 8100 60  0001 C CNN "Digi-Key PN"
 F 5 "0402" H 3330 7700 50  0000 R CNN "display_footprint"
-F 6 "50V" H 3330 7600 50  0000 R CNN "Voltage"
+F 6 "25V" H 3330 7600 50  0000 R CNN "Voltage"
 F 7 "X7R" H 3330 7500 50  0000 R CNN "Dielectric"
 F 8 "USB" H 3480 7600 50  0001 C CNN "Configuration"
@@
 F 5 "1%" V 5316 4800 50  0000 C CNN "Tolerance"
 F 6 "1/16W" V 5225 4800 50  0000 C CNN "Wattage"
-F 7 "" H 5410 5200 60  0001 C CNN "Digi-Key PN"
+F 7 "RMCF0402FT27R0CT-ND" H 5410 5200 60  0001 C CNN "Digi-Key PN"
 F 8 "USB" H 5110 4800 50  0001 C CNN "Configuration"
 	1    5110 4800
@@
 F 3 "" H 4435 3770 50  0001 C CNN
 F 4 "0402" H 4260 3770 50  0000 R CNN "display_footprint"
-F 5 "50V" H 4260 3670 50  0000 R CNN "Voltage"
+F 5 "25V" H 4260 3670 50  0000 R CNN "Voltage"
 F 6 "X7R" H 4260 3570 50  0000 R CNN "Dielectric"
-F 7 "" H 4835 4170 60  0001 C CNN "Digi-Key PN"
+F 7 "490-10698-1-ND" H 4835 4170 60  0001 C CNN "Digi-Key PN"
 F 8 "USB" H 4410 3670 50  0001 C CNN "Configuration"
 	1    4410 3670
@@
 F 5 "1%" V 5440 3240 50  0001 C CNN "Tolerance"
 F 6 "1/16W" V 5540 3240 50  0001 C CNN "Wattage"
-F 7 "" H 5240 3240 50  0001 C CNN "Digi-Key PN"
+F 7 "RMCF0402FT10R0CT-ND" H 5240 3240 50  0001 C CNN "Digi-Key PN"
 F 8 "Telemetry" V 5340 3240 50  0000 C CNN "Configuration"
 	1    5240 3240
@@
 F 5 "1%" V 4980 3240 50  0001 C CNN "Tolerance"
 F 6 "1/16W" V 5080 3240 50  0001 C CNN "Wattage"
-F 7 "" H 4780 3240 50  0001 C CNN "Digi-Key PN"
+F 7 "RMCF0402FT10R0CT-ND" H 4780 3240 50  0001 C CNN "Digi-Key PN"
 F 8 "Telemetry" V 4880 3240 50  0000 C CNN "Configuration"
 	1    4780 3240
@@
 F 5 "1%" H 4240 970 50  0000 L CNN "Tolerance"
 F 6 "1/16W" H 4240 880 50  0000 L CNN "Wattage"
+F 7 "RMCF0402FT100KCT-ND" H 4170 1010 50  0001 C CNN "Digi-Key PN"
 	1    4170 1010
 	1    0    0    -1
@@
 F 5 "1%" H 4750 970 50  0000 L CNN "Tolerance"
 F 6 "1/16W" H 4750 880 50  0000 L CNN "Wattage"
+F 7 "RMCF0402FT100KCT-ND" H 4680 1010 50  0001 C CNN "Digi-Key PN"
 	1    4680 1010
 	1    0    0    -1
@@
 F 3 "" H 4065 2020 50  0001 C CNN
 F 4 "0402" H 3890 2020 50  0000 R CNN "display_footprint"
-F 5 "50V" H 3890 1920 50  0000 R CNN "Voltage"
+F 5 "25V" H 3890 1920 50  0000 R CNN "Voltage"
 F 6 "X7R" H 3890 1820 50  0000 R CNN "Dielectric"
+F 7 "490-10698-1-ND" H 4040 1920 50  0001 C CNN "Digi-Key PN"
 	1    4040 1920
 	1    0    0    -1
@@
 F 3 "" H 4775 2020 50  0001 C CNN
 F 4 "0402" H 4600 2020 50  0000 R CNN "display_footprint"
-F 5 "50V" H 4600 1920 50  0000 R CNN "Voltage"
+F 5 "25V" H 4600 1920 50  0000 R CNN "Voltage"
 F 6 "X7R" H 4600 1820 50  0000 R CNN "Dielectric"
+F 7 "490-10698-1-ND" H 4750 1920 50  0001 C CNN "Digi-Key PN"
 	1    4750 1920
 	1    0    0    -1
@@
 F 5 "10V" H 2890 3680 50  0000 R CNN "Voltage"
 F 6 "X5R" H 2890 3580 50  0000 R CNN "Dielectric"
-F 7 "" H 3040 3680 50  0001 C CNN "Digi-Key PN"
+F 7 "1276-6830-1-ND" H 3040 3680 50  0001 C CNN "Digi-Key PN"
 F 8 "USB" H 3040 3680 50  0001 C CNN "Configuration"
 	1    3040 3680
@@
 F 5 "1%" H 1990 970 50  0000 L CNN "Tolerance"
 F 6 "1/16W" H 1990 880 50  0000 L CNN "Wattage"
+F 7 "RMCF0402FT100KCT-ND" H 1920 1010 50  0001 C CNN "Digi-Key PN"
 	1    1920 1010
 	-1   0    0    -1
@@
 F 5 "1%" H 2500 970 50  0000 L CNN "Tolerance"
 F 6 "1/16W" H 2500 880 50  0000 L CNN "Wattage"
+F 7 "RMCF0402FT100KCT-ND" H 2430 1010 50  0001 C CNN "Digi-Key PN"
 	1    2430 1010
 	-1   0    0    -1
@@
 F 6 "1/16W" V 5310 3820 50  0001 C CNN "Wattage"
 F 7 "~Telemetry" V 5110 3820 50  0000 C CNN "Configuration"
+F 8 "2019-RK73Z1ETTPCT-ND" H 5010 3820 50  0001 C CNN "Digi-Key PN"
 	1    5010 3820
 	0    -1   1    0
@@
 F 6 "1/16W" V 5310 4090 50  0001 C CNN "Wattage"
 F 7 "~Telemetry" V 5110 4090 50  0000 C CNN "Configuration"
+F 8 "2019-RK73Z1ETTPCT-ND" H 5010 4090 50  0001 C CNN "Digi-Key PN"
 	1    5010 4090
 	0    -1   1    0
@@
 F 6 "1/16W" V 5310 4360 50  0001 C CNN "Wattage"
 F 7 "~Telemetry" V 5110 4360 50  0000 C CNN "Configuration"
+F 8 "2019-RK73Z1ETTPCT-ND" H 5010 4360 50  0001 C CNN "Digi-Key PN"
 	1    5010 4360
 	0    -1   1    0
@@
 F 0 "J?" H 9800 1490 50  0000 L CNN
 F 1 "OSEPP_FTDI_01" H 9800 1390 50  0000 L CNN
-F 2 "" H 9690 1420 50  0001 C CNN
+F 2 "Connector_PinHeader_2.54mm:PinHeader_1x06_P2.54mm_Vertical" H 9690 1420 50  0001 C CNN
 F 3 "~" H 9690 1420 50  0001 C CNN
 F 4 "~USB" H 9800 1290 50  0000 L CNN "Configuration"
@@
 F 3 "" H 8365 1660 50  0001 C CNN
 F 4 "0402" H 8190 1660 50  0000 R CNN "display_footprint"
-F 5 "50V" H 8190 1560 50  0000 R CNN "Voltage"
+F 5 "25V" H 8190 1560 50  0000 R CNN "Voltage"
 F 6 "X7R" H 8190 1460 50  0000 R CNN "Dielectric"
+F 7 "490-10698-1-ND" H 8340 1560 50  0001 C CNN "Digi-Key PN"
 	1    8340 1560
 	1    0    0    -1
@@
 F 6 "1/16W" V 8770 800 50  0001 C CNN "Wattage"
 F 7 "~USB" V 8570 800 50  0000 C CNN "Configuration"
+F 8 "2019-RK73Z1ETTPCT-ND" H 8470 800 50  0001 C CNN "Digi-Key PN"
 	1    8470 800
 	0    -1   1    0

Commit message: started working on rev B PCB, a few SCH changes
Parts:
- gave numbers to parts that had none: 3
Changed lines of the file:
@@
 	6950 3470 6950 4500
 $Comp
-L Connector_Generic:Conn_01x06 J?
+L Connector_Generic:Conn_01x06 J1202
 U 1 1 5FEF27B0
 P 9690 1420
-F 0 "J?" H 9800 1490 50  0000 L CNN
+F 0 "J1202" H 9800 1490 50  0000 L CNN
 F 1 "OSEPP_FTDI_01" H 9800 1390 50  0000 L CNN
 F 2 "Connector_PinHeader_2.54mm:PinHeader_1x06_P2.54mm_Vertical" H 9690 1420 50  0001 C CNN
@@
 $EndComp
 $Comp
-L power:GND #PWR?
+L power:GND #PWR0101
 U 1 1 5FF04965
 P 9410 1800
-F 0 "#PWR?" H 9410 1550 50  0001 C CNN
+F 0 "#PWR0101" H 9410 1550 50  0001 C CNN
 F 1 "GND" H 9410 1650 50  0000 C CNN
 F 2 "" H 9410 1800 50  0001 C CNN
@@
 NoConn ~ 9490 1620
 $Comp
-L Custom_Library:+3.3V_USB #PWR?
+L Custom_Library:+3.3V_USB #PWR0102
 U 1 1 5FF0AAFA
 P 9490 1520
-F 0 "#PWR?" H 9490 1370 50  0001 C CNN
+F 0 "#PWR0102" H 9490 1370 50  0001 C CNN
 F 1 "+3.3V_USB" V 9490 1660 50  0000 L CNN
 F 2 "" H 9490 1520 50  0001 C CNN
@@
 NoConn ~ 9490 1220
 $Comp
-L Custom_Library:C_Custom C?
+L Custom_Library:C_Custom C1211
 U 1 1 5FF1CC79
 P 8340 1560
-F 0 "C?" H 8365 1660 50  0000 L CNN
+F 0 "C1211" H 8365 1660 50  0000 L CNN
 F 1 "0.1uF" H 8365 1460 50  0000 L CNN
 F 2 "Capacitors_SMD:C_0402" H 8378 1410 50  0001 C CNN
@@
 $EndComp
 $Comp
-L power:GND #PWR?
+L power:GND #PWR0103
 U 1 1 5FF1D1ED
 P 8340 1710
-F 0 "#PWR?" H 8340 1460 50  0001 C CNN
+F 0 "#PWR0103" H 8340 1460 50  0001 C CNN
 F 1 "GND" H 8340 1560 50  0000 C CNN
 F 2 "" H 8340 1710 50  0001 C CNN
@@
 $EndComp
 $Comp
-L Custom_Library:+3.3V_USB #PWR?
+L Custom_Library:+3.3V_USB #PWR0104
 U 1 1 5FF1D1F7
 P 8340 1410
-F 0 "#PWR?" H 8340 1260 50  0001 C CNN
+F 0 "#PWR0104" H 8340 1260 50  0001 C CNN
 F 1 "+3.3V_USB" H 8340 1550 50  0000 C CNN
 F 2 "" H 8340 1410 50  0001 C CNN
@@
 AR Path="/5EAE2D8A/5FF25591" Ref="R?"  Part="1"
 AR Path="/5EAE2D66/5FF25591" Ref="R?"  Part="1"
-AR Path="/5EAE2F97/5FF25591" Ref="R?"  Part="1"
-F 0 "R?" V 8370 800 50  0000 C CNN
+AR Path="/5EAE2F97/5FF25591" Ref="R1218"  Part="1"
+F 0 "R1218" V 8370 800 50  0000 C CNN
 F 1 "0" V 8470 800 50  0000 C CNN
 F 2 "Resistors_SMD:R_0402" H 8470 800 50  0001 C CNN
@@
 $EndComp
 $Comp
-L Custom_Library:+3.3V_USB #PWR?
+L Custom_Library:+3.3V_USB #PWR0105
 U 1 1 5FF25AF5
 P 8620 800
-F 0 "#PWR?" H 8620 650 50  0001 C CNN
+F 0 "#PWR0105" H 8620 650 50  0001 C CNN
 F 1 "+3.3V_USB" V 8620 940 50  0000 L CNN
 F 2 "" H 8620 800 50  0001 C CNN
