File: hdw/rev_b/Pulse_Oximeter/Display.sch (KiCad schematic (older format))
At the start: 21 parts, among them U1601 74LVC1G17, U1602 NHD-0420H1Z

Commit message: changed all passives to 0402, cleared digikey pns
Parts:
- removed C1604: 10nF, Capacitors_SMD:C_0402, symbol Custom_Library:C_Custom
- removed C1605: 1nF, Capacitors_SMD:C_0402, symbol Custom_Library:C_Custom
- removed RV1601: 10k, Potentiometer_SMD:Potentiometer_Vishay_TS53YL_Vertical, symbol Device:R_POT
- removed U1601: 74LVC1G17, TO_SOT_Packages_SMD:SOT-353_SC-70-5, symbol Custom_Library:74LVC1G17_Power
- added R?: 10k, Resistors_SMD:R_0402, symbol Custom_Library:R_Custom
- added R?: 100, Resistors_SMD:R_0402, symbol Custom_Library:R_Custom
- added U1601: 74LVC1G97, Package_TO_SOT_SMD:SOT-363_SC-70-6, symbol Custom_Library:74LVC1G97_Power_BUF
- C1601, C1603: Digi-Key PN 490-10701-1-ND -> (none)
- C1602: Digi-Key PN 490-13211-1-ND -> (none)
- R1601, R1602, R1603, R1605, R1606, R1607, R1608, R1609, R1610, R1611, R1612, R1613: Digi-Key PN RMCF0402FT10K0CT-ND -> (none)
- R1604: value 10 -> 0; Digi-Key PN 541-3964-1-ND -> (none)
Connections:
- net +3V3: now also R?.1, U1601.5 (VCC)
- net GND: now also R?.2, U1601.2 (GND), U1601.3 (GND), U1601.6 (GND)
- net LCD_BACKLIGHT: now also R1604.2; no longer R1604.1
- net LCD_BACKLIGHT_PWM: now also U1601.1
- net LCD_CONTRAST: now also R?.1, R?.2
- new net: R1604.1, U1601.4

Commit message: removed more unique components, cleaned up SCH
Parts:
- U1602: footprint Display:NHD-0420H1Z -> (none)
Changed lines of the file:
@@
 F 0 "U1602" H 5340 4670 50  0000 C CNN
 F 1 "NHD-0420H1Z" H 5790 4670 50  0000 L CNN
-F 2 "Display:NHD-0420H1Z" H 5590 3020 50  0001 C CNN
+F 2 "" H 5590 3020 50  0001 C CNN
 F 3 "http://www.newhavendisplay.com/specs/NHD-0420H1Z-FSW-GBW-33V3.pdf" H 5690 3820 50  0001 C CNN
 F 4 "NHD-0420H1Z-FSW-GBW-33V3-ND" H 5590 3920 50  0001 C CNN "Digi-Key PN"

Commit message: annotated schematic
Parts:
- U1601: Digi-Key PN (none) -> 296-SN74LVC1G97DCK3CT-ND
- gave numbers to parts that had none: 2
- renumbered R1603 to R1605, R1604 to R1608, R1608 to R1609, R1609 to R1610, R1610 to R1611, R1605 to R1612, R1611 to R1613, R1612 to R1614, R1613 to R1615

Commit message: changed display sheet to use new LCD
Parts:
- U1602: value NHD-0420H1Z -> Generic 20x04 LCD; footprint (none) -> Custom Footprints Library:20x04_LCD; Digi-Key PN NHD-0420H1Z-FSW-GBW-33V3-ND -> (none)
Changed lines of the file:
@@
 P 5590 3920
 F 0 "U1602" H 5340 4670 50  0000 C CNN
-F 1 "NHD-0420H1Z" H 5790 4670 50  0000 L CNN
-F 2 "" H 5590 3020 50  0001 C CNN
-F 3 "http://www.newhavendisplay.com/specs/NHD-0420H1Z-FSW-GBW-33V3.pdf" H 5690 3820 50  0001 C CNN
-F 4 "NHD-0420H1Z-FSW-GBW-33V3-ND" H 5590 3920 50  0001 C CNN "Digi-Key PN"
+F 1 "Generic 20x04 LCD" H 5790 4670 50  0000 L CNN
+F 2 "Custom Footprints Library:20x04_LCD" H 5590 3020 50  0001 C CNN
+F 3 "" H 5690 3820 50  0001 C CNN
 	1    5590 3920
 	1    0    0    -1

Commit message: assigned digikey PNs
Parts:
- C1601, C1603: Digi-Key PN (none) -> 490-10698-1-ND; Voltage 50V -> 25V
- C1602: Digi-Key PN (none) -> 1276-6830-1-ND; Voltage 6.3V -> 10V
- R1601, R1602, R1604, R1605, R1606, R1607, R1609, R1610, R1611, R1612, R1613, R1614, R1615: Digi-Key PN (none) -> RMCF0402FT10K0CT-ND
- R1603: Digi-Key PN (none) -> RMCF0402FT100RCT-ND
- R1608: Digi-Key PN (none) -> 2019-RK73Z1ETTPCT-ND
Changed lines of the file:
@@
 F 5 "1%" H 2900 6460 50  0000 L CNN "Tolerance"
 F 6 "1/16W" H 2910 6380 50  0000 L CNN "Wattage"
-F 7 "" H 2800 6460 50  0001 C CNN "Digi-Key PN"
+F 7 "RMCF0402FT10K0CT-ND" H 2800 6460 50  0001 C CNN "Digi-Key PN"
 	1    2800 6460
 	1    0    0    -1
@@
 F 3 "" H 3375 7030 50  0001 C CNN
 F 4 "0402" H 3200 7030 50  0000 R CNN "display_footprint"
-F 5 "50V" H 3200 6930 50  0000 R CNN "Voltage"
+F 5 "25V" H 3200 6930 50  0000 R CNN "Voltage"
 F 6 "X7R" H 3200 6830 50  0000 R CNN "Dielectric"
-F 7 "" H 3775 7430 60  0001 C CNN "Digi-Key PN"
+F 7 "490-10698-1-ND" H 3775 7430 60  0001 C CNN "Digi-Key PN"
 	1    3350 6930
 	1    0    0    -1
@@
 F 3 "" H 6895 5150 50  0001 C CNN
 F 4 "0402" H 6720 5150 50  0000 R CNN "display_footprint"
-F 5 "50V" H 6720 5050 50  0000 R CNN "Voltage"
+F 5 "25V" H 6720 5050 50  0000 R CNN "Voltage"
 F 6 "X7R" H 6720 4950 50  0000 R CNN "Dielectric"
-F 7 "" H 2960 -1830 50  0001 C CNN "Digi-Key PN"
+F 7 "490-10698-1-ND" H 2960 -1830 50  0001 C CNN "Digi-Key PN"
 	1    6870 5050
 	1    0    0    -1
@@
 F 3 "" H 6175 5150 50  0001 C CNN
 F 4 "0402" H 6000 5150 50  0000 R CNN "display_footprint"
-F 5 "6.3V" H 6000 5050 50  0000 R CNN "Voltage"
+F 5 "10V" H 6000 5050 50  0000 R CNN "Voltage"
 F 6 "X5R" H 6000 4950 50  0000 R CNN "Dielectric"
-F 7 "" H 6150 5050 50  0001 C CNN "Digi-Key PN"
+F 7 "1276-6830-1-ND" H 6150 5050 50  0001 C CNN "Digi-Key PN"
 	1    6150 5050
 	1    0    0    -1
@@
 F 5 "1%" H 4510 3100 50  0000 L CNN "Tolerance"
 F 6 "1/16W" H 4520 3020 50  0000 L CNN "Wattage"
-F 7 "" H 4410 3100 50  0001 C CNN "Digi-Key PN"
+F 7 "RMCF0402FT10K0CT-ND" H 4410 3100 50  0001 C CNN "Digi-Key PN"
 	1    4410 3100
 	1    0    0    -1
@@
 F 5 "1%" H 3160 4800 50  0001 L CNN "Tolerance"
 F 6 "1/16W" H 3170 4720 50  0001 L CNN "Wattage"
-F 7 "" H 3060 4800 50  0001 C CNN "Digi-Key PN"
+F 7 "RMCF0402FT10K0CT-ND" H 3060 4800 50  0001 C CNN "Digi-Key PN"
 	1    3060 4800
 	1    0    0    -1
@@
 F 5 "1%" H 3360 4800 50  0001 L CNN "Tolerance"
 F 6 "1/16W" H 3370 4720 50  0001 L CNN "Wattage"
-F 7 "" H 3260 4800 50  0001 C CNN "Digi-Key PN"
+F 7 "RMCF0402FT10K0CT-ND" H 3260 4800 50  0001 C CNN "Digi-Key PN"
 	1    3260 4800
 	1    0    0    -1
@@
 F 5 "1%" H 3560 4800 50  0001 L CNN "Tolerance"
 F 6 "1/16W" H 3570 4720 50  0001 L CNN "Wattage"
-F 7 "" H 3460 4800 50  0001 C CNN "Digi-Key PN"
+F 7 "RMCF0402FT10K0CT-ND" H 3460 4800 50  0001 C CNN "Digi-Key PN"
 	1    3460 4800
 	1    0    0    -1
@@
 F 5 "1%" H 3760 4800 50  0001 L CNN "Tolerance"
 F 6 "1/16W" H 3770 4720 50  0001 L CNN "Wattage"
-F 7 "" H 3660 4800 50  0001 C CNN "Digi-Key PN"
+F 7 "RMCF0402FT10K0CT-ND" H 3660 4800 50  0001 C CNN "Digi-Key PN"
 	1    3660 4800
 	1    0    0    -1
@@
 F 5 "1%" H 3960 4800 50  0001 L CNN "Tolerance"
 F 6 "1/16W" H 3970 4720 50  0001 L CNN "Wattage"
-F 7 "" H 3860 4800 50  0001 C CNN "Digi-Key PN"
+F 7 "RMCF0402FT10K0CT-ND" H 3860 4800 50  0001 C CNN "Digi-Key PN"
 	1    3860 4800
 	1    0    0    -1
@@
 F 5 "1%" H 4160 4800 50  0001 L CNN "Tolerance"
 F 6 "1/16W" H 4170 4720 50  0001 L CNN "Wattage"
-F 7 "" H 4060 4800 50  0001 C CNN "Digi-Key PN"
+F 7 "RMCF0402FT10K0CT-ND" H 4060 4800 50  0001 C CNN "Digi-Key PN"
 	1    4060 4800
 	1    0    0    -1
@@
 F 5 "1%" H 4360 4800 50  0001 L CNN "Tolerance"
 F 6 "1/16W" H 4370 4720 50  0001 L CNN "Wattage"
-F 7 "" H 4260 4800 50  0001 C CNN "Digi-Key PN"
+F 7 "RMCF0402FT10K0CT-ND" H 4260 4800 50  0001 C CNN "Digi-Key PN"
 	1    4260 4800
 	1    0    0    -1
@@
 F 5 "1%" H 4560 4800 50  0001 L CNN "Tolerance"
 F 6 "1/16W" H 4570 4720 50  0001 L CNN "Wattage"
-F 7 "" H 4460 4800 50  0001 C CNN "Digi-Key PN"
+F 7 "RMCF0402FT10K0CT-ND" H 4460 4800 50  0001 C CNN "Digi-Key PN"
 	1    4460 4800
 	1    0    0    -1
@@
 F 5 "1%" H 4760 4800 50  0001 L CNN "Tolerance"
 F 6 "1/16W" H 4770 4720 50  0001 L CNN "Wattage"
-F 7 "" H 4660 4800 50  0001 C CNN "Digi-Key PN"
+F 7 "RMCF0402FT10K0CT-ND" H 4660 4800 50  0001 C CNN "Digi-Key PN"
 	1    4660 4800
 	1    0    0    -1
@@
 F 5 "1%" H 4960 4800 50  0001 L CNN "Tolerance"
 F 6 "1/16W" H 4970 4720 50  0001 L CNN "Wattage"
-F 7 "" H 4860 4800 50  0001 C CNN "Digi-Key PN"
+F 7 "RMCF0402FT10K0CT-ND" H 4860 4800 50  0001 C CNN "Digi-Key PN"
 	1    4860 4800
 	1    0    0    -1
@@
 F 5 "1%" V 3930 6230 50  0000 C CNN "Tolerance"
 F 6 "1/16W" V 4030 6230 50  0000 C CNN "Wattage"
+F 7 "2019-RK73Z1ETTPCT-ND" H 3730 6230 50  0001 C CNN "Digi-Key PN"
 	1    3730 6230
 	0    -1   1    0
@@
 F 5 "1%" H 3340 1710 50  0000 L CNN "Tolerance"
 F 6 "1/16W" H 3350 1630 50  0000 L CNN "Wattage"
-F 7 "" H 3240 1710 50  0001 C CNN "Digi-Key PN"
+F 7 "RMCF0402FT10K0CT-ND" H 3240 1710 50  0001 C CNN "Digi-Key PN"
 	1    3240 1710
 	1    0    0    -1
@@
 F 5 "1%" H 3340 1250 50  0000 L CNN "Tolerance"
 F 6 "1/16W" H 3350 1170 50  0000 L CNN "Wattage"
+F 7 "RMCF0402FT100RCT-ND" H 3240 1250 50  0001 C CNN "Digi-Key PN"
 	1    3240 1250
 	1    0    0    -1
