File: hdw/rev_b/Pulse_Oximeter/Display.sch (KiCad schematic (older format))
At the start: 20 parts, among them U1601 74LVC1G97, U1602 Generic 20x04 LCD

Commit message: fixed a few sch issues, more PCB placement
Parts:
- added C1604, C1605: 10uF, Capacitors_SMD:C_0402, symbol Custom_Library:C_Custom
Connections:
- net +3V3: now also C1604.1, C1605.1
- net GND: now also C1604.2, C1605.2
Other:
- moved on the sheet: C1602, C1603
Changed lines of the file:
@@
 L Custom_Library:C_Custom C?
 U 1 1 5EB557B2
-P 6870 5050
+P 8060 5640
 AR Path="/5EAE2F02/5EB557B2" Ref="C?"  Part="1"
 AR Path="/5EAE4A89/5EB557B2" Ref="C1603"  Part="1"
-F 0 "C1603" H 6895 5150 50  0000 L CNN
-F 1 "0.1uF" H 6895 4950 50  0000 L CNN
-F 2 "Capacitors_SMD:C_0402" H 6908 4900 50  0001 C CNN
-F 3 "" H 6895 5150 50  0001 C CNN
-F 4 "0402" H 6720 5150 50  0000 R CNN "display_footprint"
-F 5 "25V" H 6720 5050 50  0000 R CNN "Voltage"
-F 6 "X7R" H 6720 4950 50  0000 R CNN "Dielectric"
-F 7 "490-10698-1-ND" H 2960 -1830 50  0001 C CNN "Digi-Key PN"
-	1    6870 5050
+F 0 "C1603" H 8085 5740 50  0000 L CNN
+F 1 "0.1uF" H 8085 5540 50  0000 L CNN
+F 2 "Capacitors_SMD:C_0402" H 8098 5490 50  0001 C CNN
+F 3 "" H 8085 5740 50  0001 C CNN
+F 4 "0402" H 7910 5740 50  0000 R CNN "display_footprint"
+F 5 "25V" H 7910 5640 50  0000 R CNN "Voltage"
+F 6 "X7R" H 7910 5540 50  0000 R CNN "Dielectric"
+F 7 "490-10698-1-ND" H 4150 -1240 50  0001 C CNN "Digi-Key PN"
+	1    8060 5640
 	1    0    0    -1
 $EndComp
@@
 L power:GND #PWR?
 U 1 1 5EB557DA
-P 6150 5200
+P 7340 5790
 AR Path="/5E0CF7BC/5EB557DA" Ref="#PWR?"  Part="1"
 AR Path="/5CB25152/5EB557DA" Ref="#PWR?"  Part="1"
@@
 AR Path="/5EAE2F02/5EB557DA" Ref="#PWR?"  Part="1"
 AR Path="/5EAE4A89/5EB557DA" Ref="#PWR01623"  Part="1"
-F 0 "#PWR01623" H 6150 4950 50  0001 C CNN
-F 1 "GND" H 6150 5050 50  0000 C CNN
-F 2 "" H 6150 5200 50  0001 C CNN
-F 3 "" H 6150 5200 50  0001 C CNN
-	1    6150 5200
+F 0 "#PWR01623" H 7340 5540 50  0001 C CNN
+F 1 "GND" H 7340 5640 50  0000 C CNN
+F 2 "" H 7340 5790 50  0001 C CNN
+F 3 "" H 7340 5790 50  0001 C CNN
+	1    7340 5790
 	1    0    0    -1
 $EndComp
@@
 L Custom_Library:C_Custom C?
 U 1 1 5EB557E4
-P 6150 5050
+P 7340 5640
 AR Path="/5CB7718D/5EB557E4" Ref="C?"  Part="1"
 AR Path="/5E0DC082/5EB557E4" Ref="C?"  Part="1"
@@
 AR Path="/5EAE2F02/5EB557E4" Ref="C?"  Part="1"
 AR Path="/5EAE4A89/5EB557E4" Ref="C1602"  Part="1"
-F 0 "C1602" H 6175 5150 50  0000 L CNN
-F 1 "10uF" H 6175 4950 50  0000 L CNN
-F 2 "Capacitors_SMD:C_0402" H 6188 4900 50  0001 C CNN
-F 3 "" H 6175 5150 50  0001 C CNN
-F 4 "0402" H 6000 5150 50  0000 R CNN "display_footprint"
-F 5 "10V" H 6000 5050 50  0000 R CNN "Voltage"
-F 6 "X5R" H 6000 4950 50  0000 R CNN "Dielectric"
-F 7 "1276-6830-1-ND" H 6150 5050 50  0001 C CNN "Digi-Key PN"
-	1    6150 5050
+F 0 "C1602" H 7365 5740 50  0000 L CNN
+F 1 "10uF" H 7365 5540 50  0000 L CNN
+F 2 "Capacitors_SMD:C_0402" H 7378 5490 50  0001 C CNN
+F 3 "" H 7365 5740 50  0001 C CNN
+F 4 "0402" H 7190 5740 50  0000 R CNN "display_footprint"
+F 5 "10V" H 7190 5640 50  0000 R CNN "Voltage"
+F 6 "X5R" H 7190 5540 50  0000 R CNN "Dielectric"
+F 7 "1276-6830-1-ND" H 7340 5640 50  0001 C CNN "Digi-Key PN"
+	1    7340 5640
 	1    0    0    -1
 $EndComp
@@
 L power:+3.3V #PWR?
 U 1 1 5EB557EA
-P 6150 4900
+P 7340 5490
 AR Path="/5EAE2F02/5EB557EA" Ref="#PWR?"  Part="1"
 AR Path="/5EAE4A89/5EB557EA" Ref="#PWR01622"  Part="1"
-F 0 "#PWR01622" H 6150 4750 50  0001 C CNN
-F 1 "+3.3V" H 6150 5040 50  0000 C CNN
-F 2 "" H 6150 4900 50  0001 C CNN
-F 3 "" H 6150 4900 50  0001 C CNN
-	1    6150 4900
+F 0 "#PWR01622" H 7340 5340 50  0001 C CNN
+F 1 "+3.3V" H 7340 5630 50  0000 C CNN
+F 2 "" H 7340 5490 50  0001 C CNN
+F 3 "" H 7340 5490 50  0001 C CNN
+	1    7340 5490
 	1    0    0    -1
 $EndComp
@@
 L power:+3.3V #PWR?
 U 1 1 5FE4FA0E
-P 6870 4900
+P 8060 5490
 AR Path="/5EAE2F02/5FE4FA0E" Ref="#PWR?"  Part="1"
 AR Path="/5EAE4A89/5FE4FA0E" Ref="#PWR01624"  Part="1"
-F 0 "#PWR01624" H 6870 4750 50  0001 C CNN
-F 1 "+3.3V" H 6870 5040 50  0000 C CNN
-F 2 "" H 6870 4900 50  0001 C CNN
-F 3 "" H 6870 4900 50  0001 C CNN
-	1    6870 4900
+F 0 "#PWR01624" H 8060 5340 50  0001 C CNN
+F 1 "+3.3V" H 8060 5630 50  0000 C CNN
+F 2 "" H 8060 5490 50  0001 C CNN
+F 3 "" H 8060 5490 50  0001 C CNN
+	1    8060 5490
 	1    0    0    -1
 $EndComp
@@
 L power:GND #PWR?
 U 1 1 5FE4FBCF
-P 6870 5200
+P 8060 5790
 AR Path="/5E0CF7BC/5FE4FBCF" Ref="#PWR?"  Part="1"
 AR Path="/5CB25152/5FE4FBCF" Ref="#PWR?"  Part="1"
@@
 AR Path="/5EAE2F02/5FE4FBCF" Ref="#PWR?"  Part="1"
 AR Path="/5EAE4A89/5FE4FBCF" Ref="#PWR01625"  Part="1"
-F 0 "#PWR01625" H 6870 4950 50  0001 C CNN
-F 1 "GND" H 6870 5050 50  0000 C CNN
-F 2 "" H 6870 5200 50  0001 C CNN
-F 3 "" H 6870 5200 50  0001 C CNN
-	1    6870 5200
+F 0 "#PWR01625" H 8060 5540 50  0001 C CNN
+F 1 "GND" H 8060 5640 50  0000 C CNN
+F 2 "" H 8060 5790 50  0001 C CNN
+F 3 "" H 8060 5790 50  0001 C CNN
+	1    8060 5790
 	1    0    0    -1
 $EndComp
@@
 	1    0    0    -1
 $EndComp
+$Comp
+L power:GND #PWR?
+U 1 1 60025F0D
+P 6620 5790
+AR Path="/5E0CF7BC/60025F0D" Ref="#PWR?"  Part="1"
+AR Path="/5CB25152/60025F0D" Ref="#PWR?"  Part="1"
+AR Path="/5E697934/60025F0D" Ref="#PWR?"  Part="1"
+AR Path="/5EAE2F02/60025F0D" Ref="#PWR?"  Part="1"
+AR Path="/5EAE4A89/60025F0D" Ref="#PWR01629"  Part="1"
+F 0 "#PWR01629" H 6620 5540 50  0001 C CNN
+F 1 "GND" H 6620 5640 50  0000 C CNN
+F 2 "" H 6620 5790 50  0001 C CNN
+F 3 "" H 6620 5790 50  0001 C CNN
+	1    6620 5790
+	1    0    0    -1
+$EndComp
+$Comp
+L Custom_Library:C_Custom C?
+U 1 1 600261F3
+P 6620 5640
+AR Path="/5CB7718D/600261F3" Ref="C?"  Part="1"
+AR Path="/5E0DC082/600261F3" Ref="C?"  Part="1"
+AR Path="/5E0F9110/600261F3" Ref="C?"  Part="1"
+AR Path="/5A557C58/600261F3" Ref="C?"  Part="1"
+AR Path="/5CB25152/600261F3" Ref="C?"  Part="1"
+AR Path="/5E697934/600261F3" Ref="C?"  Part="1"
+AR Path="/5EAE2F02/600261F3" Ref="C?"  Part="1"
+AR Path="/5EAE4A89/600261F3" Ref="C1605"  Part="1"
+F 0 "C1605" H 6645 5740 50  0000 L CNN
+F 1 "10uF" H 6645 5540 50  0000 L CNN
+F 2 "Capacitors_SMD:C_0402" H 6658 5490 50  0001 C CNN
+F 3 "" H 6645 5740 50  0001 C CNN
+F 4 "0402" H 6470 5740 50  0000 R CNN "display_footprint"
+F 5 "10V" H 6470 5640 50  0000 R CNN "Voltage"
+F 6 "X5R" H 6470 5540 50  0000 R CNN "Dielectric"
+F 7 "1276-6830-1-ND" H 6620 5640 50  0001 C CNN "Digi-Key PN"
+	1    6620 5640
+	1    0    0    -1
+$EndComp
+$Comp
+L power:+3.3V #PWR?
+U 1 1 600261FD
+P 6620 5490
+AR Path="/5EAE2F02/600261FD" Ref="#PWR?"  Part="1"
+AR Path="/5EAE4A89/600261FD" Ref="#PWR01628"  Part="1"
+F 0 "#PWR01628" H 6620 5340 50  0001 C CNN
+F 1 "+3.3V" H 6620 5630 50  0000 C CNN
+F 2 "" H 6620 5490 50  0001 C CNN
+F 3 "" H 6620 5490 50  0001 C CNN
+	1    6620 5490
+	1    0    0    -1
+$EndComp
+$Comp
+L power:GND #PWR?
+U 1 1 60028138
+P 5900 5790
+AR Path="/5E0CF7BC/60028138" Ref="#PWR?"  Part="1"
+AR Path="/5CB25152/60028138" Ref="#PWR?"  Part="1"
+AR Path="/5E697934/60028138" Ref="#PWR?"  Part="1"
+AR Path="/5EAE2F02/60028138" Ref="#PWR?"  Part="1"
+AR Path="/5EAE4A89/60028138" Ref="#PWR01627"  Part="1"
+F 0 "#PWR01627" H 5900 5540 50  0001 C CNN
+F 1 "GND" H 5900 5640 50  0000 C CNN
+F 2 "" H 5900 5790 50  0001 C CNN
+F 3 "" H 5900 5790 50  0001 C CNN
+	1    5900 5790
+	1    0    0    -1
+$EndComp
+$Comp
+L Custom_Library:C_Custom C?
+U 1 1 6002844E
+P 5900 5640
+AR Path="/5CB7718D/6002844E" Ref="C?"  Part="1"
+AR Path="/5E0DC082/6002844E" Ref="C?"  Part="1"
+AR Path="/5E0F9110/6002844E" Ref="C?"  Part="1"
+AR Path="/5A557C58/6002844E" Ref="C?"  Part="1"
+AR Path="/5CB25152/6002844E" Ref="C?"  Part="1"
+AR Path="/5E697934/6002844E" Ref="C?"  Part="1"
+AR Path="/5EAE2F02/6002844E" Ref="C?"  Part="1"
+AR Path="/5EAE4A89/6002844E" Ref="C1604"  Part="1"
+F 0 "C1604" H 5925 5740 50  0000 L CNN
+F 1 "10uF" H 5925 5540 50  0000 L CNN
+F 2 "Capacitors_SMD:C_0402" H 5938 5490 50  0001 C CNN
+F 3 "" H 5925 5740 50  0001 C CNN
+F 4 "0402" H 5750 5740 50  0000 R CNN "display_footprint"
+F 5 "10V" H 5750 5640 50  0000 R CNN "Voltage"
+F 6 "X5R" H 5750 5540 50  0000 R CNN "Dielectric"
+F 7 "1276-6830-1-ND" H 5900 5640 50  0001 C CNN "Digi-Key PN"
+	1    5900 5640
+	1    0    0    -1
+$EndComp
+$Comp
+L power:+3.3V #PWR?
+U 1 1 60028458
+P 5900 5490
+AR Path="/5EAE2F02/60028458" Ref="#PWR?"  Part="1"
+AR Path="/5EAE4A89/60028458" Ref="#PWR01626"  Part="1"
+F 0 "#PWR01626" H 5900 5340 50  0001 C CNN
+F 1 "+3.3V" H 5900 5630 50  0000 C CNN
+F 2 "" H 5900 5490 50  0001 C CNN
+F 3 "" H 5900 5490 50  0001 C CNN
+	1    5900 5490
+	1    0    0    -1
+$EndComp
