File: hdw/rev_b/Pulse_Oximeter/Mechanical.sch (KiCad schematic (older format))
At the start: 12 parts

Commit message: annotated schematic
Parts:
- renumbered H2301 to H2101, H2302 to H2102, H2303 to H2103, H2304 to H2104, MK2301 to MK2101, MK2302 to MK2102, MK2303 to MK2103, MK2304 to MK2104, MK2305 to MK2105, MK2306 to MK2106, MK2307 to MK2107, MK2308 to MK2108
Changed lines of the file:
@@
 $EndDescr
 $Comp
-L Mechanical:MountingHole H2301
+L Mechanical:MountingHole H2101
 U 1 1 5CC525BF
 P 4070 1580
-F 0 "H2301" H 4070 1780 50  0000 C CNN
+F 0 "H2101" H 4070 1780 50  0000 C CNN
 F 1 "MountingHole" H 4070 1705 50  0000 C CNN
 F 2 "MountingHole:MountingHole_3mm" H 4070 1580 50  0001 C CNN
@@
 $EndComp
 $Comp
-L Mechanical:MountingHole H2303
+L Mechanical:MountingHole H2103
 U 1 1 5CC5295F
 P 4820 1580
-F 0 "H2303" H 4820 1780 50  0000 C CNN
+F 0 "H2103" H 4820 1780 50  0000 C CNN
 F 1 "MountingHole" H 4820 1705 50  0000 C CNN
 F 2 "MountingHole:MountingHole_3mm" H 4820 1580 50  0001 C CNN
@@
 $EndComp
 $Comp
-L Mechanical:MountingHole H2302
+L Mechanical:MountingHole H2102
 U 1 1 5CC53950
 P 4070 2080
-F 0 "H2302" H 4070 2280 50  0000 C CNN
+F 0 "H2102" H 4070 2280 50  0000 C CNN
 F 1 "MountingHole" H 4070 2205 50  0000 C CNN
 F 2 "MountingHole:MountingHole_3mm" H 4070 2080 50  0001 C CNN
@@
 $EndComp
 $Comp
-L Mechanical:MountingHole H2304
+L Mechanical:MountingHole H2104
 U 1 1 5CC5395A
 P 4820 2080
-F 0 "H2304" H 4820 2280 50  0000 C CNN
+F 0 "H2104" H 4820 2280 50  0000 C CNN
 F 1 "MountingHole" H 4820 2205 50  0000 C CNN
 F 2 "MountingHole:MountingHole_3mm" H 4820 2080 50  0001 C CNN
@@
 $EndComp
 $Comp
-L Custom_Library:Standoff MK2301
+L Custom_Library:Standoff MK2101
 U 1 1 5CC60957
 P 4070 3560
-F 0 "MK2301" H 4070 3710 50  0000 C CNN
+F 0 "MK2101" H 4070 3710 50  0000 C CNN
 F 1 "Standoff" H 4070 3810 50  0000 C CNN
 F 2 "" H 4070 3910 50  0001 C CNN
@@
 $EndComp
 $Comp
-L Custom_Library:Standoff MK2305
+L Custom_Library:Standoff MK2105
 U 1 1 5CC60961
 P 4820 3560
-F 0 "MK2305" H 4820 3710 50  0000 C CNN
+F 0 "MK2105" H 4820 3710 50  0000 C CNN
 F 1 "Standoff" H 4820 3810 50  0000 C CNN
 F 2 "" H 4820 3910 50  0001 C CNN
@@
 $EndComp
 $Comp
-L Custom_Library:Standoff MK2302
+L Custom_Library:Standoff MK2102
 U 1 1 5CC6097F
 P 4070 4060
-F 0 "MK2302" H 4070 4210 50  0000 C CNN
+F 0 "MK2102" H 4070 4210 50  0000 C CNN
 F 1 "Standoff" H 4070 4310 50  0000 C CNN
 F 2 "" H 4070 4410 50  0001 C CNN
@@
 $EndComp
 $Comp
-L Custom_Library:Standoff MK2306
+L Custom_Library:Standoff MK2106
 U 1 1 5CC60989
 P 4820 4060
-F 0 "MK2306" H 4820 4210 50  0000 C CNN
+F 0 "MK2106" H 4820 4210 50  0000 C CNN
 F 1 "Standoff" H 4820 4310 50  0000 C CNN
 F 2 "" H 4820 4410 50  0001 C CNN
@@
 $EndComp
 $Comp
-L Custom_Library:Screw MK2303
+L Custom_Library:Screw MK2103
 U 1 1 5CC6CBF3
 P 4070 5670
-F 0 "MK2303" H 4070 5770 50  0000 C CNN
+F 0 "MK2103" H 4070 5770 50  0000 C CNN
 F 1 "Screw" H 4070 5870 50  0000 C CNN
 F 2 "" H 4070 5920 50  0001 C CNN
@@
 $EndComp
 $Comp
-L Custom_Library:Screw MK2307
+L Custom_Library:Screw MK2107
 U 1 1 5CC6D1A5
 P 4820 5670
-F 0 "MK2307" H 4820 5770 50  0000 C CNN
+F 0 "MK2107" H 4820 5770 50  0000 C CNN
 F 1 "Screw" H 4820 5870 50  0000 C CNN
 F 2 "" H 4820 5920 50  0001 C CNN
@@
 $EndComp
 $Comp
-L Custom_Library:Screw MK2304
+L Custom_Library:Screw MK2104
 U 1 1 5CC70A99
 P 4070 6170
-F 0 "MK2304" H 4070 6270 50  0000 C CNN
+F 0 "MK2104" H 4070 6270 50  0000 C CNN
 F 1 "Screw" H 4070 6370 50  0000 C CNN
 F 2 "" H 4070 6420 50  0001 C CNN
@@
 $EndComp
 $Comp
-L Custom_Library:Screw MK2308
+L Custom_Library:Screw MK2108
 U 1 1 5CC70AA3
 P 4820 6170
-F 0 "MK2308" H 4820 6270 50  0000 C CNN
+F 0 "MK2108" H 4820 6270 50  0000 C CNN
 F 1 "Screw" H 4820 6370 50  0000 C CNN
 F 2 "" H 4820 6420 50  0001 C CNN

Commit message: assigned digikey PNs
Parts:
- MK2101, MK2102, MK2105, MK2106: Digi-Key PN 1772-1220-ND -> 1772-1910-ND
Changed lines of the file:
@@
 F 2 "" H 4070 3910 50  0001 C CNN
 F 3 "" H 4070 3910 50  0001 C CNN
-F 4 "1772-1220-ND" H 4070 3560 50  0001 C CNN "Digi-Key PN"
+F 4 "1772-1910-ND" H 4070 3560 50  0001 C CNN "Digi-Key PN"
 	1    4070 3560
 	1    0    0    -1
@@
 F 2 "" H 4820 3910 50  0001 C CNN
 F 3 "" H 4820 3910 50  0001 C CNN
-F 4 "1772-1220-ND" H 4820 3560 50  0001 C CNN "Digi-Key PN"
+F 4 "1772-1910-ND" H 4820 3560 50  0001 C CNN "Digi-Key PN"
 	1    4820 3560
 	1    0    0    -1
@@
 F 2 "" H 4070 4410 50  0001 C CNN
 F 3 "" H 4070 4410 50  0001 C CNN
-F 4 "1772-1220-ND" H 4070 4060 50  0001 C CNN "Digi-Key PN"
+F 4 "1772-1910-ND" H 4070 4060 50  0001 C CNN "Digi-Key PN"
 	1    4070 4060
 	1    0    0    -1
@@
 F 2 "" H 4820 4410 50  0001 C CNN
 F 3 "" H 4820 4410 50  0001 C CNN
-F 4 "1772-1220-ND" H 4820 4060 50  0001 C CNN "Digi-Key PN"
+F 4 "1772-1910-ND" H 4820 4060 50  0001 C CNN "Digi-Key PN"
 	1    4820 4060
 	1    0    0    -1
