File: hdw/rev_b/Pulse_Oximeter/Misc_Circuits.sch (KiCad schematic (older format))
At the start: 7 parts, among them J2001 I2C, J2002 USB UART, U2001 MCP9804

Commit message: fixed some component configurations in sch, regenerated netlist
Parts:
- C2001: Configuration (none) -> Telemetry; display_footprint (none) -> 0402
Changed lines of the file:
@@
 Sheet 20 21
 Title "Pulse Oximeter"
-Date "2020-08-01"
-Rev "A"
+Date "2020-12-09"
+Rev "B"
 Comp "Drew Maatman"
 Comment1 ""
@@
 I2C_SDA
 NoConn ~ 4800 2240
-$Comp
-L Custom_Library:C_Custom C?
-U 1 1 5EBEF932
-P 5200 3390
-AR Path="/5B3E071A/5EBEF932" Ref="C?"  Part="1"
-AR Path="/5E0652BA/5EBEF932" Ref="C?"  Part="1"
-AR Path="/5E0A0E29/5EBEF932" Ref="C?"  Part="1"
-AR Path="/5E0DC084/5EBEF932" Ref="C?"  Part="1"
-AR Path="/5E0F263C/5EBEF932" Ref="C?"  Part="1"
-AR Path="/5EAE2E6F/5EBEF932" Ref="C?"  Part="1"
-AR Path="/5EBEB0C5/5EBEF932" Ref="C2001"  Part="1"
-F 0 "C2001" H 5225 3490 50  0000 L CNN
-F 1 "0.1uF" H 5225 3290 50  0000 L CNN
-F 2 "Capacitors_SMD:C_0402" H 5238 3240 50  0001 C CNN
-F 3 "" H 5225 3490 50  0001 C CNN
-F 4 "" H 5050 3490 50  0000 R CNN "display_footprint"
-F 5 "50V" H 5050 3390 50  0000 R CNN "Voltage"
-F 6 "X7R" H 5050 3290 50  0000 R CNN "Dielectric"
-F 7 "490-10701-1-ND" H 1290 -3490 50  0001 C CNN "Digi-Key PN"
-	1    5200 3390
-	1    0    0    -1
-$EndComp
 $Comp
 L power:+3.3V #PWR?
@@
 	1    0    0    -1
 $EndComp
+$Comp
+L Custom_Library:C_Custom C?
+U 1 1 5FD3C87C
+P 5200 3390
+AR Path="/5B3E071A/5FD3C87C" Ref="C?"  Part="1"
+AR Path="/5E0652BA/5FD3C87C" Ref="C?"  Part="1"
+AR Path="/5E0A0E29/5FD3C87C" Ref="C?"  Part="1"
+AR Path="/5E052856/5FD3C87C" Ref="C?"  Part="1"
+AR Path="/5EAE2D84/5FD3C87C" Ref="C?"  Part="1"
+AR Path="/5EBEB0C5/5FD3C87C" Ref="C2001"  Part="1"
+F 0 "C2001" H 5225 3490 50  0000 L CNN
+F 1 "0.1uF" H 5225 3290 50  0000 L CNN
+F 2 "Capacitors_SMD:C_0402" H 5238 3240 50  0001 C CNN
+F 3 "" H 5225 3490 50  0001 C CNN
+F 4 "0402" H 5050 3490 50  0000 R CNN "display_footprint"
+F 5 "50V" H 5050 3390 50  0000 R CNN "Voltage"
+F 6 "X7R" H 5050 3290 50  0000 R CNN "Dielectric"
+F 7 "490-10701-1-ND" H 1290 -3490 50  0001 C CNN "Digi-Key PN"
+F 8 "Telemetry" H 4670 3390 50  0000 C CNN "Configuration"
+	1    5200 3390
+	1    0    0    -1
+$EndComp

Commit message: lots of rev b changes
Parts:
- added R?: 10k, Resistors_SMD:R_0402, symbol Custom_Library:R_Custom
- added R?: 10, Resistors_SMD:R_0402, symbol Custom_Library:R_Custom
Connections:
- net +3V3: now also R?.1
- net GND: now also R?.2
- net Telemetry_Config renamed ~Telemetry_Config
- new net ~ETC_Config: R?.1, R?.2
Changed lines of the file:
@@
 	5570 5240 5570 5160
 Text GLabel 5650 5160 2    50   UnSpc ~ 0
-Telemetry_Config
+~Telemetry_Config
 Wire Wire Line
 	5650 5160 5570 5160
@@
 	1    0    0    -1
 $EndComp
+$Comp
+L Custom_Library:R_Custom R?
+U 1 1 5FDF0D57
+P 6770 4930
+AR Path="/5BB27BA3/5FDF0D57" Ref="R?"  Part="1"
+AR Path="/5BB27BF7/5FDF0D57" Ref="R?"  Part="1"
+AR Path="/5C1DE17A/5FDF0D57" Ref="R?"  Part="1"
+AR Path="/5C1E3A08/5FDF0D57" Ref="R?"  Part="1"
+AR Path="/5D779AE1/5FDF0D57" Ref="R?"  Part="1"
+AR Path="/5CB7718D/5FDF0D57" Ref="R?"  Part="1"
+AR Path="/5E0DC082/5FDF0D57" Ref="R?"  Part="1"
+AR Path="/5E0F9110/5FDF0D57" Ref="R?"  Part="1"
+AR Path="/5E9E0EA5/5FDF0D57" Ref="R?"  Part="1"
+AR Path="/5E9E0E87/5FDF0D57" Ref="R?"  Part="1"
+AR Path="/5EAE2D66/5FDF0D57" Ref="R?"  Part="1"
+AR Path="/5EAE4A89/5FDF0D57" Ref="R?"  Part="1"
+AR Path="/5EAE2F23/5FDF0D57" Ref="R?"  Part="1"
+AR Path="/5EBEB0C5/5FDF0D57" Ref="R?"  Part="1"
+F 0 "R?" H 6690 4930 50  0000 R CNN
+F 1 "10k" V 6770 4930 50  0000 C CNN
+F 2 "Resistors_SMD:R_0402" H 6770 4930 50  0001 C CNN
+F 3 "" H 6770 4930 50  0001 C CNN
+F 4 "0402" H 6870 5010 50  0000 L CNN "display_footprint"
+F 5 "1%" H 6870 4930 50  0000 L CNN "Tolerance"
+F 6 "1/16W" H 6880 4850 50  0000 L CNN "Wattage"
+F 7 "RMCF0402FT10K0CT-ND" H 6770 4930 50  0001 C CNN "Digi-Key PN"
+	1    6770 4930
+	1    0    0    -1
+$EndComp
+$Comp
+L power:+3.3V #PWR?
+U 1 1 5FDF0E95
+P 6770 4780
+F 0 "#PWR?" H 6770 4630 50  0001 C CNN
+F 1 "+3.3V" H 6770 4920 50  0000 C CNN
+F 2 "" H 6770 4780 50  0001 C CNN
+F 3 "" H 6770 4780 50  0001 C CNN
+	1    6770 4780
+	1    0    0    -1
+$EndComp
+$Comp
+L power:GND #PWR?
+U 1 1 5FDF0E9F
+P 6770 5540
+F 0 "#PWR?" H 6770 5290 50  0001 C CNN
+F 1 "GND" H 6770 5390 50  0000 C CNN
+F 2 "" H 6770 5540 50  0001 C CNN
+F 3 "" H 6770 5540 50  0001 C CNN
+	1    6770 5540
+	1    0    0    -1
+$EndComp
+Wire Wire Line
+	6770 5240 6770 5160
+Text GLabel 6850 5160 2    50   UnSpc ~ 0
+~ETC_Config
+Wire Wire Line
+	6850 5160 6770 5160
+Connection ~ 6770 5160
+Wire Wire Line
+	6770 5160 6770 5080
+$Comp
+L Custom_Library:R_Custom R?
+U 1 1 5FDF0EB3
+P 6770 5390
+AR Path="/5BB27BA3/5FDF0EB3" Ref="R?"  Part="1"
+AR Path="/5BB27BF7/5FDF0EB3" Ref="R?"  Part="1"
+AR Path="/5C1DE17A/5FDF0EB3" Ref="R?"  Part="1"
+AR Path="/5C1E3A08/5FDF0EB3" Ref="R?"  Part="1"
+AR Path="/5D779AE1/5FDF0EB3" Ref="R?"  Part="1"
+AR Path="/5CB7718D/5FDF0EB3" Ref="R?"  Part="1"
+AR Path="/5E0DC082/5FDF0EB3" Ref="R?"  Part="1"
+AR Path="/5E0F9110/5FDF0EB3" Ref="R?"  Part="1"
+AR Path="/5E9E0EA5/5FDF0EB3" Ref="R?"  Part="1"
+AR Path="/5E9E0E87/5FDF0EB3" Ref="R?"  Part="1"
+AR Path="/5EAE2D66/5FDF0EB3" Ref="R?"  Part="1"
+AR Path="/5EAE4A89/5FDF0EB3" Ref="R?"  Part="1"
+AR Path="/5EAE2F23/5FDF0EB3" Ref="R?"  Part="1"
+AR Path="/5EBEB0C5/5FDF0EB3" Ref="R?"  Part="1"
+F 0 "R?" H 6690 5390 50  0000 R CNN
+F 1 "10" V 6770 5390 50  0000 C CNN
+F 2 "Resistors_SMD:R_0402" H 6770 5390 50  0001 C CNN
+F 3 "" H 6770 5390 50  0001 C CNN
+F 4 "0402" H 6870 5470 50  0000 L CNN "display_footprint"
+F 5 "1%" H 6870 5390 50  0000 L CNN "Tolerance"
+F 6 "1/16W" H 6880 5310 50  0000 L CNN "Wattage"
+F 7 "ETC" H 6880 5230 50  0000 L CNN "Configuration"
+F 8 "541-3964-1-ND" H 6770 5390 50  0001 C CNN "Digi-Key PN"
+	1    6770 5390
+	1    0    0    -1
+$EndComp

Commit message: changed all passives to 0402, cleared digikey pns
Parts:
- C2001: Digi-Key PN 490-10701-1-ND -> (none)
- R2001, R?: Digi-Key PN RMCF0402FT10K0CT-ND -> (none)
- R2002, R?: Digi-Key PN 541-3964-1-ND -> (none)
Changed lines of the file:
@@
 F 5 "1%" H 5670 4930 50  0000 L CNN "Tolerance"
 F 6 "1/16W" H 5680 4850 50  0000 L CNN "Wattage"
-F 7 "RMCF0402FT10K0CT-ND" H 5570 4930 50  0001 C CNN "Digi-Key PN"
+F 7 "" H 5570 4930 50  0001 C CNN "Digi-Key PN"
 	1    5570 4930
 	1    0    0    -1
@@
 F 6 "1/16W" H 5680 5310 50  0000 L CNN "Wattage"
 F 7 "Telemetry" H 5680 5230 50  0000 L CNN "Configuration"
-F 8 "541-3964-1-ND" H 5570 5390 50  0001 C CNN "Digi-Key PN"
+F 8 "" H 5570 5390 50  0001 C CNN "Digi-Key PN"
 	1    5570 5390
 	1    0    0    -1
@@
 F 5 "50V" H 5050 3390 50  0000 R CNN "Voltage"
 F 6 "X7R" H 5050 3290 50  0000 R CNN "Dielectric"
-F 7 "490-10701-1-ND" H 1290 -3490 50  0001 C CNN "Digi-Key PN"
+F 7 "" H 1290 -3490 50  0001 C CNN "Digi-Key PN"
 F 8 "Telemetry" H 4670 3390 50  0000 C CNN "Configuration"
 	1    5200 3390
@@
 F 5 "1%" H 6870 4930 50  0000 L CNN "Tolerance"
 F 6 "1/16W" H 6880 4850 50  0000 L CNN "Wattage"
-F 7 "RMCF0402FT10K0CT-ND" H 6770 4930 50  0001 C CNN "Digi-Key PN"
+F 7 "" H 6770 4930 50  0001 C CNN "Digi-Key PN"
 	1    6770 4930
 	1    0    0    -1
@@
 F 6 "1/16W" H 6880 5310 50  0000 L CNN "Wattage"
 F 7 "ETC" H 6880 5230 50  0000 L CNN "Configuration"
-F 8 "541-3964-1-ND" H 6770 5390 50  0001 C CNN "Digi-Key PN"
+F 8 "" H 6770 5390 50  0001 C CNN "Digi-Key PN"
 	1    6770 5390
 	1    0    0    -1

Commit message: few little tweaks
Parts:
- added C?: 0.1uF, Capacitors_SMD:C_0402, symbol Custom_Library:C_Custom
- added U?: LTC1694, Package_TO_SOT_SMD:SOT-23-5, symbol Custom_Library:LTC1694
Connections:
- net +3V3: now also C?.1, U?.1 (VCC)
- net GND: now also C?.2, U?.2 (GND)
- net I2C_SCL: now also U?.4 (SMBUS2)
- net I2C_SDA: now also U?.5 (SMBUS1)
Other:
- note added: "Ambient Temp Sense"
- moved on the sheet: C2001, J2001, J2002, U2001

Commit message: annotated schematic
Parts:
- gave numbers to parts that had none: 4
Changed lines of the file:
@@
 $EndComp
 $Comp
-L power:+3.3V #PWR02007
+L power:+3.3V #PWR02010
 U 1 1 5EBF5632
 P 5570 4780
-F 0 "#PWR02007" H 5570 4630 50  0001 C CNN
+F 0 "#PWR02010" H 5570 4630 50  0001 C CNN
 F 1 "+3.3V" H 5570 4920 50  0000 C CNN
 F 2 "" H 5570 4780 50  0001 C CNN
@@
 $EndComp
 $Comp
-L power:GND #PWR02008
+L power:GND #PWR02011
 U 1 1 5EBF5638
 P 5570 5540
-F 0 "#PWR02008" H 5570 5290 50  0001 C CNN
+F 0 "#PWR02011" H 5570 5290 50  0001 C CNN
 F 1 "GND" H 5570 5390 50  0000 C CNN
 F 2 "" H 5570 5540 50  0001 C CNN
@@
 P 4180 2450
 AR Path="/5EAE2DDC/5EC3C1CD" Ref="#PWR?"  Part="1"
-AR Path="/5EBEB0C5/5EC3C1CD" Ref="#PWR02010"  Part="1"
-F 0 "#PWR02010" H 4180 2200 50  0001 C CNN
+AR Path="/5EBEB0C5/5EC3C1CD" Ref="#PWR02008"  Part="1"
+F 0 "#PWR02008" H 4180 2200 50  0001 C CNN
 F 1 "GND" V 4180 2300 50  0000 R CNN
 F 2 "" H 4180 2450 50  0001 C CNN
@@
 AR Path="/5EAE2E6F/5EC3C1D3" Ref="#PWR?"  Part="1"
 AR Path="/5EAE2FAC/5EC3C1D3" Ref="#PWR?"  Part="1"
-AR Path="/5EBEB0C5/5EC3C1D3" Ref="#PWR02011"  Part="1"
-F 0 "#PWR02011" H 4180 2400 50  0001 C CNN
+AR Path="/5EBEB0C5/5EC3C1D3" Ref="#PWR02009"  Part="1"
+F 0 "#PWR02009" H 4180 2400 50  0001 C CNN
 F 1 "+3.3V" V 4180 2690 50  0000 L CNN
 F 2 "" H 4180 2550 50  0001 C CNN
@@
 P 4180 2350
 AR Path="/5EAE2DDC/5EC3C90F" Ref="#PWR?"  Part="1"
-AR Path="/5EBEB0C5/5EC3C90F" Ref="#PWR02009"  Part="1"
-F 0 "#PWR02009" H 4180 2100 50  0001 C CNN
+AR Path="/5EBEB0C5/5EC3C90F" Ref="#PWR02007"  Part="1"
+F 0 "#PWR02007" H 4180 2100 50  0001 C CNN
 F 1 "GND" V 4180 2200 50  0000 R CNN
 F 2 "" H 4180 2350 50  0001 C CNN
@@
 AR Path="/5EAE4A89/5FDF0D57" Ref="R?"  Part="1"
 AR Path="/5EAE2F23/5FDF0D57" Ref="R?"  Part="1"
-AR Path="/5EBEB0C5/5FDF0D57" Ref="R?"  Part="1"
-F 0 "R?" H 6690 4930 50  0000 R CNN
+AR Path="/5EBEB0C5/5FDF0D57" Ref="R2003"  Part="1"
+F 0 "R2003" H 6690 4930 50  0000 R CNN
 F 1 "10k" V 6770 4930 50  0000 C CNN
 F 2 "Resistors_SMD:R_0402" H 6770 4930 50  0001 C CNN
@@
 $EndComp
 $Comp
-L power:+3.3V #PWR?
+L power:+3.3V #PWR02016
 U 1 1 5FDF0E95
 P 6770 4780
-F 0 "#PWR?" H 6770 4630 50  0001 C CNN
+F 0 "#PWR02016" H 6770 4630 50  0001 C CNN
 F 1 "+3.3V" H 6770 4920 50  0000 C CNN
 F 2 "" H 6770 4780 50  0001 C CNN
@@
 $EndComp
 $Comp
-L power:GND #PWR?
+L power:GND #PWR02017
 U 1 1 5FDF0E9F
 P 6770 5540
-F 0 "#PWR?" H 6770 5290 50  0001 C CNN
+F 0 "#PWR02017" H 6770 5290 50  0001 C CNN
 F 1 "GND" H 6770 5390 50  0000 C CNN
 F 2 "" H 6770 5540 50  0001 C CNN
@@
 AR Path="/5EAE4A89/5FDF0EB3" Ref="R?"  Part="1"
 AR Path="/5EAE2F23/5FDF0EB3" Ref="R?"  Part="1"
-AR Path="/5EBEB0C5/5FDF0EB3" Ref="R?"  Part="1"
-F 0 "R?" H 6690 5390 50  0000 R CNN
+AR Path="/5EBEB0C5/5FDF0EB3" Ref="R2004"  Part="1"
+F 0 "R2004" H 6690 5390 50  0000 R CNN
 F 1 "10" V 6770 5390 50  0000 C CNN
 F 2 "Resistors_SMD:R_0402" H 6770 5390 50  0001 C CNN
@@
 $EndComp
 $Comp
-L Custom_Library:LTC1694 U?
+L Custom_Library:LTC1694 U2002
 U 1 1 5FE9D912
 P 6760 2250
-F 0 "U?" H 6760 1900 50  0000 C CNN
+F 0 "U2002" H 6760 1900 50  0000 C CNN
 F 1 "LTC1694" H 6760 2600 50  0000 C CNN
 F 2 "Package_TO_SOT_SMD:SOT-23-5" H 6660 2550 60  0001 C CNN
@@
 AR Path="/5E0F263C/5FEA0F23" Ref="#PWR?"  Part="1"
 AR Path="/5EAE2E6F/5FEA0F23" Ref="#PWR?"  Part="1"
-AR Path="/5EBEB0C5/5FEA0F23" Ref="#PWR?"  Part="1"
-F 0 "#PWR?" H 6740 2860 50  0001 C CNN
+AR Path="/5EBEB0C5/5FEA0F23" Ref="#PWR02014"  Part="1"
+F 0 "#PWR02014" H 6740 2860 50  0001 C CNN
 F 1 "+3.3V" H 6740 3150 50  0000 C CNN
 F 2 "" H 6740 3010 50  0001 C CNN
@@
 AR Path="/5E0F263C/5FEA0F29" Ref="#PWR?"  Part="1"
 AR Path="/5EAE2E6F/5FEA0F29" Ref="#PWR?"  Part="1"
-AR Path="/5EBEB0C5/5FEA0F29" Ref="#PWR?"  Part="1"
-F 0 "#PWR?" H 6740 3060 50  0001 C CNN
+AR Path="/5EBEB0C5/5FEA0F29" Ref="#PWR02015"  Part="1"
+F 0 "#PWR02015" H 6740 3060 50  0001 C CNN
 F 1 "GND" H 6740 3160 50  0000 C CNN
 F 2 "" H 6740 3310 50  0001 C CNN
@@
 AR Path="/5E052856/5FEA0F34" Ref="C?"  Part="1"
 AR Path="/5EAE2D84/5FEA0F34" Ref="C?"  Part="1"
-AR Path="/5EBEB0C5/5FEA0F34" Ref="C?"  Part="1"
-F 0 "C?" H 6765 3260 50  0000 L CNN
+AR Path="/5EBEB0C5/5FEA0F34" Ref="C2002"  Part="1"
+F 0 "C2002" H 6765 3260 50  0000 L CNN
 F 1 "0.1uF" H 6765 3060 50  0000 L CNN
 F 2 "Capacitors_SMD:C_0402" H 6778 3010 50  0001 C CNN
@@
 AR Path="/5E0F263C/5FEA152A" Ref="#PWR?"  Part="1"
 AR Path="/5EAE2E6F/5FEA152A" Ref="#PWR?"  Part="1"
-AR Path="/5EBEB0C5/5FEA152A" Ref="#PWR?"  Part="1"
-F 0 "#PWR?" H 6280 2280 50  0001 C CNN
+AR Path="/5EBEB0C5/5FEA152A" Ref="#PWR02013"  Part="1"
+F 0 "#PWR02013" H 6280 2280 50  0001 C CNN
 F 1 "GND" H 6280 2380 50  0000 C CNN
 F 2 "" H 6280 2530 50  0001 C CNN
@@
 AR Path="/5E0F263C/5FEA177A" Ref="#PWR?"  Part="1"
 AR Path="/5EAE2E6F/5FEA177A" Ref="#PWR?"  Part="1"
-AR Path="/5EBEB0C5/5FEA177A" Ref="#PWR?"  Part="1"
-F 0 "#PWR?" H 6280 1820 50  0001 C CNN
+AR Path="/5EBEB0C5/5FEA177A" Ref="#PWR02012"  Part="1"
+F 0 "#PWR02012" H 6280 1820 50  0001 C CNN
 F 1 "+3.3V" H 6280 2110 50  0000 C CNN
 F 2 "" H 6280 1970 50  0001 C CNN

Commit message: assigned digikey PNs
Parts:
- C2001, C2002: Digi-Key PN (none) -> 490-10698-1-ND; Voltage 50V -> 25V
- R2001, R2003: Digi-Key PN (none) -> RMCF0402FT10K0CT-ND
- R2002, R2004: Digi-Key PN (none) -> RMCF0402FT10R0CT-ND
Changed lines of the file:
@@
 F 5 "1%" H 5670 4930 50  0000 L CNN "Tolerance"
 F 6 "1/16W" H 5680 4850 50  0000 L CNN "Wattage"
-F 7 "" H 5570 4930 50  0001 C CNN "Digi-Key PN"
+F 7 "RMCF0402FT10K0CT-ND" H 5570 4930 50  0001 C CNN "Digi-Key PN"
 	1    5570 4930
 	1    0    0    -1
@@
 F 6 "1/16W" H 5680 5310 50  0000 L CNN "Wattage"
 F 7 "Telemetry" H 5680 5230 50  0000 L CNN "Configuration"
-F 8 "" H 5570 5390 50  0001 C CNN "Digi-Key PN"
+F 8 "RMCF0402FT10R0CT-ND" H 5570 5390 50  0001 C CNN "Digi-Key PN"
 	1    5570 5390
 	1    0    0    -1
@@
 F 3 "" H 3805 3500 50  0001 C CNN
 F 4 "0402" H 3630 3500 50  0000 R CNN "display_footprint"
-F 5 "50V" H 3630 3400 50  0000 R CNN "Voltage"
+F 5 "25V" H 3630 3400 50  0000 R CNN "Voltage"
 F 6 "X7R" H 3630 3300 50  0000 R CNN "Dielectric"
-F 7 "" H -130 -3480 50  0001 C CNN "Digi-Key PN"
+F 7 "490-10698-1-ND" H -130 -3480 50  0001 C CNN "Digi-Key PN"
 F 8 "Telemetry" H 3250 3400 50  0000 C CNN "Configuration"
 	1    3780 3400
@@
 F 5 "1%" H 6870 4930 50  0000 L CNN "Tolerance"
 F 6 "1/16W" H 6880 4850 50  0000 L CNN "Wattage"
-F 7 "" H 6770 4930 50  0001 C CNN "Digi-Key PN"
+F 7 "RMCF0402FT10K0CT-ND" H 6770 4930 50  0001 C CNN "Digi-Key PN"
 	1    6770 4930
 	1    0    0    -1
@@
 F 6 "1/16W" H 6880 5310 50  0000 L CNN "Wattage"
 F 7 "ETC" H 6880 5230 50  0000 L CNN "Configuration"
-F 8 "" H 6770 5390 50  0001 C CNN "Digi-Key PN"
+F 8 "RMCF0402FT10R0CT-ND" H 6770 5390 50  0001 C CNN "Digi-Key PN"
 	1    6770 5390
 	1    0    0    -1
@@
 F 3 "" H 6765 3260 50  0001 C CNN
 F 4 "0402" H 6590 3260 50  0000 R CNN "display_footprint"
-F 5 "50V" H 6590 3160 50  0000 R CNN "Voltage"
+F 5 "25V" H 6590 3160 50  0000 R CNN "Voltage"
 F 6 "X7R" H 6590 3060 50  0000 R CNN "Dielectric"
-F 7 "" H 2830 -3720 50  0001 C CNN "Digi-Key PN"
+F 7 "490-10698-1-ND" H 2830 -3720 50  0001 C CNN "Digi-Key PN"
 F 8 "DNP" H 6210 3160 50  0000 C CNN "Configuration"
 	1    6740 3160
