File: hdw/rev_b/Pulse_Oximeter/PIC32MZ.sch (KiCad schematic (older format))
At the start: 3 parts, among them U1101 PIC32MZ0512EFE064T-I_PT

Commit message: lots of rev b changes
Connections:
- net Telemetry_Config renamed ~Telemetry_Config
Changed lines of the file:
@@
 Wire Wire Line
 	9330 2880 9630 2880
-Text GLabel 3320 5080 0    50   UnSpc ~ 0
-Telemetry_Config
+Text GLabel 3320 5080 0    40   UnSpc ~ 0
+~Telemetry_Config
 Text GLabel 3320 4280 0    50   Input ~ 0
 POS1P8_PGOOD
@@
 NoConn ~ 3320 2980
 NoConn ~ 3320 3080
+Text GLabel 1180 2380 2    50   UnSpc ~ 0
+~ETC_Config
 $EndSCHEMATC

Commit message: changed all passives to 0402, cleared digikey pns
Parts:
- R1101, R1102: Digi-Key PN RMCF0402FT10K0CT-ND -> (none)
Changed lines of the file:
@@
 F 5 "1%" H 9430 2550 50  0000 L CNN "Tolerance"
 F 6 "1/16W" H 9440 2470 50  0000 L CNN "Wattage"
-F 7 "RMCF0402FT10K0CT-ND" H 9330 2550 50  0001 C CNN "Digi-Key PN"
+F 7 "" H 9330 2550 50  0001 C CNN "Digi-Key PN"
 	1    9330 2550
 	1    0    0    -1
@@
 F 5 "1%" H 8840 2550 50  0000 L CNN "Tolerance"
 F 6 "1/16W" H 8850 2470 50  0000 L CNN "Wattage"
-F 7 "RMCF0402FT10K0CT-ND" H 8740 2550 50  0001 C CNN "Digi-Key PN"
+F 7 "" H 8740 2550 50  0001 C CNN "Digi-Key PN"
 	1    8740 2550
 	1    0    0    -1
@@
 Text GLabel 1180 2380 2    50   UnSpc ~ 0
 ~ETC_Config
+Text GLabel 1650 2700 0    50   Input ~ 0
+PGOOD_LED_EN
 $EndSCHEMATC

Commit message: annotated schematic
Connections:
- net PGOOD_LED_EN: now also U1101.29 (RB14/AN9/RPB14/SCK3/PMA1)
- net ~ETC_Config: now also U1101.28 (RB13/TDI/AN8)
- net POS12_PGOOD: now reaches U1101.23 (RB10/TMS/CVREFOUT/AN5/RPB10/PMA13)
- net POS5_USB_PGOOD: now reaches U1101.24 (RB11/TDO/AN6/PMA12)
- net POS3P3_PGOOD: now reaches U1101.27 (RB12/TCK/AN7/PMA11)
- no-connect marks 15 -> 10
Changed lines of the file:
@@
 Text GLabel 3320 1780 0    50   Output ~ 0
 POS3P3_POX_Enable
-Text GLabel 3320 1880 0    40   Output ~ 0
+Text GLabel 3320 1880 0    40   Input ~ 0
 ~POX_INT
 Text GLabel 3320 1980 0    50   Input ~ 0
@@
 NoConn ~ 3320 2080
 NoConn ~ 3320 2180
-NoConn ~ 3320 2780
-NoConn ~ 3320 2880
 NoConn ~ 3320 3780
 NoConn ~ 7520 3280
@@
 NoConn ~ 3320 2480
 NoConn ~ 3320 2580
-NoConn ~ 3320 2680
-NoConn ~ 3320 2980
-NoConn ~ 3320 3080
-Text GLabel 1180 2380 2    50   UnSpc ~ 0
+Text GLabel 3320 2980 0    40   UnSpc ~ 0
 ~ETC_Config
-Text GLabel 1650 2700 0    50   Input ~ 0
+Text GLabel 3320 3080 0    50   Output ~ 0
 PGOOD_LED_EN
+Text GLabel 3320 2680 0    50   Input ~ 0
+POS12_PGOOD
+Text GLabel 3320 2780 0    50   Input ~ 0
+POS5_USB_PGOOD
+Text GLabel 3320 2880 0    50   Input ~ 0
+POS3P3_PGOOD
 $EndSCHEMATC

Commit message: fixed PGOOD LED drivers
Connections:
- net PGOOD_LED_EN renamed PGOOD_LED_SHDN
Changed lines of the file:
@@
 Text GLabel 3320 2980 0    40   UnSpc ~ 0
 ~ETC_Config
-Text GLabel 3320 3080 0    50   Output ~ 0
-PGOOD_LED_EN
 Text GLabel 3320 2680 0    50   Input ~ 0
 POS12_PGOOD
@@
 Text GLabel 3320 2880 0    50   Input ~ 0
 POS3P3_PGOOD
+Text GLabel 3320 3080 0    50   Output ~ 0
+PGOOD_LED_SHDN
 $EndSCHEMATC

Commit message: assigned digikey PNs
Parts:
- R1101, R1102: Digi-Key PN (none) -> RMCF0402FT10K0CT-ND
Changed lines of the file:
@@
 F 5 "1%" H 9430 2550 50  0000 L CNN "Tolerance"
 F 6 "1/16W" H 9440 2470 50  0000 L CNN "Wattage"
-F 7 "" H 9330 2550 50  0001 C CNN "Digi-Key PN"
+F 7 "RMCF0402FT10K0CT-ND" H 9330 2550 50  0001 C CNN "Digi-Key PN"
 	1    9330 2550
 	1    0    0    -1
@@
 F 5 "1%" H 8840 2550 50  0000 L CNN "Tolerance"
 F 6 "1/16W" H 8850 2470 50  0000 L CNN "Wattage"
-F 7 "" H 8740 2550 50  0001 C CNN "Digi-Key PN"
+F 7 "RMCF0402FT10K0CT-ND" H 8740 2550 50  0001 C CNN "Digi-Key PN"
 	1    8740 2550
 	1    0    0    -1
