File: hdw/rev_b/Pulse_Oximeter/PIC32MZ_Bypass.sch (KiCad schematic (older format))
At the start: 23 parts

Commit message: lots of rev b changes
Parts:
- removed C901, C902, C908, C912, C916, C917: 0.1uF, Capacitors_SMD:C_0402, symbol Custom_Library:C_Custom
- removed C903, C909, C913: 10uF, Capacitors_SMD:C_0402, symbol Custom_Library:C_Custom
- removed C904, C905, C910, C914, C918, C919: 10nF, Capacitors_SMD:C_0402, symbol Custom_Library:C_Custom
- removed C906, C907, C911, C915, C920, C921: 1nF, Capacitors_SMD:C_0402, symbol Custom_Library:C_Custom
- added C? (x6): 10uF, Capacitors_SMD:C_0402, symbol Custom_Library:C_Custom
- added C? (x6): 0.1uF, Capacitors_SMD:C_0402, symbol Custom_Library:C_Custom
Connections:
- net +3.3VA_MZ: now also C?.1, C?.1
- net +3V3: now also C?.1, C?.1, C?.1, C?.1, C?.1, C?.1, C?.1, C?.1, C?.1, C?.1
- net GND: now also C?.2, C?.2, C?.2, C?.2, C?.2, C?.2, C?.2, C?.2, C?.2, C?.2
- net GNDA_MZ: now also C?.2, C?.2

Commit message: changed all passives to 0402, cleared digikey pns
Parts:
- C? (x6): Digi-Key PN 490-13211-1-ND -> (none)
- C? (x6): Digi-Key PN 490-10701-1-ND -> (none)
Changed lines of the file:
@@
 F 5 "6.3V" H 3090 4400 50  0000 R CNN "Voltage"
 F 6 "X5R" H 3090 4300 50  0000 R CNN "Dielectric"
-F 7 "490-13211-1-ND" H 3240 4400 50  0001 C CNN "Digi-Key PN"
+F 7 "" H 3240 4400 50  0001 C CNN "Digi-Key PN"
 	1    3240 4400
 	1    0    0    -1
@@
 F 5 "50V" H 2450 4400 50  0000 R CNN "Voltage"
 F 6 "X7R" H 2450 4300 50  0000 R CNN "Dielectric"
-F 7 "490-10701-1-ND" H 3025 4900 60  0001 C CNN "Digi-Key PN"
+F 7 "" H 3025 4900 60  0001 C CNN "Digi-Key PN"
 	1    2600 4400
 	1    0    0    -1
@@
 F 5 "6.3V" H 3090 3400 50  0000 R CNN "Voltage"
 F 6 "X5R" H 3090 3300 50  0000 R CNN "Dielectric"
-F 7 "490-13211-1-ND" H 3240 3400 50  0001 C CNN "Digi-Key PN"
+F 7 "" H 3240 3400 50  0001 C CNN "Digi-Key PN"
 	1    3240 3400
 	1    0    0    -1
@@
 F 5 "50V" H 2450 3400 50  0000 R CNN "Voltage"
 F 6 "X7R" H 2450 3300 50  0000 R CNN "Dielectric"
-F 7 "490-10701-1-ND" H 3025 3900 60  0001 C CNN "Digi-Key PN"
+F 7 "" H 3025 3900 60  0001 C CNN "Digi-Key PN"
 	1    2600 3400
 	1    0    0    -1
@@
 F 5 "6.3V" H 4390 3400 50  0000 R CNN "Voltage"
 F 6 "X5R" H 4390 3300 50  0000 R CNN "Dielectric"
-F 7 "490-13211-1-ND" H 4540 3400 50  0001 C CNN "Digi-Key PN"
+F 7 "" H 4540 3400 50  0001 C CNN "Digi-Key PN"
 	1    4540 3400
 	1    0    0    -1
@@
 F 5 "50V" H 3750 3400 50  0000 R CNN "Voltage"
 F 6 "X7R" H 3750 3300 50  0000 R CNN "Dielectric"
-F 7 "490-10701-1-ND" H 4325 3900 60  0001 C CNN "Digi-Key PN"
+F 7 "" H 4325 3900 60  0001 C CNN "Digi-Key PN"
 	1    3900 3400
 	1    0    0    -1
@@
 F 5 "6.3V" H 5690 3400 50  0000 R CNN "Voltage"
 F 6 "X5R" H 5690 3300 50  0000 R CNN "Dielectric"
-F 7 "490-13211-1-ND" H 5840 3400 50  0001 C CNN "Digi-Key PN"
+F 7 "" H 5840 3400 50  0001 C CNN "Digi-Key PN"
 	1    5840 3400
 	1    0    0    -1
@@
 F 5 "50V" H 5050 3400 50  0000 R CNN "Voltage"
 F 6 "X7R" H 5050 3300 50  0000 R CNN "Dielectric"
-F 7 "490-10701-1-ND" H 5625 3900 60  0001 C CNN "Digi-Key PN"
+F 7 "" H 5625 3900 60  0001 C CNN "Digi-Key PN"
 	1    5200 3400
 	1    0    0    -1
@@
 F 5 "6.3V" H 6990 3400 50  0000 R CNN "Voltage"
 F 6 "X5R" H 6990 3300 50  0000 R CNN "Dielectric"
-F 7 "490-13211-1-ND" H 7140 3400 50  0001 C CNN "Digi-Key PN"
+F 7 "" H 7140 3400 50  0001 C CNN "Digi-Key PN"
 	1    7140 3400
 	1    0    0    -1
@@
 F 5 "50V" H 6350 3400 50  0000 R CNN "Voltage"
 F 6 "X7R" H 6350 3300 50  0000 R CNN "Dielectric"
-F 7 "490-10701-1-ND" H 6925 3900 60  0001 C CNN "Digi-Key PN"
+F 7 "" H 6925 3900 60  0001 C CNN "Digi-Key PN"
 	1    6500 3400
 	1    0    0    -1
@@
 F 5 "6.3V" H 6990 4400 50  0000 R CNN "Voltage"
 F 6 "X5R" H 6990 4300 50  0000 R CNN "Dielectric"
-F 7 "490-13211-1-ND" H 7140 4400 50  0001 C CNN "Digi-Key PN"
+F 7 "" H 7140 4400 50  0001 C CNN "Digi-Key PN"
 	1    7140 4400
 	1    0    0    -1
@@
 F 5 "50V" H 6350 4400 50  0000 R CNN "Voltage"
 F 6 "X7R" H 6350 4300 50  0000 R CNN "Dielectric"
-F 7 "490-10701-1-ND" H 6925 4900 60  0001 C CNN "Digi-Key PN"
+F 7 "" H 6925 4900 60  0001 C CNN "Digi-Key PN"
 	1    6500 4400
 	1    0    0    -1

Commit message: annotated schematic
Parts:
- gave numbers to parts that had none: 12
Changed lines of the file:
@@
 $EndDescr
 $Comp
-L power:GND #PWR0910
+L power:GND #PWR0906
 U 1 1 5CB1558B
 P 4220 3630
-F 0 "#PWR0910" H 4220 3380 50  0001 C CNN
+F 0 "#PWR0906" H 4220 3380 50  0001 C CNN
 F 1 "GND" H 4220 3480 50  0000 C CNN
 F 2 "" H 4220 3630 50  0000 C CNN
@@
 $EndComp
 $Comp
-L power:GND #PWR0914
+L power:GND #PWR0908
 U 1 1 5CB1993B
 P 5520 3630
-F 0 "#PWR0914" H 5520 3380 50  0001 C CNN
+F 0 "#PWR0908" H 5520 3380 50  0001 C CNN
 F 1 "GND" H 5520 3480 50  0000 C CNN
 F 2 "" H 5520 3630 50  0000 C CNN
@@
 $EndComp
 $Comp
-L power:GND #PWR0916
+L power:GND #PWR0910
 U 1 1 5CB219B2
 P 6820 3630
-F 0 "#PWR0916" H 6820 3380 50  0001 C CNN
+F 0 "#PWR0910" H 6820 3380 50  0001 C CNN
 F 1 "GND" H 6820 3480 50  0000 C CNN
 F 2 "" H 6820 3630 50  0000 C CNN
@@
 $EndComp
 $Comp
-L power:GND #PWR0906
+L power:GND #PWR0904
 U 1 1 5CB24EB8
 P 2920 4630
-F 0 "#PWR0906" H 2920 4380 50  0001 C CNN
+F 0 "#PWR0904" H 2920 4380 50  0001 C CNN
 F 1 "GND" H 2920 4480 50  0000 C CNN
 F 2 "" H 2920 4630 50  0000 C CNN
@@
 $EndComp
 $Comp
-L power:GND #PWR0920
+L power:GND #PWR0914
 U 1 1 5CB62D81
 P 8110 4680
-F 0 "#PWR0920" H 8110 4430 50  0001 C CNN
+F 0 "#PWR0914" H 8110 4430 50  0001 C CNN
 F 1 "GND" V 8110 4530 50  0000 R CNN
 F 2 "" H 8110 4680 50  0001 C CNN
@@
 $EndComp
 $Comp
-L power:+3.3V #PWR0915
+L power:+3.3V #PWR0909
 U 1 1 5E6E2CE4
 P 6820 3170
-F 0 "#PWR0915" H 6820 3020 50  0001 C CNN
+F 0 "#PWR0909" H 6820 3020 50  0001 C CNN
 F 1 "+3.3V" H 6820 3310 50  0000 C CNN
 F 2 "" H 6820 3170 50  0001 C CNN
@@
 $EndComp
 $Comp
-L power:+3.3V #PWR0913
+L power:+3.3V #PWR0907
 U 1 1 5E6E34DC
 P 5520 3170
-F 0 "#PWR0913" H 5520 3020 50  0001 C CNN
+F 0 "#PWR0907" H 5520 3020 50  0001 C CNN
 F 1 "+3.3V" H 5520 3310 50  0000 C CNN
 F 2 "" H 5520 3170 50  0001 C CNN
@@
 $EndComp
 $Comp
-L power:+3.3V #PWR0909
+L power:+3.3V #PWR0905
 U 1 1 5E6E3A94
 P 4220 3170
-F 0 "#PWR0909" H 4220 3020 50  0001 C CNN
+F 0 "#PWR0905" H 4220 3020 50  0001 C CNN
 F 1 "+3.3V" H 4220 3310 50  0000 C CNN
 F 2 "" H 4220 3170 50  0001 C CNN
@@
 $EndComp
 $Comp
-L power:+3.3V #PWR0903
+L power:+3.3V #PWR0901
 U 1 1 5E6E4189
 P 2920 3170
-F 0 "#PWR0903" H 2920 3020 50  0001 C CNN
+F 0 "#PWR0901" H 2920 3020 50  0001 C CNN
 F 1 "+3.3V" H 2920 3310 50  0000 C CNN
 F 2 "" H 2920 3170 50  0001 C CNN
@@
 $EndComp
 $Comp
-L power:+3.3V #PWR0905
+L power:+3.3V #PWR0903
 U 1 1 5E6E46E8
 P 2920 4170
-F 0 "#PWR0905" H 2920 4020 50  0001 C CNN
+F 0 "#PWR0903" H 2920 4020 50  0001 C CNN
 F 1 "+3.3V" H 2920 4310 50  0000 C CNN
 F 2 "" H 2920 4170 50  0001 C CNN
@@
 $EndComp
 $Comp
-L power:+3.3V #PWR0919
+L power:+3.3V #PWR0913
 U 1 1 5E6E6088
 P 8110 4120
-F 0 "#PWR0919" H 8110 3970 50  0001 C CNN
+F 0 "#PWR0913" H 8110 3970 50  0001 C CNN
 F 1 "+3.3V" V 8110 4260 50  0000 L CNN
 F 2 "" H 8110 4120 50  0001 C CNN
@@
 $EndComp
 $Comp
-L Custom_Library:GNDA_MZ #PWR0918
+L Custom_Library:GNDA_MZ #PWR0912
 U 1 1 5EB1572E
 P 6820 4630
-F 0 "#PWR0918" H 6820 4380 50  0001 C CNN
+F 0 "#PWR0912" H 6820 4380 50  0001 C CNN
 F 1 "GNDA_MZ" H 6820 4480 50  0000 C CNN
 F 2 "" H 6820 4630 50  0001 C CNN
@@
 $EndComp
 $Comp
-L Custom_Library:GNDA_MZ #PWR0922
+L Custom_Library:GNDA_MZ #PWR0916
 U 1 1 5EB160DB
 P 8410 4680
-F 0 "#PWR0922" H 8410 4430 50  0001 C CNN
+F 0 "#PWR0916" H 8410 4430 50  0001 C CNN
 F 1 "GNDA_MZ" V 8410 4530 50  0000 R CNN
 F 2 "" H 8410 4680 50  0001 C CNN
@@
 $EndComp
 $Comp
-L Custom_Library:GNDA_MZ #PWR0924
+L Custom_Library:GNDA_MZ #PWR0918
 U 1 1 5EB16842
 P 9670 4680
-F 0 "#PWR0924" H 9670 4430 50  0001 C CNN
+F 0 "#PWR0918" H 9670 4430 50  0001 C CNN
 F 1 "GNDA_MZ" V 9670 4530 50  0000 R CNN
 F 2 "" H 9670 4680 50  0001 C CNN
@@
 $EndComp
 $Comp
-L Custom_Library:+3.3VA_MZ #PWR0917
+L Custom_Library:+3.3VA_MZ #PWR0911
 U 1 1 5EB17B0F
 P 6820 4170
-F 0 "#PWR0917" H 6820 4020 50  0001 C CNN
+F 0 "#PWR0911" H 6820 4020 50  0001 C CNN
 F 1 "+3.3VA_MZ" H 6820 4310 50  0000 C CNN
 F 2 "" H 6820 4170 50  0001 C CNN
@@
 $EndComp
 $Comp
-L Custom_Library:+3.3VA_MZ #PWR0921
+L Custom_Library:+3.3VA_MZ #PWR0915
 U 1 1 5EB18347
 P 8410 4120
-F 0 "#PWR0921" H 8410 3970 50  0001 C CNN
+F 0 "#PWR0915" H 8410 3970 50  0001 C CNN
 F 1 "+3.3VA_MZ" V 8410 4260 50  0000 L CNN
 F 2 "" H 8410 4120 50  0001 C CNN
@@
 $EndComp
 $Comp
-L Custom_Library:+3.3VA_MZ #PWR0923
+L Custom_Library:+3.3VA_MZ #PWR0917
 U 1 1 5EB18B8A
 P 9670 4120
-F 0 "#PWR0923" H 9670 3970 50  0001 C CNN
+F 0 "#PWR0917" H 9670 3970 50  0001 C CNN
 F 1 "+3.3VA_MZ" V 9670 4260 50  0000 L CNN
 F 2 "" H 9670 4120 50  0001 C CNN
@@
 AR Path="/5CB25152/5FDD7A6A" Ref="C?"  Part="1"
 AR Path="/5E697934/5FDD7A6A" Ref="C?"  Part="1"
-AR Path="/5EAE2F02/5FDD7A6A" Ref="C?"  Part="1"
+AR Path="/5EAE2F02/5FDD7A6A" Ref="C904"  Part="1"
 AR Path="/5EAE3021/5FDD7A6A" Ref="C?"  Part="1"
 AR Path="/5EAE30C7/5FDD7A6A" Ref="C?"  Part="1"
-F 0 "C?" H 3265 4500 50  0000 L CNN
+F 0 "C904" H 3265 4500 50  0000 L CNN
 F 1 "10uF" H 3265 4300 50  0000 L CNN
 F 2 "Capacitors_SMD:C_0402" H 3278 4250 50  0001 C CNN
@@
 AR Path="/5EAE2D66/5FDD7A7A" Ref="C?"  Part="1"
 AR Path="/5EAE30C7/5FDD7A7A" Ref="C?"  Part="1"
-AR Path="/5EAE2F02/5FDD7A7A" Ref="C?"  Part="1"
-F 0 "C?" H 2625 4500 50  0000 L CNN
+AR Path="/5EAE2F02/5FDD7A7A" Ref="C902"  Part="1"
+F 0 "C902" H 2625 4500 50  0000 L CNN
 F 1 "0.1uF" H 2625 4300 50  0000 L CNN
 F 2 "Capacitors_SMD:C_0402" H 2638 4250 50  0001 C CNN
@@
 	2920 4210 3240 4210
 $Comp
-L power:GND #PWR0904
+L power:GND #PWR0902
 U 1 1 5CB29D2D
 P 2920 3630
-F 0 "#PWR0904" H 2920 3380 50  0001 C CNN
+F 0 "#PWR0902" H 2920 3380 50  0001 C CNN
 F 1 "GND" H 2920 3480 50  0000 C CNN
 F 2 "" H 2920 3630 50  0000 C CNN
@@
 AR Path="/5CB25152/5FDE4A40" Ref="C?"  Part="1"
 AR Path="/5E697934/5FDE4A40" Ref="C?"  Part="1"
-AR Path="/5EAE2F02/5FDE4A40" Ref="C?"  Part="1"
+AR Path="/5EAE2F02/5FDE4A40" Ref="C903"  Part="1"
 AR Path="/5EAE3021/5FDE4A40" Ref="C?"  Part="1"
 AR Path="/5EAE30C7/5FDE4A40" Ref="C?"  Part="1"
-F 0 "C?" H 3265 3500 50  0000 L CNN
+F 0 "C903" H 3265 3500 50  0000 L CNN
 F 1 "10uF" H 3265 3300 50  0000 L CNN
 F 2 "Capacitors_SMD:C_0402" H 3278 3250 50  0001 C CNN
@@
 AR Path="/5EAE2D66/5FDE4A4A" Ref="C?"  Part="1"
 AR Path="/5EAE30C7/5FDE4A4A" Ref="C?"  Part="1"
-AR Path="/5EAE2F02/5FDE4A4A" Ref="C?"  Part="1"
-F 0 "C?" H 2625 3500 50  0000 L CNN
+AR Path="/5EAE2F02/5FDE4A4A" Ref="C901"  Part="1"
+F 0 "C901" H 2625 3500 50  0000 L CNN
 F 1 "0.1uF" H 2625 3300 50  0000 L CNN
 F 2 "Capacitors_SMD:C_0402" H 2638 3250 50  0001 C CNN
@@
 AR Path="/5CB25152/5FDE5889" Ref="C?"  Part="1"
 AR Path="/5E697934/5FDE5889" Ref="C?"  Part="1"
-AR Path="/5EAE2F02/5FDE5889" Ref="C?"  Part="1"
+AR Path="/5EAE2F02/5FDE5889" Ref="C906"  Part="1"
 AR Path="/5EAE3021/5FDE5889" Ref="C?"  Part="1"
 AR Path="/5EAE30C7/5FDE5889" Ref="C?"  Part="1"
-F 0 "C?" H 4565 3500 50  0000 L CNN
+F 0 "C906" H 4565 3500 50  0000 L CNN
 F 1 "10uF" H 4565 3300 50  0000 L CNN
 F 2 "Capacitors_SMD:C_0402" H 4578 3250 50  0001 C CNN
@@
 AR Path="/5EAE2D66/5FDE5893" Ref="C?"  Part="1"
 AR Path="/5EAE30C7/5FDE5893" Ref="C?"  Part="1"
-AR Path="/5EAE2F02/5FDE5893" Ref="C?"  Part="1"
-F 0 "C?" H 3925 3500 50  0000 L CNN
+AR Path="/5EAE2F02/5FDE5893" Ref="C905"  Part="1"
+F 0 "C905" H 3925 3500 50  0000 L CNN
 F 1 "0.1uF" H 3925 3300 50  0000 L CNN
 F 2 "Capacitors_SMD:C_0402" H 3938 3250 50  0001 C CNN
@@
 AR Path="/5CB25152/5FDE65F0" Ref="C?"  Part="1"
 AR Path="/5E697934/5FDE65F0" Ref="C?"  Part="1"
-AR Path="/5EAE2F02/5FDE65F0" Ref="C?"  Part="1"
+AR Path="/5EAE2F02/5FDE65F0" Ref="C908"  Part="1"
 AR Path="/5EAE3021/5FDE65F0" Ref="C?"  Part="1"
 AR Path="/5EAE30C7/5FDE65F0" Ref="C?"  Part="1"
-F 0 "C?" H 5865 3500 50  0000 L CNN
+F 0 "C908" H 5865 3500 50  0000 L CNN
 F 1 "10uF" H 5865 3300 50  0000 L CNN
 F 2 "Capacitors_SMD:C_0402" H 5878 3250 50  0001 C CNN
@@
 AR Path="/5EAE2D66/5FDE65FA" Ref="C?"  Part="1"
 AR Path="/5EAE30C7/5FDE65FA" Ref="C?"  Part="1"
-AR Path="/5EAE2F02/5FDE65FA" Ref="C?"  Part="1"
-F 0 "C?" H 5225 3500 50  0000 L CNN
+AR Path="/5EAE2F02/5FDE65FA" Ref="C907"  Part="1"
+F 0 "C907" H 5225 3500 50  0000 L CNN
 F 1 "0.1uF" H 5225 3300 50  0000 L CNN
 F 2 "Capacitors_SMD:C_0402" H 5238 3250 50  0001 C CNN
@@
 AR Path="/5CB25152/5FDE7609" Ref="C?"  Part="1"
 AR Path="/5E697934/5FDE7609" Ref="C?"  Part="1"
-AR Path="/5EAE2F02/5FDE7609" Ref="C?"  Part="1"
+AR Path="/5EAE2F02/5FDE7609" Ref="C911"  Part="1"
 AR Path="/5EAE3021/5FDE7609" Ref="C?"  Part="1"
 AR Path="/5EAE30C7/5FDE7609" Ref="C?"  Part="1"
-F 0 "C?" H 7165 3500 50  0000 L CNN
+F 0 "C911" H 7165 3500 50  0000 L CNN
 F 1 "10uF" H 7165 3300 50  0000 L CNN
 F 2 "Capacitors_SMD:C_0402" H 7178 3250 50  0001 C CNN
@@
 AR Path="/5EAE2D66/5FDE7613" Ref="C?"  Part="1"
 AR Path="/5EAE30C7/5FDE7613" Ref="C?"  Part="1"
-AR Path="/5EAE2F02/5FDE7613" Ref="C?"  Part="1"
-F 0 "C?" H 6525 3500 50  0000 L CNN
+AR Path="/5EAE2F02/5FDE7613" Ref="C909"  Part="1"
+F 0 "C909" H 6525 3500 50  0000 L CNN
 F 1 "0.1uF" H 6525 3300 50  0000 L CNN
 F 2 "Capacitors_SMD:C_0402" H 6538 3250 50  0001 C CNN
@@
 AR Path="/5CB25152/5FDE9E30" Ref="C?"  Part="1"
 AR Path="/5E697934/5FDE9E30" Ref="C?"  Part="1"
-AR Path="/5EAE2F02/5FDE9E30" Ref="C?"  Part="1"
+AR Path="/5EAE2F02/5FDE9E30" Ref="C912"  Part="1"
 AR Path="/5EAE3021/5FDE9E30" Ref="C?"  Part="1"
 AR Path="/5EAE30C7/5FDE9E30" Ref="C?"  Part="1"
-F 0 "C?" H 7165 4500 50  0000 L CNN
+F 0 "C912" H 7165 4500 50  0000 L CNN
 F 1 "10uF" H 7165 4300 50  0000 L CNN
 F 2 "Capacitors_SMD:C_0402" H 7178 4250 50  0001 C CNN
@@
 AR Path="/5EAE2D66/5FDE9E3A" Ref="C?"  Part="1"
 AR Path="/5EAE30C7/5FDE9E3A" Ref="C?"  Part="1"
-AR Path="/5EAE2F02/5FDE9E3A" Ref="C?"  Part="1"
-F 0 "C?" H 6525 4500 50  0000 L CNN
+AR Path="/5EAE2F02/5FDE9E3A" Ref="C910"  Part="1"
+F 0 "C910" H 6525 4500 50  0000 L CNN
 F 1 "0.1uF" H 6525 4300 50  0000 L CNN
 F 2 "Capacitors_SMD:C_0402" H 6538 4250 50  0001 C CNN

Commit message: assigned digikey PNs
Parts:
- C901, C902, C905, C907, C909, C910: Digi-Key PN (none) -> 490-10698-1-ND; Voltage 50V -> 25V
- C903, C904, C906, C908, C911, C912: Digi-Key PN (none) -> 1276-6830-1-ND; Voltage 6.3V -> 10V
Changed lines of the file:
@@
 F 3 "" H 3265 4500 50  0001 C CNN
 F 4 "0402" H 3090 4500 50  0000 R CNN "display_footprint"
-F 5 "6.3V" H 3090 4400 50  0000 R CNN "Voltage"
+F 5 "10V" H 3090 4400 50  0000 R CNN "Voltage"
 F 6 "X5R" H 3090 4300 50  0000 R CNN "Dielectric"
-F 7 "" H 3240 4400 50  0001 C CNN "Digi-Key PN"
+F 7 "1276-6830-1-ND" H 3240 4400 50  0001 C CNN "Digi-Key PN"
 	1    3240 4400
 	1    0    0    -1
@@
 F 3 "" H 2625 4500 50  0001 C CNN
 F 4 "0402" H 2450 4500 50  0000 R CNN "display_footprint"
-F 5 "50V" H 2450 4400 50  0000 R CNN "Voltage"
+F 5 "25V" H 2450 4400 50  0000 R CNN "Voltage"
 F 6 "X7R" H 2450 4300 50  0000 R CNN "Dielectric"
-F 7 "" H 3025 4900 60  0001 C CNN "Digi-Key PN"
+F 7 "490-10698-1-ND" H 3025 4900 60  0001 C CNN "Digi-Key PN"
 	1    2600 4400
 	1    0    0    -1
@@
 F 3 "" H 3265 3500 50  0001 C CNN
 F 4 "0402" H 3090 3500 50  0000 R CNN "display_footprint"
-F 5 "6.3V" H 3090 3400 50  0000 R CNN "Voltage"
+F 5 "10V" H 3090 3400 50  0000 R CNN "Voltage"
 F 6 "X5R" H 3090 3300 50  0000 R CNN "Dielectric"
-F 7 "" H 3240 3400 50  0001 C CNN "Digi-Key PN"
+F 7 "1276-6830-1-ND" H 3240 3400 50  0001 C CNN "Digi-Key PN"
 	1    3240 3400
 	1    0    0    -1
@@
 F 3 "" H 2625 3500 50  0001 C CNN
 F 4 "0402" H 2450 3500 50  0000 R CNN "display_footprint"
-F 5 "50V" H 2450 3400 50  0000 R CNN "Voltage"
+F 5 "25V" H 2450 3400 50  0000 R CNN "Voltage"
 F 6 "X7R" H 2450 3300 50  0000 R CNN "Dielectric"
-F 7 "" H 3025 3900 60  0001 C CNN "Digi-Key PN"
+F 7 "490-10698-1-ND" H 3025 3900 60  0001 C CNN "Digi-Key PN"
 	1    2600 3400
 	1    0    0    -1
@@
 F 3 "" H 4565 3500 50  0001 C CNN
 F 4 "0402" H 4390 3500 50  0000 R CNN "display_footprint"
-F 5 "6.3V" H 4390 3400 50  0000 R CNN "Voltage"
+F 5 "10V" H 4390 3400 50  0000 R CNN "Voltage"
 F 6 "X5R" H 4390 3300 50  0000 R CNN "Dielectric"
-F 7 "" H 4540 3400 50  0001 C CNN "Digi-Key PN"
+F 7 "1276-6830-1-ND" H 4540 3400 50  0001 C CNN "Digi-Key PN"
 	1    4540 3400
 	1    0    0    -1
@@
 F 3 "" H 3925 3500 50  0001 C CNN
 F 4 "0402" H 3750 3500 50  0000 R CNN "display_footprint"
-F 5 "50V" H 3750 3400 50  0000 R CNN "Voltage"
+F 5 "25V" H 3750 3400 50  0000 R CNN "Voltage"
 F 6 "X7R" H 3750 3300 50  0000 R CNN "Dielectric"
-F 7 "" H 4325 3900 60  0001 C CNN "Digi-Key PN"
+F 7 "490-10698-1-ND" H 4325 3900 60  0001 C CNN "Digi-Key PN"
 	1    3900 3400
 	1    0    0    -1
@@
 F 3 "" H 5865 3500 50  0001 C CNN
 F 4 "0402" H 5690 3500 50  0000 R CNN "display_footprint"
-F 5 "6.3V" H 5690 3400 50  0000 R CNN "Voltage"
+F 5 "10V" H 5690 3400 50  0000 R CNN "Voltage"
 F 6 "X5R" H 5690 3300 50  0000 R CNN "Dielectric"
-F 7 "" H 5840 3400 50  0001 C CNN "Digi-Key PN"
+F 7 "1276-6830-1-ND" H 5840 3400 50  0001 C CNN "Digi-Key PN"
 	1    5840 3400
 	1    0    0    -1
@@
 F 3 "" H 5225 3500 50  0001 C CNN
 F 4 "0402" H 5050 3500 50  0000 R CNN "display_footprint"
-F 5 "50V" H 5050 3400 50  0000 R CNN "Voltage"
+F 5 "25V" H 5050 3400 50  0000 R CNN "Voltage"
 F 6 "X7R" H 5050 3300 50  0000 R CNN "Dielectric"
-F 7 "" H 5625 3900 60  0001 C CNN "Digi-Key PN"
+F 7 "490-10698-1-ND" H 5625 3900 60  0001 C CNN "Digi-Key PN"
 	1    5200 3400
 	1    0    0    -1
@@
 F 3 "" H 7165 3500 50  0001 C CNN
 F 4 "0402" H 6990 3500 50  0000 R CNN "display_footprint"
-F 5 "6.3V" H 6990 3400 50  0000 R CNN "Voltage"
+F 5 "10V" H 6990 3400 50  0000 R CNN "Voltage"
 F 6 "X5R" H 6990 3300 50  0000 R CNN "Dielectric"
-F 7 "" H 7140 3400 50  0001 C CNN "Digi-Key PN"
+F 7 "1276-6830-1-ND" H 7140 3400 50  0001 C CNN "Digi-Key PN"
 	1    7140 3400
 	1    0    0    -1
@@
 F 3 "" H 6525 3500 50  0001 C CNN
 F 4 "0402" H 6350 3500 50  0000 R CNN "display_footprint"
-F 5 "50V" H 6350 3400 50  0000 R CNN "Voltage"
+F 5 "25V" H 6350 3400 50  0000 R CNN "Voltage"
 F 6 "X7R" H 6350 3300 50  0000 R CNN "Dielectric"
-F 7 "" H 6925 3900 60  0001 C CNN "Digi-Key PN"
+F 7 "490-10698-1-ND" H 6925 3900 60  0001 C CNN "Digi-Key PN"
 	1    6500 3400
 	1    0    0    -1
@@
 F 3 "" H 7165 4500 50  0001 C CNN
 F 4 "0402" H 6990 4500 50  0000 R CNN "display_footprint"
-F 5 "6.3V" H 6990 4400 50  0000 R CNN "Voltage"
+F 5 "10V" H 6990 4400 50  0000 R CNN "Voltage"
 F 6 "X5R" H 6990 4300 50  0000 R CNN "Dielectric"
-F 7 "" H 7140 4400 50  0001 C CNN "Digi-Key PN"
+F 7 "1276-6830-1-ND" H 7140 4400 50  0001 C CNN "Digi-Key PN"
 	1    7140 4400
 	1    0    0    -1
@@
 F 3 "" H 6525 4500 50  0001 C CNN
 F 4 "0402" H 6350 4500 50  0000 R CNN "display_footprint"
-F 5 "50V" H 6350 4400 50  0000 R CNN "Voltage"
+F 5 "25V" H 6350 4400 50  0000 R CNN "Voltage"
 F 6 "X7R" H 6350 4300 50  0000 R CNN "Dielectric"
-F 7 "" H 6925 4900 60  0001 C CNN "Digi-Key PN"
+F 7 "490-10698-1-ND" H 6925 4900 60  0001 C CNN "Digi-Key PN"
 	1    6500 4400
 	1    0    0    -1
