File: hdw/rev_b/Pulse_Oximeter/PIC32MZ_Clocking.sch (KiCad schematic (older format))
At the start: 10 parts, among them X1001 ASE-8.000MHz

Commit message: lots of rev B sch progress
Parts:
- L1001, X1001: Configuration (none) -> EXT_OSC
Changed lines of the file:
@@
 F 3 "http://www.abracon.com/Oscillators/ASV.pdf" H 5410 2700 50  0001 C CNN
 F 4 "	535-9558-1-ND" H 5510 2700 50  0001 C CNN "Digi-Key PN"
+F 5 "EXT_OSC" H 5510 2130 50  0000 C CNN "Configuration"
 	1    5510 2700
 	1    0    0    -1
@@
 AR Path="/5E697952/5E053473" Ref="L?"  Part="1"
 AR Path="/5EAE2F15/5E053473" Ref="L1001"  Part="1"
-F 0 "L1001" V 4890 1825 50  0000 C CNN
-F 1 "600R 0.5A" V 5190 1800 50  0000 C CNN
+F 0 "L1001" V 4640 1810 50  0000 C CNN
+F 1 "600R 0.5A" V 4740 1810 50  0000 C CNN
 F 2 "Inductors_SMD:L_0402" V 4970 1800 50  0001 C CNN
 F 3 "~" H 5040 1800 50  0001 C CNN
 F 4 "490-5441-1-ND" H -3150 -1290 50  0001 C CNN "Digi-Key PN"
+F 5 "EXT_OSC" V 4840 1810 50  0000 C CNN "Configuration"
 	1    5040 1800
 	0    1    1    0

Commit message: merged, more cleanups
Parts:
- removed C1001: 0.1uF, Capacitors_SMD:C_0402, symbol Custom_Library:C_Custom
- removed C1003: 10nF, Capacitors_SMD:C_0402, symbol Custom_Library:C_Custom
- removed C1005: 1nF, Capacitors_SMD:C_0402, symbol Custom_Library:C_Custom
- added C?: 10uF, Capacitors_SMD:C_0402, symbol Custom_Library:C_Custom
- added C?: 0.1uF, Capacitors_SMD:C_0402, symbol Custom_Library:C_Custom
Connections:
- net GND: now also C?.2, C?.2
- net at L1001.1, X1001.4 (Vdd): now also C?.1, C?.1
Changed lines of the file:
@@
 PIC32MZ_POSC_EC_Enable
-$Comp
-L power:GND #PWR?
-U 1 1 5E03ADCE
-P 6400 2300
-AR Path="/5CB25152/5E03ADCE" Ref="#PWR?"  Part="1"
-AR Path="/5E01BCC3/5E03ADCE" Ref="#PWR?"  Part="1"
-AR Path="/5E697952/5E03ADCE" Ref="#PWR?"  Part="1"
-AR Path="/5EAE2F15/5E03ADCE" Ref="#PWR01006"  Part="1"
-F 0 "#PWR01006" H 6400 2050 50  0001 C CNN
-F 1 "GND" H 6400 2150 50  0000 C CNN
-F 2 "" H 6400 2300 50  0000 C CNN
-F 3 "" H 6400 2300 50  0000 C CNN
-	1    6400 2300
-	1    0    0    -1
-$EndComp
-$Comp
-L Custom_Library:C_Custom C?
-U 1 1 5E03ADD8
-P 6080 2070
-AR Path="/5CB25152/5E03ADD8" Ref="C?"  Part="1"
-AR Path="/5E01BCC3/5E03ADD8" Ref="C?"  Part="1"
-AR Path="/5E697952/5E03ADD8" Ref="C?"  Part="1"
-AR Path="/5EAE2F15/5E03ADD8" Ref="C1001"  Part="1"
-F 0 "C1001" H 6105 2170 50  0000 L CNN
-F 1 "0.1uF" H 6105 1970 50  0000 L CNN
-F 2 "Capacitors_SMD:C_0402" H 6118 1920 50  0001 C CNN
-F 3 "" H 6105 2170 50  0001 C CNN
-F 4 "0402" H 5930 2170 50  0000 R CNN "display_footprint"
-F 5 "50V" H 5930 2070 50  0000 R CNN "Voltage"
-F 6 "X7R" H 5930 1970 50  0000 R CNN "Dielectric"
-F 7 "490-10701-1-ND" H 2170 -4810 50  0001 C CNN "Digi-Key PN"
-	1    6080 2070
-	1    0    0    -1
-$EndComp
-$Comp
-L Custom_Library:C_Custom C?
-U 1 1 5E03ADE2
-P 6720 2070
-AR Path="/5CB25152/5E03ADE2" Ref="C?"  Part="1"
-AR Path="/5E01BCC3/5E03ADE2" Ref="C?"  Part="1"
-AR Path="/5E697952/5E03ADE2" Ref="C?"  Part="1"
-AR Path="/5EAE2F15/5E03ADE2" Ref="C1005"  Part="1"
-F 0 "C1005" H 6745 2170 50  0000 L CNN
-F 1 "1nF" H 6745 1970 50  0000 L CNN
-F 2 "Capacitors_SMD:C_0402" H 6758 1920 50  0001 C CNN
-F 3 "" H 6745 2170 50  0001 C CNN
-F 4 "0402" H 6570 2170 50  0001 R CNN "display_footprint"
-F 5 "50V" H 6570 2070 50  0001 R CNN "Voltage"
-F 6 "X7R" H 6570 1970 50  0001 R CNN "Dielectric"
-F 7 "399-1032-1-ND" H 2170 -4810 50  0001 C CNN "Digi-Key PN"
-	1    6720 2070
-	1    0    0    -1
-$EndComp
-$Comp
-L Custom_Library:C_Custom C?
-U 1 1 5E03ADEC
-P 6400 2070
-AR Path="/5CB25152/5E03ADEC" Ref="C?"  Part="1"
-AR Path="/5E01BCC3/5E03ADEC" Ref="C?"  Part="1"
-AR Path="/5E697952/5E03ADEC" Ref="C?"  Part="1"
-AR Path="/5EAE2F15/5E03ADEC" Ref="C1003"  Part="1"
-F 0 "C1003" H 6425 2170 50  0000 L CNN
-F 1 "10nF" H 6425 1970 50  0000 L CNN
-F 2 "Capacitors_SMD:C_0402" H 6438 1920 50  0001 C CNN
-F 3 "" H 6425 2170 50  0001 C CNN
-F 4 "0402" H 6250 2170 50  0001 R CNN "display_footprint"
-F 5 "50V" H 6250 2070 50  0001 R CNN "Voltage"
-F 6 "X7R" H 6250 1970 50  0001 R CNN "Dielectric"
-F 7 "490-13295-1-ND" H 2170 -4810 50  0001 C CNN "Digi-Key PN"
-	1    6400 2070
-	1    0    0    -1
-$EndComp
-Wire Wire Line
-	6080 1880 6080 1920
-Connection ~ 6400 1880
-Wire Wire Line
-	6720 1880 6720 1920
-Wire Wire Line
-	6080 1880 6400 1880
-Wire Wire Line
-	6080 2260 6080 2220
-Connection ~ 6400 2260
-Wire Wire Line
-	6720 2260 6720 2220
-Wire Wire Line
-	6080 2260 6400 2260
-Wire Wire Line
-	6400 2220 6400 2260
-Wire Wire Line
-	6400 1880 6720 1880
-Wire Wire Line
-	6400 1880 6400 1920
-Wire Wire Line
-	6400 2260 6720 2260
-Wire Wire Line
-	6400 2260 6400 2300
 $Comp
 L Device:Ferrite_Bead L?
@@
 Wire Wire Line
 	5510 1800 5510 2400
-Wire Wire Line
-	5510 1800 6400 1800
-Wire Wire Line
-	6400 1800 6400 1880
 Connection ~ 5510 1800
 Wire Wire Line
@@
 	2840 5130 2760 5130
 Connection ~ 2760 5130
+$Comp
+L Custom_Library:C_Custom C?
+U 1 1 5FE10797
+P 6730 2030
+AR Path="/5CB7718D/5FE10797" Ref="C?"  Part="1"
+AR Path="/5E0DC082/5FE10797" Ref="C?"  Part="1"
+AR Path="/5E0F9110/5FE10797" Ref="C?"  Part="1"
+AR Path="/5A557C58/5FE10797" Ref="C?"  Part="1"
+AR Path="/5CB25152/5FE10797" Ref="C?"  Part="1"
+AR Path="/5E697934/5FE10797" Ref="C?"  Part="1"
+AR Path="/5EAE2F02/5FE10797" Ref="C?"  Part="1"
+AR Path="/5EAE3021/5FE10797" Ref="C?"  Part="1"
+AR Path="/5EAE30C7/5FE10797" Ref="C?"  Part="1"
+AR Path="/5EAE2F15/5FE10797" Ref="C?"  Part="1"
+F 0 "C?" H 6755 2130 50  0000 L CNN
+F 1 "10uF" H 6755 1930 50  0000 L CNN
+F 2 "Capacitors_SMD:C_0402" H 6768 1880 50  0001 C CNN
+F 3 "" H 6755 2130 50  0001 C CNN
+F 4 "0402" H 6580 2130 50  0000 R CNN "display_footprint"
+F 5 "6.3V" H 6580 2030 50  0000 R CNN "Voltage"
+F 6 "X5R" H 6580 1930 50  0000 R CNN "Dielectric"
+F 7 "490-13211-1-ND" H 6730 2030 50  0001 C CNN "Digi-Key PN"
+	1    6730 2030
+	1    0    0    -1
+$EndComp
+$Comp
+L Custom_Library:C_Custom C?
+U 1 1 5FE107A1
+P 6090 2030
+AR Path="/5BAAE16C/5FE107A1" Ref="C?"  Part="1"
+AR Path="/5BB181D8/5FE107A1" Ref="C?"  Part="1"
+AR Path="/5BB2595E/5FE107A1" Ref="C?"  Part="1"
+AR Path="/5BAAE0FA/5FE107A1" Ref="C?"  Part="1"
+AR Path="/5BB86F23/5FE107A1" Ref="C?"  Part="1"
+AR Path="/5C1D5C9E/5FE107A1" Ref="C?"  Part="1"
+AR Path="/5CB6F1ED/5FE107A1" Ref="C?"  Part="1"
+AR Path="/5E939CFF/5FE107A1" Ref="C?"  Part="1"
+AR Path="/5E9E0E87/5FE107A1" Ref="C?"  Part="1"
+AR Path="/5EAE2D66/5FE107A1" Ref="C?"  Part="1"
+AR Path="/5EAE30C7/5FE107A1" Ref="C?"  Part="1"
+AR Path="/5EAE2F02/5FE107A1" Ref="C?"  Part="1"
+AR Path="/5EAE2F15/5FE107A1" Ref="C?"  Part="1"
+F 0 "C?" H 6115 2130 50  0000 L CNN
+F 1 "0.1uF" H 6115 1930 50  0000 L CNN
+F 2 "Capacitors_SMD:C_0402" H 6128 1880 50  0001 C CNN
+F 3 "" H 6115 2130 50  0001 C CNN
+F 4 "0402" H 5940 2130 50  0000 R CNN "display_footprint"
+F 5 "50V" H 5940 2030 50  0000 R CNN "Voltage"
+F 6 "X7R" H 5940 1930 50  0000 R CNN "Dielectric"
+F 7 "490-10701-1-ND" H 6515 2530 60  0001 C CNN "Digi-Key PN"
+	1    6090 2030
+	1    0    0    -1
+$EndComp
+$Comp
+L power:GND #PWR?
+U 1 1 5FE10E08
+P 6090 2180
+F 0 "#PWR?" H 6090 1930 50  0001 C CNN
+F 1 "GND" H 6090 2030 50  0000 C CNN
+F 2 "" H 6090 2180 50  0001 C CNN
+F 3 "" H 6090 2180 50  0001 C CNN
+	1    6090 2180
+	1    0    0    -1
+$EndComp
+$Comp
+L power:GND #PWR?
+U 1 1 5FE10FFC
+P 6730 2180
+F 0 "#PWR?" H 6730 1930 50  0001 C CNN
+F 1 "GND" H 6730 2030 50  0000 C CNN
+F 2 "" H 6730 2180 50  0001 C CNN
+F 3 "" H 6730 2180 50  0001 C CNN
+	1    6730 2180
+	1    0    0    -1
+$EndComp
+Wire Wire Line
+	6090 1880 6090 1800
+Wire Wire Line
+	6090 1800 5510 1800
+Wire Wire Line
+	6090 1800 6730 1800
+Wire Wire Line
+	6730 1800 6730 1880
+Connection ~ 6090 1800
 $EndSCHEMATC

Commit message: changed all passives to 0402, cleared digikey pns
Parts:
- C?: Digi-Key PN 490-13211-1-ND -> (none)
- C?: Digi-Key PN 490-10701-1-ND -> (none)
- R1001, R1004, R1006: Digi-Key PN RMCF0402FT10K0CT-ND -> (none)
- R1002: Digi-Key PN 541-100LCT-ND -> (none)
Changed lines of the file:
@@
 F 5 "1%" H 6630 2930 50  0000 L CNN "Tolerance"
 F 6 "1/16W" H 6630 2860 50  0000 L CNN "Wattage"
-F 7 "RMCF0402FT10K0CT-ND" H 6560 2930 50  0001 C CNN "Digi-Key PN"
+F 7 "" H 6560 2930 50  0001 C CNN "Digi-Key PN"
 	1    6560 2930
 	-1   0    0    -1
@@
 F 5 "1%" V 6310 2700 50  0001 C CNN "Tolerance"
 F 6 "1/16W" V 6410 2700 50  0001 C CNN "Wattage"
-F 7 "541-100LCT-ND" H 6410 3100 60  0001 C CNN "Digi-Key PN"
+F 7 "" H 6410 3100 60  0001 C CNN "Digi-Key PN"
 	1    6110 2700
 	0    -1   1    0
@@
 F 5 "1%" H 5030 2930 50  0000 L CNN "Tolerance"
 F 6 "1/16W" H 5030 2860 50  0000 L CNN "Wattage"
-F 7 "RMCF0402FT10K0CT-ND" H 4960 2930 50  0001 C CNN "Digi-Key PN"
+F 7 "" H 4960 2930 50  0001 C CNN "Digi-Key PN"
 	1    4960 2930
 	-1   0    0    -1
@@
 F 5 "1%" H 2830 5360 50  0000 L CNN "Tolerance"
 F 6 "1/16W" H 2830 5290 50  0000 L CNN "Wattage"
-F 7 "RMCF0402FT10K0CT-ND" H 2760 5360 50  0001 C CNN "Digi-Key PN"
+F 7 "" H 2760 5360 50  0001 C CNN "Digi-Key PN"
 	1    2760 5360
 	-1   0    0    -1
@@
 F 5 "6.3V" H 6580 2030 50  0000 R CNN "Voltage"
 F 6 "X5R" H 6580 1930 50  0000 R CNN "Dielectric"
-F 7 "490-13211-1-ND" H 6730 2030 50  0001 C CNN "Digi-Key PN"
+F 7 "" H 6730 2030 50  0001 C CNN "Digi-Key PN"
 	1    6730 2030
 	1    0    0    -1
@@
 F 5 "50V" H 5940 2030 50  0000 R CNN "Voltage"
 F 6 "X7R" H 5940 1930 50  0000 R CNN "Dielectric"
-F 7 "490-10701-1-ND" H 6515 2530 60  0001 C CNN "Digi-Key PN"
+F 7 "" H 6515 2530 60  0001 C CNN "Digi-Key PN"
 	1    6090 2030
 	1    0    0    -1

Commit message: annotated schematic
Parts:
- C1001, C1002: renamed from C?; Digi-Key PN (none) -> DNP
- L1001, X1001: Configuration EXT_OSC -> DNP
- R1002: renamed from R1001; Configuration (none) -> DNP
- R1003: renamed from R1002; Digi-Key PN (none) -> DNP
- renumbered R1006 to R1001
Changed lines of the file:
@@
 F 3 "http://www.abracon.com/Oscillators/ASV.pdf" H 5410 2700 50  0001 C CNN
 F 4 "	535-9558-1-ND" H 5510 2700 50  0001 C CNN "Digi-Key PN"
-F 5 "EXT_OSC" H 5510 2130 50  0000 C CNN "Configuration"
+F 5 "DNP" H 5510 2130 50  0000 C CNN "Configuration"
 	1    5510 2700
 	1    0    0    -1
@@
 AR Path="/5E01BCC3/5E021EFB" Ref="#PWR?"  Part="1"
 AR Path="/5E697952/5E021EFB" Ref="#PWR?"  Part="1"
-AR Path="/5EAE2F15/5E021EFB" Ref="#PWR01008"  Part="1"
-F 0 "#PWR01008" H 6560 2830 50  0001 C CNN
+AR Path="/5EAE2F15/5E021EFB" Ref="#PWR01006"  Part="1"
+F 0 "#PWR01006" H 6560 2830 50  0001 C CNN
 F 1 "GND" H 6560 2930 50  0000 C CNN
 F 2 "" H 6560 3080 50  0001 C CNN
@@
 AR Path="/5E01BCC3/5E024C29" Ref="R?"  Part="1"
 AR Path="/5E697952/5E024C29" Ref="R?"  Part="1"
-AR Path="/5EAE2F15/5E024C29" Ref="R1002"  Part="1"
-F 0 "R1002" V 6070 2560 50  0000 R CNN
+AR Path="/5EAE2F15/5E024C29" Ref="R1003"  Part="1"
+F 0 "R1003" V 6070 2560 50  0000 R CNN
 F 1 "100" V 6110 2700 50  0000 C CNN
 F 2 "Resistors_SMD:R_0402" H 6110 2700 50  0001 C CNN
@@
 F 5 "1%" V 6310 2700 50  0001 C CNN "Tolerance"
 F 6 "1/16W" V 6410 2700 50  0001 C CNN "Wattage"
-F 7 "" H 6410 3100 60  0001 C CNN "Digi-Key PN"
+F 7 "DNP" V 6000 2700 60  0000 C CNN "Digi-Key PN"
 	1    6110 2700
 	0    -1   1    0
@@
 AR Path="/5E01BCC3/5E0269C4" Ref="R?"  Part="1"
 AR Path="/5E697952/5E0269C4" Ref="R?"  Part="1"
-AR Path="/5EAE2F15/5E0269C4" Ref="R1001"  Part="1"
-F 0 "R1001" H 4900 2930 50  0000 R CNN
+AR Path="/5EAE2F15/5E0269C4" Ref="R1002"  Part="1"
+F 0 "R1002" H 4900 2930 50  0000 R CNN
 F 1 "10k" V 4960 2930 50  0000 C CNN
 F 2 "Resistors_SMD:R_0402" H 4960 2930 50  0001 C CNN
@@
 F 5 "1%" H 5030 2930 50  0000 L CNN "Tolerance"
 F 6 "1/16W" H 5030 2860 50  0000 L CNN "Wattage"
-F 7 "" H 4960 2930 50  0001 C CNN "Digi-Key PN"
+F 7 "DNP" H 5350 2930 50  0000 C CNN "Configuration"
 	1    4960 2930
 	-1   0    0    -1
@@
 F 3 "~" H 5040 1800 50  0001 C CNN
 F 4 "490-5441-1-ND" H -3150 -1290 50  0001 C CNN "Digi-Key PN"
-F 5 "EXT_OSC" V 4840 1810 50  0000 C CNN "Configuration"
+F 5 "DNP" V 4840 1810 50  0000 C CNN "Configuration"
 	1    5040 1800
 	0    1    1    0
@@
 	5510 1730 5510 1800
 $Comp
-L power:+3.3V #PWR01001
+L power:+3.3V #PWR01002
 U 1 1 5E6E8CA9
 P 4530 1720
-F 0 "#PWR01001" H 4530 1570 50  0001 C CNN
+F 0 "#PWR01002" H 4530 1570 50  0001 C CNN
 F 1 "+3.3V" H 4530 1860 50  0000 C CNN
 F 2 "" H 4530 1720 50  0001 C CNN
@@
 AR Path="/5E01BCC3/5EC05874" Ref="R?"  Part="1"
 AR Path="/5E697952/5EC05874" Ref="R?"  Part="1"
-AR Path="/5EAE2F15/5EC05874" Ref="R1006"  Part="1"
-F 0 "R1006" H 2700 5360 50  0000 R CNN
+AR Path="/5EAE2F15/5EC05874" Ref="R1001"  Part="1"
+F 0 "R1001" H 2700 5360 50  0000 R CNN
 F 1 "10k" V 2760 5360 50  0000 C CNN
 F 2 "Resistors_SMD:R_0402" H 2760 5360 50  0001 C CNN
@@
 $EndComp
 $Comp
-L power:GND #PWR0101
+L power:GND #PWR01001
 U 1 1 5EC063B5
 P 2760 5510
-F 0 "#PWR0101" H 2760 5260 50  0001 C CNN
+F 0 "#PWR01001" H 2760 5260 50  0001 C CNN
 F 1 "GND" H 2760 5360 50  0000 C CNN
 F 2 "" H 2760 5510 50  0001 C CNN
@@
 AR Path="/5EAE3021/5FE10797" Ref="C?"  Part="1"
 AR Path="/5EAE30C7/5FE10797" Ref="C?"  Part="1"
-AR Path="/5EAE2F15/5FE10797" Ref="C?"  Part="1"
-F 0 "C?" H 6755 2130 50  0000 L CNN
+AR Path="/5EAE2F15/5FE10797" Ref="C1002"  Part="1"
+F 0 "C1002" H 6755 2130 50  0000 L CNN
 F 1 "10uF" H 6755 1930 50  0000 L CNN
 F 2 "Capacitors_SMD:C_0402" H 6768 1880 50  0001 C CNN
@@
 F 5 "6.3V" H 6580 2030 50  0000 R CNN "Voltage"
 F 6 "X5R" H 6580 1930 50  0000 R CNN "Dielectric"
-F 7 "" H 6730 2030 50  0001 C CNN "Digi-Key PN"
+F 7 "DNP" H 7050 2030 50  0000 C CNN "Digi-Key PN"
 	1    6730 2030
 	1    0    0    -1
@@
 AR Path="/5EAE30C7/5FE107A1" Ref="C?"  Part="1"
 AR Path="/5EAE2F02/5FE107A1" Ref="C?"  Part="1"
-AR Path="/5EAE2F15/5FE107A1" Ref="C?"  Part="1"
-F 0 "C?" H 6115 2130 50  0000 L CNN
+AR Path="/5EAE2F15/5FE107A1" Ref="C1001"  Part="1"
+F 0 "C1001" H 6115 2130 50  0000 L CNN
 F 1 "0.1uF" H 6115 1930 50  0000 L CNN
 F 2 "Capacitors_SMD:C_0402" H 6128 1880 50  0001 C CNN
@@
 F 5 "50V" H 5940 2030 50  0000 R CNN "Voltage"
 F 6 "X7R" H 5940 1930 50  0000 R CNN "Dielectric"
-F 7 "" H 6515 2530 60  0001 C CNN "Digi-Key PN"
+F 7 "DNP" H 5670 2030 50  0000 C CNN "Digi-Key PN"
 	1    6090 2030
 	1    0    0    -1
 $EndComp
 $Comp
-L power:GND #PWR?
+L power:GND #PWR01005
 U 1 1 5FE10E08
 P 6090 2180
-F 0 "#PWR?" H 6090 1930 50  0001 C CNN
+F 0 "#PWR01005" H 6090 1930 50  0001 C CNN
 F 1 "GND" H 6090 2030 50  0000 C CNN
 F 2 "" H 6090 2180 50  0001 C CNN
@@
 $EndComp
 $Comp
-L power:GND #PWR?
+L power:GND #PWR01007
 U 1 1 5FE10FFC
 P 6730 2180
-F 0 "#PWR?" H 6730 1930 50  0001 C CNN
+F 0 "#PWR01007" H 6730 1930 50  0001 C CNN
 F 1 "GND" H 6730 2030 50  0000 C CNN
 F 2 "" H 6730 2180 50  0001 C CNN

Commit message: assigned digikey PNs
Parts:
- C1001: Digi-Key PN DNP -> 490-10698-1-ND; Voltage 50V -> 25V
- C1002: Digi-Key PN DNP -> 1276-6830-1-ND; Voltage 6.3V -> 10V
- R1001, R1002, R1004: Digi-Key PN (none) -> RMCF0402FT10K0CT-ND
- R1003: Digi-Key PN DNP -> RMCF0402FT100RCT-ND
Changed lines of the file:
@@
 F 5 "1%" H 6630 2930 50  0000 L CNN "Tolerance"
 F 6 "1/16W" H 6630 2860 50  0000 L CNN "Wattage"
-F 7 "" H 6560 2930 50  0001 C CNN "Digi-Key PN"
+F 7 "RMCF0402FT10K0CT-ND" H 6560 2930 50  0001 C CNN "Digi-Key PN"
 	1    6560 2930
 	-1   0    0    -1
@@
 F 5 "1%" V 6310 2700 50  0001 C CNN "Tolerance"
 F 6 "1/16W" V 6410 2700 50  0001 C CNN "Wattage"
-F 7 "DNP" V 6000 2700 60  0000 C CNN "Digi-Key PN"
+F 7 "RMCF0402FT100RCT-ND" V 6000 2700 60  0000 C CNN "Digi-Key PN"
 	1    6110 2700
 	0    -1   1    0
@@
 F 6 "1/16W" H 5030 2860 50  0000 L CNN "Wattage"
 F 7 "DNP" H 5350 2930 50  0000 C CNN "Configuration"
+F 8 "RMCF0402FT10K0CT-ND" H 4960 2930 50  0001 C CNN "Digi-Key PN"
 	1    4960 2930
 	-1   0    0    -1
@@
 F 5 "1%" H 2830 5360 50  0000 L CNN "Tolerance"
 F 6 "1/16W" H 2830 5290 50  0000 L CNN "Wattage"
-F 7 "" H 2760 5360 50  0001 C CNN "Digi-Key PN"
+F 7 "RMCF0402FT10K0CT-ND" H 2760 5360 50  0001 C CNN "Digi-Key PN"
 	1    2760 5360
 	-1   0    0    -1
@@
 F 3 "" H 6755 2130 50  0001 C CNN
 F 4 "0402" H 6580 2130 50  0000 R CNN "display_footprint"
-F 5 "6.3V" H 6580 2030 50  0000 R CNN "Voltage"
+F 5 "10V" H 6580 2030 50  0000 R CNN "Voltage"
 F 6 "X5R" H 6580 1930 50  0000 R CNN "Dielectric"
-F 7 "DNP" H 7050 2030 50  0000 C CNN "Digi-Key PN"
+F 7 "1276-6830-1-ND" H 7050 2030 50  0000 C CNN "Digi-Key PN"
 	1    6730 2030
 	1    0    0    -1
@@
 F 3 "" H 6115 2130 50  0001 C CNN
 F 4 "0402" H 5940 2130 50  0000 R CNN "display_footprint"
-F 5 "50V" H 5940 2030 50  0000 R CNN "Voltage"
+F 5 "25V" H 5940 2030 50  0000 R CNN "Voltage"
 F 6 "X7R" H 5940 1930 50  0000 R CNN "Dielectric"
-F 7 "DNP" H 5670 2030 50  0000 C CNN "Digi-Key PN"
+F 7 "490-10698-1-ND" H 5670 2030 50  0000 C CNN "Digi-Key PN"
 	1    6090 2030
 	1    0    0    -1
