File: hdw/rev_b/Pulse_Oximeter/POS1P8_Telemetry.sch (KiCad schematic (older format))
At the start: 7 parts, among them U702 MCP9804, U703 INA219BxDCN

Commit message: fixed some component configurations in sch, regenerated netlist
Parts:
- C703, C704, C705: Configuration (none) -> Telemetry; display_footprint (none) -> 0402
Changed lines of the file:
@@
 Sheet 7 21
 Title "Pulse Oximeter"
-Date "2020-08-01"
-Rev "A"
+Date "2020-12-09"
+Rev "B"
 Comp "Drew Maatman"
 Comment1 ""
@@
 NoConn ~ 5030 4840
 $Comp
-L Custom_Library:C_Custom C?
-U 1 1 5E2AA9A5
-P 5430 5990
-AR Path="/5B3E071A/5E2AA9A5" Ref="C?"  Part="1"
-AR Path="/5E0652BA/5E2AA9A5" Ref="C?"  Part="1"
-AR Path="/5E0A0E29/5E2AA9A5" Ref="C?"  Part="1"
-AR Path="/5E0DC084/5E2AA9A5" Ref="C?"  Part="1"
-AR Path="/5E0F263C/5E2AA9A5" Ref="C?"  Part="1"
-AR Path="/5EAE2E6F/5E2AA9A5" Ref="C703"  Part="1"
-F 0 "C703" H 5455 6090 50  0000 L CNN
-F 1 "0.1uF" H 5455 5890 50  0000 L CNN
-F 2 "Capacitors_SMD:C_0402" H 5468 5840 50  0001 C CNN
-F 3 "" H 5455 6090 50  0001 C CNN
-F 4 "" H 5280 6090 50  0000 R CNN "display_footprint"
-F 5 "50V" H 5280 5990 50  0000 R CNN "Voltage"
-F 6 "X7R" H 5280 5890 50  0000 R CNN "Dielectric"
-F 7 "490-10701-1-ND" H 1520 -890 50  0001 C CNN "Digi-Key PN"
-	1    5430 5990
-	1    0    0    -1
-$EndComp
-$Comp
 L power:+3.3V #PWR?
 U 1 1 5E2AA9A9
@@
 I2C_SCL
 $Comp
-L Custom_Library:C_Custom C?
-U 1 1 5E1C2940
-P 7470 3180
-AR Path="/5B3E071A/5E1C2940" Ref="C?"  Part="1"
-AR Path="/5E0652BA/5E1C2940" Ref="C?"  Part="1"
-AR Path="/5E0A0E29/5E1C2940" Ref="C?"  Part="1"
-AR Path="/5E052856/5E1C2940" Ref="C?"  Part="1"
-AR Path="/5EAE2E6F/5E1C2940" Ref="C705"  Part="1"
-F 0 "C705" H 7495 3280 50  0000 L CNN
-F 1 "0.1uF" H 7495 3080 50  0000 L CNN
-F 2 "Capacitors_SMD:C_0402" H 7508 3030 50  0001 C CNN
-F 3 "" H 7495 3280 50  0001 C CNN
-F 4 "" H 7320 3280 50  0000 R CNN "display_footprint"
-F 5 "50V" H 7320 3180 50  0000 R CNN "Voltage"
-F 6 "X7R" H 7320 3080 50  0000 R CNN "Dielectric"
-F 7 "490-10701-1-ND" H 3560 -3700 50  0001 C CNN "Digi-Key PN"
-	1    7470 3180
-	1    0    0    -1
-$EndComp
-$Comp
 L power:+3.3V #PWR?
 U 1 1 5EC52D17
@@
 Wire Wire Line
 	6590 2050 6590 1970
-$Comp
-L Custom_Library:C_Custom C?
-U 1 1 5EC52D19
-P 6590 2200
-AR Path="/5B3E071A/5EC52D19" Ref="C?"  Part="1"
-AR Path="/5E0652BA/5EC52D19" Ref="C?"  Part="1"
-AR Path="/5E0A0E29/5EC52D19" Ref="C?"  Part="1"
-AR Path="/5E052856/5EC52D19" Ref="C?"  Part="1"
-AR Path="/5EAE2E6F/5EC52D19" Ref="C704"  Part="1"
-F 0 "C704" H 6615 2300 50  0000 L CNN
-F 1 "0.1uF" H 6615 2100 50  0000 L CNN
-F 2 "Capacitors_SMD:C_0402" H 6628 2050 50  0001 C CNN
-F 3 "" H 6615 2300 50  0001 C CNN
-F 4 "" H 6440 2300 50  0000 R CNN "display_footprint"
-F 5 "50V" H 6440 2200 50  0000 R CNN "Voltage"
-F 6 "X7R" H 6440 2100 50  0000 R CNN "Dielectric"
-F 7 "490-10701-1-ND" H 2680 -4680 50  0001 C CNN "Digi-Key PN"
-	1    6590 2200
-	1    0    0    -1
-$EndComp
 Wire Wire Line
 	6150 2430 6590 2430
@@
 	0    1    -1   0
 $EndComp
+$Comp
+L Custom_Library:C_Custom C?
+U 1 1 5FD2CD38
+P 6590 2200
+AR Path="/5B3E071A/5FD2CD38" Ref="C?"  Part="1"
+AR Path="/5E0652BA/5FD2CD38" Ref="C?"  Part="1"
+AR Path="/5E0A0E29/5FD2CD38" Ref="C?"  Part="1"
+AR Path="/5E052856/5FD2CD38" Ref="C?"  Part="1"
+AR Path="/5EAE2D84/5FD2CD38" Ref="C?"  Part="1"
+AR Path="/5EAE2E6F/5FD2CD38" Ref="C704"  Part="1"
+F 0 "C704" H 6615 2300 50  0000 L CNN
+F 1 "0.1uF" H 6615 2100 50  0000 L CNN
+F 2 "Capacitors_SMD:C_0402" H 6628 2050 50  0001 C CNN
+F 3 "" H 6615 2300 50  0001 C CNN
+F 4 "0402" H 6440 2300 50  0000 R CNN "display_footprint"
+F 5 "50V" H 6440 2200 50  0000 R CNN "Voltage"
+F 6 "X7R" H 6440 2100 50  0000 R CNN "Dielectric"
+F 7 "490-10701-1-ND" H 2680 -4680 50  0001 C CNN "Digi-Key PN"
+F 8 "Telemetry" H 6060 2200 50  0000 C CNN "Configuration"
+	1    6590 2200
+	1    0    0    -1
+$EndComp
+$Comp
+L Custom_Library:C_Custom C?
+U 1 1 5FD2EE9B
+P 7470 3180
+AR Path="/5B3E071A/5FD2EE9B" Ref="C?"  Part="1"
+AR Path="/5E0652BA/5FD2EE9B" Ref="C?"  Part="1"
+AR Path="/5E0A0E29/5FD2EE9B" Ref="C?"  Part="1"
+AR Path="/5E052856/5FD2EE9B" Ref="C?"  Part="1"
+AR Path="/5EAE2D84/5FD2EE9B" Ref="C?"  Part="1"
+AR Path="/5EAE2E6F/5FD2EE9B" Ref="C705"  Part="1"
+F 0 "C705" H 7495 3280 50  0000 L CNN
+F 1 "0.1uF" H 7495 3080 50  0000 L CNN
+F 2 "Capacitors_SMD:C_0402" H 7508 3030 50  0001 C CNN
+F 3 "" H 7495 3280 50  0001 C CNN
+F 4 "0402" H 7320 3280 50  0000 R CNN "display_footprint"
+F 5 "50V" H 7320 3180 50  0000 R CNN "Voltage"
+F 6 "X7R" H 7320 3080 50  0000 R CNN "Dielectric"
+F 7 "490-10701-1-ND" H 3560 -3700 50  0001 C CNN "Digi-Key PN"
+F 8 "Telemetry" H 6940 3180 50  0000 C CNN "Configuration"
+	1    7470 3180
+	1    0    0    -1
+$EndComp
+$Comp
+L Custom_Library:C_Custom C?
+U 1 1 5FD2F371
+P 5430 5990
+AR Path="/5B3E071A/5FD2F371" Ref="C?"  Part="1"
+AR Path="/5E0652BA/5FD2F371" Ref="C?"  Part="1"
+AR Path="/5E0A0E29/5FD2F371" Ref="C?"  Part="1"
+AR Path="/5E052856/5FD2F371" Ref="C?"  Part="1"
+AR Path="/5EAE2D84/5FD2F371" Ref="C?"  Part="1"
+AR Path="/5EAE2E6F/5FD2F371" Ref="C703"  Part="1"
+F 0 "C703" H 5455 6090 50  0000 L CNN
+F 1 "0.1uF" H 5455 5890 50  0000 L CNN
+F 2 "Capacitors_SMD:C_0402" H 5468 5840 50  0001 C CNN
+F 3 "" H 5455 6090 50  0001 C CNN
+F 4 "0402" H 5280 6090 50  0000 R CNN "display_footprint"
+F 5 "50V" H 5280 5990 50  0000 R CNN "Voltage"
+F 6 "X7R" H 5280 5890 50  0000 R CNN "Dielectric"
+F 7 "490-10701-1-ND" H 1520 -890 50  0001 C CNN "Digi-Key PN"
+F 8 "Telemetry" H 4900 5990 50  0000 C CNN "Configuration"
+	1    5430 5990
+	1    0    0    -1
+$EndComp
 $EndSCHEMATC

Commit message: changed all passives to 0402, cleared digikey pns
Parts:
- C703, C704, C705: Digi-Key PN 490-10701-1-ND -> (none)
Changed lines of the file:
@@
 F 5 "50V" H 6440 2200 50  0000 R CNN "Voltage"
 F 6 "X7R" H 6440 2100 50  0000 R CNN "Dielectric"
-F 7 "490-10701-1-ND" H 2680 -4680 50  0001 C CNN "Digi-Key PN"
+F 7 "" H 2680 -4680 50  0001 C CNN "Digi-Key PN"
 F 8 "Telemetry" H 6060 2200 50  0000 C CNN "Configuration"
 	1    6590 2200
@@
 F 5 "50V" H 7320 3180 50  0000 R CNN "Voltage"
 F 6 "X7R" H 7320 3080 50  0000 R CNN "Dielectric"
-F 7 "490-10701-1-ND" H 3560 -3700 50  0001 C CNN "Digi-Key PN"
+F 7 "" H 3560 -3700 50  0001 C CNN "Digi-Key PN"
 F 8 "Telemetry" H 6940 3180 50  0000 C CNN "Configuration"
 	1    7470 3180
@@
 F 5 "50V" H 5280 5990 50  0000 R CNN "Voltage"
 F 6 "X7R" H 5280 5890 50  0000 R CNN "Dielectric"
-F 7 "490-10701-1-ND" H 1520 -890 50  0001 C CNN "Digi-Key PN"
+F 7 "" H 1520 -890 50  0001 C CNN "Digi-Key PN"
 F 8 "Telemetry" H 4900 5990 50  0000 C CNN "Configuration"
 	1    5430 5990

Commit message: annotated schematic
Parts:
- renumbered C703 to C701, C704 to C702, C705 to C703, DOC702 to DOC701, DOC703 to DOC702, U702 to U701, U703 to U702
Changed lines of the file:
@@
 AR Path="/5E0DC084/5EC52D1B" Ref="#PWR?"  Part="1"
 AR Path="/5E0F263C/5EC52D1B" Ref="#PWR?"  Part="1"
-AR Path="/5EAE2E6F/5EC52D1B" Ref="#PWR0707"  Part="1"
-F 0 "#PWR0707" H 5430 5170 50  0001 C CNN
+AR Path="/5EAE2E6F/5EC52D1B" Ref="#PWR0702"  Part="1"
+F 0 "#PWR0702" H 5430 5170 50  0001 C CNN
 F 1 "GND" H 5430 5270 50  0000 C CNN
 F 2 "" H 5430 5420 50  0001 C CNN
@@
 AR Path="/5E0DC084/5EC52D1C" Ref="#PWR?"  Part="1"
 AR Path="/5E0F263C/5EC52D1C" Ref="#PWR?"  Part="1"
-AR Path="/5EAE2E6F/5EC52D1C" Ref="#PWR0706"  Part="1"
-F 0 "#PWR0706" H 5430 4190 50  0001 C CNN
+AR Path="/5EAE2E6F/5EC52D1C" Ref="#PWR0701"  Part="1"
+F 0 "#PWR0701" H 5430 4190 50  0001 C CNN
 F 1 "+3.3V" H 5430 4480 50  0000 C CNN
 F 2 "" H 5430 4340 50  0001 C CNN
@@
 AR Path="/5E0DC084/5E0BDB9D" Ref="U?"  Part="1"
 AR Path="/5E0F263C/5E0BDB9D" Ref="U?"  Part="1"
-AR Path="/5EAE2E6F/5E0BDB9D" Ref="U702"  Part="1"
-F 0 "U702" H 5180 5290 50  0000 C CNN
+AR Path="/5EAE2E6F/5E0BDB9D" Ref="U701"  Part="1"
+F 0 "U701" H 5180 5290 50  0000 C CNN
 F 1 "MCP9804" H 5830 5290 50  0000 C CNN
 F 2 "Package_DFN_QFN:DFN-8-1EP_3x2mm_P0.5mm_EP1.3x1.5mm" H 4330 4340 50  0001 C CNN
@@
 AR Path="/5E0DC084/5E2AA9A9" Ref="#PWR?"  Part="1"
 AR Path="/5E0F263C/5E2AA9A9" Ref="#PWR?"  Part="1"
-AR Path="/5EAE2E6F/5E2AA9A9" Ref="#PWR0708"  Part="1"
-F 0 "#PWR0708" H 5430 5690 50  0001 C CNN
+AR Path="/5EAE2E6F/5E2AA9A9" Ref="#PWR0703"  Part="1"
+F 0 "#PWR0703" H 5430 5690 50  0001 C CNN
 F 1 "+3.3V" H 5430 5980 50  0000 C CNN
 F 2 "" H 5430 5840 50  0001 C CNN
@@
 AR Path="/5E0DC084/5EC52D1F" Ref="#PWR?"  Part="1"
 AR Path="/5E0F263C/5EC52D1F" Ref="#PWR?"  Part="1"
-AR Path="/5EAE2E6F/5EC52D1F" Ref="#PWR0709"  Part="1"
-F 0 "#PWR0709" H 5430 5890 50  0001 C CNN
+AR Path="/5EAE2E6F/5EC52D1F" Ref="#PWR0704"  Part="1"
+F 0 "#PWR0704" H 5430 5890 50  0001 C CNN
 F 1 "GND" H 5430 5990 50  0000 C CNN
 F 2 "" H 5430 6140 50  0001 C CNN
@@
 AR Path="/5E0A0E29/5E1C292F" Ref="#PWR?"  Part="1"
 AR Path="/5E052856/5E1C292F" Ref="#PWR?"  Part="1"
-AR Path="/5EAE2E6F/5E1C292F" Ref="#PWR0714"  Part="1"
-F 0 "#PWR0714" H 7470 2360 50  0001 C CNN
+AR Path="/5EAE2E6F/5E1C292F" Ref="#PWR0709"  Part="1"
+F 0 "#PWR0709" H 7470 2360 50  0001 C CNN
 F 1 "GND" H 7470 2460 50  0000 C CNN
 F 2 "" H 7470 2610 50  0001 C CNN
@@
 AR Path="/5E0A0E29/5E1C2935" Ref="#PWR?"  Part="1"
 AR Path="/5E052856/5E1C2935" Ref="#PWR?"  Part="1"
-AR Path="/5EAE2E6F/5E1C2935" Ref="#PWR0713"  Part="1"
-F 0 "#PWR0713" H 7470 1660 50  0001 C CNN
+AR Path="/5EAE2E6F/5E1C2935" Ref="#PWR0708"  Part="1"
+F 0 "#PWR0708" H 7470 1660 50  0001 C CNN
 F 1 "+3.3V" H 7470 1950 50  0000 C CNN
 F 2 "" H 7470 1810 50  0001 C CNN
@@
 AR Path="/5E0A0E29/5EC52D17" Ref="#PWR?"  Part="1"
 AR Path="/5E052856/5EC52D17" Ref="#PWR?"  Part="1"
-AR Path="/5EAE2E6F/5EC52D17" Ref="#PWR0715"  Part="1"
-F 0 "#PWR0715" H 7470 2880 50  0001 C CNN
+AR Path="/5EAE2E6F/5EC52D17" Ref="#PWR0710"  Part="1"
+F 0 "#PWR0710" H 7470 2880 50  0001 C CNN
 F 1 "+3.3V" H 7470 3170 50  0000 C CNN
 F 2 "" H 7470 3030 50  0001 C CNN
@@
 AR Path="/5E0A0E29/5EC52D18" Ref="#PWR?"  Part="1"
 AR Path="/5E052856/5EC52D18" Ref="#PWR?"  Part="1"
-AR Path="/5EAE2E6F/5EC52D18" Ref="#PWR0716"  Part="1"
-F 0 "#PWR0716" H 7470 3080 50  0001 C CNN
+AR Path="/5EAE2E6F/5EC52D18" Ref="#PWR0711"  Part="1"
+F 0 "#PWR0711" H 7470 3080 50  0001 C CNN
 F 1 "GND" H 7470 3180 50  0000 C CNN
 F 2 "" H 7470 3330 50  0001 C CNN
@@
 	6150 1970 6590 1970
 $Comp
-L Analog_ADC:INA219BxDCN U703
+L Analog_ADC:INA219BxDCN U702
 U 1 1 5EC52D1A
 P 7470 2210
-F 0 "U703" H 7220 2560 50  0000 C CNN
+F 0 "U702" H 7220 2560 50  0000 C CNN
 F 1 "INA219BxDCN" H 7720 2560 50  0000 C CNN
 F 2 "Package_TO_SOT_SMD:SOT-23-8" H 8120 1860 50  0001 C CNN
@@
 AR Path="/5E052856/5EC3148F" Ref="DOC?"  Part="1"
 AR Path="/5EAE2DDC/5EC3148F" Ref="DOC?"  Part="1"
-AR Path="/5EAE2E6F/5EC3148F" Ref="DOC703"  Part="1"
-F 0 "DOC703" H 8370 3300 60  0001 C CNN
+AR Path="/5EAE2E6F/5EC3148F" Ref="DOC702"  Part="1"
+F 0 "DOC702" H 8370 3300 60  0001 C CNN
 F 1 "0x44" H 7920 3050 60  0000 L CNN
 F 2 "" H 8370 3400 60  0001 C CNN
@@
 P 7870 2410
 AR Path="/5EAE2DDC/5EC31495" Ref="#PWR?"  Part="1"
-AR Path="/5EAE2E6F/5EC31495" Ref="#PWR0718"  Part="1"
-F 0 "#PWR0718" H 7870 2160 50  0001 C CNN
+AR Path="/5EAE2E6F/5EC31495" Ref="#PWR0713"  Part="1"
+F 0 "#PWR0713" H 7870 2160 50  0001 C CNN
 F 1 "GND" V 7870 2260 50  0000 R CNN
 F 2 "" H 7870 2410 50  0001 C CNN
@@
 AR Path="/5E0A0E29/5EC31886" Ref="#PWR?"  Part="1"
 AR Path="/5E052856/5EC31886" Ref="#PWR?"  Part="1"
-AR Path="/5EAE2E6F/5EC31886" Ref="#PWR0717"  Part="1"
-F 0 "#PWR0717" H 7870 2160 50  0001 C CNN
+AR Path="/5EAE2E6F/5EC31886" Ref="#PWR0712"  Part="1"
+F 0 "#PWR0712" H 7870 2160 50  0001 C CNN
 F 1 "+3.3V" V 7870 2450 50  0000 L CNN
 F 2 "" H 7870 2310 50  0001 C CNN
@@
 AR Path="/5E0F263C/5EC37016" Ref="DOC?"  Part="1"
 AR Path="/5EAE2DDC/5EC37016" Ref="DOC?"  Part="1"
-AR Path="/5EAE2E6F/5EC37016" Ref="DOC702"  Part="1"
-F 0 "DOC702" H 6330 6110 60  0001 C CNN
+AR Path="/5EAE2E6F/5EC37016" Ref="DOC701"  Part="1"
+F 0 "DOC701" H 6330 6110 60  0001 C CNN
 F 1 "0x1A" H 5880 5860 60  0000 L CNN
 F 2 "" H 6330 6210 60  0001 C CNN
@@
 P 5830 4940
 AR Path="/5EAE2DDC/5EC3701C" Ref="#PWR?"  Part="1"
-AR Path="/5EAE2E6F/5EC3701C" Ref="#PWR0710"  Part="1"
-F 0 "#PWR0710" H 5830 4690 50  0001 C CNN
+AR Path="/5EAE2E6F/5EC3701C" Ref="#PWR0705"  Part="1"
+F 0 "#PWR0705" H 5830 4690 50  0001 C CNN
 F 1 "GND" V 5830 4790 50  0000 R CNN
 F 2 "" H 5830 4940 50  0001 C CNN
@@
 P 5830 5140
 AR Path="/5EAE2DDC/5EC37022" Ref="#PWR?"  Part="1"
-AR Path="/5EAE2E6F/5EC37022" Ref="#PWR0712"  Part="1"
-F 0 "#PWR0712" H 5830 4890 50  0001 C CNN
+AR Path="/5EAE2E6F/5EC37022" Ref="#PWR0707"  Part="1"
+F 0 "#PWR0707" H 5830 4890 50  0001 C CNN
 F 1 "GND" V 5830 4990 50  0000 R CNN
 F 2 "" H 5830 5140 50  0001 C CNN
@@
 AR Path="/5E0F263C/5EC37028" Ref="#PWR?"  Part="1"
 AR Path="/5EAE2DDC/5EC37028" Ref="#PWR?"  Part="1"
-AR Path="/5EAE2E6F/5EC37028" Ref="#PWR0711"  Part="1"
-F 0 "#PWR0711" H 5830 4890 50  0001 C CNN
+AR Path="/5EAE2E6F/5EC37028" Ref="#PWR0706"  Part="1"
+F 0 "#PWR0706" H 5830 4890 50  0001 C CNN
 F 1 "+3.3V" V 5830 5180 50  0000 L CNN
 F 2 "" H 5830 5040 50  0001 C CNN
@@
 AR Path="/5E052856/5FD2CD38" Ref="C?"  Part="1"
 AR Path="/5EAE2D84/5FD2CD38" Ref="C?"  Part="1"
-AR Path="/5EAE2E6F/5FD2CD38" Ref="C704"  Part="1"
-F 0 "C704" H 6615 2300 50  0000 L CNN
+AR Path="/5EAE2E6F/5FD2CD38" Ref="C702"  Part="1"
+F 0 "C702" H 6615 2300 50  0000 L CNN
 F 1 "0.1uF" H 6615 2100 50  0000 L CNN
 F 2 "Capacitors_SMD:C_0402" H 6628 2050 50  0001 C CNN
@@
 AR Path="/5E052856/5FD2EE9B" Ref="C?"  Part="1"
 AR Path="/5EAE2D84/5FD2EE9B" Ref="C?"  Part="1"
-AR Path="/5EAE2E6F/5FD2EE9B" Ref="C705"  Part="1"
-F 0 "C705" H 7495 3280 50  0000 L CNN
+AR Path="/5EAE2E6F/5FD2EE9B" Ref="C703"  Part="1"
+F 0 "C703" H 7495 3280 50  0000 L CNN
 F 1 "0.1uF" H 7495 3080 50  0000 L CNN
 F 2 "Capacitors_SMD:C_0402" H 7508 3030 50  0001 C CNN
@@
 AR Path="/5E052856/5FD2F371" Ref="C?"  Part="1"
 AR Path="/5EAE2D84/5FD2F371" Ref="C?"  Part="1"
-AR Path="/5EAE2E6F/5FD2F371" Ref="C703"  Part="1"
-F 0 "C703" H 5455 6090 50  0000 L CNN
+AR Path="/5EAE2E6F/5FD2F371" Ref="C701"  Part="1"
+F 0 "C701" H 5455 6090 50  0000 L CNN
 F 1 "0.1uF" H 5455 5890 50  0000 L CNN
 F 2 "Capacitors_SMD:C_0402" H 5468 5840 50  0001 C CNN

Commit message: assigned digikey PNs
Parts:
- C701, C702, C703: Digi-Key PN (none) -> 490-10698-1-ND; Voltage 50V -> 25V
Changed lines of the file:
@@
 F 3 "" H 6615 2300 50  0001 C CNN
 F 4 "0402" H 6440 2300 50  0000 R CNN "display_footprint"
-F 5 "50V" H 6440 2200 50  0000 R CNN "Voltage"
+F 5 "25V" H 6440 2200 50  0000 R CNN "Voltage"
 F 6 "X7R" H 6440 2100 50  0000 R CNN "Dielectric"
-F 7 "" H 2680 -4680 50  0001 C CNN "Digi-Key PN"
+F 7 "490-10698-1-ND" H 2680 -4680 50  0001 C CNN "Digi-Key PN"
 F 8 "Telemetry" H 6060 2200 50  0000 C CNN "Configuration"
 	1    6590 2200
@@
 F 3 "" H 7495 3280 50  0001 C CNN
 F 4 "0402" H 7320 3280 50  0000 R CNN "display_footprint"
-F 5 "50V" H 7320 3180 50  0000 R CNN "Voltage"
+F 5 "25V" H 7320 3180 50  0000 R CNN "Voltage"
 F 6 "X7R" H 7320 3080 50  0000 R CNN "Dielectric"
-F 7 "" H 3560 -3700 50  0001 C CNN "Digi-Key PN"
+F 7 "490-10698-1-ND" H 3560 -3700 50  0001 C CNN "Digi-Key PN"
 F 8 "Telemetry" H 6940 3180 50  0000 C CNN "Configuration"
 	1    7470 3180
@@
 F 3 "" H 5455 6090 50  0001 C CNN
 F 4 "0402" H 5280 6090 50  0000 R CNN "display_footprint"
-F 5 "50V" H 5280 5990 50  0000 R CNN "Voltage"
+F 5 "25V" H 5280 5990 50  0000 R CNN "Voltage"
 F 6 "X7R" H 5280 5890 50  0000 R CNN "Dielectric"
-F 7 "" H 1520 -890 50  0001 C CNN "Digi-Key PN"
+F 7 "490-10698-1-ND" H 1520 -890 50  0001 C CNN "Digi-Key PN"
 F 8 "Telemetry" H 4900 5990 50  0000 C CNN "Configuration"
 	1    5430 5990
