File: hdw/rev_b/Pulse_Oximeter/Pulse_Oximeter.kicad_pcb (KiCad board)
At the start: 4 copper layers, 100 x 50 mm, 267 parts, among them J1201 USB_B_Mini, J2001 I2C, J2002 USB UART, J201 +12V IN, J801 PICKIT3, Q201 Si4946BEY, Q401 BSS214NW, Q402 ZXMS6004FFTA, Q801 BSS214NW, SW1702 Cap_Touch, SW801 MRST, U1101 PIC32MZ0512EFE064T-I_PT, U1201 TLV6700, U1202 FT234XD, U1203 TPD3S014DBVR, U1301 INA219BxDCN, U1302 MCP9804, U1401 DS1683, U1501 TPS22929D, U1502 TCA9803, U1503 MAX30102, U1601 74LVC1G17, U1602 NHD-0420H1Z, U1702 TPS71530, U1704 AT42QT1010-TSHR, U1706 74LVC1G17, U1801 TPS71530, U1802 74LVC1G06, U1803 74LVC1G06, U1805 74LVC1G06, U1806 74LVC1G06, U1901 74LVC1G06, U1902 74LVC1G06, U1903 74LVC1G06, U1904 74LVC1G06, U2001 MCP9804, U201 LTC4365DDB, U301 INA219BxDCN, U302 MCP9804, U401 TPS62150, U502 MCP9804, U503 INA219BxDCN, U601 TPS7A91, U702 MCP9804, U703 INA219BxDCN, X1001 ASE-8.000MHz

Commit message: fixed some component configurations in sch, regenerated netlist
Parts:
- L1201: value 600R 0.5A -> DNP
- R1604: value 499 -> 10
Connections:
- R1604 pad 1: Net-(R1604-Pad1) -> LCD_BACKLIGHT
- R1604 pad 2: LCD_BACKLIGHT -> Net-(R1604-Pad2)
- U1601 pad 4: Net-(R1604-Pad1) -> Net-(R1604-Pad2)
Routing:
- net LCD_BACKLIGHT: track 2.30 -> 0.61 mm
- net Net-(R1604-Pad1): track 1.23 -> 0.00 mm

Commit message: started working on rev B PCB, a few SCH changes
Parts:
- removed C1003, C1604, C914, C918, C919: 10nF, Capacitors_SMD:C_0402
- removed C1005, C1513, C1605, C915, C920, C921: 1nF, Capacitors_SMD:C_0402
- removed C1514, C1706, C1708, C604, C913: 10uF, Capacitors_SMD:C_0402
- removed C1710, C1805, C1806, C204, C504, C505, C605, C704, C705, C916, C917: 0.1uF, Capacitors_SMD:C_0402
- removed C205: 100uF, Capacitors_Tantalum_SMD:CP_Tantalum_Case-X_EIA-7343-43_Reflow
- removed D1805: Green, LEDs:LED_0402
- removed G***: Microchip_Logo, Custom Footprints Library:Microchip_Logo
- removed G***: PIC32_Logo, Custom Footprints Library:PIC32_Logo
- removed G***: Owl_1_Logo, Custom Footprints Library:Owl_1_Logo
- removed H2301, H2302, H2303, H2304: MountingHole, MountingHole:MountingHole_3mm
- removed J2001: I2C, Connector_PinHeader_2.54mm:PinHeader_1x03_P2.54mm_Vertical
- removed J2002: USB UART, Connector_PinHeader_2.54mm:PinHeader_1x03_P2.54mm_Vertical
- removed Q201: Si4946BEY, Package_SO:SOIC-8_3.9x4.9mm_P1.27mm
- removed R1006, R1706: 10k, Resistors_SMD:R_0402
- removed REF**: Symbol_Barrel_Polarity, Symbol:Symbol_Barrel_Polarity
- removed RV1601: 10k, Potentiometer_SMD:Potentiometer_Vishay_TS53YL_Vertical
- removed SW1702: Cap_Touch, Custom Footprints Library:Capacitive_Touch_Pad
- removed U1704: AT42QT1010-TSHR, TO_SOT_Packages_SMD:SOT-23-6
- removed U1706: 74LVC1G17, TO_SOT_Packages_SMD:SOT-353_SC-70-5
- removed U1805, U1806: 74LVC1G06, TO_SOT_Packages_SMD:SOT-353_SC-70-5
- removed U503, U703: INA219BxDCN, Package_TO_SOT_SMD:SOT-23-8
- added C1002: 10uF, Capacitors_SMD:C_0402, F.Cu at (338.0, 139.2)
- added C1210: 0.1uF, Capacitors_SMD:C_0402, F.Cu at (248.6, 117.5)
- added C1211: 0.1uF, Capacitors_SMD:C_0402, F.Cu at (241.9, 121.7)
- added C1701: 10nF, Capacitors_SMD:C_0402, F.Cu at (419.7, 101.4)
- added C1703: 10uF, Capacitors_SMD:C_0402, F.Cu at (419.7, 103.4)
- added C2002: 0.1uF, Capacitors_SMD:C_0402, F.Cu at (305.4, 136.8)
- added C407: 10uF, Capacitors_SMD:C_1206, F.Cu at (327.3, 54.3)
- added C501: 0.1uF, Capacitors_SMD:C_0402, F.Cu at (335.1, 39.1)
- added C502: 0.1uF, Capacitors_SMD:C_0402, F.Cu at (338.2, 40.1)
- added C701: 0.1uF, Capacitors_SMD:C_0402, B.Cu at (64.8, 106.7)
- added C702: 0.1uF, Capacitors_SMD:C_0402, B.Cu at (61.5, 102.5)
- added D1803: Green, LEDs:LED_0402, F.Cu at (437.8, 147.3)
- added H2101: MountingHole, MountingHole:MountingHole_3mm, F.Cu at (285.8, 119.9)
- added H2102: MountingHole, MountingHole:MountingHole_3mm, F.Cu at (285.8, 127.5)
- added H2103: MountingHole, MountingHole:MountingHole_3mm, F.Cu at (293.3, 119.9)
- added H2104: MountingHole, MountingHole:MountingHole_3mm, F.Cu at (293.3, 127.5)
- added J1202: OSEPP_FTDI_01, Connector_PinHeader_2.54mm:PinHeader_1x06_P2.54mm_Vertical, F.Cu at (234.0, 110.5)
- added L1501: 600R 0.5A, Inductors_SMD:L_0402, F.Cu at (351.5, 127.6)
- added L1502: 600R 0.5A, Inductors_SMD:L_0402, F.Cu at (346.7, 133.8)
- added R1003: 100, Resistors_SMD:R_0402, F.Cu at (340.8, 139.2)
- added R1211: 0, Resistors_SMD:R_0402, F.Cu at (247.4, 124.1)
- added R1212: 0, Resistors_SMD:R_0402, F.Cu at (254.1, 116.1)
- added R1213: 27, Resistors_SMD:R_0402, F.Cu at (251.1, 119.8)
- added R1214: 27, Resistors_SMD:R_0402, F.Cu at (261.6, 109.3)
- added R1215: 10, Resistors_SMD:R_0402, F.Cu at (258.7, 111.7)
- added R1216: 100k, Resistors_SMD:R_0402, F.Cu at (247.7, 121.8)
- added R1217: 100k, Resistors_SMD:R_0402, F.Cu at (256.3, 114.0)
- added R1218: 0, Resistors_SMD:R_0402, F.Cu at (244.8, 124.1)
- added R1614: 10k, Resistors_SMD:R_0402, F.Cu at (401.5, 144.5)
- added R1615: 10k, Resistors_SMD:R_0402, F.Cu at (398.8, 148.8)
- added R1701: 1k, Resistors_SMD:R_0402, F.Cu at (420.4, 109.9)
- added R1703: 10k, Resistors_SMD:R_0402, F.Cu at (422.0, 105.6)
- added R1803: 1k, Resistors_SMD:R_0402, F.Cu at (440.7, 145.3)
- added R2003: 10k, Resistors_SMD:R_0402, F.Cu at (307.8, 138.9)
- added R2004: 10, Resistors_SMD:R_0402, F.Cu at (305.2, 138.9)
- added R214: 10k, Resistors_SMD:R_0402, F.Cu at (60.1, 86.9)
- added R215: 1k, Resistors_SMD:R_0402, F.Cu at (66.2, 89.4)
- added R216: 1k, Resistors_SMD:R_0402, F.Cu at (64.5, 89.4)
- added R217: 1k, Resistors_SMD:R_0402, F.Cu at (64.5, 88.4)
- added R218: 10k, Resistors_SMD:R_0402, F.Cu at (65.0, 86.9)
- added R219: 10k, Resistors_SMD:R_0402, F.Cu at (63.0, 86.9)
- added R220: 10k, Resistors_SMD:R_0402, F.Cu at (64.0, 86.9)
- added R401: 10k, Resistors_SMD:R_0402, F.Cu at (348.2, 53.5)
- added R402: 0, Resistors_SMD:R_0402, F.Cu at (339.1, 61.6)
- added R404: 10k, Resistors_SMD:R_0402, F.Cu at (351.2, 49.2)
- added R412: 0, Resistors_SMD:R_0402, F.Cu at (342.9, 53.0)
- added R413: 0, Resistors_SMD:R_0402, F.Cu at (335.9, 59.5)
- added R414: 10, Resistors_SMD:R_0402, F.Cu at (348.5, 49.2)
- added R415: 562k, Resistors_SMD:R_0402, F.Cu at (338.5, 59.5)
- added R416: 180k, Resistors_SMD:R_0402, F.Cu at (342.9, 55.2)
- added R603: 100, Resistors_SMD:R_0402, F.Cu at (63.4, 105.7)
- added R604: 100, Resistors_SMD:R_0402, F.Cu at (63.4, 104.6)
- added R605: 10, Resistors_SMD:R_0402, F.Cu at (61.6, 103.0)
- added SW1701: Cap_Touch, Custom Footprints Library:Capacitive_Touch_Pad, F.Cu at (407.6, 106.1)
- added U1204: TPD3S014DBVR, TO_SOT_Packages_SMD:SOT-23-6, F.Cu at (254.9, 110.5)
- added U1701: AT42QT1010-TSHR, TO_SOT_Packages_SMD:SOT-23-6, F.Cu at (415.8, 102.7)
- added U1804: 74LVC1G97, Package_TO_SOT_SMD:SOT-363_SC-70-6, F.Cu at (429.9, 144.0)
- added U2002: LTC1694, Package_TO_SOT_SMD:SOT-23-5, F.Cu at (301.4, 138.1)
- added U402: TPS62152, Package_DFN_QFN:QFN-16-1EP_3x3mm_P0.5mm_EP1.8x1.8mm, F.Cu at (332.7, 55.4)
- added U501: MCP9804, Package_DFN_QFN:DFN-8-1EP_3x2mm_P0.5mm_EP1.3x1.5mm, F.Cu at (336.2, 36.3)
- added U701: MCP9804, Package_DFN_QFN:DFN-8-1EP_3x2mm_P0.5mm_EP1.3x1.5mm, B.Cu at (64.5, 109.4)
- C1203, C1502, C908, C912: value 0.1uF -> 10uF
- C1204: value 4.7uF -> 0.1uF
- C1205, C1702, C1803, C1901, C1902, C1903, C1904, C503, C601, C603, J1201, L1202, R1001, R1004, R1501, R1704, R1901, R1902, R1905, R1906, U1201: moved to F.Cu
- C1208: value 47pF -> 0.1uF
- C1209: value 0.1uF -> 47pF; moved to F.Cu
- C1501, C1802: value 10uF -> 0.1uF; moved to F.Cu
- C1506, C1509, C403, C904: value 10nF -> 10uF
- C1510, C906, C911: value 1nF -> 10uF
- C1512, C202, C905, C910: value 10nF -> 0.1uF
- C1704: value 10nF -> 0.1uF; moved to F.Cu
- C201, C404: value 0.1uF -> 10nF
- C203: value 1nF -> 100uF; footprint Capacitors_SMD:C_0402 -> Capacitors_Tantalum_SMD:CP_Tantalum_Case-X_EIA-7343-43_Reflow
- C401: value 10uF -> 0.1uF; footprint Capacitors_SMD:C_1206 -> Capacitors_SMD:C_0402
- C402: footprint Capacitors_SMD:C_0402 -> Capacitors_SMD:C_1206
- C405: value 100uF -> 0.1uF; footprint Capacitors_SMD:C_1206 -> Capacitors_SMD:C_0402
- C406: value 0.1uF -> 10uF; footprint Capacitors_SMD:C_0402 -> Capacitors_SMD:C_1206
- C602: value 0.1uF -> 10nF; moved to F.Cu
- C703: moved to B.Cu
- C907: value 1nF -> 0.1uF
- C909: value 10uF -> 0.1uF
- D401: value BAT48JFILM -> Red; footprint Diode_SMD:D_SOD-323 -> LEDs:LED_0402
- J801: value PICKIT3 -> PICKIT4; footprint Custom Footprints Library:PICKIT3_Header -> Custom Footprints Library:PICKIT4_Header
- L1201: value DNP -> 600R 0.5A; moved to F.Cu
- Q401, Q801: footprint Package_TO_SOT_SMD:SOT-323_SC-70 -> TO_SOT_Packages_SMD:SOT-323_SC-70
- Q402: value ZXMS6004FFTA -> BSS214NW; footprint Package_TO_SOT_SMD:SOT-23 -> TO_SOT_Packages_SMD:SOT-323_SC-70
- R1002: value 100 -> 10k
- R1201: value 487k -> 1k; moved to F.Cu
- R1202: value 6.04k -> 487k; moved to F.Cu
- R1203: value 40.2k -> 6.04k; moved to F.Cu
- R1204: value 10k -> 40.2k; moved to F.Cu
- R1205, R205, R206: value 10 -> 10k; moved to F.Cu
- R1206: value 0.02 -> 100k; footprint Resistors_SMD:R_0612 -> Resistors_SMD:R_0402; moved to F.Cu
- R1207: value 27 -> 100k
- R1208: value 27 -> 10
- R1209, R606: value 10 -> 0.02; footprint Resistors_SMD:R_0402 -> Resistors_SMD:R_0612; moved to F.Cu
- R1210: value 1k -> 0
- R1503: value 10k -> 0; moved to F.Cu
- R1504, R1608: value 10k -> 0
- R1603: value 10k -> 100
- R1604, R212, R403: value 10 -> 10k
- R1702: value 499 -> 1k; moved to F.Cu
- R1801: value 1k -> 10k
- R201: value 6.04M -> 100k
- R202: value 86.6k -> 10k
- R203: value 243k -> 100k
- R204: value 243k -> 1k
- R207: value 13.7k -> 10
- R208: value 5.23k -> 0.02; footprint Resistors_SMD:R_0402 -> Resistors_SMD:R_0612; moved to F.Cu
- R209: value 10 -> 0
- R210, R408: value 0.02 -> 0; footprint Resistors_SMD:R_0612 -> Resistors_SMD:R_0402
- R211: value 5.23k -> 0
- R213: value 10k -> 10
- R407, R801, R803: value 10 -> 100
- R410: value 562k -> 0.02; footprint Resistors_SMD:R_0402 -> Resistors_SMD:R_0612
- R411: value 180k -> 0
- R607: value 0.02 -> 0; footprint Resistors_SMD:R_0612 -> Resistors_SMD:R_0402; moved to F.Cu
- R608: value 10 -> 0; moved to F.Cu
- R609: value 1.87k -> 0; moved to F.Cu
- R610: value 1.5k -> 10; moved to F.Cu
- TP202, TP203: value TP -> TP_Pad
- U1203: value TPD3S014DBVR -> TXB0102DCU; footprint TO_SOT_Packages_SMD:SOT-23-6 -> Package_SO:VSSOP-8_2.4x2.1mm_P0.5mm; moved to F.Cu
- U1601: value 74LVC1G17 -> 74LVC1G97; footprint TO_SOT_Packages_SMD:SOT-353_SC-70-5 -> Package_TO_SOT_SMD:SOT-363_SC-70-6
- U1602: value NHD-0420H1Z -> Generic 20x04 LCD; footprint Display:NHD-0420H1Z -> Custom Footprints Library:20x04_LCD
- U1702: value TPS71530 -> 74LVC1G97; footprint Package_TO_SOT_SMD:SOT-353_SC-70-5 -> Package_TO_SOT_SMD:SOT-363_SC-70-6; moved to F.Cu
- U1801: value TPS71530 -> 74LVC1G97; footprint Package_TO_SOT_SMD:SOT-353_SC-70-5 -> Package_TO_SOT_SMD:SOT-363_SC-70-6
- U1802, U1803, U1901, U1902, U1903, U1904: value 74LVC1G06 -> 74LVC1G97; footprint TO_SOT_Packages_SMD:SOT-353_SC-70-5 -> Package_TO_SOT_SMD:SOT-363_SC-70-6
- U201: value LTC4365DDB -> TPS26600RHFT; footprint Housings_DFN_QFN:DFN-8-1EP_2x3mm_Pitch0.5mm -> Housings_DFN_QFN:QFN-24-1EP_4x5mm_Pitch0.5mm
- U401: value TPS62150 -> 74LVC1G97; footprint Package_DFN_QFN:QFN-16-1EP_3x3mm_P0.5mm_EP1.8x1.8mm -> Package_TO_SOT_SMD:SOT-363_SC-70-6
- U502: value MCP9804 -> INA219BxDCN; footprint Package_DFN_QFN:DFN-8-1EP_3x2mm_P0.5mm_EP1.3x1.5mm -> Package_TO_SOT_SMD:SOT-23-8; moved to F.Cu
- U601: value TPS7A91 -> TPS7A7200RGTR; footprint Package_DFN_QFN:Texas_S-PDSO-N10_EP1.2x2mm -> Package_DFN_QFN:QFN-16-1EP_3x3mm_P0.5mm_EP1.75x1.75mm; moved to F.Cu
- U702: value MCP9804 -> INA219BxDCN; footprint Package_DFN_QFN:DFN-8-1EP_3x2mm_P0.5mm_EP1.3x1.5mm -> Package_TO_SOT_SMD:SOT-23-8; moved to B.Cu
- moved R1608 292.3 mm to (400.4, 142.3)
- moved R1611 289.5 mm to (398.8, 144.5)
- moved R1613 288.9 mm to (398.8, 146.7)
- moved R1610 288.0 mm to (396.2, 146.7)
- moved R1612 287.4 mm to (396.2, 148.8)
- moved R1609 286.6 mm to (393.5, 148.8)
- moved R1604 286.1 mm to (397.8, 142.3), turned to 0 degrees
- moved R1601 282.4 mm to (395.1, 142.3)
- moved R1801 282.3 mm to (443.3, 145.4)
- moved R1804 280.0 mm to (443.7, 143.2)
- moved R1805 279.2 mm to (440.7, 147.4)
- moved D1801 279.1 mm to (440.9, 143.1)
- moved C1802 278.9 mm to (437.8, 143.2), turned to 0 degrees
- moved U1601 276.9 mm to (388.6, 143.1), turned to 0 degrees
- moved U1802 276.7 mm to (434.2, 147.9)
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Connections:
- net Telemetry_Config renamed ~Telemetry_Config
- C1201 pad 1: +3V3 -> +3.3V_USB
- C1202 pad 1: +3V3 -> +5V_USB
- C1204 pad 1: +5V_USB -> +3V3
- C1206 pad 1: Net-(C1206-Pad1) -> +3.3V_USB
- C1208 pad 1: /USB UART Bridge/CONN_USB- -> +3V3
- C1209 pad 1: Net-(C1209-Pad1) -> /USB UART Bridge/CONN_USB-
- C1506 pad 1: POS3P3_POX_ADC -> Net-(C1506-Pad1)
- C1507 pad 1: +1.8V -> Net-(C1507-Pad1)
- C1508 pad 1: +1.8V -> POS3P3_POX_ADC
- C1509 pad 1: +1.8V -> Net-(C1506-Pad1)
- C1510 pad 1: +1.8V -> Net-(C1507-Pad1)
- C1511 pad 1: +3.3V_POX -> Net-(C1506-Pad1)
- C1512 pad 1: +3.3V_POX -> Net-(C1507-Pad1)
- C1704 pad 1: Net-(C1704-Pad1) -> +3V3
- C1704 pad 2: Net-(C1704-Pad2) -> GND
- C1801 pad 1: +12V -> +3V3
- C1802 pad 1: Net-(C1802-Pad1) -> +3V3
- C201 pad 1: +12Vin -> Net-(C201-Pad1)
- C201 pad 2: GND -> Net-(C201-Pad2)
- C203 pad 1: +12Vin -> +12V
- C401 pad 1: +12V -> +3V3
- C402 pad 1: Net-(C402-Pad1) -> +12V
- C404 pad 1: +12V -> Net-(C404-Pad1)
- C405 pad 1: Net-(C405-Pad1) -> +12V
- C406 pad 1: +3V3 -> Net-(C406-Pad1)
- C910 pad 1: +3V3 -> +3.3VA_MZ
- C910 pad 2: GND -> GNDA_MZ
- C912 pad 1: +3V3 -> +3.3VA_MZ
- C912 pad 2: GND -> GNDA_MZ
- D401 pad 1: Net-(C402-Pad1) -> Net-(C403-Pad1)
- D401 pad 2: +3V3 -> Net-(D401-Pad2)
- J1201 pad 4: Net-(J1201-Pad4) -> (no net)
- J801 pad 6: Net-(J801-Pad6) -> (no net)
- L1201 pad 2: Net-(C1209-Pad1) -> Net-(L1201-Pad2)
- L401 pad 2: Net-(C405-Pad1) -> Net-(C406-Pad1)
- Q402 pad 3: +3V3 -> Net-(Q402-Pad3)
- R1001 pad 1: PIC32MZ_POSC_EC_Enable -> PIC32MZ_REFCLK1
- R1002 pad 1: Net-(R1002-Pad1) -> PIC32MZ_POSC_EC_Enable
- R1002 pad 2: PIC32MZ_POSC_EC -> GND
- R1201 pad 2: Net-(R1201-Pad2) -> Net-(D1201-Pad2)
- R1202 pad 1: Net-(R1201-Pad2) -> +5V_USB
- R1203 pad 2: GND -> Net-(R1203-Pad2)
- R1204 pad 1: +3V3 -> Net-(R1203-Pad2)
- R1204 pad 2: POS5_USB_PGOOD -> GND
- R1205 pad 1: POS5_USB_SNS- -> +3V3
- R1205 pad 2: +5V_USB -> POS5_USB_PGOOD
- R1206 pad 1: +5V_USB -> +3V3
- R1206 pad 2: Net-(R1206-Pad2) -> USB_UART_TX
- R1207 pad 1: /USB UART Bridge/CONN_USB+ -> +3V3
- R1207 pad 2: /USB UART Bridge/BRIDGE_USB+ -> USB_UART_RX
- R1208 pad 1: /USB UART Bridge/CONN_USB- -> POS5_USB_SNS-
- R1208 pad 2: /USB UART Bridge/BRIDGE_USB- -> +5V_USB
- R1209 pad 1: POS5_USB_SNS+ -> +5V_USB
- R1209 pad 2: Net-(R1206-Pad2) -> Net-(R1209-Pad2)
- R1210 pad 2: Net-(D1201-Pad2) -> Net-(R1209-Pad2)
- R1503 pad 1: +3.3V_POX -> I2C_SCL
- R1503 pad 2: POS3P3_POX_ADC -> Net-(R1503-Pad2)
- R1504 pad 1: POS3P3_POX_ADC -> I2C_SDA
- R1504 pad 2: GND -> Net-(R1504-Pad2)
- R1505 pad 1: +1.8V -> +3.3V_POX
- R1505 pad 2: Net-(R1505-Pad2) -> POS3P3_POX_ADC
- R1506 pad 1: +1.8V -> POS3P3_POX_ADC
- R1506 pad 2: Net-(R1506-Pad2) -> GND
- R1603 pad 1: LCD_PMP_R_W -> +3V3
- R1603 pad 2: GND -> LCD_CONTRAST
- R1604 pad 1: LCD_BACKLIGHT -> LCD_CONTRAST
- R1604 pad 2: Net-(R1604-Pad2) -> GND
- R1605 pad 1: +3V3 -> LCD_PMP_R_W
- R1605 pad 2: LCD_PMP_E -> GND
- R1608 pad 1: LCD_PMP_DB2 -> Net-(R1608-Pad1)
- R1608 pad 2: GND -> LCD_BACKLIGHT
- R1609 pad 1: LCD_PMP_DB3 -> LCD_PMP_DB2
- R1610 pad 1: LCD_PMP_DB4 -> LCD_PMP_DB3
- R1611 pad 1: LCD_PMP_DB5 -> LCD_PMP_DB4
- R1612 pad 1: LCD_PMP_DB6 -> +3V3
- R1612 pad 2: GND -> LCD_PMP_E
- R1613 pad 1: LCD_PMP_DB7 -> LCD_PMP_DB5
- R1702 pad 2: Net-(C1704-Pad2) -> Net-(R1701-Pad2)
- R1704 pad 1: Net-(R1704-Pad1) -> Net-(C1703-Pad1)
- R1704 pad 2: GND -> Net-(R1703-Pad1)
- R1801 pad 1: Net-(C1802-Pad1) -> PGOOD_LED_SHDN
- R1801 pad 2: Net-(D1801-Pad2) -> GND
- R1802 pad 2: Net-(D1802-Pad2) -> Net-(D1801-Pad2)
- R1804 pad 2: Net-(D1804-Pad2) -> Net-(D1803-Pad2)
- R1805 pad 2: Net-(D1805-Pad2) -> Net-(D1804-Pad2)
- R202 pad 1: Net-(R201-Pad2) -> Net-(R202-Pad1)
- R202 pad 2: Net-(R202-Pad2) -> Net-(C201-Pad2)
- R203 pad 1: Net-(R202-Pad2) -> +12Vin
- R203 pad 2: GND -> Net-(R201-Pad2)
- R204 pad 1: +12Vin -> Net-(R201-Pad2)
- R204 pad 2: Net-(R204-Pad2) -> Net-(R202-Pad1)
- R205 pad 1: Net-(R205-Pad1) -> Net-(R202-Pad1)
- R205 pad 2: Net-(Q201-Pad2) -> Net-(C201-Pad2)
- R206 pad 1: Net-(Q201-Pad4) -> +12Vin
- R206 pad 2: Net-(R205-Pad1) -> Net-(R206-Pad2)
- R207 pad 1: +12V -> POS12_SNS+
- R207 pad 2: POS12_PGOOD -> Net-(R207-Pad2)
- R208 pad 1: POS12_PGOOD -> Net-(R207-Pad2)
- R208 pad 2: GND -> +12V
- R209 pad 1: POS12_SNS+ -> Net-(R207-Pad2)
- R209 pad 2: Net-(Q201-Pad5) -> +12V
- R210 pad 1: Net-(Q201-Pad5) -> Net-(R207-Pad2)
- R211 pad 1: Net-(R205-Pad1) -> Net-(R207-Pad2)
- R211 pad 2: Net-(C204-Pad1) -> +12V
- R212 pad 1: POS12_SNS- -> Net-(R212-Pad1)
- R212 pad 2: +12V -> Net-(C201-Pad2)
- R213 pad 1: +12V -> POS12_SNS-
- R213 pad 2: GND -> +12V
- R403 pad 1: POS3P3_RUN -> +3V3
- R403 pad 2: POS12_PGOOD -> Net-(R403-Pad2)
- R405 pad 1: +3V3 -> +12V
- R405 pad 2: POS3P3_PGOOD -> Net-(D401-Pad2)
- R406 pad 1: Net-(C402-Pad1) -> Net-(C403-Pad1)
- R407 pad 1: POS3P3_SNS_OUT+ -> +3V3
- R407 pad 2: Net-(C405-Pad1) -> Net-(Q402-Pad3)
- R408 pad 1: Net-(C405-Pad1) -> Net-(R408-Pad1)
- R408 pad 2: +3V3 -> GND
- R409 pad 1: POS3P3_SNS_OUT- -> POS3P3_SNS_OUT+
- R409 pad 2: +3V3 -> Net-(C406-Pad1)
- R410 pad 1: +3V3 -> Net-(C406-Pad1)
- R410 pad 2: Net-(R410-Pad2) -> +3V3
- R411 pad 1: Net-(R410-Pad2) -> Net-(C406-Pad1)
- R411 pad 2: GND -> Net-(R411-Pad2)
- R606 pad 1: POS1P8_SNS_OUT+ -> Net-(C603-Pad1)
- R606 pad 2: Net-(C603-Pad1) -> +1.8V
- R608 pad 1: POS1P8_SNS_OUT- -> Net-(C603-Pad1)
- R609 pad 1: +1.8V -> Net-(C603-Pad1)
- R609 pad 2: Net-(R609-Pad2) -> +1.8V
- R610 pad 1: Net-(R609-Pad2) -> POS1P8_SNS_OUT-
- R610 pad 2: GND -> +1.8V
- R801 pad 1: Net-(R801-Pad1) -> Net-(Q801-Pad1)
- R801 pad 2: Net-(Q801-Pad1) -> Net-(R801-Pad2)
- R803 pad 1: Net-(Q801-Pad3) -> Net-(C802-Pad1)
- R803 pad 2: Net-(C802-Pad1) -> Net-(Q801-Pad3)
- SW801 pad 2: Net-(R801-Pad1) -> Net-(R801-Pad2)
- U1101 pad 10: Net-(U1101-Pad10) -> (no net)
- U1101 pad 11: Net-(U1101-Pad11) -> (no net)
- U1101 pad 12: Net-(U1101-Pad12) -> (no net)
- U1101 pad 21: Net-(U1101-Pad21) -> (no net)
- U1101 pad 22: Net-(U1101-Pad22) -> (no net)
- U1101 pad 23: Net-(U1101-Pad23) -> POS12_PGOOD
- U1101 pad 24: Net-(U1101-Pad24) -> POS5_USB_PGOOD
- U1101 pad 27: Net-(U1101-Pad27) -> POS3P3_PGOOD
- U1101 pad 28: Net-(U1101-Pad28) -> ~ETC_Config
- U1101 pad 29: Net-(U1101-Pad29) -> PGOOD_LED_SHDN
- U1101 pad 33: Net-(U1101-Pad33) -> (no net)
- U1101 pad 36: Net-(U1101-Pad36) -> (no net)
- U1101 pad 37: Net-(U1101-Pad37) -> (no net)
- U1101 pad 38: Net-(U1101-Pad38) -> (no net)
- U1101 pad 4: Net-(U1101-Pad4) -> (no net)
- U1101 pad 48: Net-(U1101-Pad48) -> (no net)
- U1201 pad 3: Net-(R1201-Pad2) -> Net-(R1202-Pad2)
- U1201 pad 4: Net-(R1202-Pad2) -> Net-(R1203-Pad2)
- U1202 pad 10: USB_UART_TX -> USB_UART_TX_BUF
- U1202 pad 11: Net-(U1202-Pad11) -> (no net)
- U1202 pad 2: Net-(U1202-Pad2) -> (no net)
- U1202 pad 3: Net-(C1206-Pad1) -> +3.3V_USB
- U1202 pad 7: USB_UART_RX -> USB_UART_RX_BUF
- U1202 pad 8: Net-(U1202-Pad8) -> (no net)
- U1202 pad 9: +3V3 -> +3.3V_USB
- U1203 pad 1: Net-(C1209-Pad1) -> USB_UART_TX_BUF
- U1203 pad 3: Net-(C1209-Pad1) -> +3V3
- U1203 pad 4: Net-(R1206-Pad2) -> USB_UART_TX
- U1203 pad 5: /USB UART Bridge/CONN_USB- -> USB_UART_RX
- U1203 pad 6: /USB UART Bridge/CONN_USB+ -> POS5_USB_PGOOD
- U1302 pad 3: Net-(U1302-Pad3) -> (no net)
- U1401 pad 2: Net-(U1401-Pad2) -> (no net)
- U1401 pad 3: Net-(U1401-Pad3) -> (no net)
- U1401 pad 7: Net-(U1401-Pad7) -> (no net)
- U1502 pad 6: Net-(R1506-Pad2) -> Net-(R1504-Pad2)
- U1502 pad 7: Net-(R1505-Pad2) -> Net-(R1503-Pad2)
- U1503 pad 1: Net-(U1503-Pad1) -> (no net)
- U1503 pad 10: +3.3V_POX -> Net-(C1506-Pad1)
- U1503 pad 11: +1.8V -> Net-(C1507-Pad1)
- U1503 pad 14: Net-(U1503-Pad14) -> (no net)
- U1503 pad 2: Net-(R1505-Pad2) -> Net-(R1503-Pad2)
- U1503 pad 3: Net-(R1506-Pad2) -> Net-(R1504-Pad2)
- U1503 pad 5: Net-(U1503-Pad5) -> (no net)
- U1503 pad 6: Net-(U1503-Pad6) -> (no net)
- U1503 pad 7: Net-(U1503-Pad7) -> (no net)
- U1503 pad 8: Net-(U1503-Pad8) -> (no net)
- U1503 pad 9: +3.3V_POX -> Net-(C1506-Pad1)
- U1601 pad 1: (no net) -> LCD_BACKLIGHT_PWM
- U1601 pad 2: LCD_BACKLIGHT_PWM -> GND
- U1601 pad 4: Net-(R1604-Pad2) -> Net-(R1608-Pad1)
- U1702 pad 1: Net-(U1702-Pad1) -> Net-(C1703-Pad1)
- U1702 pad 3: Net-(U1702-Pad3) -> GND
- U1702 pad 4: +3V3 -> Cap_Touch_Power
- U1702 pad 5: Net-(C1706-Pad1) -> +3V3
- U1801 pad 1: Net-(U1801-Pad1) -> +3V3
- U1801 pad 3: Net-(U1801-Pad3) -> PGOOD_LED_SHDN
- U1801 pad 4: +12V -> Net-(D1801-Pad1)
- U1801 pad 5: Net-(C1802-Pad1) -> +3V3
- U1802 pad 1: (no net) -> +3V3
- U1802 pad 2: POS12_PGOOD -> GND
- U1802 pad 3: GND -> PGOOD_LED_SHDN
- U1802 pad 4: Net-(D1801-Pad1) -> Net-(D1802-Pad1)
- U1802 pad 5: Net-(C1802-Pad1) -> +3V3
- U1803 pad 1: (no net) -> +3V3
- U1803 pad 2: POS5_USB_PGOOD -> GND
- U1803 pad 3: GND -> PGOOD_LED_SHDN
- U1803 pad 4: Net-(D1802-Pad1) -> Net-(D1803-Pad1)
- U1901 pad 1: (no net) -> +3V3
- U1901 pad 2: Heartbeat_LED -> GND
- U1902 pad 1: (no net) -> +3V3
- U1902 pad 2: Error_LED -> GND
- U1903 pad 1: (no net) -> +3V3
- U1903 pad 2: Reset_LED -> GND
- U1904 pad 1: (no net) -> +3V3
- U1904 pad 2: CPU_Trap_LED -> GND
- U2001 pad 3: Net-(U2001-Pad3) -> (no net)
- U201 pad 1: GND -> (no net)
- U201 pad 2: Net-(R202-Pad2) -> (no net)
- U201 pad 3: Net-(R201-Pad2) -> (no net)
- U201 pad 4: +12Vin -> (no net)
- U201 pad 5: Net-(R205-Pad1) -> (no net)
- U201 pad 6: Net-(Q201-Pad5) -> (no net)
- U201 pad 7: POS12_PGOOD -> (no net)
- U201 pad 8: Net-(R204-Pad2) -> +12Vin
- U201 pad 9: GND -> +12Vin
- U302 pad 3: Net-(U302-Pad3) -> (no net)
- U401 pad 1: Net-(L401-Pad1) -> GND
- U401 pad 2: Net-(L401-Pad1) -> GND
- U401 pad 3: Net-(L401-Pad1) -> POS3P3_RUN
- U401 pad 5: Net-(R410-Pad2) -> +3V3
- U401 pad 6: GND -> Net-(R403-Pad2)
- U502 pad 1: I2C_SDA -> POS3P3_SNS_OUT+
- U502 pad 2: I2C_SCL -> POS3P3_SNS_OUT-
- U502 pad 3: Net-(U502-Pad3) -> GND
- U502 pad 4: GND -> +3V3
- U502 pad 5: GND -> I2C_SCL
- U502 pad 6: GND -> I2C_SDA
- U502 pad 7: +3V3 -> I2C_SDA
- U502 pad 8: +3V3 -> GND
- U601 pad 1: Net-(C603-Pad1) -> +1.8V
- U601 pad 10: +3V3 -> (no net)
- U601 pad 11: GND -> Net-(C602-Pad1)
- U601 pad 2: Net-(C603-Pad1) -> (no net)
- U601 pad 3: Net-(R609-Pad2) -> POS1P8_PGOOD
- U601 pad 4: GND -> (no net)
- U601 pad 5: POS1P8_PGOOD -> GND
- U601 pad 6: +3V3 -> (no net)
- U601 pad 7: POS1P8_RUN -> GND
- U601 pad 8: Net-(C602-Pad1) -> GND
- U601 pad 9: +3V3 -> GND
- U702 pad 1: I2C_SDA -> POS1P8_SNS_OUT+
- U702 pad 2: I2C_SCL -> POS1P8_SNS_OUT-
- U702 pad 3: Net-(U702-Pad3) -> GND
- U702 pad 4: GND -> +3V3
- U702 pad 5: GND -> I2C_SCL
- U702 pad 6: +3V3 -> I2C_SDA
- X1001 pad 3: Net-(R1002-Pad1) -> Net-(R1003-Pad1)
Routing:
- net I2C_SCL: track 249.5 -> 18.4 mm, vias 10 -> 1
- net I2C_SDA: track 238.5 -> 26.1 mm, vias 7 -> 1
- net GND: track 249.3 -> 64.2 mm, vias 102 -> 6
- net +3V3: track 145.3 -> 21.8 mm, vias 54 -> 2
- net USB_UART_TX: track 120.0 -> 0.00 mm, vias 3 -> 0
- net USB_UART_RX: track 87.7 -> 0.00 mm, vias 6 -> 0
- net POS1P8_PGOOD: track 83.4 -> 0.00 mm, vias 2 -> 0
- net POS1P8_RUN: track 71.3 -> 0.00 mm, vias 2 -> 0
- net LCD_PMP_DB1: track 67.4 -> 0.00 mm
- net LCD_PMP_DB0: track 60.0 -> 0.00 mm, vias 1 -> 0
- net ~PIC32MZ_MCLR: track 58.9 -> 0.00 mm, vias 2 -> 0
- net POS3P3_POX_ADC: track 57.6 -> 0.71 mm, vias 1 -> 0
- net LCD_PMP_E: track 54.3 -> 0.00 mm, vias 1 -> 0
- net LCD_PMP_R_W: track 52.8 -> 0.00 mm, vias 1 -> 0
- net +12V: track 49.6 -> 0.00 mm, vias 2 -> 0
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- removed copper zone on F.Cu, net +12V
- removed copper zone on F.Cu, net +12Vin
- removed copper zone on B.Cu, net +3V3
- removed copper zone on F.Cu, net +3V3
- removed copper zone on PWR, net +3V3
- removed copper zone on GND, net GND
- removed copper zone on F.Cu, net Net-(C405-Pad1)
- removed copper zone on B.Cu, net Net-(C603-Pad1)
- removed copper zone on F.Cu, net Net-(L401-Pad1)
- removed copper zone on F.Cu, net Net-(Q201-Pad5)
Other:
- board outline removed
- board text removed: "GND"
- board text removed: "I2C"
- board text removed: "RX"
- board text removed: "SCL"
- board text removed: "SDA"
- board text removed: "TX"
- board text removed: "USB UART"

Commit message: fixed a few sch issues, more PCB placement
Parts:
- added C1604: 10uF, Capacitors_SMD:C_0402, F.Cu at (103.6, 13.5)
- added C1605: 10uF, Capacitors_SMD:C_0402, F.Cu at (103.6, 14.4)
- added C1801: 0.1uF, Capacitors_SMD:C_0402, F.Cu at (18.0, 82.4)
- added R1705: 10k, Resistors_SMD:R_0402, B.Cu at (79.0, 104.7)
- C1701, R1002, R1004, R1602, R1605, R1606, R1607, R1609, R1610, R1611, R1612, R1613, R1614, R1615, R1702, R1703, R1704, R1801, R1901, R1902, R1905, R1906, SW1701, U1701, U1702: moved to B.Cu
- moved R1801 430.2 mm to (18.0, 80.5), turned to 90 degrees
- moved R1804 426.0 mm to (21.1, 90.0)
- moved D1801 424.3 mm to (21.1, 81.1)
- moved R1803 423.9 mm to (21.1, 85.0)
- moved R1802 423.0 mm to (21.1, 79.9)
- moved R1805 422.8 mm to (21.1, 95.1)
- moved C1803 422.8 mm to (18.0, 92.5), turned to 180 degrees
- moved U1801 420.9 mm to (18.0, 80.5)
- moved D1802 420.9 mm to (21.1, 86.2)
- moved U1802 420.8 mm to (18.0, 85.6)
- moved D1803 420.5 mm to (21.1, 91.2)
- moved D1804 417.9 mm to (21.1, 96.3)
- moved C1804 417.7 mm to (18.0, 97.6), turned to 180 degrees
- moved C1802 416.1 mm to (18.0, 87.4), turned to 180 degrees
- moved U1803 415.8 mm to (18.0, 90.7)
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- renumbered C1801 to C1802, C1802 to C1803, C1803 to C1804
Routing:
- net GND: track 64.2 -> 50.7 mm, vias 6 -> 5
- net I2C_SDA: track 26.1 -> 15.0 mm
- net PIC32MZ_REFCLK1: track 7.85 -> 11.4 mm
- net Net-(R1504-Pad2): track 0.00 -> 2.63 mm
- net Net-(R1503-Pad2): track 0.00 -> 2.57 mm
- net +3V3: track 21.8 -> 19.7 mm, vias 2 -> 1
- net +1.8V: track 2.66 -> 0.89 mm, vias 1 -> 0
- net Net-(C1506-Pad1): track 1.69 -> 0.00 mm
- net +3.3V_USB: track 2.04 -> 3.41 mm
- net Net-(D1201-Pad2): track 0.00 -> 0.97 mm
- net +5V_USB: track 1.94 -> 2.83 mm
- net /USB UART Bridge/BRIDGE_USB+: track 0.72 -> 0.00 mm
Other:
- board text added: "Pulse Oximeter REV B TBD"
- board text removed: "Pulse Oximeter REV A June 2020"

Commit message: finished arranging pcb by sheet
Parts:
- C1201, C1202, C1203, C1204, C1206, C1207, C1209, C1301, C1302, C1303, C403, C501, D1201, D401, Q401, Q402, R1201, R1213, R1214, R401, R402, R404, R405, R406, R407, R411, R412, R413, U1202, U1203, U1301, U1302, U501: moved to B.Cu
- moved D1201 219.9 mm to (253.2, 119.6)
- moved R1201 219.9 mm to (253.2, 121.6)
- moved TP1201 218.6 mm to (254.6, 116.5)
- moved R1207 215.5 mm to (259.3, 120.2)
- moved C1302 214.5 mm to (249.8, 119.8), turned to 0 degrees
- moved C1208 213.3 mm to (257.0, 118.9)
- moved U1301 212.4 mm to (249.8, 122.1), turned to 0 degrees
- moved C1301 209.6 mm to (247.4, 122.7), turned to 90 degrees
- moved C1202 207.3 mm to (246.9, 116.0)
- moved C1203 205.5 mm to (246.0, 116.0)
- moved C1201 205.1 mm to (245.8, 122.7)
- moved U1202 204.6 mm to (245.6, 119.4)
- moved C1206 203.7 mm to (245.1, 116.0)
- moved C1303 203.3 mm to (244.9, 122.7)
- moved R1208 202.3 mm to (245.9, 121.7), turned to 90 degrees
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Connections:
- R411 pad 2: Net-(R411-Pad2) -> +3V3
- R412 pad 2: Net-(R411-Pad2) -> +3V3
- R413 pad 2: Net-(R411-Pad2) -> +3V3

Commit message: board outline, arranged functional blocks
Parts:
- added REF**: Symbol_Barrel_Polarity, Symbol:Symbol_Barrel_Polarity, B.Cu at (108.8, 132.1)
- C1201, C1202, C1203, C1204, C1206, C1207, C1209, C1301, C1302, C1303, D1201, R1201, R1213, R1214, U1202, U1203, U1301, U1302: moved to F.Cu
- C1205, C1208, C1210, C1211, C1502, J1201, J1202, L1201, L1202, R1202, R1203, R1204, R1205, R1206, R1207, R1208, R1209, R1210, R1211, R1212, R1215, R1216, R1217, R1218, U1201, U1204: moved to B.Cu
- moved H2102 200.6 mm to (100.1, 136.1)
- moved H2101 196.0 mm to (100.1, 63.1)
- moved R1207 123.4 mm to (136.2, 111.0), turned to 270 degrees
- moved R1206 122.0 mm to (137.5, 111.0), turned to 270 degrees
- moved H2104 121.9 mm to (190.1, 136.1)
- moved C1210 120.9 mm to (136.3, 113.2), turned to 90 degrees
- moved U1203 120.3 mm to (136.9, 113.2), turned to 180 degrees
- moved C1208 119.7 mm to (137.5, 113.2), turned to 270 degrees
- moved R1216 118.7 mm to (136.2, 115.4), turned to 90 degrees
- moved R1201 118.5 mm to (134.8, 117.0), turned to 0 degrees
- moved R1217 117.3 mm to (137.5, 115.4), turned to 90 degrees
- moved D1201 116.5 mm to (136.8, 117.0), turned to 180 degrees
- moved U1301 115.5 mm to (134.3, 120.5), turned to 90 degrees
- moved H2103 114.3 mm to (190.1, 63.1)
- moved C1301 113.7 mm to (133.7, 122.9), turned to 0 degrees
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Other:
- board outline added: 100 x 83 mm
- board text added: "PIC KIT 4"
- board text added: "REFCLK1 (1MHz)"
- board text added: "Reset"
- board text added: "TODO: Set date Set board info like via, trakc numbers, etc"
- board text added: "Track Segments: TBD Nets: TBD Vias: TBD Components: TBD"
- board text removed: "REFCLK1"
- board text removed: "Reset/ Prog"
- board text removed: "Track Segments: 1787 Nets: 160 Vias: 256 Components: 276"

Commit message: started routing
Parts:
- moved J1202 3.61 mm to (157.9, 123.8)
- moved C1211 3.61 mm to (149.0, 121.3)
- moved R1218 3.61 mm to (149.0, 120.1)
- moved R601 3.47 mm to (144.0, 127.2), turned to 0 degrees
- turned C503 to 270 degrees
- turned R213 to 270 degrees
Routing:
- net +3V3: track 19.7 -> 108.7 mm, vias 1 -> 21
- net GND: track 50.7 -> 136.4 mm, vias 5 -> 37
- net PIC32MZ_POSC_EC_Enable: track 0.00 -> 13.9 mm, vias 0 -> 1
- net POS3P3_SNS_OUT-: track 0.00 -> 4.87 mm
- net Net-(R403-Pad2): track 0.00 -> 4.65 mm
- net PIC32MZ_POSC_EC: track 0.00 -> 4.40 mm, vias 0 -> 1
- net Net-(R408-Pad1): track 0.00 -> 4.22 mm
- net LCD_CONTRAST: track 0.00 -> 4.06 mm
- net GNDA_MZ: track 0.00 -> 3.93 mm
- net +3.3VA_MZ: track 0.00 -> 3.91 mm
- net Net-(C1001-Pad1): track 0.00 -> 3.74 mm
- net LCD_BACKLIGHT: track 0.00 -> 3.62 mm
- net LCD_PMP_R_W: track 0.00 -> 3.62 mm
- net LCD_PMP_RS: track 0.00 -> 3.62 mm
- net LCD_PMP_DB5: track 0.00 -> 3.62 mm
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- added copper zone on PWR, net +3V3
- added copper zone on GND, net GND

Commit message: added POX LED, much more routing
Parts:
- added C1513: 0.1uF, Capacitors_SMD:C_0402, B.Cu at (187.0, 124.9)
- added D1501: Green, LEDs:LED_0402, B.Cu at (184.0, 123.6)
- added R1508: 1k, Resistors_SMD:R_0402, B.Cu at (184.0, 122.4)
- added U1504: 74LVC1G97, Package_TO_SOT_SMD:SOT-363_SC-70-6, B.Cu at (187.0, 123.1)
- C1211, R1218, R411, R412, R413: moved to F.Cu
- moved J1202 13.1 mm to (144.7, 124.0), turned to 270 degrees
- moved REF** 6.12 mm to (107.1, 126.2), turned to 270 degrees
- moved R411 5.59 mm to (110.2, 109.7)
- moved R412 3.56 mm to (111.3, 109.7)
- moved TP401 3.37 mm to (108.4, 107.2)
- moved C502 3.05 mm to (107.1, 111.5)
- moved C503 3.05 mm to (104.1, 113.9)
- moved R409 3.05 mm to (108.7, 110.2)
- moved R414 3.05 mm to (108.7, 109.2)
- moved U502 3.05 mm to (106.4, 113.9)
- moved C303 1.72 mm to (110.8, 122.8)
- moved U302 1.72 mm to (111.5, 124.6)
- moved R413 1.52 mm to (112.3, 109.7)
- moved C203 1.22 mm to (121.9, 128.6)
- moved C1211 0.28 mm to (149.2, 121.5)
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Connections:
- J1201 pad 4: (no net) -> Net-(J1201-Pad4)
- J1202 pad 1: (no net) -> Net-(J1202-Pad1)
- J1202 pad 5: (no net) -> Net-(J1202-Pad5)
- J801 pad 6: (no net) -> Net-(J801-Pad6)
- J801 pad 7: (no net) -> Net-(J801-Pad7)
- J801 pad 8: (no net) -> Net-(J801-Pad8)
- U1101 pad 10: (no net) -> Net-(U1101-Pad10)
- U1101 pad 11: (no net) -> Net-(U1101-Pad11)
- U1101 pad 12: (no net) -> Net-(U1101-Pad12)
- U1101 pad 21: (no net) -> Net-(U1101-Pad21)
- U1101 pad 22: (no net) -> Net-(U1101-Pad22)
- U1101 pad 33: (no net) -> Net-(U1101-Pad33)
- U1101 pad 36: (no net) -> Net-(U1101-Pad36)
- U1101 pad 37: (no net) -> Net-(U1101-Pad37)
- U1101 pad 38: (no net) -> Net-(U1101-Pad38)
- U1101 pad 4: (no net) -> Net-(U1101-Pad4)
- U1101 pad 48: (no net) -> Net-(U1101-Pad48)
- U1202 pad 11: (no net) -> Net-(U1202-Pad11)
- U1202 pad 2: (no net) -> Net-(U1202-Pad2)
- U1202 pad 8: (no net) -> Net-(U1202-Pad8)
- U1302 pad 3: (no net) -> Net-(U1302-Pad3)
- U1401 pad 2: (no net) -> Net-(U1401-Pad2)
- U1401 pad 3: (no net) -> Net-(U1401-Pad3)
- U1401 pad 7: (no net) -> Net-(U1401-Pad7)
- U1503 pad 1: (no net) -> Net-(U1503-Pad1)
- U1503 pad 14: (no net) -> Net-(U1503-Pad14)
- U1503 pad 5: (no net) -> Net-(U1503-Pad5)
- U1503 pad 6: (no net) -> Net-(U1503-Pad6)
- U1503 pad 7: (no net) -> Net-(U1503-Pad7)
- U1503 pad 8: (no net) -> Net-(U1503-Pad8)
- U2001 pad 3: (no net) -> Net-(U2001-Pad3)
- U2002 pad 3: (no net) -> Net-(U2002-Pad3)
- U201 pad 1: (no net) -> Net-(U201-Pad1)
- U201 pad 11: (no net) -> Net-(U201-Pad11)
- U201 pad 13: (no net) -> Net-(U201-Pad13)
- U201 pad 16: (no net) -> Net-(U201-Pad16)
- U201 pad 2: (no net) -> Net-(U201-Pad2)
- U201 pad 21: (no net) -> Net-(U201-Pad21)
- U201 pad 3: (no net) -> Net-(U201-Pad3)
- U201 pad 4: (no net) -> Net-(U201-Pad4)
- U201 pad 5: (no net) -> Net-(U201-Pad5)
- U201 pad 6: (no net) -> Net-(U201-Pad6)
- U201 pad 7: (no net) -> Net-(U201-Pad7)
- U302 pad 3: (no net) -> Net-(U302-Pad3)
- U501 pad 3: (no net) -> Net-(U501-Pad3)
- U601 pad 10: (no net) -> Net-(U601-Pad10)
- U601 pad 2: (no net) -> Net-(U601-Pad2)
- U601 pad 4: (no net) -> Net-(U601-Pad4)
- U601 pad 6: (no net) -> Net-(U601-Pad6)
- U701 pad 3: (no net) -> Net-(U701-Pad3)
Routing:
- net GND: track 136.4 -> 208.0 mm, vias 37 -> 89
- net +3V3: track 108.7 -> 163.4 mm, vias 21 -> 63
- net PIC32MZ_ICSPCLK: track 0.00 -> 51.1 mm
- net PIC32MZ_ICSPDAT: track 0.00 -> 50.0 mm
- net ~PIC32MZ_MCLR: track 0.00 -> 36.8 mm
- net POS3P3_RUN: track 0.00 -> 12.4 mm, vias 0 -> 1
- net +5V_USB: track 2.83 -> 9.58 mm
- net POS12_PGOOD: track 0.00 -> 6.49 mm
- net Net-(C201-Pad2): track 0.00 -> 6.01 mm, vias 0 -> 7
- net Net-(C1506-Pad1): track 0.00 -> 5.78 mm, vias 0 -> 1
- net Net-(R1209-Pad2): track 0.00 -> 5.75 mm
- net Net-(C1507-Pad1): track 0.00 -> 4.52 mm, vias 0 -> 1
- net +12V: track 2.59 -> 6.36 mm
- net POS1P8_PGOOD: track 0.00 -> 3.57 mm
- net POS5_USB_SNS+: track 1.40 -> 4.92 mm, vias 0 -> 1
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- added copper zone on F.Cu, net +1.8V
- added copper zone on F.Cu, net +12V
- added copper zone on F.Cu, net +12Vin
- added copper zone on F.Cu, net +3V3
- added copper zone on B.Cu, net GND
- added copper zone on GND, net Net-(C201-Pad2)
- added copper zone on F.Cu, net Net-(C406-Pad1)
- added copper zone on F.Cu, net Net-(C603-Pad1)
- added copper zone on F.Cu, net Net-(L401-Pad1)
- added copper zone on F.Cu, net Net-(R207-Pad2)
Other:
- board text added: "GND"
- board text added: "OSEPP-FTDI-01"
- board text added: "POX DATA"
- board text added: "Place Finger Here < ---------"
- board text added: "RX"
- board text added: "TODO: Set date Set board info like via, track count, etc Add deleted extra features that aren't in netlist"
- board text added: "TX"
- board text added: "VDD"
- board text removed: "TODO: Set date Set board info like via, trakc numbers, etc"

Commit message: much more point to point manual routing
Connections:
- U1101 pad 43: Error_LED -> CPU_Trap_LED
- U1101 pad 44: CPU_Trap_LED -> Error_LED
Routing:
- net +3.3V_USB: track 3.41 -> 60.6 mm, vias 0 -> 3
- net LCD_PMP_RS: track 3.62 -> 49.9 mm
- net GND: track 208.0 -> 248.9 mm, vias 89 -> 106
- net Reset_LED: track 3.02 -> 38.0 mm, vias 1 -> 3
- net LCD_PMP_R_W: track 3.62 -> 38.2 mm
- net LCD_PMP_E: track 3.62 -> 36.2 mm, vias 0 -> 2
- net Heartbeat_LED: track 2.30 -> 34.7 mm, vias 1 -> 3
- net LCD_PMP_DB0: track 3.62 -> 35.4 mm
- net LCD_PMP_DB1: track 3.62 -> 34.8 mm
- net CPU_Trap_LED: track 2.30 -> 31.9 mm
- net LCD_PMP_DB2: track 3.62 -> 32.1 mm
- net +3V3: track 163.4 -> 190.4 mm, vias 63 -> 74
- net LCD_PMP_DB3: track 3.62 -> 30.6 mm
- net LCD_PMP_DB5: track 3.62 -> 28.7 mm
- net LCD_PMP_DB6: track 3.62 -> 28.1 mm
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