File: rev_b/hdw/Pulse_Oximeter/Display.sch (KiCad schematic (older format))
At the start: 22 parts, among them U1601 74LVC1G97, U1602 Generic 20x04 LCD

Commit message: fixed LCD contrast resistors
Parts:
- renumbered R1604 to R1603, R1603 to R1604
Connections:
- net +3V3: now also R1603.1; no longer R1604.1
- net GND: now also R1604.2; no longer R1603.2
- net LCD_CONTRAST: now also R1603.2, R1604.1; no longer R1603.1, R1604.2
Other:
- moved on the sheet: R1603, R1604
Changed lines of the file:
@@
 L Custom_Library:R_Custom R?
 U 1 1 5FE5C1AA
-P 3240 1710
+P 3240 1250
 AR Path="/5BB27BA3/5FE5C1AA" Ref="R?"  Part="1"
 AR Path="/5BB27BF7/5FE5C1AA" Ref="R?"  Part="1"
@@
 AR Path="/5E9E0E87/5FE5C1AA" Ref="R?"  Part="1"
 AR Path="/5EAE2D66/5FE5C1AA" Ref="R?"  Part="1"
-AR Path="/5EAE4A89/5FE5C1AA" Ref="R1604"  Part="1"
-F 0 "R1604" H 3160 1710 50  0000 R CNN
-F 1 "10k" V 3240 1710 50  0000 C CNN
-F 2 "Resistors_SMD:R_0402" H 3240 1710 50  0001 C CNN
-F 3 "" H 3240 1710 50  0001 C CNN
-F 4 "0402" H 3340 1790 50  0000 L CNN "display_footprint"
-F 5 "1%" H 3340 1710 50  0000 L CNN "Tolerance"
-F 6 "1/16W" H 3350 1630 50  0000 L CNN "Wattage"
-F 7 "RMCF0402FT10K0CT-ND" H 3240 1710 50  0001 C CNN "Digi-Key PN"
-	1    3240 1710
+AR Path="/5EAE4A89/5FE5C1AA" Ref="R1603"  Part="1"
+F 0 "R1603" H 3160 1250 50  0000 R CNN
+F 1 "10k" V 3240 1250 50  0000 C CNN
+F 2 "Resistors_SMD:R_0402" H 3240 1250 50  0001 C CNN
+F 3 "" H 3240 1250 50  0001 C CNN
+F 4 "0402" H 3340 1330 50  0000 L CNN "display_footprint"
+F 5 "1%" H 3340 1250 50  0000 L CNN "Tolerance"
+F 6 "1/16W" H 3350 1170 50  0000 L CNN "Wattage"
+F 7 "RMCF0402FT10K0CT-ND" H 3240 1250 50  0001 C CNN "Digi-Key PN"
+	1    3240 1250
 	1    0    0    -1
 $EndComp
@@
 L Custom_Library:R_Custom R?
 U 1 1 5FE5E503
-P 3240 1250
+P 3240 1710
 AR Path="/5BB27BA3/5FE5E503" Ref="R?"  Part="1"
 AR Path="/5BB27BF7/5FE5E503" Ref="R?"  Part="1"
@@
 AR Path="/5EAE2D66/5FE5E503" Ref="R?"  Part="1"
 AR Path="/5EAE2E5F/5FE5E503" Ref="R?"  Part="1"
-AR Path="/5EAE4A89/5FE5E503" Ref="R1603"  Part="1"
-F 0 "R1603" H 3160 1250 50  0000 R CNN
-F 1 "100" V 3240 1250 50  0000 C CNN
-F 2 "Resistors_SMD:R_0402" H 3240 1250 50  0001 C CNN
-F 3 "" H 3240 1250 50  0001 C CNN
-F 4 "0402" H 3340 1330 50  0000 L CNN "display_footprint"
-F 5 "1%" H 3340 1250 50  0000 L CNN "Tolerance"
-F 6 "1/16W" H 3350 1170 50  0000 L CNN "Wattage"
-F 7 "RMCF0402FT100RCT-ND" H 3240 1250 50  0001 C CNN "Digi-Key PN"
-	1    3240 1250
+AR Path="/5EAE4A89/5FE5E503" Ref="R1604"  Part="1"
+F 0 "R1604" H 3160 1710 50  0000 R CNN
+F 1 "100" V 3240 1710 50  0000 C CNN
+F 2 "Resistors_SMD:R_0402" H 3240 1710 50  0001 C CNN
+F 3 "" H 3240 1710 50  0001 C CNN
+F 4 "0402" H 3340 1790 50  0000 L CNN "display_footprint"
+F 5 "1%" H 3340 1710 50  0000 L CNN "Tolerance"
+F 6 "1/16W" H 3350 1630 50  0000 L CNN "Wattage"
+F 7 "RMCF0402FT100RCT-ND" H 3240 1710 50  0001 C CNN "Digi-Key PN"
+	1    3240 1710
 	1    0    0    -1
 $EndComp
