File: rev_b/hdw/Pulse_Oximeter/Pulse_Oximeter.kicad_pcb (KiCad board)
At the start: 4 copper layers, 100 x 83 mm, 292 parts, among them J1201 USB_B_Mini, J1202 OSEPP_FTDI_01, J201 +12V IN, J801 PICKIT4, Q401 BSS214NW, Q402 BSS214NW, Q801 BSS214NW, SW1701 Cap_Touch, SW801 MRST, U1101 PIC32MZ0512EFE064T-I_PT, U1201 TLV6700, U1202 FT234XD, U1203 TXB0102DCU, U1204 TPD3S014DBVR, U1301 INA219BxDCN, U1302 MCP9804, U1401 DS1683, U1501 TPS22929D, U1502 TCA9803, U1503 MAX30102, U1504 74LVC1G97, U1601 74LVC1G97, U1602 Generic 20x04 LCD, U1701 AT42QT1010-TSHR, U1702 74LVC1G97, U1801 74LVC1G97, U1802 74LVC1G97, U1803 74LVC1G97, U1804 74LVC1G97, U1901 74LVC1G97, U1902 74LVC1G97, U1903 74LVC1G97, U1904 74LVC1G97, U2001 MCP9804, U2002 LTC1694, U201 TPS26600RHFT, U301 INA219BxDCN, U302 MCP9804, U401 74LVC1G97, U402 TPS62152, U501 MCP9804, U502 INA219BxDCN, U601 TPS7A7200RGTR, U701 MCP9804, U702 INA219BxDCN, X1001 ASE-8.000MHz

Commit message: fixed LCD contrast resistors
Parts:
- R1603: value 100 -> 10k
- R1604: value 10k -> 100
